Commit message: Added IMU, still testing: looks like we can measure accelerations but we can not see gravity vector

File: coman_urdf/urdf/coman_robot.urdf.xacro (robot description, xacro)
@@ -7,4 +7,23 @@
   -->
   <include filename="$(find coman_urdf)/urdf/coman.urdf.xacro" />
+  <link name="imu_link">
+    <inertial>
+      <mass value="0.01"/>
+      <origin xyz="0 0 0"/>
+      <inertia ixx="1.0E-6" ixy="0" ixz="0" iyy="1.0E-6" iyz="0" izz="1.0E-6"/>
+    </inertial>
+    <visual>
+      <origin rpy="0 0 0" xyz="0 0 0"/>
+      <geometry>
+        <box size="0.01 0.01 0.01"/>
+      </geometry>
+    </visual>
+  </link>
+  <joint name="imu_joint" type="fixed">
+    <parent link="Waist"/>
+    <child link="imu_link"/>
+    <origin xyz="0 0 0" rpy="0 0 0"/>
+  </joint>
+  <include filename="$(find coman_urdf)/urdf/microstrain_3dmgx2_imu.gazebo.xacro" />
   <include filename="$(find coman_urdf)/urdf/coman_transmission.urdf.xacro" />
   <include filename="$(find coman_urdf)/urdf/coman.gazebo" />

File: coman_urdf/urdf/coman_transmission.urdf.xacro (robot description, xacro)
@@ -14,12 +14,4 @@
   <joint name="WaistLat"/>
   <actuator name="WaistLat_motor">
-    <hardwareInterface>EffortJointInterface</hardwareInterface>
-    <mechanicalReduction>100</mechanicalReduction>
-  </actuator>
-</transmission>
-<transmission name="WaistYaw_simple_trans">
-  <type>transmission_interface/SimpleTransmission</type>
-  <joint name="WaistYaw"/>
-  <actuator name="WaistYaw_motor">
     <hardwareInterface>EffortJointInterface</hardwareInterface>
     <mechanicalReduction>100</mechanicalReduction>

Commit message: Added position of IMU from CAD

File: coman_urdf/urdf/coman_robot.urdf.xacro (robot description, xacro)
@@ -24,5 +24,5 @@
     <parent link="Waist"/>
     <child link="imu_link"/>
-    <origin xyz="0 0 0" rpy="0 0 0"/>
+    <origin xyz="-0.072 -0.0068 0.044" rpy="0 0 0"/>
   </joint>
   <xacro:include filename="$(find coman_urdf)/urdf/microstrain_3dmgx2_imu.gazebo.xacro" />
