Commit message: Fixed bug in soft hand. Updated PIDs arm

File: coman_urdf/urdf/soft_hand.urdf.xacro (robot description, xacro)
@@ -20,5 +20,5 @@
      <origin xyz="0 0 0" rpy="0 0 0"/>
      <geometry>
-       <box size="0.05 0.05 0.05" />
+       <box size="0.07 0.07 0.07" />
      </geometry>
    </collision>
@@ -42,5 +42,5 @@
      <origin xyz="0 0 0" rpy="0 0 0"/>
      <geometry>
-       <box size="0.05 0.05 0.05" />
+       <box size="0.07 0.07 0.07" />
      </geometry>
    </collision>
