Commit message: Removed the duplicate coman_plain robot description in favour of a xacro-based conditional description of the robot. The parts of the description that depend on either ROS or YARP can be deactivated by setting the GAZEBO_COMAN_USES_ROS and GAZEBO_COMAN_USES_YARP environment variables during compilation. They can be either 0 or 1. A small dirty python script has been added to circumvent the gzsdf bug preventing the gazebo force_torque sensors described in a urdf to show in the final sdf file. The README.md file has been modified to list the added requirements to run the script (python-bs4). Lastly, the version of the model in manifest.xml has been bumped to 13.10.31 (date based version number).

File: coman_urdf/urdf/coman.gazebo.xacro (robot description, xacro)
@@ -1,4 +1,11 @@
 <?xml version="1.0"?>
-<robot>
+<robot xmlns:xacro="http://ros.org/wiki/xacro">
+    <xacro:if value="$(optenv GAZEBO_COMAN_USES_ROS false)">
+      <gazebo>
+        <plugin name="gazebo_ros_control" filename="libgazebo_ros_control.so">
+          <robotNamespace>/COMAN</robotNamespace>
+        </plugin>
+      </gazebo>
+    </xacro:if>
 <!-- contact model for foot surface -->
    <gazebo reference="LFoot">
@@ -49,16 +56,6 @@
    <gazebo reference="RAnkSag">
     <cfmDamping>1</cfmDamping>
-<!--
     <provideFeedback>true</provideFeedback>
-    <sensor type="force_torque" name="RAnkSag_FT">
-	<always_on>true</always_on>
-	<visualize>true</visualize>
-	<update_rate>1000</update_rate>
-        <plugin name="gazebo_RAnkSag_FT" filename="libFakebotForceTorquePlugin.so">
-	  <boardId>1</boardId>
-        </plugin>
-    </sensor>
--->
-   </gazebo>
+  </gazebo>
    <gazebo reference="LHipSag">
     <cfmDamping>1</cfmDamping>
@@ -78,15 +75,5 @@
    <gazebo reference="LAnkSag">
     <cfmDamping>1</cfmDamping>
-<!--
     <provideFeedback>true</provideFeedback>
-    <sensor type="force_torque" name="LAnkSag_FT">
-	<always_on>true</always_on>
-	<visualize>true</visualize>
-	<update_rate>1000</update_rate>
-        <plugin name="gazebo_LAnkSag_FT" filename="libFakebotForceTorquePlugin.so">
- 	  <boardId>2</boardId>
-        </plugin>
-    </sensor>
--->
    </gazebo>
    <gazebo reference="RShSag">
@@ -101,15 +88,4 @@
    <gazebo reference="RElbj">
     <cfmDamping>1</cfmDamping>
-<!--
-    <provideFeedback>true</provideFeedback>
-    <sensor type="force_torque" name="RElbj_FT">
-	<always_on>true</always_on>
-	<visualize>true</visualize>
-	<update_rate>1000</update_rate>
-        <plugin name="gazebo_RAnkSag_FT" filename="libFakebotForceTorquePlugin.so">
-	  <boardId>3</boardId>
-        </plugin>
-    </sensor>
--->
    </gazebo>
    <gazebo reference="LShSag">
@@ -124,41 +100,4 @@
    <gazebo reference="LElbj">
     <cfmDamping>1</cfmDamping>
-<!--
-    <provideFeedback>true</provideFeedback>
-    <sensor type="force_torque" name="LElbj_FT">
-	<always_on>true</always_on>
-	<visualize>true</visualize>
-	<update_rate>1000</update_rate>
-        <plugin name="gazebo_RAnkSag_FT" filename="libFakebotForceTorquePlugin.so">
-	  <boardId>4</boardId>
-        </plugin>
-    </sensor>
--->
-   </gazebo>
-   <gazebo reference="imu_link">
-    <sensor name="imu_sensor" type="imu">
-     <always_on>1</always_on>
-     <update_rate>1000</update_rate>
-     <visualize>true</visualize>
-     <topic>__default_topic__</topic>
-     <imu>
-      <!--noise>
-       <type>gaussian</type>
-        <rate>
-         <mean>0.0</mean>
-         <stddev>2e-4</stddev>
-         <bias_mean>0.0000075</bias_mean>
-         <bias_stddev>0.0000008</bias_stddev>
-        </rate>
-        <accel>
-         <mean>0.0</mean>
-         <stddev>1.7e-2</stddev>
-         <bias_mean>0.1</bias_mean>
-         <bias_stddev>0.001</bias_stddev>
-        </accel>
-      </noise-->
-     </imu>
-     <plugin name="coman_yarp_gazebo_plugin_IMU" filename="libfakebotIMUplugin.so"/>
-    </sensor>
    </gazebo>
 </robot>

File: coman_urdf/urdf/coman_robot.urdf.xacro (robot description, xacro)
@@ -6,5 +6,5 @@
   This file groups files to use COMAN in GAZEBO
   -->
-  <include filename="$(find coman_urdf)/urdf/coman.urdf.xacro" />
+  <xacro:include filename="$(find coman_urdf)/urdf/coman.urdf.xacro" />
 <!-- IMU, needs to be checked effective position and orientation. For now it maches the same poisition/orientation of Waist link -->
   <link name="imu_link">
@@ -26,6 +26,7 @@
     <origin xyz="0 0 0" rpy="0 0 0"/>
   </joint>
-  <include filename="$(find coman_urdf)/urdf/microstrain_3dmgx2_imu.gazebo.xacro" />
-  <include filename="$(find coman_urdf)/urdf/coman_transmission.urdf.xacro" />
-  <include filename="$(find coman_urdf)/urdf/coman.gazebo" />
+  <xacro:include filename="$(find coman_urdf)/urdf/microstrain_3dmgx2_imu.gazebo.xacro" />
+  <xacro:include filename="$(find coman_urdf)/urdf/coman_transmission.urdf.xacro" />
+  <xacro:include filename="$(find coman_urdf)/urdf/coman.gazebo.xacro" />
+  <origin xyz="0.0 0.0 0.521" rpy="0 0 0" />
 </robot>

File: coman_urdf/urdf/microstrain_3dmgx2_imu.gazebo.xacro (robot description, xacro)
@@ -6,18 +6,50 @@
   This file groups files to use COMAN in GAZEBO
   -->
-  <gazebo>
-    <plugin name="quadrotor_imu_sim" filename="libhector_gazebo_ros_imu.so">
-      <updateRate>100.0</updateRate>
-      <bodyName>imu_link</bodyName>
-      <topicName>COMAN/raw_imu</topicName>
-      <rpyOffsets>0 0 0</rpyOffsets> <!-- deprecated -->
-      <gaussianNoise>0</gaussianNoise>  <!-- deprecated -->
-      <accelDrift>0.5 0.5 0.5</accelDrift>
-      <accelGaussianNoise>0.35 0.35 0.3</accelGaussianNoise>
-      <rateDrift>0.1 0.1 0.1</rateDrift>
-      <rateGaussianNoise>0.05 0.05 0.015</rateGaussianNoise>
-      <headingDrift>0.1</headingDrift>
-      <headingGaussianNoise>0.05</headingGaussianNoise>
-    </plugin>
-  </gazebo>
+  <xacro:if value="$(optenv GAZEBO_COMAN_USES_ROS false)">
+    <gazebo>
+        <plugin name="quadrotor_imu_sim" filename="libhector_gazebo_ros_imu.so">
+          <updateRate>100.0</updateRate>
+          <bodyName>imu_link</bodyName>
+          <topicName>COMAN/raw_imu</topicName>
+          <rpyOffsets>0 0 0</rpyOffsets> <!-- deprecated -->
+          <gaussianNoise>0</gaussianNoise>  <!-- deprecated -->
+          <accelDrift>0.5 0.5 0.5</accelDrift>
+          <accelGaussianNoise>0.35 0.35 0.3</accelGaussianNoise>
+          <rateDrift>0.1 0.1 0.1</rateDrift>
+          <rateGaussianNoise>0.05 0.05 0.015</rateGaussianNoise>
+          <headingDrift>0.1</headingDrift>
+          <headingGaussianNoise>0.05</headingGaussianNoise>
+        </plugin>
+      </gazebo>
+  </xacro:if>
+  <xacro:if value="$(optenv GAZEBO_COMAN_USES_YARP true)">
+    <gazebo reference="imu_link">
+        <sensor name="imu_sensor" type="imu">
+         <always_on>1</always_on>
+         <update_rate>1000</update_rate>
+         <visualize>true</visualize>
+         <topic>__default_topic__</topic>
+         <imu>
+          <!--
+          <noise>
+           <type>gaussian</type>
+            <rate>
+             <mean>0.0</mean>
+             <stddev>2e-4</stddev>
+             <bias_mean>0.0000075</bias_mean>
+             <bias_stddev>0.0000008</bias_stddev>
+            </rate>
+            <accel>
+             <mean>0.0</mean>
+             <stddev>1.7e-2</stddev>
+             <bias_mean>0.1</bias_mean>
+             <bias_stddev>0.001</bias_stddev>
+            </accel>
+          </noise>
+          -->
+         </imu>
+         <plugin name="coman_yarp_gazebo_plugin_IMU" filename="libfakebotIMUplugin.so"/>
+        </sensor>
+       </gazebo>
+  </xacro:if>
 </robot>

Commit message: Added hands in simulation with relative .ini files. Fixed coman.gazebo.xacro issues.

File: coman_urdf/urdf/coman.gazebo.xacro (robot description, xacro)
@@ -1,5 +1,5 @@
 <?xml version="1.0"?>
 <robot xmlns:xacro="http://ros.org/wiki/xacro">
-    <xacro:if value="$(optenv GAZEBO_COMAN_USES_ROS false)">
+    <xacro:if value="${GAZEBO_COMAN_USES_ROS}">
       <gazebo>
         <plugin name="gazebo_ros_control" filename="libgazebo_ros_control.so">
@@ -30,4 +30,6 @@
    </gazebo>
 <!-- contact model for hand surface -->
+<xacro:if value="${GAZEBO_COMAN_USES_7DOF_FOREARMS_DRC_14}">
+    <xacro:if value="${GAZEBO_COMAN_USES_SOFTHANDS_DRC_sw1_14}">
    <gazebo reference="LSoftHand">
      <kp>1000000.0</kp>
@@ -50,4 +52,6 @@
      <cfmDamping>1</cfmDamping>
    </gazebo>
+  </xacro:if>
+</xacro:if>
 <!-- Other parameters... -->
    <gazebo reference="WaistSag">
@@ -127,4 +131,5 @@
     <provideFeedback>true</provideFeedback>
    </gazebo>
+<xacro:if value="${GAZEBO_COMAN_USES_7DOF_FOREARMS_DRC_14}">
    <gazebo reference="RForearmPlate">
     <cfmDamping>1</cfmDamping>
@@ -139,4 +144,13 @@
     <provideFeedback>true</provideFeedback>
    </gazebo>
+</xacro:if>
+<xacro:if value="${GAZEBO_COMAN_USES_7DOF_FOREARMS_DRC_14}">
+    <xacro:if value="${GAZEBO_COMAN_USES_SOFTHANDS_DRC_sw1_14}">
+      <gazebo reference="r_handj">
+        <cfmDamping>1</cfmDamping>
+        <provideFeedback>true</provideFeedback>
+      </gazebo>
+    </xacro:if>
+</xacro:if>
    <gazebo reference="LShSag">
     <cfmDamping>1</cfmDamping>
@@ -155,4 +169,5 @@
     <provideFeedback>true</provideFeedback>
    </gazebo>
+<xacro:if value="${GAZEBO_COMAN_USES_7DOF_FOREARMS_DRC_14}">
    <gazebo reference="LForearmPlate">
     <cfmDamping>1</cfmDamping>
@@ -167,3 +182,12 @@
     <provideFeedback>true</provideFeedback>
    </gazebo>
+</xacro:if>
+<xacro:if value="${GAZEBO_COMAN_USES_7DOF_FOREARMS_DRC_14}">
+    <xacro:if value="${GAZEBO_COMAN_USES_SOFTHANDS_DRC_sw1_14}">
+      <gazebo reference="l_handj">
+        <cfmDamping>1</cfmDamping>
+        <provideFeedback>true</provideFeedback>
+      </gazebo>
+    </xacro:if>
+</xacro:if>
 </robot>

File: coman_urdf/urdf/coman.urdf (robot description, URDF)
Before this commit: robot COMAN, 43 links, 42 joints
Joints:
- joint l_handj: parent l_wrist -> LWrMot3
- joint r_handj: parent r_wrist -> RWrMot3

File: coman_urdf/urdf/coman.urdf.xacro (robot description, xacro)
@@ -476,6 +476,6 @@
   </xacro:if>
 <!-- ********************HANDS********************* -->
-  <xacro:if value="$(optenv GAZEBO_COMAN_USES_7DOF_FOREARMS_DRC_14 true)">
-    <xacro:if value="$(optenv GAZEBO_COMAN_USES_SOFTHANDS_DRC_sw1_14 true)">
+  <xacro:if value="${GAZEBO_COMAN_USES_7DOF_FOREARMS_DRC_14}">
+    <xacro:if value="${GAZEBO_COMAN_USES_SOFTHANDS_DRC_sw1_14}">
       <xacro:include filename="$(find coman_urdf)/urdf/soft_hand.urdf.xacro" />
     </xacro:if>
@@ -755,8 +755,8 @@
   </xacro:if>
 <!-- ********************RIGHT HAND****************** -->
-  <xacro:if value="$(optenv GAZEBO_COMAN_USES_7DOF_FOREARMS_DRC_14 true)">
-    <xacro:if value="$(optenv GAZEBO_COMAN_USES_SOFTHANDS_DRC_sw1_14 true)">
+  <xacro:if value="${GAZEBO_COMAN_USES_7DOF_FOREARMS_DRC_14}">
+    <xacro:if value="${GAZEBO_COMAN_USES_SOFTHANDS_DRC_sw1_14}">
       <joint name="r_handj" type="revolute">
-        <parent link="r_wrist"/>
+        <parent link="RWrMot3"/>
         <child link="RSoftHand"/>
         <origin xyz="0 0 -0.04" rpy="0 0 0"/>
@@ -807,8 +807,8 @@
   </xacro:if>
 <!-- ********************LEFT HAND******************** -->
-  <xacro:if value="$(optenv GAZEBO_COMAN_USES_7DOF_FOREARMS_DRC_14 true)">
-    <xacro:if value="$(optenv GAZEBO_COMAN_USES_SOFTHANDS_DRC_sw1_14 true)">
+  <xacro:if value="${GAZEBO_COMAN_USES_7DOF_FOREARMS_DRC_14}">
+    <xacro:if value="${GAZEBO_COMAN_USES_SOFTHANDS_DRC_sw1_14}">
       <joint name="l_handj" type="revolute">
-        <parent link="l_wrist"/>
+        <parent link="LWrMot3"/>
         <child link="LSoftHand"/>
         <origin xyz="0 0 -0.04" rpy="0 0 0"/>

Commit message: Deleted for now contact model for hands. Set 5Nm max torque in forehands and wrists.

File: coman_urdf/urdf/coman.gazebo.xacro (robot description, xacro)
@@ -30,4 +30,5 @@
    </gazebo>
 <!-- contact model for hand surface -->
+<!--
 <xacro:if value="${GAZEBO_COMAN_USES_7DOF_FOREARMS_DRC_14}">
     <xacro:if value="${GAZEBO_COMAN_USES_SOFTHANDS_DRC_sw1_14}">
@@ -54,4 +55,5 @@
   </xacro:if>
 </xacro:if>
+-->
 <!-- Other parameters... -->
    <gazebo reference="WaistSag">

File: coman_urdf/urdf/coman_hands.urdf (robot description, URDF)
Before this commit: robot COMAN, 45 links, 44 joints
Joints:
- joint LForearmPlate: limit lower=-1.5708 upper=1.5708 effort=50 velocity=4.0 -> lower=-1.5708 upper=1.5708 effort=5 velocity=4.0
- joint LWrj1: limit lower=-0.524 upper=0.524 effort=50 velocity=4.0 -> lower=-0.524 upper=0.524 effort=5 velocity=4.0
- joint LWrj2: limit lower=-0.785375 upper=1.395 effort=50 velocity=4.0 -> lower=-0.785375 upper=1.395 effort=5 velocity=4.0
- joint RForearmPlate: limit lower=-1.5708 upper=1.5708 effort=50 velocity=4.0 -> lower=-1.5708 upper=1.5708 effort=5 velocity=4.0
- joint RWrj1: limit lower=-0.524 upper=0.524 effort=50 velocity=4.0 -> lower=-0.524 upper=0.524 effort=5 velocity=4.0
- joint RWrj2: limit lower=-1.395 upper=0.785375 effort=50 velocity=4.0 -> lower=-1.395 upper=0.785375 effort=5 velocity=4.0
