Commit message: Updated coman gazebo database

File: coman_urdf/urdf/coman_hands.urdf (robot description, URDF)
Before this commit: robot COMAN, 45 links, 44 joints
Links:
- link LElb: geometry collision mesh filename=package://coman_urdf/meshes/collada/simple/forearms/elbow.s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 scale=1.0 1.0 1.0; visual mesh filename=package://coman_urdf/meshes/collada/forearms/elbow.dae scale=1.0 1.0 1.0
- link LForearm: geometry collision mesh filename=package://coman_urdf/meshes/collada/simple/forearms/forearm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 scale=1.0 1.0 1.0; visual mesh filename=package://coman_urdf/meshes/collada/forearms/forearm_lowpol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 scale=0.1 0.1 0.1
- link RElb: geometry collision mesh filename=package://coman_urdf/meshes/collada/simple/forearms/elbow.s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 scale=1.0 1.0 1.0; visual mesh filename=package://coman_urdf/meshes/collada/forearms/elbow.dae scale=1.0 1.0 1.0
- link RForearm: geometry collision mesh filename=package://coman_urdf/meshes/collada/simple/forearms/forearm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 scale=1.0 1.0 1.0; visual mesh filename=package://coman_urdf/meshes/collada/forearms/forearm_lowpol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 scale=0.1 0.1 0.1
- link Xtion_cam_body: geometry collision mesh filename=package://coman_urdf/meshes/collada/simple/Xtion/xtion_cam_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 scale=0.001 0.001 0.001; visual mesh filename=package://coman_urdf/meshes/collada/Xtion/xtion_cam_body.dae scale=0.001 0.001 0.001
