Commit message: Small changin in the gazebo part. Now maximum allowed velocity is 4 rad/sec. Increasing of PID values

File: coman_urdf/urdf/coman.urdf (robot description, URDF)
Before this commit: robot COMAN, 34 links, 33 joints
Joints:
- joint LAnkLat: limit lower=-0.6109 upper=0.6109 effort=30 velocity=3.0 -> lower=-0.6109 upper=0.6109 effort=50 velocity=4.0
- joint LAnkSag: limit lower=-1.2217 upper=1.2217 effort=30 velocity=3.0 -> lower=-1.2217 upper=1.2217 effort=50 velocity=4.0
- joint LElbj: limit lower=-2.3562 upper=0.0 effort=30 velocity=3.0 -> lower=-2.3562 upper=0.0 effort=50 velocity=4.0
- joint LHipLat: limit lower=-0.4363 upper=1.0472 effort=30 velocity=3.0 -> lower=-0.4363 upper=1.0472 effort=50 velocity=4.0
- joint LHipSag: limit lower=-1.9199 upper=0.7854 effort=30 velocity=3.0 -> lower=-1.9199 upper=0.7854 effort=50 velocity=4.0
- joint LHipYaw: limit lower=-0.8727 upper=0.8727 effort=30 velocity=3.0 -> lower=-0.8727 upper=0.8727 effort=50 velocity=4.0
- joint LKneeSag: limit lower=-0.1745 upper=1.9199 effort=30 velocity=3.0 -> lower=-0.1745 upper=1.9199 effort=50 velocity=4.0
- joint LShLat: limit lower=-0.31415 upper=2.094 effort=30 velocity=3.0 -> lower=-0.31415 upper=2.094 effort=50 velocity=4.0
- joint LShSag: limit lower=-3.4034 upper=1.6581 effort=30 velocity=3.0 -> lower=-3.4034 upper=1.6581 effort=50 velocity=4.0
- joint LShYaw: limit lower=-1.5708 upper=1.5708 effort=30 velocity=3.0 -> lower=-1.5708 upper=1.5708 effort=50 velocity=4.0
- joint RAnkLat: limit lower=-0.6109 upper=0.6109 effort=30 velocity=3.0 -> lower=-0.6109 upper=0.6109 effort=50 velocity=4.0
- joint RAnkSag: limit lower=-1.2217 upper=1.2217 effort=30 velocity=3.0 -> lower=-1.2217 upper=1.2217 effort=50 velocity=4.0
- joint RElbj: limit lower=-2.3562 upper=0.0 effort=30 velocity=3.0 -> lower=-2.3562 upper=0.0 effort=50 velocity=4.0
- joint RHipLat: limit lower=-1.0472 upper=0.4363 effort=30 velocity=3.0 -> lower=-1.0472 upper=0.4363 effort=50 velocity=4.0
- joint RHipSag: limit lower=-1.9199 upper=0.7854 effort=30 velocity=3.0 -> lower=-1.9199 upper=0.7854 effort=50 velocity=4.0
- joint RHipYaw: limit lower=-0.8727 upper=0.8727 effort=30 velocity=3.0 -> lower=-0.8727 upper=0.8727 effort=50 velocity=4.0
- joint RKneeSag: limit lower=-0.1745 upper=1.9199 effort=30 velocity=3.0 -> lower=-0.1745 upper=1.9199 effort=50 velocity=4.0
- joint RShLat: limit lower=-2.094 upper=0.31415 effort=30 velocity=3.0 -> lower=-2.094 upper=0.31415 effort=50 velocity=4.0
- joint RShSag: limit lower=-3.4034 upper=1.6581 effort=30 velocity=3.0 -> lower=-3.4034 upper=1.6581 effort=50 velocity=4.0
- joint RShYaw: limit lower=-1.5708 upper=1.5708 effort=30 velocity=3.0 -> lower=-1.5708 upper=1.5708 effort=50 velocity=4.0
- joint WaistLat: limit lower=-0.3491 upper=0.8727 effort=30 velocity=3.0 -> lower=-0.3491 upper=0.8727 effort=50 velocity=4.0
- joint WaistSag: limit lower=-0.5236 upper=0.5235 effort=30 velocity=3.0 -> lower=-0.5236 upper=0.5235 effort=50 velocity=4.0
- joint WaistYaw: limit lower=-1.3963 upper=1.3962 effort=30 velocity=3.0 -> lower=-1.3963 upper=1.3962 effort=50 velocity=4.0

File: coman_urdf/urdf/coman.urdf.xacro (robot description, xacro)
@@ -546,5 +546,5 @@
     <origin xyz="0.020281504 0 0.11912053" rpy="0 0 0" />
     <axis xyz="0.939692608 0 0.3420201433" />
-    <limit velocity="3.0" effort="50" lower="-0.5236" upper="0.5235" />
+    <limit velocity="4.0" effort="50" lower="-0.5236" upper="0.5235" />
   </joint>
   <joint name="WaistLat" type="revolute"> <!-- Wrong name! need to fix this... -->
@@ -553,5 +553,5 @@
     <origin xyz="0 0 0" rpy="0 0 0" />
     <axis xyz="0 1 0" />
-    <limit velocity="3.0" effort="50" lower="-0.3491" upper="0.8727" />
+    <limit velocity="4.0" effort="50" lower="-0.3491" upper="0.8727" />
   </joint>
   <joint name="WaistYaw" type="revolute">
@@ -560,5 +560,5 @@
     <origin xyz="0 0 0.04749999" rpy="0 0 0" />
     <axis xyz="0 0 1" />
-    <limit velocity="3.0" effort="50" lower="-1.3963" upper="1.3962" />
+    <limit velocity="4.0" effort="50" lower="-1.3963" upper="1.3962" />
   </joint>
 <!-- ********************RIGHT LEG******************** -->
@@ -568,5 +568,5 @@
     <origin xyz="0.0 -0.023 0.0" rpy="0 0 0" />
     <axis xyz="0 1 0" />
-    <limit velocity="3.0" effort="50" lower="-1.9199" upper="0.7854" />
+    <limit velocity="4.0" effort="50" lower="-1.9199" upper="0.7854" />
   </joint>
   <joint name="RHipLat" type="revolute">
@@ -575,5 +575,5 @@
     <origin xyz="0.0 -0.0496 0.0" rpy="0 0 0" />
     <axis xyz="1 0 0" />
-    <limit velocity="3.0" effort="50" lower="-1.0472" upper="0.4363" />
+    <limit velocity="4.0" effort="50" lower="-1.0472" upper="0.4363" />
   </joint>
   <joint name="RHipYaw" type="revolute">
@@ -582,5 +582,5 @@
     <origin xyz="0.0 0.0 -0.1024" rpy="0 0 0" />
     <axis xyz="0 0 1" />
-    <limit velocity="3.0" effort="50" lower="-0.8727" upper="0.8727" />
+    <limit velocity="4.0" effort="50" lower="-0.8727" upper="0.8727" />
   </joint>
   <joint name="RKneeSag" type="revolute">
@@ -589,5 +589,5 @@
     <origin xyz="0.0 0.0 -0.1234" rpy="0 0 0" />
     <axis xyz="0 1 0" />
-    <limit velocity="3.0" effort="50" lower="-0.1745" upper="1.9199" />
+    <limit velocity="4.0" effort="50" lower="-0.1745" upper="1.9199" />
   </joint>
   <joint name="RAnkLat" type="revolute">
@@ -596,5 +596,5 @@
     <origin xyz="0.0 0.0 -0.201" rpy="0 0 0" />
     <axis xyz="1 0 0" />
-    <limit velocity="3.0" effort="50" lower="-0.6109" upper="0.6109" />
+    <limit velocity="4.0" effort="50" lower="-0.6109" upper="0.6109" />
   </joint>
   <joint name="RAnkSag" type="revolute">
@@ -603,5 +603,5 @@
     <origin xyz="0.0 0.0 0.0" rpy="0 0 0" />
     <axis xyz="0 1 0" />
-    <limit velocity="3.0" effort="50" lower="-1.2217" upper="1.2217" />
+    <limit velocity="4.0" effort="50" lower="-1.2217" upper="1.2217" />
   </joint>
 <!-- ********************LEFT LEG******************** -->
@@ -611,5 +611,5 @@
     <origin xyz="0.0 0.023 0.0" rpy="0 0 0" />
     <axis xyz="0 1 0" />
-    <limit velocity="3.0" effort="50" lower="-1.9199" upper="0.7854" />
+    <limit velocity="4.0" effort="50" lower="-1.9199" upper="0.7854" />
   </joint>
   <joint name="LHipLat" type="revolute">
@@ -618,5 +618,5 @@
     <origin xyz="0.0 0.0496 0.0" rpy="0 0 0" />
     <axis xyz="1 0 0" />
-    <limit velocity="3.0" effort="50" lower="-0.4363" upper="1.0472" />
+    <limit velocity="4.0" effort="50" lower="-0.4363" upper="1.0472" />
   </joint>
   <joint name="LHipYaw" type="revolute">
@@ -625,5 +625,5 @@
     <origin xyz="0.0 0.0 -0.1024" rpy="0 0 0" />
     <axis xyz="0 0 1" />
-    <limit velocity="3.0" effort="50" lower="-0.8727" upper="0.8727" />
+    <limit velocity="4.0" effort="50" lower="-0.8727" upper="0.8727" />
   </joint>
   <joint name="LKneeSag" type="revolute">
@@ -632,5 +632,5 @@
     <origin xyz="0.0 0.0 -0.1234" rpy="0 0 0" />
     <axis xyz="0 1 0" />
-    <limit velocity="3.0" effort="50" lower="-0.1745" upper="1.9199" />
+    <limit velocity="4.0" effort="50" lower="-0.1745" upper="1.9199" />
   </joint>
   <joint name="LAnkLat" type="revolute">
@@ -639,5 +639,5 @@
     <origin xyz="0.0 0.0 -0.201" rpy="0 0 0" />
     <axis xyz="1 0 0" />
-    <limit velocity="3.0" effort="50" lower="-0.6109" upper="0.6109" />
+    <limit velocity="4.0" effort="50" lower="-0.6109" upper="0.6109" />
   </joint>
   <joint name="LAnkSag" type="revolute">
@@ -646,5 +646,5 @@
     <origin xyz="0.0 0.0 0.0" rpy="0 0 0" />
     <axis xyz="0 1 0" />
-    <limit velocity="3.0" effort="50" lower="-1.2217" upper="1.2217" />
+    <limit velocity="4.0" effort="50" lower="-1.2217" upper="1.2217" />
   </joint>
 <!-- ********************RIGHT ARM******************** -->
@@ -654,5 +654,5 @@
     <origin xyz="-0.014976503999999998 -0.0825 0.15770847" rpy="0 0 0" />
     <axis xyz="0 1 0" />
-    <limit velocity="3.0" effort="50" lower="-3.4034" upper="1.6581" />
+    <limit velocity="4.0" effort="50" lower="-3.4034" upper="1.6581" />
   </joint>
   <joint name="RShLat" type="revolute">
@@ -661,5 +661,5 @@
     <origin xyz="0.0 -0.07329999999999999 0.0" rpy="0 0 0" />
     <axis xyz="1 0 0" />
-    <limit velocity="3.0" effort="50" lower="-2.094" upper="0.31415" />
+    <limit velocity="4.0" effort="50" lower="-2.094" upper="0.31415" />
   </joint>
   <joint name="RShYaw" type="revolute">
@@ -668,5 +668,5 @@
     <origin xyz="0.0 0.0 -0.04480846999999999" rpy="0 0 0" />
     <axis xyz="0 0 1" />
-    <limit velocity="3.0" effort="50" lower="-1.5708" upper="1.5708" />
+    <limit velocity="4.0" effort="50" lower="-1.5708" upper="1.5708" />
   </joint>
   <joint name="RElbj" type="revolute">
@@ -675,5 +675,5 @@
     <origin xyz="0.0 0.0 -0.13519152999999998" rpy="0 0 0" />
     <axis xyz="0 1 0" />
-    <limit velocity="3.0" effort="50" lower="-2.3562" upper="0.0" />
+    <limit velocity="4.0" effort="50" lower="-2.3562" upper="0.0" />
   </joint>
 <!-- ********************LEFT ARM******************** -->
@@ -683,5 +683,5 @@
     <origin xyz="-0.014976503999999998 0.0825 0.15770847" rpy="0 0 0" />
     <axis xyz="0 1 0" />
-    <limit velocity="3.0" effort="50" lower="-3.4034" upper="1.6581" />
+    <limit velocity="4.0" effort="50" lower="-3.4034" upper="1.6581" />
   </joint>
   <joint name="LShLat" type="revolute">
@@ -690,5 +690,5 @@
     <origin xyz="0.0 0.07329999999999999 0.0" rpy="0 0 0" />
     <axis xyz="1 0 0" />
-    <limit velocity="3.0" effort="50" lower="-0.31415" upper="2.094" />
+    <limit velocity="4.0" effort="50" lower="-0.31415" upper="2.094" />
   </joint>
   <joint name="LShYaw" type="revolute">
@@ -697,5 +697,5 @@
     <origin xyz="0.0 0.0 -0.04480846999999999" rpy="0 0 0" />
     <axis xyz="0 0 1" />
-    <limit velocity="3.0" effort="50" lower="-1.5708" upper="1.5708" />
+    <limit velocity="4.0" effort="50" lower="-1.5708" upper="1.5708" />
   </joint>
   <joint name="LElbj" type="revolute">
@@ -704,5 +704,5 @@
     <origin xyz="0.0 0.0 -0.13519152999999998" rpy="0 0 0" />
     <axis xyz="0 1 0" />
-    <limit velocity="3.0" effort="50" lower="-2.3562" upper="0.0" />
+    <limit velocity="4.0" effort="50" lower="-2.3562" upper="0.0" />
   </joint>
 </robot>

Commit message: Solved small bug in coman kinematic chain

File: coman_urdf/urdf/coman.urdf (robot description, URDF)
Before this commit: robot COMAN, 34 links, 33 joints
Links:
- link RElb: geometry collision mesh filename=package://coman_urdf/meshes/collada/simple/simple_asm0001_c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 scale=0.03937 0.03937 0.03937; visual mesh filename=package://coman_urdf/meshes/collada/asm0001_collada_11_prt.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 scale=0.03937 0.03937 0.03937
Joints:
- joint LElbj: origin xyz=0.0 0.0 -0.13519152999999998 rpy=0 0 0 -> xyz=0.015 0.0 -0.13519152999999998 rpy=0 0 0
- joint RElbj: origin xyz=0.0 0.0 -0.13519152999999998 rpy=0 0 0 -> xyz=0.015 0.0 -0.13519152999999998 rpy=0 0 0
- joint l_wrist_joint: origin xyz=0 0 -0.22 rpy=0 0 0 -> xyz=-0.015 0 -0.22 rpy=0 0 0
- joint r_wrist_joint: origin xyz=0 0 -0.22 rpy=0 0 0 -> xyz=-0.015 0 -0.22 rpy=0 0 0

File: coman_urdf/urdf/coman.urdf.xacro (robot description, xacro)
@@ -400,13 +400,13 @@
     </inertial>
     <visual>
-      <origin xyz="-0.005305 0.1558 -0.664329" rpy="0 0 -3.14159265359"/>
+      <origin xyz="-0.020305 -0.1558 -0.664329" rpy="0 0 -3.14159265359"/>
       <geometry name="RElb_visual">
-        <mesh filename="package://coman_urdf/meshes/collada/asm0001_collada_21_prt.dae" scale="0.03937 0.03937 0.03937" />
-      </geometry>
-    </visual>
-    <collision>
-      <origin xyz="-0.005305 0.1558 -0.664329" rpy="0 0 -3.14159265359"/>
+        <mesh filename="package://coman_urdf/meshes/collada/asm0001_collada_11_prt.dae" scale="0.03937 0.03937 0.03937" />
+      </geometry>
+    </visual>
+    <collision>
+      <origin xyz="-0.020305 -0.1558 -0.664329" rpy="0 0 -3.14159265359"/>
       <geometry name="RElb_collision">
-        <mesh filename="package://coman_urdf/meshes/collada/simple/simple_asm0001_collada_21_prt.dae" scale="0.03937 0.03937 0.03937" />
+        <mesh filename="package://coman_urdf/meshes/collada/simple/simple_asm0001_collada_11_prt.dae" scale="0.03937 0.03937 0.03937" />
       </geometry>
     </collision>
@@ -477,5 +477,5 @@
     </inertial>
     <visual>
-      <origin xyz="-0.005305 -0.1558 -0.664329" rpy="0 0 -3.14159265359"/>
+      <origin xyz="-0.020305 -0.1558 -0.664329" rpy="0 0 -3.14159265359"/>
       <geometry name="LElb_visual">
         <mesh filename="package://coman_urdf/meshes/collada/asm0001_collada_11_prt.dae" scale="0.03937 0.03937 0.03937" />
@@ -483,5 +483,5 @@
     </visual>
     <collision>
-      <origin xyz="-0.005305 -0.1558 -0.664329" rpy="0 0 -3.14159265359"/>
+      <origin xyz="-0.020305 -0.1558 -0.664329" rpy="0 0 -3.14159265359"/>
       <geometry name="LElb_collision">
         <mesh filename="package://coman_urdf/meshes/collada/simple/simple_asm0001_collada_11_prt.dae" scale="0.03937 0.03937 0.03937" />
@@ -498,10 +498,10 @@
     <parent link="LElb"/>
     <child link="l_wrist"/>
-    <origin xyz="0 0 -0.22" rpy="0 0 0" />
+    <origin xyz="-0.015 0 -0.22" rpy="0 0 0" />
   </joint>
   <joint name="r_wrist_joint" type="fixed">
     <parent link="RElb"/>
     <child link="r_wrist"/>
-    <origin xyz="0 0 -0.22" rpy="0 0 0" />
+    <origin xyz="-0.015 0 -0.22" rpy="0 0 0" />
   </joint>
   <joint name="l_ankle_joint" type="fixed">
@@ -673,5 +673,5 @@
     <parent link="RShy"/>
     <child link="RElb"/>
-    <origin xyz="0.0 0.0 -0.13519152999999998" rpy="0 0 0" />
+    <origin xyz="0.015 0.0 -0.13519152999999998" rpy="0 0 0" />
     <axis xyz="0 1 0" />
     <limit velocity="4.0" effort="50" lower="-2.3562" upper="0.0" />
@@ -702,5 +702,5 @@
     <parent link="LShy"/>
     <child link="LElb"/>
-    <origin xyz="0.0 0.0 -0.13519152999999998" rpy="0 0 0" />
+    <origin xyz="0.015 0.0 -0.13519152999999998" rpy="0 0 0" />
     <axis xyz="0 1 0" />
     <limit velocity="4.0" effort="50" lower="-2.3562" upper="0.0" />

Commit message: Added acrbon fiber forearm link information (inertia,mass and CoG) and fixed forearm_joint. All dynamic parameters are computed considering the inertia of a cylinder, these parameters, for now, are not precise as in CAD

File: coman_urdf/urdf/coman.urdf (robot description, URDF)
Before this commit: robot COMAN, 34 links, 33 joints
Links:
- added link LForearm, mass 0.263
- added link RForearm, mass 0.263
Joints:
- added joint LForearmPlate: type fixed, parent LElb, child LForearm, origin xyz=-0.015 0.0 -0.05 rpy=0 0 0
- added joint RForearmPlate: type fixed, parent RElb, child RForearm, origin xyz=-0.015 0.0 -0.05 rpy=0 0 0

Commit message: See previous commit

File: coman_urdf/urdf/coman.urdf (robot description, URDF)
Before this commit: robot COMAN, 36 links, 35 joints
Links:
- removed link LForearm
- removed link RForearm
- link LElb: geometry collision mesh filename=package://coman_urdf/meshes/collada/simple/forearms/elbow.d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 scale=1.0 1.0 1.0; visual mesh filename=package://coman_urdf/meshes/collada/forearms/elbow.dae scale=1.0 1.0 1.0
- link RElb: geometry collision mesh filename=package://coman_urdf/meshes/collada/simple/forearms/elbow.d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 scale=1.0 1.0 1.0; visual mesh filename=package://coman_urdf/meshes/collada/forearms/elbow.dae scale=1.0 1.0 1.0
Joints:
- removed joint LForearmPlate
- removed joint RForearmPlate

File: coman_urdf/urdf/coman.urdf.xacro (robot description, xacro)
@@ -460,4 +460,23 @@
     </inertial>
     <visual>
+      <origin xyz="0 0 0" rpy="-1.570796326795 1.570796326795 0"/>
+      <geometry name="RElb_visual">
+        <mesh filename="package://coman_urdf/meshes/collada/forearms/elbow.dae" scale="1.0 1.0 1.0" />
+      </geometry>
+    </visual>
+    <collision>
+      <origin xyz="0 0 0" rpy="-1.570796326795 1.570796326795 0"/>
+      <geometry name="RElb_collision">
+        <mesh filename="package://coman_urdf/meshes/collada/simple/forearms/elbow.dae" scale="1.0 1.0 1.0" />
+      </geometry>
+    </collision>
+  </link>
+  <!--link name ="RElb">
+    <inertial>
+      <origin xyz="-6.5553403E-4 -9.3464748E-4 -9.3101289E-4" rpy="0 0 0"/>
+      <mass value="0.63306933"/>
+      <inertia ixx="2.2599075E-4"  ixy="-2.6376470E-7"  ixz="-9.8007285E-6" iyy="2.7781302E-4" iyz="-2.0435288E-6" izz="2.1878992E-4" />
+    </inertial>
+    <visual>
       <origin xyz="-0.020305 -0.1558 -0.664329" rpy="0 0 -3.14159265359"/>
       <geometry name="RElb_visual">
@@ -478,5 +497,5 @@
       <inertia ixx="6.913E-4"  ixy="0.0"  ixz="0.0" iyy="6.913E-4" iyz="0.0" izz="4.0425E-5" />
     </inertial>
-  </link>
+  </link-->
 <!-- ********************LEFT ARM******************** -->
   <link name ="LShp">
@@ -541,4 +560,23 @@
       <origin xyz="-6.5553403E-4 9.3464748E-4 -9.3101289E-4" rpy="0 0 0"/>
       <mass value="0.63306933"/>
+      <inertia ixx="2.2599075E-4"  ixy="2.6376470E-7"  ixz="-9.8007285E-6" iyy="2.7781302E-4" iyz="2.0435288E-6" izz="2.1878992E-4" />
+    </inertial>
+    <visual>
+      <origin xyz="0 0 0" rpy="-1.570796326795 1.570796326795 0"/>
+      <geometry name="LElb_visual">
+        <mesh filename="package://coman_urdf/meshes/collada/forearms/elbow.dae" scale="1.0 1.0 1.0" />
+      </geometry>
+    </visual>
+    <collision>
+      <origin xyz="0 0 0" rpy="-1.570796326795 1.570796326795 0"/>
+      <geometry name="LElb_collision">
+        <mesh filename="package://coman_urdf/meshes/collada/simple/forearms/elbow.dae" scale="1.0 1.0 1.0" />
+      </geometry>
+    </collision>
+  </link>
+  <!--link name ="LElb">
+    <inertial>
+      <origin xyz="-6.5553403E-4 9.3464748E-4 -9.3101289E-4" rpy="0 0 0"/>
+      <mass value="0.63306933"/>
       <inertia ixx="2.2599075E-4"  ixy="2.637647E-7"  ixz="-9.8007285E-6" iyy="2.7781302E-4" iyz="2.0435288E-6" izz="2.1878992E-4" />
     </inertial>
@@ -562,5 +600,5 @@
       <inertia ixx="6.913E-4"  ixy="0.0"  ixz="0.0" iyy="6.913E-4" iyz="0.0" izz="4.0425E-5" />
     </inertial>
-  </link>
+  </link-->
 <!-- ********************JOINTS******************** -->
   <joint name="base_joint" type="fixed">
@@ -811,9 +849,9 @@
     <dynamics friction="0" damping="3.0"/>
   </joint>
-  <joint name="RForearmPlate" type="fixed">
+  <!--joint name="RForearmPlate" type="fixed">
     <parent link="RElb"/>
     <child link="RForearm"/>
     <origin xyz="-0.015 0.0 -0.05" rpy="0 0 0"/>
-  </joint>
+  </joint-->
 <!-- ********************LEFT ARM******************** -->
   <joint name="LShSag" type="revolute">
@@ -849,8 +887,8 @@
     <dynamics friction="0" damping="3.0"/>
   </joint>
-  <joint name="LForearmPlate" type="fixed">
+  <!--joint name="LForearmPlate" type="fixed">
     <parent link="LElb"/>
     <child link="LForearm"/>
     <origin xyz="-0.015 0.0 -0.05" rpy="0 0 0"/>
-  </joint>
+  </joint-->
 </robot>

Commit message: Added forearm with fixed joint. Next step is to make that joint rotative.

File: coman_urdf/urdf/coman.urdf (robot description, URDF)
Before this commit: robot COMAN, 34 links, 33 joints
Links:
- added link LForearm, mass 0.263; collision mesh filename=package://coman_urdf/meshes/collada/simple/forearms/forearm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 scale=1.0 1.0 1.0; visual mesh filename=package://coman_urdf/meshes/collada/forearms/forearm.dae scale=1.0 1.0 1.0
- added link RForearm, mass 0.263; collision mesh filename=package://coman_urdf/meshes/collada/simple/forearms/forearm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 scale=1.0 1.0 1.0; visual mesh filename=package://coman_urdf/meshes/collada/forearms/forearm.dae scale=1.0 1.0 1.0
Joints:
- added joint LForearmPlate: type fixed, parent LElb, child LForearm, origin xyz=-0.015 0.0 -0.05 rpy=0 0 0
- added joint RForearmPlate: type fixed, parent RElb, child RForearm, origin xyz=-0.015 0.0 -0.05 rpy=0 0 0

File: coman_urdf/urdf/coman.urdf.xacro (robot description, xacro)
@@ -472,4 +472,24 @@
     </collision>
   </link>
+  <!-- ## WRONG NUMBERS FOR INERTIAL!!! FIX THEM!! ## -->
+  <link name ="RForearm">
+    <inertial>
+      <origin xyz="0 0 -0.085" rpy="0 0 0"/>
+      <mass value="0.263"/>
+      <inertia ixx="6.913E-4"  ixy="0.0"  ixz="0.0" iyy="6.913E-4" iyz="0.0" izz="4.0425E-5" />
+    </inertial>
+    <visual>
+      <origin xyz="0 0 0.015" rpy="0 3.14159265359 1.570796326795"/>
+      <geometry name="RForearm_visual">
+        <mesh filename="package://coman_urdf/meshes/collada/forearms/forearm.dae" scale="1.0 1.0 1.0" />
+      </geometry>
+    </visual>
+    <collision>
+      <origin xyz="0 0 0.015" rpy="0 3.14159265359 1.570796326795"/>
+      <geometry name="RForearm_collision">
+        <mesh filename="package://coman_urdf/meshes/collada/simple/forearms/forearm.dae" scale="1.0 1.0 1.0" />
+      </geometry>
+    </collision>
+  </link>
   <!--link name ="RElb">
     <inertial>
@@ -572,4 +592,24 @@
       <geometry name="LElb_collision">
         <mesh filename="package://coman_urdf/meshes/collada/simple/forearms/elbow.dae" scale="1.0 1.0 1.0" />
+      </geometry>
+    </collision>
+  </link>
+  <!-- ## WRONG NUMBERS FOR INERTIAL!!! FIX THEM!! ## -->
+  <link name ="LForearm">
+    <inertial>
+      <origin xyz="0 0 -0.085" rpy="0 0 0"/>
+      <mass value="0.263"/>
+      <inertia ixx="6.913E-4"  ixy="0.0"  ixz="0.0" iyy="6.913E-4" iyz="0.0" izz="4.0425E-5" />
+    </inertial>
+    <visual>
+      <origin xyz="0 0 0.015" rpy="0 3.14159265359 1.570796326795"/>
+      <geometry name="LForearm_visual">
+        <mesh filename="package://coman_urdf/meshes/collada/forearms/forearm.dae" scale="1.0 1.0 1.0" />
+      </geometry>
+    </visual>
+    <collision>
+      <origin xyz="0 0 0.015" rpy="0 3.14159265359 1.570796326795"/>
+      <geometry name="LForearm_collision">
+        <mesh filename="package://coman_urdf/meshes/collada/simple/forearms/forearm.dae" scale="1.0 1.0 1.0" />
       </geometry>
     </collision>
@@ -849,4 +889,9 @@
     <dynamics friction="0" damping="3.0"/>
   </joint>
+  <joint name="RForearmPlate" type="fixed">
+    <parent link="RElb"/>
+    <child link="RForearm"/>
+    <origin xyz="-0.015 0.0 -0.05" rpy="0 0 0"/>
+  </joint>
   <!--joint name="RForearmPlate" type="fixed">
     <parent link="RElb"/>
@@ -887,4 +932,9 @@
     <dynamics friction="0" damping="3.0"/>
   </joint>
+    <joint name="LForearmPlate" type="fixed">
+    <parent link="LElb"/>
+    <child link="LForearm"/>
+    <origin xyz="-0.015 0.0 -0.05" rpy="0 0 0"/>
+  </joint>
   <!--joint name="LForearmPlate" type="fixed">
     <parent link="LElb"/>
