Commit message: Added revolute YAW joint to move the forearm. Joint limits are +/- 90 deg (check if it is true). Tried in RVIZ.

File: coman_urdf/urdf/coman.urdf (robot description, URDF)
Before this commit: robot COMAN, 36 links, 35 joints
Joints:
- joint LForearmPlate: axis (none) -> 0 0 1; limit (none) -> lower=-1.5708 upper=1.5708 effort=50 velocity=4.0; type fixed -> revolute
- joint RForearmPlate: axis (none) -> 0 0 1; limit (none) -> lower=-1.5708 upper=1.5708 effort=50 velocity=4.0; type fixed -> revolute

File: coman_urdf/urdf/coman.urdf.xacro (robot description, xacro)
@@ -889,8 +889,11 @@
     <dynamics friction="0" damping="3.0"/>
   </joint>
-  <joint name="RForearmPlate" type="fixed">
+  <joint name="RForearmPlate" type="revolute">
     <parent link="RElb"/>
     <child link="RForearm"/>
     <origin xyz="-0.015 0.0 -0.05" rpy="0 0 0"/>
+    <axis xyz="0 0 1" />
+    <limit velocity="4.0" effort="50" lower="-1.5708" upper="1.5708" />
+    <dynamics friction="0" damping="3.0"/>
   </joint>
   <!--joint name="RForearmPlate" type="fixed">
@@ -932,8 +935,11 @@
     <dynamics friction="0" damping="3.0"/>
   </joint>
-    <joint name="LForearmPlate" type="fixed">
+    <joint name="LForearmPlate" type="revolute">
     <parent link="LElb"/>
     <child link="LForearm"/>
     <origin xyz="-0.015 0.0 -0.05" rpy="0 0 0"/>
+    <axis xyz="0 0 1" />
+    <limit velocity="4.0" effort="50" lower="-1.5708" upper="1.5708" />
+    <dynamics friction="0" damping="3.0"/>
   </joint>
   <!--joint name="LForearmPlate" type="fixed">

Commit message: Added dynamic in joint forearm. With actual inertial parameter the model explodes if damping is more than the one set

File: coman_urdf/urdf/coman.urdf (robot description, URDF)
Before this commit: robot COMAN, 36 links, 35 joints
Joints:
- joint LForearmPlate: origin xyz=-0.015 0.0 -0.05 rpy=0 0 0 -> xyz=-0.015 0.0 -0.051 rpy=0 0 0
- joint RForearmPlate: origin xyz=-0.015 0.0 -0.05 rpy=0 0 0 -> xyz=-0.015 0.0 -0.051 rpy=0 0 0

File: coman_urdf/urdf/coman.urdf.xacro (robot description, xacro)
@@ -892,8 +892,8 @@
     <parent link="RElb"/>
     <child link="RForearm"/>
-    <origin xyz="-0.015 0.0 -0.05" rpy="0 0 0"/>
+    <origin xyz="-0.015 0.0 -0.051" rpy="0 0 0"/>
     <axis xyz="0 0 1" />
     <limit velocity="4.0" effort="50" lower="-1.5708" upper="1.5708" />
-    <dynamics friction="0" damping="3.0"/>
+    <dynamics friction="0" damping="0.03"/>
   </joint>
   <!--joint name="RForearmPlate" type="fixed">
@@ -935,11 +935,11 @@
     <dynamics friction="0" damping="3.0"/>
   </joint>
-    <joint name="LForearmPlate" type="revolute">
+  <joint name="LForearmPlate" type="revolute">
     <parent link="LElb"/>
     <child link="LForearm"/>
-    <origin xyz="-0.015 0.0 -0.05" rpy="0 0 0"/>
+    <origin xyz="-0.015 0.0 -0.051" rpy="0 0 0"/>
     <axis xyz="0 0 1" />
     <limit velocity="4.0" effort="50" lower="-1.5708" upper="1.5708" />
-    <dynamics friction="0" damping="3.0"/>
+    <dynamics friction="0" damping="0.03"/>
   </joint>
   <!--joint name="LForearmPlate" type="fixed">

Commit message: Fixed bug for l_ankle/r_ankle

File: coman_urdf/urdf/coman.urdf (robot description, URDF)
Before this commit: robot COMAN, 36 links, 35 joints
Joints:
- joint l_ankle_joint: parent LHipMot -> LFoot
- joint r_ankle_joint: parent RHipMot -> RFoot

File: coman_urdf/urdf/coman.urdf.xacro (robot description, xacro)
@@ -658,10 +658,10 @@
   </joint>
   <joint name="l_ankle_joint" type="fixed">
-    <parent link="LHipMot"/>
+    <parent link="LFoot"/>
     <child link="l_ankle"/>
     <origin xyz="0 0 0" rpy="0 0 0" />
   </joint>
   <joint name="r_ankle_joint" type="fixed">
-    <parent link="RHipMot"/>
+    <parent link="RFoot"/>
     <child link="r_ankle"/>
     <origin xyz="0 0 0" rpy="0 0 0" />
