Commit message: First commit to include full forearm and a cube representing the hand.

File: coman_urdf/urdf/coman.urdf (robot description, URDF)
Before this commit: robot COMAN, 36 links, 35 joints
Links:
- added link LWrMot2, mass 0.26070556; collision mesh filename=package://coman_urdf/meshes/collada/simple/forearms/simple_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 scale=0.001 0.001 0.001; visual mesh filename=package://coman_urdf/meshes/collada/forearms/fa_asm_3_right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 scale=0.001 0.001 0.001
- added link LWrMot3, mass 0.054007518; collision mesh filename=package://coman_urdf/meshes/collada/simple/forearms/simple_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 scale=0.001 0.001 0.001; visual mesh filename=package://coman_urdf/meshes/collada/forearms/fa_hand_interf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 scale=0.001 0.001 0.001
- added link RWrMot2, mass 0.26070556; collision mesh filename=package://coman_urdf/meshes/collada/simple/forearms/simple_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 scale=0.001 0.001 0.001; visual mesh filename=package://coman_urdf/meshes/collada/forearms/fa_asm_3_right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 scale=0.001 0.001 0.001
- added link RWrMot3, mass 0.054007518; collision mesh filename=package://coman_urdf/meshes/collada/simple/forearms/simple_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 scale=0.001 0.001 0.001; visual mesh filename=package://coman_urdf/meshes/collada/forearms/fa_hand_interf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 scale=0.001 0.001 0.001
- link LForearm: mass 0.263 -> 0.93351655; geometry collision mesh filename=package://coman_urdf/meshes/collada/simple/forearms/forearm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 scale=1.0 1.0 1.0; visual mesh filename=package://coman_urdf/meshes/collada/forearms/forearm.dae scale=0.001 0.001 0.001
- link RForearm: mass 0.263 -> 0.93351655; geometry collision mesh filename=package://coman_urdf/meshes/collada/simple/forearms/forearm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 scale=1.0 1.0 1.0; visual mesh filename=package://coman_urdf/meshes/collada/forearms/forearm.dae scale=0.001 0.001 0.001
Joints:
- added joint LWrj1: type revolute, parent LForearm, child LWrMot2, origin xyz=0 0 -0.14368 rpy=0 0 0, axis 0 1 0, limit lower=-0.524 upper=0.524 effort=50 velocity=4.0
- added joint LWrj2: type revolute, parent LWrMot2, child LWrMot3, origin xyz=0 0 0.0 rpy=0 0 0, axis 1 0 0, limit lower=-0.785375 upper=1.395 effort=50 velocity=4.0
- added joint RWrj1: type revolute, parent RForearm, child RWrMot2, origin xyz=0 0 -0.14368 rpy=0 0 0, axis 0 1 0, limit lower=-0.524 upper=0.524 effort=50 velocity=4.0
- added joint RWrj2: type revolute, parent RWrMot2, child RWrMot3, origin xyz=0 0 0.0 rpy=0 0 0, axis 1 0 0, limit lower=-1.395 upper=0.785375 effort=50 velocity=4.0
- joint l_wrist_joint: origin xyz=-0.015 0 -0.22 rpy=0 0 0 -> xyz=0 0 0 rpy=0 0 0; parent LElb -> LWrMot3
- joint r_wrist_joint: origin xyz=-0.015 0 -0.22 rpy=0 0 0 -> xyz=0 0 0 rpy=0 0 0; parent RElb -> RWrMot3

File: coman_urdf/urdf/coman.urdf.xacro (robot description, xacro)
@@ -473,4 +473,43 @@
   </link>
   <!-- ## WRONG NUMBERS FOR INERTIAL!!! FIX THEM!! ## -->
+  <!-- In ROBOTRAN this link is named RFArm -->
+  <link name ="RForearm">
+    <inertial>
+      <origin xyz="0 0 -0.085" rpy="0 0 0"/>
+      <mass value="0.93351655"/>
+      <inertia ixx="0.001"  ixy="0.0"  ixz="0.0" iyy="0.001" iyz="0.0" izz="0.001" />
+    </inertial>
+    <visual>
+      <origin xyz="0 0 0.015" rpy="-1.570796326795 0 1.570796326795"/>
+      <geometry name="RForearm_visual">
+        <mesh filename="package://coman_urdf/meshes/collada/forearms/forearm.dae" scale="0.001 0.001 0.001" />
+      </geometry>
+    </visual>
+    <collision>
+      <origin xyz="0 0 0.015" rpy="0 3.14159265359 1.570796326795"/>
+      <geometry name="RForearm_collision">
+        <mesh filename="package://coman_urdf/meshes/collada/simple/forearms/forearm.dae" scale="1.0 1.0 1.0" />
+      </geometry>
+    </collision>
+  </link>
+  <!--link name ="RElb">
+    <inertial>
+      <origin xyz="-6.5553403E-4 -9.3464748E-4 -9.3101289E-4" rpy="0 0 0"/>
+      <mass value="0.63306933"/>
+      <inertia ixx="2.2599075E-4"  ixy="-2.6376470E-7"  ixz="-9.8007285E-6" iyy="2.7781302E-4" iyz="-2.0435288E-6" izz="2.1878992E-4" />
+    </inertial>
+    <visual>
+      <origin xyz="-0.020305 -0.1558 -0.664329" rpy="0 0 -3.14159265359"/>
+      <geometry name="RElb_visual">
+        <mesh filename="package://coman_urdf/meshes/collada/asm0001_collada_11_prt.dae" scale="0.03937 0.03937 0.03937" />
+      </geometry>
+    </visual>
+    <collision>
+      <origin xyz="-0.020305 -0.1558 -0.664329" rpy="0 0 -3.14159265359"/>
+      <geometry name="RElb_collision">
+        <mesh filename="package://coman_urdf/meshes/collada/simple/simple_asm0001_collada_11_prt.dae" scale="0.03937 0.03937 0.03937" />
+      </geometry>
+    </collision>
+  </link>
   <link name ="RForearm">
     <inertial>
@@ -479,26 +518,154 @@
       <inertia ixx="6.913E-4"  ixy="0.0"  ixz="0.0" iyy="6.913E-4" iyz="0.0" izz="4.0425E-5" />
     </inertial>
-    <visual>
+  </link-->
+  <!-- ## WRONG NUMBERS FOR INERTIAL!!! FIX THEM!! ## -->
+  <!-- Here I have used the inertia of a full cylinder with r = 0.02 [m] and h = 0.07 [m] -->
+  <link name="RWrMot2">
+    <inertial>
+      <origin xyz="0 0 0" rpy="0 0 0"/>
+      <mass value="0.26070556"/>
+      <inertia ixx="0.000132"  ixy="0"  ixz="0" iyy="0.000132" iyz="0" izz="5.213E-5" />
+    </inertial>
+    <visual>
+      <origin xyz="0.025 0 0" rpy="0 1.570796326795 3.14159265359"/>
+      <geometry name="RWrMot2_visual">
+        <mesh filename="package://coman_urdf/meshes/collada/forearms/fa_asm_3_right_sw0001.dae" scale="0.001 0.001 0.001" />
+      </geometry>
+    </visual>
+    <collision>
+      <origin xyz="0.025 0 0" rpy="0 1.570796326795 3.14159265359"/>
+      <geometry name="RWrMot2_collision">
+        <mesh filename="package://coman_urdf/meshes/collada/simple/forearms/simple_fa_asm_3_right_sw0001.dae" scale="0.001 0.001 0.001" />
+      </geometry>
+    </collision>
+  </link>
+  <!-- ## WRONG NUMBERS FOR INERTIAL!!! FIX THEM!! ## -->
+  <!-- Here I have used the inertia of a concave cylinder with r = 0.02 [m] -->
+  <link name="RWrMot3">
+    <inertial>
+      <origin xyz="0 0 0" rpy="0 0 0"/>
+      <mass value="0.054007518"/>
+      <inertia ixx="2.16E-5"  ixy="0"  ixz="0" iyy="2.16E-5" iyz="0" izz="2.16E-5" />
+    </inertial>
+    <visual>
+      <origin xyz="0.025 -0.012 -0.02" rpy="0 3.14159265359 1.570796326795"/>
+      <geometry name="RWrMot3_visual">
+        <mesh filename="package://coman_urdf/meshes/collada/forearms/fa_hand_interface_rig_sw0001.dae" scale="0.001 0.001 0.001" />
+      </geometry>
+    </visual>
+    <collision>
+      <origin xyz="0.025 -0.012 -0.02" rpy="0 3.14159265359 1.570796326795"/>
+      <geometry name="RWrMot3_collision">
+        <mesh filename="package://coman_urdf/meshes/collada/simple/forearms/simple_fa_hand_interface_rig_sw0001.dae" scale="0.001 0.001 0.001" />
+      </geometry>
+    </collision>
+  </link>
+<!-- ********************LEFT ARM******************** -->
+  <link name ="LShp">
+    <inertial>
+      <origin xyz="0.0099500565 0.038682024 1.6446924E-4" rpy="0 0 0"/>
+      <mass value="0.56782202"/>
+      <inertia ixx="7.8337456E-4"  ixy="-1.9035768E-4"  ixz="-3.0037676E-6" iyy="6.3399921E-4" iyz="-4.3840774E-6" izz="0.001008054" />
+    </inertial>
+    <visual>
+      <origin xyz="-0.005305 -0.0825 -0.844329" rpy="0 0 -3.14159265359"/>
+      <geometry name="LShp_visual">
+        <mesh filename="package://coman_urdf/meshes/collada/asm0001_collada_14_prt.dae" scale="0.03937 0.03937 0.03937" />
+      </geometry>
+    </visual>
+    <collision>
+      <origin xyz="-0.005305 -0.0825 -0.844329" rpy="0 0 -3.14159265359"/>
+      <geometry name="LShp_collision">
+        <mesh filename="package://coman_urdf/meshes/collada/simple/simple_asm0001_collada_14_prt.dae" scale="0.03937 0.03937 0.03937" />
+      </geometry>
+    </collision>
+  </link>
+  <link name ="LShr">
+    <inertial>
+      <origin xyz="-0.0038936743 -2.2022151E-6 -0.0048616005" rpy="0 0 0"/>
+      <mass value="0.77683752"/>
+      <inertia ixx="4.5812904E-4"  ixy="2.4111086E-7"  ixz="9.2521185E-6" iyy="4.3089204E-4" iyz="4.721695E-7" izz="3.4174855E-4" />
+    </inertial>
+    <visual>
+      <origin xyz="-0.005305 -0.1558 -0.844329" rpy="0 0 -3.14159265359"/>
+      <geometry name="LShr_visual">
+        <mesh filename="package://coman_urdf/meshes/collada/asm0001_collada_13_prt.dae" scale="0.03937 0.03937 0.03937" />
+      </geometry>
+    </visual>
+    <collision>
+      <origin xyz="-0.005305 -0.1558 -0.844329" rpy="0 0 -3.14159265359"/>
+      <geometry name="LShr_collision">
+        <mesh filename="package://coman_urdf/meshes/collada/simple/simple_asm0001_collada_13_prt.dae" scale="0.03937 0.03937 0.03937" />
+      </geometry>
+    </collision>
+  </link>
+  <link name ="LShy">
+    <inertial>
+      <origin xyz="0.0022714213 0.0071091517 -0.057455221" rpy="0 0 0"/>
+      <mass value="1.0462304"/>
+      <inertia ixx="0.0030934574"  ixy="-6.6702837E-5"  ixz="3.0222291E-4" iyy="0.0029181573" iyz="5.2663661E-4" izz="8.0830389E-4" />
+    </inertial>
+    <visual>
+      <origin xyz="-0.005305 -0.1558 -0.79952053" rpy="0 0 -3.14159265359"/>
+      <geometry name="LShy_visual">
+        <mesh filename="package://coman_urdf/meshes/collada/asm0001_collada_12_prt.dae" scale="0.03937 0.03937 0.03937" />
+      </geometry>
+    </visual>
+    <collision>
+      <origin xyz="-0.005305 -0.1558 -0.79952053" rpy="0 0 -3.14159265359"/>
+      <geometry name="LShy_collision">
+        <mesh filename="package://coman_urdf/meshes/collada/simple/simple_asm0001_collada_12_prt.dae" scale="0.03937 0.03937 0.03937" />
+      </geometry>
+    </collision>
+  </link>
+  <link name ="LElb">
+    <inertial>
+      <origin xyz="-6.5553403E-4 9.3464748E-4 -9.3101289E-4" rpy="0 0 0"/>
+      <mass value="0.63306933"/>
+      <inertia ixx="2.2599075E-4"  ixy="2.6376470E-7"  ixz="-9.8007285E-6" iyy="2.7781302E-4" iyz="2.0435288E-6" izz="2.1878992E-4" />
+    </inertial>
+    <visual>
+      <origin xyz="0 0 0" rpy="-1.570796326795 1.570796326795 0"/>
+      <geometry name="LElb_visual">
+        <mesh filename="package://coman_urdf/meshes/collada/forearms/elbow.dae" scale="1.0 1.0 1.0" />
+      </geometry>
+    </visual>
+    <collision>
+      <origin xyz="0 0 0" rpy="-1.570796326795 1.570796326795 0"/>
+      <geometry name="LElb_collision">
+        <mesh filename="package://coman_urdf/meshes/collada/simple/forearms/elbow.dae" scale="1.0 1.0 1.0" />
+      </geometry>
+    </collision>
+  </link>
+  <!-- ## WRONG NUMBERS FOR INERTIAL!!! FIX THEM!! ## -->
+  <!-- In ROBOTRAN this link is named LFARM -->
+  <link name ="LForearm">
+    <inertial>
+      <origin xyz="0 0 -0.085" rpy="0 0 0"/>
+      <mass value="0.93351655"/>
+      <inertia ixx="0.001"  ixy="0.0"  ixz="0.0" iyy="0.001" iyz="0.0" izz="0.001" />
+    </inertial>
+    <visual>
+      <origin xyz="0 0 0.015" rpy="-1.570796326795 0 1.570796326795"/>
+      <geometry name="LForearm_visual">
+        <mesh filename="package://coman_urdf/meshes/collada/forearms/forearm.dae" scale="0.001 0.001 0.001" />
+      </geometry>
+    </visual>
+    <collision>
       <origin xyz="0 0 0.015" rpy="0 3.14159265359 1.570796326795"/>
-      <geometry name="RForearm_visual">
-        <mesh filename="package://coman_urdf/meshes/collada/forearms/forearm.dae" scale="1.0 1.0 1.0" />
-      </geometry>
-    </visual>
-    <collision>
-      <origin xyz="0 0 0.015" rpy="0 3.14159265359 1.570796326795"/>
-      <geometry name="RForearm_collision">
+      <geometry name="LForearm_collision">
         <mesh filename="package://coman_urdf/meshes/collada/simple/forearms/forearm.dae" scale="1.0 1.0 1.0" />
       </geometry>
     </collision>
   </link>
-  <!--link name ="RElb">
-    <inertial>
-      <origin xyz="-6.5553403E-4 -9.3464748E-4 -9.3101289E-4" rpy="0 0 0"/>
+  <!--link name ="LElb">
+    <inertial>
+      <origin xyz="-6.5553403E-4 9.3464748E-4 -9.3101289E-4" rpy="0 0 0"/>
       <mass value="0.63306933"/>
-      <inertia ixx="2.2599075E-4"  ixy="-2.6376470E-7"  ixz="-9.8007285E-6" iyy="2.7781302E-4" iyz="-2.0435288E-6" izz="2.1878992E-4" />
+      <inertia ixx="2.2599075E-4"  ixy="2.637647E-7"  ixz="-9.8007285E-6" iyy="2.7781302E-4" iyz="2.0435288E-6" izz="2.1878992E-4" />
     </inertial>
     <visual>
       <origin xyz="-0.020305 -0.1558 -0.664329" rpy="0 0 -3.14159265359"/>
-      <geometry name="RElb_visual">
+      <geometry name="LElb_visual">
         <mesh filename="package://coman_urdf/meshes/collada/asm0001_collada_11_prt.dae" scale="0.03937 0.03937 0.03937" />
       </geometry>
@@ -506,10 +673,10 @@
     <collision>
       <origin xyz="-0.020305 -0.1558 -0.664329" rpy="0 0 -3.14159265359"/>
-      <geometry name="RElb_collision">
+      <geometry name="LElb_collision">
         <mesh filename="package://coman_urdf/meshes/collada/simple/simple_asm0001_collada_11_prt.dae" scale="0.03937 0.03937 0.03937" />
       </geometry>
     </collision>
   </link>
-  <link name ="RForearm">
+  <link name ="LForearm">
     <inertial>
       <origin xyz="0 0 -0.085" rpy="0 0 0"/>
@@ -518,127 +685,46 @@
     </inertial>
   </link-->
-<!-- ********************LEFT ARM******************** -->
-  <link name ="LShp">
-    <inertial>
-      <origin xyz="0.0099500565 0.038682024 1.6446924E-4" rpy="0 0 0"/>
-      <mass value="0.56782202"/>
-      <inertia ixx="7.8337456E-4"  ixy="-1.9035768E-4"  ixz="-3.0037676E-6" iyy="6.3399921E-4" iyz="-4.3840774E-6" izz="0.001008054" />
-    </inertial>
-    <visual>
-      <origin xyz="-0.005305 -0.0825 -0.844329" rpy="0 0 -3.14159265359"/>
-      <geometry name="LShp_visual">
-        <mesh filename="package://coman_urdf/meshes/collada/asm0001_collada_14_prt.dae" scale="0.03937 0.03937 0.03937" />
-      </geometry>
-    </visual>
-    <collision>
-      <origin xyz="-0.005305 -0.0825 -0.844329" rpy="0 0 -3.14159265359"/>
-      <geometry name="LShp_collision">
-        <mesh filename="package://coman_urdf/meshes/collada/simple/simple_asm0001_collada_14_prt.dae" scale="0.03937 0.03937 0.03937" />
-      </geometry>
-    </collision>
-  </link>
-  <link name ="LShr">
-    <inertial>
-      <origin xyz="-0.0038936743 -2.2022151E-6 -0.0048616005" rpy="0 0 0"/>
-      <mass value="0.77683752"/>
-      <inertia ixx="4.5812904E-4"  ixy="2.4111086E-7"  ixz="9.2521185E-6" iyy="4.3089204E-4" iyz="4.721695E-7" izz="3.4174855E-4" />
-    </inertial>
-    <visual>
-      <origin xyz="-0.005305 -0.1558 -0.844329" rpy="0 0 -3.14159265359"/>
-      <geometry name="LShr_visual">
-        <mesh filename="package://coman_urdf/meshes/collada/asm0001_collada_13_prt.dae" scale="0.03937 0.03937 0.03937" />
-      </geometry>
-    </visual>
-    <collision>
-      <origin xyz="-0.005305 -0.1558 -0.844329" rpy="0 0 -3.14159265359"/>
-      <geometry name="LShr_collision">
-        <mesh filename="package://coman_urdf/meshes/collada/simple/simple_asm0001_collada_13_prt.dae" scale="0.03937 0.03937 0.03937" />
-      </geometry>
-    </collision>
-  </link>
-  <link name ="LShy">
-    <inertial>
-      <origin xyz="0.0022714213 0.0071091517 -0.057455221" rpy="0 0 0"/>
-      <mass value="1.0462304"/>
-      <inertia ixx="0.0030934574"  ixy="-6.6702837E-5"  ixz="3.0222291E-4" iyy="0.0029181573" iyz="5.2663661E-4" izz="8.0830389E-4" />
-    </inertial>
-    <visual>
-      <origin xyz="-0.005305 -0.1558 -0.79952053" rpy="0 0 -3.14159265359"/>
-      <geometry name="LShy_visual">
-        <mesh filename="package://coman_urdf/meshes/collada/asm0001_collada_12_prt.dae" scale="0.03937 0.03937 0.03937" />
-      </geometry>
-    </visual>
-    <collision>
-      <origin xyz="-0.005305 -0.1558 -0.79952053" rpy="0 0 -3.14159265359"/>
-      <geometry name="LShy_collision">
-        <mesh filename="package://coman_urdf/meshes/collada/simple/simple_asm0001_collada_12_prt.dae" scale="0.03937 0.03937 0.03937" />
-      </geometry>
-    </collision>
-  </link>
-  <link name ="LElb">
-    <inertial>
-      <origin xyz="-6.5553403E-4 9.3464748E-4 -9.3101289E-4" rpy="0 0 0"/>
-      <mass value="0.63306933"/>
-      <inertia ixx="2.2599075E-4"  ixy="2.6376470E-7"  ixz="-9.8007285E-6" iyy="2.7781302E-4" iyz="2.0435288E-6" izz="2.1878992E-4" />
-    </inertial>
-    <visual>
-      <origin xyz="0 0 0" rpy="-1.570796326795 1.570796326795 0"/>
-      <geometry name="LElb_visual">
-        <mesh filename="package://coman_urdf/meshes/collada/forearms/elbow.dae" scale="1.0 1.0 1.0" />
-      </geometry>
-    </visual>
-    <collision>
-      <origin xyz="0 0 0" rpy="-1.570796326795 1.570796326795 0"/>
-      <geometry name="LElb_collision">
-        <mesh filename="package://coman_urdf/meshes/collada/simple/forearms/elbow.dae" scale="1.0 1.0 1.0" />
-      </geometry>
-    </collision>
-  </link>
   <!-- ## WRONG NUMBERS FOR INERTIAL!!! FIX THEM!! ## -->
-  <link name ="LForearm">
-    <inertial>
-      <origin xyz="0 0 -0.085" rpy="0 0 0"/>
-      <mass value="0.263"/>
-      <inertia ixx="6.913E-4"  ixy="0.0"  ixz="0.0" iyy="6.913E-4" iyz="0.0" izz="4.0425E-5" />
-    </inertial>
-    <visual>
-      <origin xyz="0 0 0.015" rpy="0 3.14159265359 1.570796326795"/>
-      <geometry name="LForearm_visual">
-        <mesh filename="package://coman_urdf/meshes/collada/forearms/forearm.dae" scale="1.0 1.0 1.0" />
-      </geometry>
-    </visual>
-    <collision>
-      <origin xyz="0 0 0.015" rpy="0 3.14159265359 1.570796326795"/>
-      <geometry name="LForearm_collision">
-        <mesh filename="package://coman_urdf/meshes/collada/simple/forearms/forearm.dae" scale="1.0 1.0 1.0" />
-      </geometry>
-    </collision>
-  </link>
-  <!--link name ="LElb">
-    <inertial>
-      <origin xyz="-6.5553403E-4 9.3464748E-4 -9.3101289E-4" rpy="0 0 0"/>
-      <mass value="0.63306933"/>
-      <inertia ixx="2.2599075E-4"  ixy="2.637647E-7"  ixz="-9.8007285E-6" iyy="2.7781302E-4" iyz="2.0435288E-6" izz="2.1878992E-4" />
-    </inertial>
-    <visual>
-      <origin xyz="-0.020305 -0.1558 -0.664329" rpy="0 0 -3.14159265359"/>
-      <geometry name="LElb_visual">
-        <mesh filename="package://coman_urdf/meshes/collada/asm0001_collada_11_prt.dae" scale="0.03937 0.03937 0.03937" />
-      </geometry>
-    </visual>
-    <collision>
-      <origin xyz="-0.020305 -0.1558 -0.664329" rpy="0 0 -3.14159265359"/>
-      <geometry name="LElb_collision">
-        <mesh filename="package://coman_urdf/meshes/collada/simple/simple_asm0001_collada_11_prt.dae" scale="0.03937 0.03937 0.03937" />
-      </geometry>
-    </collision>
-  </link>
-  <link name ="LForearm">
-    <inertial>
-      <origin xyz="0 0 -0.085" rpy="0 0 0"/>
-      <mass value="0.263"/>
-      <inertia ixx="6.913E-4"  ixy="0.0"  ixz="0.0" iyy="6.913E-4" iyz="0.0" izz="4.0425E-5" />
-    </inertial>
-  </link-->
+  <!-- Here I have used the inertia of a full cylinder with r = 0.02 [m] and h = 0.07 [m] -->
+  <link name="LWrMot2">
+    <inertial>
+      <origin xyz="0 0 0" rpy="0 0 0"/>
+      <mass value="0.26070556"/>
+      <inertia ixx="0.000132"  ixy="0"  ixz="0" iyy="0.000132" iyz="0" izz="5.213E-5" />
+    </inertial>
+    <visual>
+      <origin xyz="0.025 0 0" rpy="0 1.570796326795 3.14159265359"/>
+      <geometry name="LWrMot2_visual">
+        <mesh filename="package://coman_urdf/meshes/collada/forearms/fa_asm_3_right_sw0001.dae" scale="0.001 0.001 0.001" />
+      </geometry>
+    </visual>
+    <collision>
+      <origin xyz="0.025 0 0" rpy="0 1.570796326795 3.14159265359"/>
+      <geometry name="LWrMot2_collision">
+        <mesh filename="package://coman_urdf/meshes/collada/simple/forearms/simple_fa_asm_3_right_sw0001.dae" scale="0.001 0.001 0.001" />
+      </geometry>
+    </collision>
+  </link>
+  <!-- ## WRONG NUMBERS FOR INERTIAL!!! FIX THEM!! ## -->
+  <!-- Here I have used the inertia of a concave cylinder with r = 0.02 [m] -->
+  <link name="LWrMot3">
+    <inertial>
+      <origin xyz="0 0 0" rpy="0 0 0"/>
+      <mass value="0.054007518"/>
+      <inertia ixx="2.16E-5"  ixy="0"  ixz="0" iyy="2.16E-5" iyz="0" izz="2.16E-5" />
+    </inertial>
+    <visual>
+      <origin xyz="0.025 -0.012 -0.02" rpy="0 3.14159265359 1.570796326795"/>
+      <geometry name="LWrMot3_visual">
+        <mesh filename="package://coman_urdf/meshes/collada/forearms/fa_hand_interface_rig_sw0001.dae" scale="0.001 0.001 0.001" />
+      </geometry>
+    </visual>
+    <collision>
+      <origin xyz="0.025 -0.012 -0.02" rpy="0 3.14159265359 1.570796326795"/>
+      <geometry name="LWrMot3_collision">
+        <mesh filename="package://coman_urdf/meshes/collada/simple/forearms/simple_fa_hand_interface_rig_sw0001.dae" scale="0.001 0.001 0.001" />
+      </geometry>
+    </collision>
+  </link>
 <!-- ********************JOINTS******************** -->
   <joint name="base_joint" type="fixed">
@@ -648,12 +734,12 @@
   </joint>
   <joint name="l_wrist_joint" type="fixed">
-    <parent link="LElb"/>
+    <parent link="LWrMot3"/>
     <child link="l_wrist"/>
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
File: coman_urdf/urdf/coman_robot.urdf.xacro (robot description, xacro)
@@ -7,5 +7,17 @@
   -->
   <xacro:include filename="$(find coman_urdf)/urdf/coman.urdf.xacro" />
-<!-- IMU, needs to be checked effective position and orientation. For now it maches the same poisition/orientation of Waist link -->
+<!-- Hands! -->
+  <xacro:include filename="$(find coman_urdf)/urdf/soft_hand.urdf.xacro" />
+  <joint name="r_handj" type="fixed">
+    <parent link="r_wrist"/>
+    <child link="RSoftHand"/>
+    <origin xyz="0 0 -0.04" rpy="0 0 0"/>
+  </joint>
+  <joint name="l_handj" type="fixed">
+    <parent link="l_wrist"/>
+    <child link="LSoftHand"/>
+    <origin xyz="0 0 -0.04" rpy="0 0 0"/>
+  </joint>
+<!-- IMU -->
   <link name="imu_link">
     <inertial>

Commit message: Added gaze joint and repositioned torso at same height of shoulder

File: coman_urdf/urdf/coman.urdf (robot description, URDF)
Before this commit: robot COMAN, 40 links, 39 joints
Links:
- added link gaze
Joints:
- added joint gaze_joint: type fixed, parent torso, child gaze, origin xyz=0 0 0.1 rpy=0 0 0
- joint torso_joint: origin xyz=0 0 0 rpy=0 0 0 -> xyz=-0.014976503999999998 0 0.15770847 rpy=0 0 0

File: coman_urdf/urdf/coman.urdf.xacro (robot description, xacro)
@@ -27,4 +27,6 @@
 <!-- The coordinate frame called torso is attached to the lowest body of the model which is a parent of l_gripper, r_gripper and gaze. -->
  <link name="torso"/>
+<!-- Head -->
+ <link name="gaze"/>
 <!-- ********************TORSO******************** -->
 <!-- first real link of the robot, inertial reference frame -->
@@ -776,5 +778,10 @@
     <parent link="DWYTorso"/>
     <child link="torso"/>
-    <origin xyz="0 0 0" rpy="0 0 0" />
+    <origin xyz="-0.014976503999999998 0 0.15770847" rpy="0 0 0" />
+  </joint>
+  <joint name="gaze_joint" type="fixed">
+    <parent link="torso"/>
+    <child link="gaze"/>
+    <origin xyz="0 0 0.1" rpy="0 0 0" />
   </joint>
 <!-- ********************TORSO******************** -->
