Commit message: Added new feet. Added flags to compile coman with and without forearms, with and without hands, with old feet and with new feet

File: coman_urdf/urdf/coman.urdf (robot description, URDF)
Before this commit: robot COMAN, 41 links, 40 joints
Links:
- link LFoot: geometry collision box size=0.2 0.12 0.04; visual box size=0.2 0.12 0.04
- link RFoot: geometry collision box size=0.2 0.12 0.04; visual box size=0.2 0.12 0.04

File: coman_urdf/urdf/coman.urdf.xacro (robot description, xacro)
@@ -8,4 +8,5 @@
   Velocity and effort limits are fake!
 -->
+<!-- Adding macros for feet-->
 <!-- ********************LINKS******************** -->
 <!-- This links are defined in order to be compliant with http://www.ros.org/reps/rep-0120.html#coordinate-frames
@@ -204,23 +205,10 @@
   </link>
   <xacro:unless value="$(optenv GAZEBO_COMAN_USES_ACCURATE_FT false)">
-    <link name ="RFoot">
-      <inertial>
-        <origin xyz="0.00969210464 -0.0090460227 -0.043062308" rpy="0 0 0"/>
-        <mass value="0.66646684"/>
-        <inertia ixx="0.0012944808"  ixy="-9.2387693E-5"  ixz="2.0080105E-4" iyy="0.0015851846" iyz="2.7599327E-4" izz="0.0013326766" />
-      </inertial>
-      <visual>
-        <origin xyz="0.0 0.0726 -0.0932" rpy="0 0 -3.14159265359"/>
-        <geometry name="RFoot_visual">
-          <mesh filename="package://coman_urdf/meshes/collada/asm0001_collada_15_prt.dae" scale="0.03937 0.03937 0.03937" />
-        </geometry>
-      </visual>
-      <collision>
-        <origin xyz="0.0 0.0726 -0.0932" rpy="0 0 -3.14159265359"/>
-        <geometry name="RFoot_collision">
-          <mesh filename="package://coman_urdf/meshes/collada/simple/simple_asm0001_collada_15_prt.dae" scale="0.03937 0.03937 0.03937" />
-        </geometry>
-      </collision>
-    </link>
+    <xacro:if value="$(optenv GAZEBO_COMAN_USES_ROUND_FEET_13 true)">
+      <xacro:include filename="$(find coman_urdf)/urdf/feet/round_feet_13/round_foot_R_13.urdf.xacro" />
+    </xacro:if>
+    <xacro:if value="$(optenv GAZEBO_COMAN_USES_SIMPLE_FEET_DRC_sw1_14 false)">
+      <xacro:include filename="$(find coman_urdf)/urdf/feet/simple_feet_DRC_sw1_14/simple_foot_R_DRC_sw1_14.urdf.xacro" />
+    </xacro:if>
   </xacro:unless>
   <xacro:if value="$(optenv GAZEBO_COMAN_USES_ACCURATE_FT false)">
@@ -232,23 +220,10 @@
       </inertial>
     </link>
-    <link name ="RFoot">
-      <inertial>
-        <origin xyz="0.00969210464 -0.0090460227 -0.0282" rpy="0 0 0"/>
-        <mass value="0.404"/>
-        <inertia ixx="0.0012944808"  ixy="-9.2387693E-5"  ixz="2.0080105E-4" iyy="0.0015851846" iyz="2.7599327E-4" izz="0.0013326766" />
-      </inertial>
-      <visual>
-        <origin xyz="0.0 0.0726 -0.0282" rpy="0 0 -3.14159265359"/>
-        <geometry name="RFoot_visual">
-          <mesh filename="package://coman_urdf/meshes/collada/asm0001_collada_15_prt.dae" scale="0.03937 0.03937 0.03937" />
-        </geometry>
-      </visual>
-      <collision>
-        <origin xyz="0.0 0.0726 -0.0282" rpy="0 0 -3.14159265359"/>
-        <geometry name="RFoot_collision">
-          <mesh filename="package://coman_urdf/meshes/collada/simple/simple_asm0001_collada_15_prt.dae" scale="0.03937 0.03937 0.03937" />
-        </geometry>
-      </collision>
-    </link>
+    <xacro:if value="$(optenv GAZEBO_COMAN_USES_ROUND_FEET_13 true)">
+      <xacro:include filename="$(find coman_urdf)/urdf/feet/round_feet_13/accurate_FT_round_foot_R_13.urdf.xacro" />
+    </xacro:if>
+    <xacro:if value="$(optenv GAZEBO_COMAN_USES_SIMPLE_FEET_DRC_sw1_14 false)">
+      <xacro:include filename="$(find coman_urdf)/urdf/feet/simple_feet_DRC_sw1_14/accurate_FT_simple_foot_R_DRC_sw1_14.urdf.xacro" />
+    </xacro:if>
   </xacro:if>
 <!-- ********************LEFT LEG******************** -->
@@ -349,23 +324,10 @@
   </link>
   <xacro:unless value="$(optenv GAZEBO_COMAN_USES_ACCURATE_FT false)">
-    <link name ="LFoot">
-      <inertial>
-        <origin xyz="0.0096921046 0.0090460227 -0.043062308" rpy="0 0 0"/>
-        <mass value="0.66646684"/>
-        <inertia ixx="0.0012944808"  ixy="9.2387693E-5"  ixz="2.0080105E-4" iyy="0.0015851846" iyz="-2.7599327E-4" izz="0.0013326766" />
-      </inertial>
-      <visual>
-        <origin xyz="0.0 -0.0726 -0.0932" rpy="0 0 -3.14159265359"/>
-        <geometry name="LFoot_visual">
-          <mesh filename="package://coman_urdf/meshes/collada/asm0001_collada_01_prt.dae" scale="0.03937 0.03937 0.03937" />
-        </geometry>
-      </visual>
-      <collision>
-        <origin xyz="0.0 -0.0726 -0.0932" rpy="0 0 -3.14159265359"/>
-        <geometry name="LFoot_collision">
-          <mesh filename="package://coman_urdf/meshes/collada/simple/simple_asm0001_collada_01_prt.dae" scale="0.03937 0.03937 0.03937" />
-        </geometry>
-      </collision>
-    </link>
+    <xacro:if value="$(optenv GAZEBO_COMAN_USES_ROUND_FEET_13 true)">
+      <xacro:include filename="$(find coman_urdf)/urdf/feet/round_feet_13/round_foot_L_13.urdf.xacro" />
+    </xacro:if>
+    <xacro:if value="$(optenv GAZEBO_COMAN_USES_SIMPLE_FEET_DRC_sw1_14 false)">
+      <xacro:include filename="$(find coman_urdf)/urdf/feet/simple_feet_DRC_sw1_14/simple_foot_L_DRC_sw1_14.urdf.xacro" />
+    </xacro:if>
   </xacro:unless>
   <xacro:if value="$(optenv GAZEBO_COMAN_USES_ACCURATE_FT false)">
@@ -377,23 +339,10 @@
       </inertial>
     </link>
-    <link name ="LFoot">
-      <inertial>
-        <origin xyz="0.0096921046 0.0090460227 -0.0282" rpy="0 0 0"/>
-        <mass value="0.404"/>
-        <inertia ixx="0.0012944808"  ixy="9.2387693E-5"  ixz="2.0080105E-4" iyy="0.0015851846" iyz="-2.7599327E-4" izz="0.0013326766" />
-      </inertial>
-      <visual>
-        <origin xyz="0.0 -0.0726 -0.0282" rpy="0 0 -3.14159265359"/>
-        <geometry name="LFoot_visual">
-          <mesh filename="package://coman_urdf/meshes/collada/asm0001_collada_01_prt.dae" scale="0.03937 0.03937 0.03937" />
-        </geometry>
-      </visual>
-      <collision>
-        <origin xyz="0.0 -0.0726 -0.0282" rpy="0 0 -3.14159265359"/>
-        <geometry name="LFoot_collision">
-          <mesh filename="package://coman_urdf/meshes/collada/simple/simple_asm0001_collada_01_prt.dae" scale="0.03937 0.03937 0.03937" />
-        </geometry>
-      </collision>
-    </link>
+    <xacro:if value="$(optenv GAZEBO_COMAN_USES_ROUND_FEET_13 true)">
+      <xacro:include filename="$(find coman_urdf)/urdf/feet/round_feet_13/accurate_FT_round_foot_L_13.urdf.xacro" />
+    </xacro:if>
+    <xacro:if value="$(optenv GAZEBO_COMAN_USES_SIMPLE_FEET_DRC_sw1_14 false)">
+      <xacro:include filename="$(find coman_urdf)/urdf/feet/simple_feet_DRC_sw1_14/accurate_FT_simple_foot_L_DRC_sw1_14.urdf.xacro" />
+    </xacro:if>
   </xacro:if>
 <!-- ********************RIGHT ARM******************** -->
@@ -455,112 +404,10 @@
     </collision>
   </link>
-  <link name ="RElb">
-    <inertial>
-      <origin xyz="-6.5553403E-4 -9.3464748E-4 -9.3101289E-4" rpy="0 0 0"/>
-      <mass value="0.63306933"/>
-      <inertia ixx="2.2599075E-4"  ixy="-2.6376470E-7"  ixz="-9.8007285E-6" iyy="2.7781302E-4" iyz="-2.0435288E-6" izz="2.1878992E-4" />
-    </inertial>
-    <visual>
-      <origin xyz="0 0 0" rpy="-1.570796326795 1.570796326795 0"/>
-      <geometry name="RElb_visual">
-        <mesh filename="package://coman_urdf/meshes/collada/forearms/elbow.dae" scale="1.0 1.0 1.0" />
-      </geometry>
-    </visual>
-    <collision>
-      <origin xyz="0 0 0" rpy="-1.570796326795 1.570796326795 0"/>
-      <geometry name="RElb_collision">
-        <mesh filename="package://coman_urdf/meshes/collada/simple/forearms/elbow.dae" scale="1.0 1.0 1.0" />
-      </geometry>
-    </collision>
-  </link>
-  <!-- ## WRONG NUMBERS FOR INERTIAL!!! FIX THEM!! ## -->
-  <!-- In ROBOTRAN this link is named RFArm -->
-  <link name ="RForearm">
-    <inertial>
-      <origin xyz="0 0 -0.085" rpy="0 0 0"/>
-      <mass value="0.93351655"/>
-      <inertia ixx="0.001"  ixy="0.0"  ixz="0.0" iyy="0.001" iyz="0.0" izz="0.001" />
-    </inertial>
-    <visual>
-      <origin xyz="0 0 0.015" rpy="-1.570796326795 0 1.570796326795"/>
-      <geometry name="RForearm_visual">
-        <mesh filename="package://coman_urdf/meshes/collada/forearms/forearm.dae" scale="0.001 0.001 0.001" />
-      </geometry>
-    </visual>
-    <collision>
-      <origin xyz="0 0 0.015" rpy="0 3.14159265359 1.570796326795"/>
-      <geometry name="RForearm_collision">
-        <mesh filename="package://coman_urdf/meshes/collada/simple/forearms/forearm.dae" scale="1.0 1.0 1.0" />
-      </geometry>
-    </collision>
-  </link>
-  <!--link name ="RElb">
-    <inertial>
-      <origin xyz="-6.5553403E-4 -9.3464748E-4 -9.3101289E-4" rpy="0 0 0"/>
-      <mass value="0.63306933"/>
-      <inertia ixx="2.2599075E-4"  ixy="-2.6376470E-7"  ixz="-9.8007285E-6" iyy="2.7781302E-4" iyz="-2.0435288E-6" izz="2.1878992E-4" />
-    </inertial>
-    <visual>
-      <origin xyz="-0.020305 -0.1558 -0.664329" rpy="0 0 -3.14159265359"/>
-      <geometry name="RElb_visual">
-        <mesh filename="package://coman_urdf/meshes/collada/asm0001_collada_11_prt.dae" scale="0.03937 0.03937 0.03937" />
-      </geometry>
-    </visual>
-    <collision>
-      <origin xyz="-0.020305 -0.1558 -0.664329" rpy="0 0 -3.14159265359"/>
-      <geometry name="RElb_collision">
-        <mesh filename="package://coman_urdf/meshes/collada/simple/simple_asm0001_collada_11_prt.dae" scale="0.03937 0.03937 0.03937" />
-      </geometry>
-    </collision>
-  </link>
-  <link name ="RForearm">
-    <inertial>
-      <origin xyz="0 0 -0.085" rpy="0 0 0"/>
-      <mass value="0.263"/>
-      <inertia ixx="6.913E-4"  ixy="0.0"  ixz="0.0" iyy="6.913E-4" iyz="0.0" izz="4.0425E-5" />
-    </inertial>
-  </link-->
-  <!-- ## WRONG NUMBERS FOR INERTIAL!!! FIX THEM!! ## -->
-  <!-- Here I have used the inertia of a full cylinder with r = 0.02 [m] and h = 0.07 [m] -->
-  <link name="RWrMot2">
-    <inertial>
-      <origin xyz="0 0 0" rpy="0 0 0"/>
-      <mass value="0.26070556"/>
-      <inertia ixx="0.000132"  ixy="0"  ixz="0" iyy="0.000132" iyz="0" izz="5.213E-5" />
-    </inertial>
-    <visual>
-      <origin xyz="0.025 0 0" rpy="0 1.570796326795 3.14159265359"/>
-      <geometry name="RWrMot2_visual">
-        <mesh filename="package://coman_urdf/meshes/collada/forearms/fa_asm_3_right_sw0001.dae" scale="0.001 0.001 0.001" />
-      </geometry>
-    </visual>
-    <collision>
-      <origin xyz="0.025 0 0" rpy="0 1.570796326795 3.14159265359"/>
-      <geometry name="RWrMot2_collision">
-        <mesh filename="package://coman_urdf/meshes/collada/simple/forearms/simple_fa_asm_3_right_sw0001.dae" scale="0.001 0.001 0.001" />
-      </geometry>
-    </collision>
-  </link>
-  <!-- ## WRONG NUMBERS FOR INERTIAL!!! FIX THEM!! ## -->
-  <!-- Here I have used the inertia of a concave cylinder with r = 0.02 [m] -->
-  <link name="RWrMot3">
-    <inertial>
-      <origin xyz="0 0 0" rpy="0 0 0"/>
-      <mass value="0.054007518"/>
-      <inertia ixx="2.16E-5"  ixy="0"  ixz="0" iyy="2.16E-5" iyz="0" izz="2.16E-5" />
-    </inertial>
-    <visual>
-      <origin xyz="0.025 -0.012 -0.02" rpy="0 3.14159265359 1.570796326795"/>
-      <geometry name="RWrMot3_visual">
-        <mesh filename="package://coman_urdf/meshes/collada/forearms/fa_hand_interface_rig_sw0001.dae" scale="0.001 0.001 0.001" />
-      </geometry>
-    </visual>
-    <collision>
-      <origin xyz="0.025 -0.012 -0.02" rpy="0 3.14159265359 1.570796326795"/>
-      <geometry name="RWrMot3_collision">
-        <mesh filename="package://coman_urdf/meshes/collada/simple/forearms/simple_fa_hand_interface_rig_sw0001.dae" scale="0.001 0.001 0.001" />
-      </geometry>
-    </collision>
-  </link>
+  <xacro:if value="$(optenv GAZEBO_COMAN_USES_NO_FOREARMS true)">
+      <xacro:include filename="$(find coman_urdf)/urdf/forearms/no_forearms/links/no_forearms_R.urdf.xacro" />
+  </xacro:if>
+  <xacro:if value="$(optenv GAZEBO_COMAN_USES_7DOF_FOREARMS_DRC_14 false)">
+      <xacro:include filename="$(find coman_urdf)/urdf/forearms/7DOF_forearms_DRC_14/links/7DOF_forearms_R_DRC_14.urdf.xacro" />
+  </xacro:if>
 <!-- ********************LEFT ARM******************** -->
   <link name ="LShp">
@@ -621,112 +468,10 @@
     </collision>
   </link>
-  <link name ="LElb">
-    <inertial>
-      <origin xyz="-6.5553403E-4 9.3464748E-4 -9.3101289E-4" rpy="0 0 0"/>
-      <mass value="0.63306933"/>
-      <inertia ixx="2.2599075E-4"  ixy="2.6376470E-7"  ixz="-9.8007285E-6" iyy="2.7781302E-4" iyz="2.0435288E-6" izz="2.1878992E-4" />
-    </inertial>
-    <visual>
-      <origin xyz="0 0 0" rpy="-1.570796326795 1.570796326795 0"/>
-      <geometry name="LElb_visual">
-        <mesh filename="package://coman_urdf/meshes/collada/forearms/elbow.dae" scale="1.0 1.0 1.0" />
-      </geometry>
-    </visual>
-    <collision>
-      <origin xyz="0 0 0" rpy="-1.570796326795 1.570796326795 0"/>
-      <geometry name="LElb_collision">
-        <mesh filename="package://coman_urdf/meshes/collada/simple/forearms/elbow.dae" scale="1.0 1.0 1.0" />
-      </geometry>
-    </collision>
-  </link>
-  <!-- ## WRONG NUMBERS FOR INERTIAL!!! FIX THEM!! ## -->
-  <!-- In ROBOTRAN this link is named LFARM -->
-  <link name ="LForearm">
-    <inertial>
-      <origin xyz="0 0 -0.085" rpy="0 0 0"/>
-      <mass value="0.93351655"/>
-      <inertia ixx="0.001"  ixy="0.0"  ixz="0.0" iyy="0.001" iyz="0.0" izz="0.001" />
-    </inertial>
-    <visual>
-      <origin xyz="0 0 0.015" rpy="-1.570796326795 0 1.570796326795"/>
-      <geometry name="LForearm_visual">
-        <mesh filename="package://coman_urdf/meshes/collada/forearms/forearm.dae" scale="0.001 0.001 0.001" />
-      </geometry>
-    </visual>
-    <collision>
-      <origin xyz="0 0 0.015" rpy="0 3.14159265359 1.570796326795"/>
-      <geometry name="LForearm_collision">
-        <mesh filename="package://coman_urdf/meshes/collada/simple/forearms/forearm.dae" scale="1.0 1.0 1.0" />
-      </geometry>
-    </collision>
-  </link>
-  <!--link name ="LElb">
-    <inertial>
-      <origin xyz="-6.5553403E-4 9.3464748E-4 -9.3101289E-4" rpy="0 0 0"/>
-      <mass value="0.63306933"/>
-      <inertia ixx="2.2599075E-4"  ixy="2.637647E-7"  ixz="-9.8007285E-6" iyy="2.7781302E-4" iyz="2.0435288E-6" izz="2.1878992E-4" />
-    </inertial>
-    <visual>
-      <origin xyz="-0.020305 -0.1558 -0.664329" rpy="0 0 -3.14159265359"/>
-      <geometry name="LElb_visual">
-        <mesh filename="package://coman_urdf/meshes/collada/asm0001_collada_11_prt.dae" scale="0.03937 0.03937 0.03937" />
-      </geometry>
-    </visual>
-    <collision>
-      <origin xyz="-0.020305 -0.1558 -0.664329" rpy="0 0 -3.14159265359"/>
-      <geometry name="LElb_collision">
-        <mesh filename="package://coman_urdf/meshes/collada/simple/simple_asm0001_collada_11_prt.dae" scale="0.03937 0.03937 0.03937" />
-      </geometry>
-    </collision>
-  </link>
-  <link name ="LForearm">
-    <inertial>
-      <origin xyz="0 0 -0.085" rpy="0 0 0"/>
-      <mass value="0.263"/>
-      <inertia ixx="6.913E-4"  ixy="0.0"  ixz="0.0" iyy="6.913E-4" iyz="0.0" izz="4.0425E-5" />
-    </inertial>
-  </link-->
-  <!-- ## WRONG NUMBERS FOR INERTIAL!!! FIX THEM!! ## -->
-  <!-- Here I have used the inertia of a full cylinder with r = 0.02 [m] and h = 0.07 [m] -->
-  <link name="LWrMot2">
-    <inertial>
-      <origin xyz="0 0 0" rpy="0 0 0"/>
-      <mass value="0.26070556"/>
-      <inertia ixx="0.000132"  ixy="0"  ixz="0" iyy="0.000132" iyz="0" izz="5.213E-5" />
-    </inertial>
-    <visual>
-      <origin xyz="0.025 0 0" rpy="0 1.570796326795 3.14159265359"/>
-      <geometry name="LWrMot2_visual">
-        <mesh filename="package://coman_urdf/meshes/collada/forearms/fa_asm_3_right_sw0001.dae" scale="0.001 0.001 0.001" />
-      </geometry>
-    </visual>
-    <collision>
-      <origin xyz="0.025 0 0" rpy="0 1.570796326795 3.14159265359"/>
-      <geometry name="LWrMot2_collision">
-        <mesh filename="package://coman_urdf/meshes/collada/simple/forearms/simple_fa_asm_3_right_sw0001.dae" scale="0.001 0.001 0.001" />
-      </geometry>
-    </collision>
-  </link>
-  <!-- ## WRONG NUMBERS FOR INERTIAL!!! FIX THEM!! ## -->
-  <!-- Here I have used the inertia of a concave cylinder with r = 0.02 [m] -->
-  <link name="LWrMot3">
-    <inertial>
-      <origin xyz="0 0 0" rpy="0 0 0"/>
-      <mass value="0.054007518"/>
-      <inertia ixx="2.16E-5"  ixy="0"  ixz="0" iyy="2.16E-5" iyz="0" izz="2.16E-5" />
-    </inertial>
-    <visual>
-      <origin xyz="0.025 -0.012 -0.02" rpy="0 3.14159265359 1.570796326795"/>
-      <geometry name="LWrMot3_visual">
-        <mesh filename="package://coman_urdf/meshes/collada/forearms/fa_hand_interface_rig_sw0001.dae" scale="0.001 0.001 0.001" />
-      </geometry>
-    </visual>
-    <collision>
-      <origin xyz="0.025 -0.012 -0.02" rpy="0 3.14159265359 1.570796326795"/>
-      <geometry name="LWrMot3_collision">
-        <mesh filename="package://coman_urdf/meshes/collada/simple/forearms/simple_fa_hand_interface_rig_sw0001.dae" scale="0.001 0.001 0.001" />
-      </geometry>
-    </collision>
-  </link>
+  <xacro:if value="$(optenv GAZEBO_COMAN_USES_NO_FOREARMS true)">
+      <xacro:include filename="$(find coman_urdf)/urdf/forearms/no_forearms/links/no_forearms_L.urdf.xacro" />
+  </xacro:if>
+  <xacro:if value="$(optenv GAZEBO_COMAN_USES_7DOF_FOREARMS_DRC_14 false)">
+      <xacro:include filename="$(find coman_urdf)/urdf/forearms/7DOF_forearms_DRC_14/links/7DOF_forearms_L_DRC_14.urdf.xacro" />
+  </xacro:if>
 <!-- ********************JOINTS******************** -->
   <joint name="base_joint" type="fixed">
@@ -740,14 +485,16 @@
     <origin xyz="0 0 0" rpy="0 0 0" />
   </joint>
-  <joint name="r_wrist_joint" type="fixed">
-    <parent link="RWrMot3"/>
-    <child link="r_wrist"/>
-    <origin xyz="0 0 0" rpy="0 0 0" />
-  </joint>
-  <joint name="l_ankle_joint" type="fixed">
-    <parent link="LFoot"/>
-    <child link="l_ankle"/>
-    <origin xyz="0 0 0" rpy="0 0 0" />
-  </joint>
+  <xacro:if value="$(optenv GAZEBO_COMAN_USES_7DOF_FOREARMS_DRC_14 false)">
+    <joint name="r_wrist_joint" type="fixed">
+      <parent link="RWrMot3"/>
+      <child link="r_wrist"/>
+      <origin xyz="0 0 0" rpy="0 0 0" />
+    </joint>
+    <joint name="l_ankle_joint" type="fixed">
+      <parent link="LFoot"/>
+      <child link="l_ankle"/>
+      <origin xyz="0 0 0" rpy="0 0 0" />
+    </joint>
+  </xacro:if>
   <joint name="r_ankle_joint" type="fixed">
     <parent link="RFoot"/>
@@ -982,33 +729,10 @@
     <dynamics friction="0" damping="3.0"/>
   </joint>
-  <joint name="RForearmPlate" type="revolute">
-    <parent link="RElb"/>
-    <child link="RForearm"/>
-    <origin xyz="-0.015 0.0 -0.051" rpy="0 0 0"/>
-    <axis xyz="0 0 1" />
-    <limit velocity="4.0" effort="50" lower="-1.5708" upper="1.5708" />
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
File: coman_urdf/urdf/coman_robot.urdf.xacro (robot description, xacro)
@@ -8,15 +8,19 @@
   <xacro:include filename="$(find coman_urdf)/urdf/coman.urdf.xacro" />
 <!-- Hands! -->
-  <xacro:include filename="$(find coman_urdf)/urdf/soft_hand.urdf.xacro" />
-  <joint name="r_handj" type="fixed">
-    <parent link="r_wrist"/>
-    <child link="RSoftHand"/>
-    <origin xyz="0 0 -0.04" rpy="0 0 0"/>
-  </joint>
-  <joint name="l_handj" type="fixed">
-    <parent link="l_wrist"/>
-    <child link="LSoftHand"/>
-    <origin xyz="0 0 -0.04" rpy="0 0 0"/>
-  </joint>
+  <xacro:if value="$(optenv GAZEBO_COMAN_USES_7DOF_FOREARMS_DRC_14 false)">
+    <xacro:if value="$(optenv GAZEBO_COMAN_USES_SOFTHANDS_DRC_sw1_14 false)">
+      <xacro:include filename="$(find coman_urdf)/urdf/soft_hand.urdf.xacro" />
+      <joint name="r_handj" type="fixed">
+        <parent link="r_wrist"/>
+        <child link="RSoftHand"/>
+        <origin xyz="0 0 -0.04" rpy="0 0 0"/>
+      </joint>
+      <joint name="l_handj" type="fixed">
+        <parent link="l_wrist"/>
+        <child link="LSoftHand"/>
+        <origin xyz="0 0 -0.04" rpy="0 0 0"/>
+      </joint>
+    </xacro:if>
+  </xacro:if>
 <!-- IMU -->
   <link name="imu_link">

Commit message: Changed script. IMPORTANT now the script has to be called as: ". create_urdf_and_sdf.sh"

File: coman_urdf/urdf/coman.urdf (robot description, URDF)
Before this commit: robot COMAN, 41 links, 40 joints
Links:
- link LFoot: geometry collision box size=0.2 0.1 0.04; visual box size=0.2 0.1 0.04
- link RFoot: geometry collision box size=0.2 0.1 0.04; visual box size=0.2 0.1 0.04

File: coman_urdf/urdf/coman_robot.urdf.xacro (robot description, xacro)
@@ -8,6 +8,6 @@
   <xacro:include filename="$(find coman_urdf)/urdf/coman.urdf.xacro" />
 <!-- Hands! -->
-  <xacro:if value="$(optenv GAZEBO_COMAN_USES_7DOF_FOREARMS_DRC_14 false)">
-    <xacro:if value="$(optenv GAZEBO_COMAN_USES_SOFTHANDS_DRC_sw1_14 false)">
+  <xacro:if value="$(optenv GAZEBO_COMAN_USES_7DOF_FOREARMS_DRC_14 true)">
+    <xacro:if value="$(optenv GAZEBO_COMAN_USES_SOFTHANDS_DRC_sw1_14 true)">
       <xacro:include filename="$(find coman_urdf)/urdf/soft_hand.urdf.xacro" />
       <joint name="r_handj" type="fixed">
@@ -43,5 +43,5 @@
   </joint>
   <xacro:include filename="$(find coman_urdf)/urdf/microstrain_3dmgx2_imu.gazebo.xacro" />
-  <xacro:if value="$(optenv GAZEBO_COMAN_USES_ROS true)">
+  <xacro:if value="$(optenv GAZEBO_COMAN_USES_ROS false)">
   	<xacro:include filename="$(find coman_urdf)/urdf/coman_transmission.urdf.xacro" />
   </xacro:if>
