Commit message: Added hand joint as revolute. Added Hand inside coman.urdf (before it was in coman_robot.urdf)

File: coman_urdf/urdf/coman.urdf (robot description, URDF)
Before this commit: robot COMAN, 41 links, 40 joints
Links:
- added link LSoftHand, mass 0.3; collision box size=0.07 0.07 0.07; visual box size=0.07 0.07 0.07
- added link RSoftHand, mass 0.3; collision box size=0.07 0.07 0.07; visual box size=0.07 0.07 0.07
Joints:
- added joint l_handj: type revolute, parent l_wrist, child LSoftHand, origin xyz=0 0 -0.04 rpy=0 0 0, axis 1 0 0, limit lower=-1.57075 upper=0.0 effort=5 velocity=4.0
- added joint r_handj: type revolute, parent r_wrist, child RSoftHand, origin xyz=0 0 -0.04 rpy=0 0 0, axis 1 0 0, limit lower=0.0 upper=1.57075 effort=5 velocity=4.0

File: coman_urdf/urdf/coman.urdf.xacro (robot description, xacro)
@@ -475,4 +475,10 @@
       <xacro:include filename="$(find coman_urdf)/urdf/forearms/7DOF_forearms_DRC_14/links/7DOF_forearms_L_DRC_14.urdf.xacro" />
   </xacro:if>
+<!-- ********************HANDS********************* -->
+  <xacro:if value="$(optenv GAZEBO_COMAN_USES_7DOF_FOREARMS_DRC_14 true)">
+    <xacro:if value="$(optenv GAZEBO_COMAN_USES_SOFTHANDS_DRC_sw1_14 true)">
+      <xacro:include filename="$(find coman_urdf)/urdf/soft_hand.urdf.xacro" />
+    </xacro:if>
+  </xacro:if>
 <!-- ********************JOINTS******************** -->
   <joint name="base_joint" type="fixed">
@@ -748,4 +754,17 @@
       <xacro:include filename="$(find coman_urdf)/urdf/forearms/7DOF_forearms_DRC_14/joints/7DOF_forearms_R_DRC_14.urdf.xacro" />
   </xacro:if>
+<!-- ********************RIGHT HAND****************** -->
+  <xacro:if value="$(optenv GAZEBO_COMAN_USES_7DOF_FOREARMS_DRC_14 true)">
+    <xacro:if value="$(optenv GAZEBO_COMAN_USES_SOFTHANDS_DRC_sw1_14 true)">
+      <joint name="r_handj" type="revolute">
+        <parent link="r_wrist"/>
+        <child link="RSoftHand"/>
+        <origin xyz="0 0 -0.04" rpy="0 0 0"/>
+        <axis xyz="1 0 0" />
+        <limit velocity="4.0" effort="5" lower="0.0" upper="1.57075" />
+        <dynamics friction="0" damping="3.0"/>
+      </joint>
+      </xacro:if>
+  </xacro:if>
 <!-- ********************LEFT ARM******************** -->
   <joint name="LShSag" type="revolute">
@@ -787,3 +806,16 @@
       <xacro:include filename="$(find coman_urdf)/urdf/forearms/7DOF_forearms_DRC_14/joints/7DOF_forearms_L_DRC_14.urdf.xacro" />
   </xacro:if>
+<!-- ********************LEFT HAND******************** -->
+  <xacro:if value="$(optenv GAZEBO_COMAN_USES_7DOF_FOREARMS_DRC_14 true)">
+    <xacro:if value="$(optenv GAZEBO_COMAN_USES_SOFTHANDS_DRC_sw1_14 true)">
+      <joint name="l_handj" type="revolute">
+        <parent link="l_wrist"/>
+        <child link="LSoftHand"/>
+        <origin xyz="0 0 -0.04" rpy="0 0 0"/>
+        <axis xyz="1 0 0" />
+        <limit velocity="4.0" effort="5" lower="-1.57075" upper="0.0" />
+        <dynamics friction="0" damping="3.0"/>
+      </joint>
+    </xacro:if>
+  </xacro:if>
 </robot>

File: coman_urdf/urdf/coman_robot.urdf.xacro (robot description, xacro)
@@ -7,20 +7,4 @@
   -->
   <xacro:include filename="$(find coman_urdf)/urdf/coman.urdf.xacro" />
-<!-- Hands! -->
-  <xacro:if value="$(optenv GAZEBO_COMAN_USES_7DOF_FOREARMS_DRC_14 true)">
-    <xacro:if value="$(optenv GAZEBO_COMAN_USES_SOFTHANDS_DRC_sw1_14 true)">
-      <xacro:include filename="$(find coman_urdf)/urdf/soft_hand.urdf.xacro" />
-      <joint name="r_handj" type="fixed">
-        <parent link="r_wrist"/>
-        <child link="RSoftHand"/>
-        <origin xyz="0 0 -0.04" rpy="0 0 0"/>
-      </joint>
-      <joint name="l_handj" type="fixed">
-        <parent link="l_wrist"/>
-        <child link="LSoftHand"/>
-        <origin xyz="0 0 -0.04" rpy="0 0 0"/>
-      </joint>
-    </xacro:if>
-  </xacro:if>
 <!-- IMU -->
   <link name="imu_link">

File: coman_urdf/urdf/soft_hand.urdf.xacro (robot description, xacro)
@@ -5,5 +5,5 @@
     <inertial>
       <origin xyz="0 0 0" rpy="0 0 0"/>
-      <mass value="0.2"/>
+      <mass value="0.3"/>
       <inertia ixx="0.001"  ixy="0"  ixz="0" iyy="0.001" iyz="0" izz="0.001" />
     </inertial>
@@ -27,5 +27,5 @@
     <inertial>
       <origin xyz="0 0 0" rpy="0 0 0"/>
-      <mass value="0.2"/>
+      <mass value="0.3"/>
       <inertia ixx="0.001"  ixy="0"  ixz="0" iyy="0.001" iyz="0" izz="0.001" />
     </inertial>

Commit message: Added FT Sensors to forearms

File: coman_urdf/urdf/coman.urdf (robot description, URDF)
Before this commit: robot COMAN, 43 links, 42 joints
Joints:
- joint LForearmPlate: origin xyz=-0.015 0.0 -0.051 rpy=0 0 0 -> xyz=-0.015 0.0 -0.1078 rpy=0 0 0
- joint LWrj1: origin xyz=0 0 -0.14368 rpy=0 0 0 -> xyz=0 0 -0.08688 rpy=0 0 0
- joint RForearmPlate: origin xyz=-0.015 0.0 -0.051 rpy=0 0 0 -> xyz=-0.015 0.0 -0.1078 rpy=0 0 0
- joint RWrj1: origin xyz=0 0 -0.14368 rpy=0 0 0 -> xyz=0 0 -0.08688 rpy=0 0 0

File: coman_urdf/urdf/forearms/7DOF_forearms_DRC_14/7DOF_forearms_DRC_14.urdf.xacro (robot description, xacro)
@@ -1,4 +1,10 @@
 <?xml version="1.0"?>
 <robot xmlns:xacro="http://ros.org/wiki/xacro">
+<!-- distance from last motor to FT sensor
+		The value needs to be subtracted to the *FOrearmPlate joint z origin,
+		and in order to be compensated in the following joint and link,
+		it neeeds to be added in return to the following joint (*Wrj1) z origin
+		and to the z displacement of mass, visual and collision of *Forearm -->
+<xacro:property name="Wrj1_to_FT" value="0.0568" />
 <!-- ****************LINKS**************** -->
 <!-- ****************LEFT FOREARM**************** -->
@@ -26,10 +32,10 @@
       <link name ="LForearm">
         <inertial>
-          <origin xyz="0 0 -0.085" rpy="0 0 0"/>
+          <origin xyz="0 0 ${-0.085 + Wrj1_to_FT}" rpy="0 0 0"/>
           <mass value="0.93351655"/>
           <inertia ixx="0.001"  ixy="0.0"  ixz="0.0" iyy="0.001" iyz="0.0" izz="0.001" />
         </inertial>
         <visual>
-          <origin xyz="0 0 0.015" rpy="-1.570796326795 0 1.570796326795"/>
+          <origin xyz="0 0 ${0.015 + Wrj1_to_FT}" rpy="-1.570796326795 0 1.570796326795"/>
           <geometry name="LForearm_visual">
             <mesh filename="package://coman_urdf/meshes/collada/forearms/forearm.dae" scale="0.001 0.001 0.001" />
@@ -37,5 +43,5 @@
         </visual>
         <collision>
-          <origin xyz="0 0 0.015" rpy="0 3.14159265359 1.570796326795"/>
+          <origin xyz="0 0 ${0.015 + Wrj1_to_FT}" rpy="0 3.14159265359 1.570796326795"/>
           <geometry name="LForearm_collision">
             <mesh filename="package://coman_urdf/meshes/collada/simple/forearms/forearm.dae" scale="1.0 1.0 1.0" />
@@ -109,10 +115,10 @@
       <link name ="RForearm">
         <inertial>
-          <origin xyz="0 0 -0.085" rpy="0 0 0"/>
+          <origin xyz="0 0 ${-0.085 + Wrj1_to_FT}" rpy="0 0 0"/>
           <mass value="0.93351655"/>
           <inertia ixx="0.001"  ixy="0.0"  ixz="0.0" iyy="0.001" iyz="0.0" izz="0.001" />
         </inertial>
         <visual>
-          <origin xyz="0 0 0.015" rpy="-1.570796326795 0 1.570796326795"/>
+          <origin xyz="0 0 ${0.015 + Wrj1_to_FT}" rpy="-1.570796326795 0 1.570796326795"/>
           <geometry name="RForearm_visual">
             <mesh filename="package://coman_urdf/meshes/collada/forearms/forearm.dae" scale="0.001 0.001 0.001" />
@@ -120,5 +126,5 @@
         </visual>
         <collision>
-          <origin xyz="0 0 0.015" rpy="0 3.14159265359 1.570796326795"/>
+          <origin xyz="0 0 ${0.015 + Wrj1_to_FT}" rpy="0 3.14159265359 1.570796326795"/>
           <geometry name="RForearm_collision">
             <mesh filename="package://coman_urdf/meshes/collada/simple/forearms/forearm.dae" scale="1.0 1.0 1.0" />
@@ -173,5 +179,5 @@
     <parent link="LElb"/>
     <child link="LForearm"/>
-    <origin xyz="-0.015 0.0 -0.051" rpy="0 0 0"/>
+    <origin xyz="-0.015 0.0 ${-0.051 - Wrj1_to_FT}" rpy="0 0 0"/>
     <axis xyz="0 0 1" />
     <limit velocity="4.0" effort="50" lower="-1.5708" upper="1.5708" />
@@ -181,5 +187,5 @@
     <parent link="LForearm"/>
     <child link="LWrMot2"/>
-    <origin xyz="0 0 -0.14368" rpy="0 0 0"/>
+    <origin xyz="0 0 ${-0.14368 + Wrj1_to_FT}" rpy="0 0 0"/>
     <axis xyz="0 1 0"/>
     <limit velocity="4.0" effort="50" lower="-0.524" upper="0.524" />
@@ -198,5 +204,5 @@
     <parent link="RElb"/>
     <child link="RForearm"/>
-    <origin xyz="-0.015 0.0 -0.051" rpy="0 0 0"/>
+    <origin xyz="-0.015 0.0 ${-0.051 - Wrj1_to_FT}" rpy="0 0 0"/>
     <axis xyz="0 0 1" />
     <limit velocity="4.0" effort="50" lower="-1.5708" upper="1.5708" />
@@ -206,5 +212,5 @@
     <parent link="RForearm"/>
     <child link="RWrMot2"/>
-    <origin xyz="0 0 -0.14368" rpy="0 0 0"/>
+    <origin xyz="0 0 ${-0.14368 + Wrj1_to_FT}" rpy="0 0 0"/>
     <axis xyz="0 1 0"/>
     <limit velocity="4.0" effort="50" lower="-0.524" upper="0.524" />

Commit message: Added xtion in urdf (to finish...)

File: coman_urdf/urdf/coman.urdf (robot description, URDF)
Before this commit: robot COMAN, 43 links, 42 joints
Links:
- added link Xtion_body, mass 0.89258227; collision mesh filename=package://coman_urdf/meshes/collada/simple/Xtion/xtion_base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 scale=0.03937 0.03937 0.03937; visual mesh filename=package://coman_urdf/meshes/collada/Xtion/xtion_base.dae scale=0.03937 0.03937 0.03937
- added link Xtion_cam_body, mass 0.89258227; collision mesh filename=package://coman_urdf/meshes/collada/Xtion/xtion_cam_body.dae scale=0.001 0.001 0.001; visual mesh filename=package://coman_urdf/meshes/collada/Xtion/xtion_cam_body.dae scale=0.001 0.001 0.001
Joints:
- added joint Xtion_body_joint: type fixed, parent torso, child Xtion_body, origin xyz=0 0 0 rpy=0 0 0
- added joint Xtion_cam_body_joint: type fixed, parent Xtion_body, child Xtion_cam_body, origin xyz=0.08 0 0.44 rpy=0 0 0
- joint gaze_joint: origin xyz=0 0 0.1 rpy=0 0 0 -> xyz=0 0 0.0 rpy=0 0 0; parent torso -> Xtion_cam_body

File: coman_urdf/urdf/coman.urdf.xacro (robot description, xacro)
@@ -30,5 +30,45 @@
  <link name="torso"/>
 <!-- Head -->
- <link name="gaze"/>
+<xacro:if value="${GAZEBO_COMAN_USES_XTION}">
+	<link name ="Xtion_body">
+    <inertial>
+      <origin xyz="0.0 0.0 0.0" rpy="0 0 0"/>
+      <mass value="0.89258227"/>
+      <inertia ixx="0.0001"  ixy="0.0"  ixz="0.0" iyy="0.0001" iyz="0.0" izz="0.0001" />
+    </inertial>
+    <visual>
+      <origin xyz="-0.005305004 0.0 -0.844329" rpy="0 0 -3.14159265359"/>
+      <geometry name="Xtion_body_visual">
+        <mesh filename="package://coman_urdf/meshes/collada/Xtion/xtion_base.dae" scale="0.03937 0.03937 0.03937" />
+      </geometry>
+    </visual>
+    <collision>
+      <origin xyz="-0.005305004 0.0 -0.844329" rpy="0 0 -3.14159265359"/>
+      <geometry name="Xtion_body_collision">
+        <mesh filename="package://coman_urdf/meshes/collada/simple/Xtion/xtion_base.dae" scale="0.03937 0.03937 0.03937" />
+      </geometry>
+    </collision>
+  </link>
+  <link name ="Xtion_cam_body">
+    <inertial>
+      <origin xyz="0.0 0.0 0.0" rpy="0 0 0"/>
+      <mass value="0.89258227"/>
+      <inertia ixx="0.0001"  ixy="0.0"  ixz="0.0" iyy="0.0001" iyz="0.0" izz="0.0001" />
+    </inertial>
+    <visual>
+      <origin xyz="-0.085305004 0.0 -1.284329" rpy="0 0 -3.14159265359"/>
+      <geometry name="Xtion_cam_body_visual">
+        <mesh filename="package://coman_urdf/meshes/collada/Xtion/xtion_cam_body.dae" scale="0.001 0.001 0.001" />
+      </geometry>
+    </visual>
+    <collision>
+      <origin xyz="-0.085305004 0.0 -1.284329" rpy="0 0 -3.14159265359"/>
+      <geometry name="Xtion_cam_body_collision">
+        <mesh filename="package://coman_urdf/meshes/collada/Xtion/xtion_cam_body.dae" scale="0.001 0.001 0.001" />
+      </geometry>
+    </collision>
+  </link>
+</xacro:if>
+<link name="gaze"/>
 <!-- ************ COMAN BASE ************** -->
 <xacro:include filename="$(find coman_urdf)//urdf/coman_base.urdf.xacro"/>

File: coman_urdf/urdf/coman_base.urdf.xacro (robot description, xacro)
@@ -481,9 +481,28 @@
     <origin xyz="-0.014976503999999998 0 0.15770847" rpy="0 0 0" />
   </joint>
-  <joint name="gaze_joint" type="fixed">
-    <parent link="torso"/>
-    <child link="gaze"/>
-    <origin xyz="0 0 0.1" rpy="0 0 0" />
-  </joint>
+<xacro:if value="${GAZEBO_COMAN_USES_XTION}">
+        <joint name="Xtion_body_joint" type="fixed">
+    		<parent link="torso"/>
+    		<child link="Xtion_body"/>
+    		<origin xyz="0 0 0" rpy="0 0 0" />
+  	</joint>
+        <joint name="Xtion_cam_body_joint" type="fixed">
+    		<parent link="Xtion_body"/>
+    		<child link="Xtion_cam_body"/>
+    		<origin xyz="0.08 0 0.44" rpy="0 0 0" />
+  	</joint>
+        <joint name="gaze_joint" type="fixed">
+    		<parent link="Xtion_cam_body"/>
+    		<child link="gaze"/>
+    		<origin xyz="0 0 0.0" rpy="0 0 0" />
+  	</joint>
+</xacro:if>
+<xacro:unless value="${GAZEBO_COMAN_USES_XTION}">
+ 	<joint name="gaze_joint" type="fixed">
+    		<parent link="torso"/>
+    		<child link="gaze"/>
+    		<origin xyz="0 0 0.1" rpy="0 0 0" />
+  	</joint>
+</xacro:unless>
 <!-- ********************TORSO******************** -->
   <joint name="WaistSag" type="revolute"> <!-- Wrong name! need to fix this... -->

File: coman_urdf/urdf/coman_config.urdf.xacro (robot description, xacro)
@@ -99,3 +99,21 @@
 -->
 <xacro:property name="GAZEBO_COMAN_USES_ACCURATE_FT" value="false" />
+<!--
+####################################################
+##
+##  Xtion SELECTION
+##
+##
+## options:
+## 1) COMAN classic without the staff to carry the sensor.
+##      Torso frame is connected to gaze link through a gaze_joint "fixed"
+## 2) COMAN with staff and xtion sensor. Torso frame is connected to a xtion_staff_link through
+##      a xtion_staff_joint "fixed". Xtion_staff_link is then connected to gaze_link through gaze_joint "fixed".
+##
+####################################################
+#
+# 1/2 (true/false)
+#
+-->
+<xacro:property name="GAZEBO_COMAN_USES_XTION" value="true" />
 </robot>

Commit message: Added kinect ref frame and new bodies. ACCURATE!!!!

File: coman_urdf/urdf/coman.urdf (robot description, URDF)
Before this commit: robot COMAN, 45 links, 44 joints
Links:
- link Xtion_body: mass 0.89258227 -> 0.39
- link Xtion_cam_body: mass 0.89258227 -> 0.2
Joints:
- joint Xtion_body_joint: parent torso -> DWYTorso
- joint Xtion_cam_body_joint: origin xyz=0.08 0 0.44 rpy=0 0 0 -> xyz=0.071 0 0.591 rpy=0 1.396 0
- joint gaze_joint: origin xyz=0 0 0.0 rpy=0 0 0 -> xyz=0.015 0 0.022 rpy=0 0 0

File: coman_urdf/urdf/coman.urdf.xacro (robot description, xacro)
@@ -33,10 +33,10 @@
 	<link name ="Xtion_body">
     <inertial>
-      <origin xyz="0.0 0.0 0.0" rpy="0 0 0"/>
-      <mass value="0.89258227"/>
-      <inertia ixx="0.0001"  ixy="0.0"  ixz="0.0" iyy="0.0001" iyz="0.0" izz="0.0001" />
+      <origin xyz="0.047 0.0 0.40" rpy="0 0 0"/>
+      <mass value="0.39"/>
+      <inertia ixx="0.01"  ixy="3.34E-7"  ixz="-2.66E-4" iyy="0.009" iyz="1.97E-6" izz="5.1E-4" />
     </inertial>
     <visual>
-      <origin xyz="-0.005305004 0.0 -0.844329" rpy="0 0 -3.14159265359"/>
+      <origin xyz="-0.020281504 0.0 -0.68662053" rpy="0 0 -3.14159265359"/>
       <geometry name="Xtion_body_visual">
         <mesh filename="package://coman_urdf/meshes/collada/Xtion/xtion_base.dae" scale="0.03937 0.03937 0.03937" />
@@ -44,5 +44,5 @@
     </visual>
     <collision>
-      <origin xyz="-0.005305004 0.0 -0.844329" rpy="0 0 -3.14159265359"/>
+      <origin xyz="-0.020281504 0.0 -0.68662053" rpy="0 0 -3.14159265359"/>
       <geometry name="Xtion_body_collision">
         <mesh filename="package://coman_urdf/meshes/collada/simple/Xtion/xtion_base.dae" scale="0.03937 0.03937 0.03937" />
@@ -52,10 +52,10 @@
   <link name ="Xtion_cam_body">
     <inertial>
-      <origin xyz="0.0 0.0 0.0" rpy="0 0 0"/>
-      <mass value="0.89258227"/>
-      <inertia ixx="0.0001"  ixy="0.0"  ixz="0.0" iyy="0.0001" iyz="0.0" izz="0.0001" />
+      <origin xyz="0.0 0.0 0.0225" rpy="0 0 0"/>
+      <mass value="0.2"/>
+      <inertia ixx="0.00053"  ixy="0.0"  ixz="0.0" iyy="0.00008" iyz="0.0" izz="0.00053" />
     </inertial>
     <visual>
-      <origin xyz="-0.085305004 0.0 -1.284329" rpy="0 0 -3.14159265359"/>
+      <origin xyz="-0.0915 0.0 -1.2778" rpy="0 0 -3.14159265359"/>
       <geometry name="Xtion_cam_body_visual">
         <mesh filename="package://coman_urdf/meshes/collada/Xtion/xtion_cam_body.dae" scale="0.001 0.001 0.001" />
@@ -63,5 +63,5 @@
     </visual>
     <collision>
-      <origin xyz="-0.085305004 0.0 -1.284329" rpy="0 0 -3.14159265359"/>
+      <origin xyz="-0.0915 0.0 -1.2778" rpy="0 0 -3.14159265359"/>
       <geometry name="Xtion_cam_body_collision">
         <mesh filename="package://coman_urdf/meshes/collada/Xtion/xtion_cam_body.dae" scale="0.001 0.001 0.001" />

File: coman_urdf/urdf/coman_base.urdf.xacro (robot description, xacro)
@@ -483,5 +483,5 @@
 <xacro:if value="${GAZEBO_COMAN_USES_XTION}">
         <joint name="Xtion_body_joint" type="fixed">
-    		<parent link="torso"/>
+    		<parent link="DWYTorso"/>
     		<child link="Xtion_body"/>
     		<origin xyz="0 0 0" rpy="0 0 0" />
@@ -490,10 +490,13 @@
     		<parent link="Xtion_body"/>
     		<child link="Xtion_cam_body"/>
-    		<origin xyz="0.08 0 0.44" rpy="0 0 0" />
+		<origin xyz="0.071 0 0.591" rpy="0 1.396 0" />
+		<!--axis xyz="0 1 0" />
+    		<limit velocity="4.0" effort="5" lower="-0.4145" upper="1.57075" />
+    		<dynamics friction="0" damping="3.0"/-->
   	</joint>
         <joint name="gaze_joint" type="fixed">
     		<parent link="Xtion_cam_body"/>
     		<child link="gaze"/>
-    		<origin xyz="0 0 0.0" rpy="0 0 0" />
+    		<origin xyz="0.015 0 0.022" rpy="0 0 0" />
   	</joint>
 </xacro:if>

Commit message: Added fixed posed SoftHand in robo model. Need to be tested yet in simulation.

File: coman_urdf/urdf/coman.urdf (robot description, URDF)
Before this commit: robot COMAN, 45 links, 44 joints
Links:
- link LSoftHand: geometry collision mesh filename=package://coman_urdf/meshes/collada/simple/forearms/L_soft_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 scale=1E-3 1E-3 1E-3; visual mesh filename=package://coman_urdf/meshes/collada/forearms/L_soft_hand_op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 scale=1E-3 1E-3 1E-3
- link RSoftHand: geometry collision mesh filename=package://coman_urdf/meshes/collada/simple/forearms/R_soft_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 scale=1E-3 1E-3 1E-3; visual mesh filename=package://coman_urdf/meshes/collada/forearms/R_soft_hand_op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 scale=1E-3 1E-3 1E-3
Joints:
- joint l_handj: axis 1 0 0 -> (none); limit lower=-1.57075 upper=0.0 effort=5 velocity=4.0 -> (none); origin xyz=0 0 -0.04 rpy=0 0 0 -> xyz=0 0 -0.064 rpy=0 0 0; type revolute -> fixed
- joint r_handj: axis 1 0 0 -> (none); limit lower=0.0 upper=1.57075 effort=5 velocity=4.0 -> (none); origin xyz=0 0 -0.04 rpy=0 0 0 -> xyz=0 0 -0.064 rpy=0 0 0; type revolute -> fixed

File: coman_urdf/urdf/coman.urdf.xacro (robot description, xacro)
@@ -92,6 +92,18 @@
       <origin xyz="0 0 0" rpy="0 0 0" />
     </joint>
+    <xacro:include filename="$(find coman_urdf)/urdf/soft_hand.urdf.xacro" />
+    <xacro:unless value="${GAZEBO_COMAN_USES_SOFTHANDS_DRC_sw1_14}">
+      <joint name="r_handj" type="fixed">
+        <parent link="RWrMot3"/>
+        <child link="RSoftHand"/>
+        <origin xyz="0 0 -0.064" rpy="0 0 0"/>
+      </joint>
+      <joint name="l_handj" type="fixed">
+        <parent link="LWrMot3"/>
+        <child link="LSoftHand"/>
+        <origin xyz="0 0 -0.064" rpy="0 0 0"/>
+      </joint>
+    </xacro:unless>
     <xacro:if value="${GAZEBO_COMAN_USES_SOFTHANDS_DRC_sw1_14}">
-      <xacro:include filename="$(find coman_urdf)/urdf/soft_hand.urdf.xacro" />
       <joint name="r_handj" type="revolute">
         <parent link="RWrMot3"/>

File: coman_urdf/urdf/coman_config.urdf.xacro (robot description, xacro)
@@ -35,5 +35,4 @@
 #
 <xacro:property name="GAZEBO_COMAN_USES_NO_FOREARMS" value="true" />
-<xacro:property name="GAZEBO_COMAN_USES_NO_HANDS" value="false" />
 <xacro:property name="GAZEBO_COMAN_USES_7DOF_FOREARMS_DRC_14" value="true" />
 <xacro:property name="GAZEBO_COMAN_USES_SOFTHANDS_DRC_sw1_14" value="false" />
@@ -41,7 +40,6 @@
 -->
 <xacro:property name="GAZEBO_COMAN_USES_NO_FOREARMS" value="false" />
-<xacro:property name="GAZEBO_COMAN_USES_NO_HANDS" value="false" />
 <xacro:property name="GAZEBO_COMAN_USES_7DOF_FOREARMS_DRC_14" value="true" />
-<xacro:property name="GAZEBO_COMAN_USES_SOFTHANDS_DRC_sw1_14" value="true" />
+<xacro:property name="GAZEBO_COMAN_USES_SOFTHANDS_DRC_sw1_14" value="false" />
 <!--
 ####################################################

File: coman_urdf/urdf/soft_hand.urdf.xacro (robot description, xacro)
@@ -1,4 +1,45 @@
 <?xml version="1.0"?>
 <robot xmlns:xacro="http://ros.org/wiki/xacro" name="SoftHand">
+<xacro:unless value="${GAZEBO_COMAN_USES_SOFTHANDS_DRC_sw1_14}">
+<link name="RSoftHand">
+    <inertial>
+      <origin xyz="0 0 0" rpy="0 0 0"/>
+      <mass value="0.3"/>
+      <inertia ixx="0.001"  ixy="0"  ixz="0" iyy="0.001" iyz="0" izz="0.001" />
+    </inertial>
+    <visual>
+      <origin xyz="0 0.01 -0.04" rpy="0 0 3.14159265359"/>
+      <geometry name="RSoftHand_visual">
+        <mesh filename="package://coman_urdf/meshes/collada/forearms/R_soft_hand_open.dae" scale="1E-3 1E-3 1E-3" />
+      </geometry>
+   </visual>
+   <collision>
+      <origin xyz="0 0.01 -0.04" rpy="0 0 3.14159265359"/>
+      <geometry name="RSoftHand_collision">
+        <mesh filename="package://coman_urdf/meshes/collada/simple/forearms/R_soft_hand_open.dae" scale="1E-3 1E-3 1E-3" />
+      </geometry>
+   </collision>
+  </link>
+  <link name="LSoftHand">
+    <inertial>
+      <origin xyz="0 0 0" rpy="0 0 0"/>
+      <mass value="0.3"/>
+      <inertia ixx="0.001"  ixy="0"  ixz="0" iyy="0.001" iyz="0" izz="0.001" />
+    </inertial>
+    <visual>
+      <origin xyz="0.007 -0.012 -0.04" rpy="0 0 ${3.14159265359/2}"/>
+      <geometry name="LSoftHand_visual">
+        <mesh filename="package://coman_urdf/meshes/collada/forearms/L_soft_hand_open.dae" scale="1E-3 1E-3 1E-3" />
+      </geometry>
+   </visual>
+   <collision>
+     <origin xyz="0.007 -0.012 -0.04" rpy="0 0 ${3.14159265359/2}"/>
+      <geometry name="LSoftHand_collision">
+        <mesh filename="package://coman_urdf/meshes/collada/simple/forearms/L_soft_hand_open.dae" scale="1E-3 1E-3 1E-3" />
+      </geometry>
+   </collision>
+  </link>
+</xacro:unless>
+<xacro:if value="${GAZEBO_COMAN_USES_SOFTHANDS_DRC_sw1_14}">
 <!-- ## WRONG NUMBERS FOR... ok lasciamo perde... FIX THEM!! ## -->
   <link name="RSoftHand">
@@ -46,3 +87,4 @@
    </collision>
   </link>
+</xacro:if>
 </robot>
