Commit message: Default model has to be with hands

File: coman_urdf/urdf/coman.urdf (robot description, URDF)
Before this commit: robot COMAN, 45 links, 44 joints
Links:
- link LSoftHand: geometry collision box size=0.07 0.07 0.07; visual box size=0.07 0.07 0.07
- link RSoftHand: geometry collision box size=0.07 0.07 0.07; visual box size=0.07 0.07 0.07
Joints:
- joint l_handj: axis (none) -> 1 0 0; limit (none) -> lower=-1.57075 upper=0.0 effort=5 velocity=4.0; origin xyz=0 0 -0.064 rpy=0 0 0 -> xyz=0 0 -0.04 rpy=0 0 0; type fixed -> revolute
- joint r_handj: axis (none) -> 1 0 0; limit (none) -> lower=0.0 upper=1.57075 effort=5 velocity=4.0; origin xyz=0 0 -0.064 rpy=0 0 0 -> xyz=0 0 -0.04 rpy=0 0 0; type fixed -> revolute

File: coman_urdf/urdf/coman_config.urdf.xacro (robot description, xacro)
@@ -40,13 +40,13 @@
 -->
 <!-- 2) 7DOFS_FOREARMS -->
+<!--
 <xacro:property name="GAZEBO_COMAN_USES_NO_FOREARMS" value="false" />
 <xacro:property name="GAZEBO_COMAN_USES_7DOF_FOREARMS_DRC_14" value="true" />
 <xacro:property name="GAZEBO_COMAN_USES_SOFTHANDS_DRC_sw1_14" value="false" />
+-->
 <!-- 3) 7DOFS_FOREARMS + SOFT_HANDS -->
-<!--
 <xacro:property name="GAZEBO_COMAN_USES_NO_FOREARMS" value="false" />
 <xacro:property name="GAZEBO_COMAN_USES_7DOF_FOREARMS_DRC_14" value="true" />
 <xacro:property name="GAZEBO_COMAN_USES_SOFTHANDS_DRC_sw1_14" value="true" />
--->
 <!--
 ####################################################

Commit message: Set model back without hands. Set rotation of gaze to 0 0 0 for xtion

File: coman_urdf/urdf/coman.urdf (robot description, URDF)
Before this commit: robot COMAN, 45 links, 44 joints
Links:
- link LSoftHand: geometry collision mesh filename=package://coman_urdf/meshes/collada/simple/forearms/L_soft_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 scale=1E-3 1E-3 1E-3; visual mesh filename=package://coman_urdf/meshes/collada/forearms/L_soft_hand_op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 scale=1E-3 1E-3 1E-3
- link RSoftHand: geometry collision mesh filename=package://coman_urdf/meshes/collada/simple/forearms/R_soft_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 scale=1E-3 1E-3 1E-3; visual mesh filename=package://coman_urdf/meshes/collada/forearms/R_soft_hand_op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 scale=1E-3 1E-3 1E-3
Joints:
- joint Xtion_cam_body_joint: origin xyz=0.071 0 0.591 rpy=0 1.396 0 -> xyz=0.071 0 0.591 rpy=0 0 0
- joint l_handj: axis 1 0 0 -> (none); limit lower=-1.57075 upper=0.0 effort=5 velocity=4.0 -> (none); origin xyz=0 0 -0.04 rpy=0 0 0 -> xyz=0 0 -0.064 rpy=0 0 0; type revolute -> fixed
- joint r_handj: axis 1 0 0 -> (none); limit lower=0.0 upper=1.57075 effort=5 velocity=4.0 -> (none); origin xyz=0 0 -0.04 rpy=0 0 0 -> xyz=0 0 -0.064 rpy=0 0 0; type revolute -> fixed

File: coman_urdf/urdf/coman_base.urdf.xacro (robot description, xacro)
@@ -490,5 +490,6 @@
     		<parent link="Xtion_body"/>
     		<child link="Xtion_cam_body"/>
-		<origin xyz="0.071 0 0.591" rpy="0 1.396 0" />
+		<!-- origin xyz="0.071 0 0.591" rpy="0 1.396 0" / -->
+                <origin xyz="0.071 0 0.591" rpy="0 0 0" />
 		<!--axis xyz="0 1 0" />
     		<limit velocity="4.0" effort="5" lower="-0.4145" upper="1.57075" />

File: coman_urdf/urdf/coman_config.urdf.xacro (robot description, xacro)
@@ -40,13 +40,13 @@
 -->
 <!-- 2) 7DOFS_FOREARMS -->
+<xacro:property name="GAZEBO_COMAN_USES_NO_FOREARMS" value="false" />
+<xacro:property name="GAZEBO_COMAN_USES_7DOF_FOREARMS_DRC_14" value="true" />
+<xacro:property name="GAZEBO_COMAN_USES_SOFTHANDS_DRC_sw1_14" value="false" />
+<!-- 3) 7DOFS_FOREARMS + SOFT_HANDS -->
 <!--
 <xacro:property name="GAZEBO_COMAN_USES_NO_FOREARMS" value="false" />
 <xacro:property name="GAZEBO_COMAN_USES_7DOF_FOREARMS_DRC_14" value="true" />
-<xacro:property name="GAZEBO_COMAN_USES_SOFTHANDS_DRC_sw1_14" value="false" />
+<xacro:property name="GAZEBO_COMAN_USES_SOFTHANDS_DRC_sw1_14" value="true" />
 -->
-<!-- 3) 7DOFS_FOREARMS + SOFT_HANDS -->
-<xacro:property name="GAZEBO_COMAN_USES_NO_FOREARMS" value="false" />
-<xacro:property name="GAZEBO_COMAN_USES_7DOF_FOREARMS_DRC_14" value="true" />
-<xacro:property name="GAZEBO_COMAN_USES_SOFTHANDS_DRC_sw1_14" value="true" />
 <!--
 ####################################################

Commit message: Small update of position of fixed soft hands (added 6 mm in z tanslation).

File: coman_urdf/urdf/coman.urdf (robot description, URDF)
Before this commit: robot COMAN, 45 links, 44 joints
Joints:
- joint l_handj: origin xyz=0 0 -0.064 rpy=0 0 0 -> xyz=0 0 -0.07 rpy=0 0 0
- joint r_handj: origin xyz=0 0 -0.064 rpy=0 0 0 -> xyz=0 0 -0.07 rpy=0 0 0

File: coman_urdf/urdf/coman.urdf.xacro (robot description, xacro)
@@ -97,10 +97,10 @@
         <parent link="RWrMot3"/>
         <child link="RSoftHand"/>
-        <origin xyz="0 0 -0.064" rpy="0 0 0"/>
+        <origin xyz="0 0 -0.07" rpy="0 0 0"/>
       </joint>
       <joint name="l_handj" type="fixed">
         <parent link="LWrMot3"/>
         <child link="LSoftHand"/>
-        <origin xyz="0 0 -0.064" rpy="0 0 0"/>
+        <origin xyz="0 0 -0.07" rpy="0 0 0"/>
       </joint>
     </xacro:unless>

Commit message: Merged devel_all_models to master

File: coman_urdf/urdf/coman.urdf (robot description, URDF)
Before this commit: robot COMAN, 45 links, 44 joints
Links:
- link LSoftHand: geometry collision mesh filename=package://coman_urdf/meshes/collada/simple/forearms/L_soft_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 scale=1E-3 1E-3 1E-3; visual mesh filename=package://coman_urdf/meshes/collada/forearms/L_soft_hand_op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 scale=1E-3 1E-3 1E-3
- link RSoftHand: geometry collision mesh filename=package://coman_urdf/meshes/collada/simple/forearms/R_soft_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 scale=1E-3 1E-3 1E-3; visual mesh filename=package://coman_urdf/meshes/collada/forearms/R_soft_hand_op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 scale=1E-3 1E-3 1E-3
Joints:
- joint l_handj: axis 1 0 0 -> (none); limit lower=-1.57075 upper=0.0 effort=5 velocity=4.0 -> (none); origin xyz=0 0 -0.04 rpy=0 0 0 -> xyz=0 0 -0.07 rpy=0 0 0; type revolute -> fixed
- joint r_handj: axis 1 0 0 -> (none); limit lower=0.0 upper=1.57075 effort=5 velocity=4.0 -> (none); origin xyz=0 0 -0.04 rpy=0 0 0 -> xyz=0 0 -0.07 rpy=0 0 0; type revolute -> fixed

File: coman_urdf/urdf/coman_config.urdf.xacro (robot description, xacro)
@@ -1,6 +1,6 @@
 <?xml version="1.0"?>
 <robot xmlns:xacro="http://ros.org/wiki/xacro" name="COMAN">
-<xacro:property name="model_name" value="IIT Coman" />
-<xacro:property name="model_version" value="1.0" />
+<xacro:property name="model_name" value="IIT Coman w/ Softhand" />
+<xacro:property name="model_version" value="0.1" />
 <!--
 ####################################################
@@ -42,13 +42,13 @@
 -->
 <!-- 2) 7DOFS_FOREARMS -->
+<!--
 <xacro:property name="GAZEBO_COMAN_USES_NO_FOREARMS" value="false" />
 <xacro:property name="GAZEBO_COMAN_USES_7DOF_FOREARMS_DRC_14" value="true" />
 <xacro:property name="GAZEBO_COMAN_USES_SOFTHANDS_DRC_sw1_14" value="false" />
+-->
 <!-- 3) 7DOFS_FOREARMS + SOFT_HANDS -->
-<!--
 <xacro:property name="GAZEBO_COMAN_USES_NO_FOREARMS" value="false" />
 <xacro:property name="GAZEBO_COMAN_USES_7DOF_FOREARMS_DRC_14" value="true" />
 <xacro:property name="GAZEBO_COMAN_USES_SOFTHANDS_DRC_sw1_14" value="true" />
--->
 <!--
 ####################################################

Commit message: CHanged torque max in forearm and wrists joints

File: coman_urdf/urdf/coman.urdf (robot description, URDF)
Before this commit: robot COMAN, 45 links, 44 joints
Joints:
- joint LForearmPlate: limit lower=-1.5708 upper=1.5708 effort=50 velocity=4.0 -> lower=-1.5708 upper=1.5708 effort=5 velocity=4.0
- joint LWrj1: limit lower=-0.524 upper=0.524 effort=50 velocity=4.0 -> lower=-0.524 upper=0.524 effort=5 velocity=4.0
- joint LWrj2: limit lower=-0.785375 upper=1.395 effort=50 velocity=4.0 -> lower=-0.785375 upper=1.395 effort=5 velocity=4.0
- joint RForearmPlate: limit lower=-1.5708 upper=1.5708 effort=50 velocity=4.0 -> lower=-1.5708 upper=1.5708 effort=5 velocity=4.0
- joint RWrj1: limit lower=-0.524 upper=0.524 effort=50 velocity=4.0 -> lower=-0.524 upper=0.524 effort=5 velocity=4.0
- joint RWrj2: limit lower=-1.395 upper=0.785375 effort=50 velocity=4.0 -> lower=-1.395 upper=0.785375 effort=5 velocity=4.0

File: coman_urdf/urdf/forearms/7DOF_forearms_DRC_14/7DOF_forearms_DRC_14.urdf.xacro (robot description, xacro)
@@ -181,5 +181,5 @@
     <origin xyz="-0.015 0.0 ${-0.051 - Wrj1_to_FT}" rpy="0 0 0"/>
     <axis xyz="0 0 1" />
-    <limit velocity="4.0" effort="50" lower="-1.5708" upper="1.5708" />
+    <limit velocity="4.0" effort="5" lower="-1.5708" upper="1.5708" />
     <dynamics friction="0" damping="0.03"/>
   </joint>
@@ -189,5 +189,5 @@
     <origin xyz="0 0 ${-0.14368 + Wrj1_to_FT}" rpy="0 0 0"/>
     <axis xyz="0 1 0"/>
-    <limit velocity="4.0" effort="50" lower="-0.524" upper="0.524" />
+    <limit velocity="4.0" effort="5" lower="-0.524" upper="0.524" />
     <dynamics friction="0" damping="0.03"/>
   </joint>
@@ -197,5 +197,5 @@
     <origin xyz="0 0 0.0" rpy="0 0 0"/>
     <axis xyz="1 0 0"/>
-    <limit velocity="4.0" effort="50" lower="-0.785375" upper="1.395" />
+    <limit velocity="4.0" effort="5" lower="-0.785375" upper="1.395" />
     <dynamics friction="0" damping="0.03"/>
   </joint>
@@ -206,5 +206,5 @@
     <origin xyz="-0.015 0.0 ${-0.051 - Wrj1_to_FT}" rpy="0 0 0"/>
     <axis xyz="0 0 1" />
-    <limit velocity="4.0" effort="50" lower="-1.5708" upper="1.5708" />
+    <limit velocity="4.0" effort="5" lower="-1.5708" upper="1.5708" />
     <dynamics friction="0" damping="0.03"/>
   </joint>
@@ -214,5 +214,5 @@
     <origin xyz="0 0 ${-0.14368 + Wrj1_to_FT}" rpy="0 0 0"/>
     <axis xyz="0 1 0"/>
-    <limit velocity="4.0" effort="50" lower="-0.524" upper="0.524" />
+    <limit velocity="4.0" effort="5" lower="-0.524" upper="0.524" />
     <dynamics friction="0" damping="0.03"/>
   </joint>
@@ -222,5 +222,5 @@
     <origin xyz="0 0 0.0" rpy="0 0 0"/>
     <axis xyz="1 0 0"/>
-    <limit velocity="4.0" effort="50" lower="-1.395" upper="0.785375" />
+    <limit velocity="4.0" effort="5" lower="-1.395" upper="0.785375" />
     <dynamics friction="0" damping="0.03"/>
   </joint>

Commit message: Changed imu orientation according to measurement

File: coman_urdf/urdf/coman.urdf (robot description, URDF)
Before this commit: robot COMAN, 45 links, 44 joints
Links:
- link LElb: geometry collision mesh filename=package://coman_urdf/meshes/collada/simple/forearms/elbow.s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 scale=1.0 1.0 1.0; visual mesh filename=package://coman_urdf/meshes/collada/forearms/elbow.dae scale=1.0 1.0 1.0
- link LForearm: geometry collision mesh filename=package://coman_urdf/meshes/collada/simple/forearms/forearm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 scale=1.0 1.0 1.0; visual mesh filename=package://coman_urdf/meshes/collada/forearms/forearm_lowpol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 scale=0.1 0.1 0.1
- link LSoftHand: geometry collision mesh filename=package://coman_urdf/meshes/collada/simple/forearms/L_soft_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 scale=1E-3 1E-3 1E-3; visual mesh filename=package://coman_urdf/meshes/collada/forearms/L_soft_hand_op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 scale=0.1 0.1 0.1
- link RElb: geometry collision mesh filename=package://coman_urdf/meshes/collada/simple/forearms/elbow.s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 scale=1.0 1.0 1.0; visual mesh filename=package://coman_urdf/meshes/collada/forearms/elbow.dae scale=1.0 1.0 1.0
- link RForearm: geometry collision mesh filename=package://coman_urdf/meshes/collada/simple/forearms/forearm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 scale=1.0 1.0 1.0; visual mesh filename=package://coman_urdf/meshes/collada/forearms/forearm_lowpol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 scale=0.1 0.1 0.1
- link RSoftHand: geometry collision mesh filename=package://coman_urdf/meshes/collada/simple/forearms/R_soft_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 scale=1E-3 1E-3 1E-3; visual mesh filename=package://coman_urdf/meshes/collada/forearms/R_soft_hand_op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 scale=0.1 0.1 0.1
- link Xtion_cam_body: geometry collision mesh filename=package://coman_urdf/meshes/collada/simple/Xtion/xtion_cam_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 scale=0.001 0.001 0.001; visual mesh filename=package://coman_urdf/meshes/collada/Xtion/xtion_cam_body.dae scale=0.001 0.001 0.001

File: coman_urdf/urdf/coman_robot.urdf.xacro (robot description, xacro)
@@ -24,5 +24,5 @@
     <parent link="Waist"/>
     <child link="imu_link"/>
-    <origin xyz="-0.072 -0.0068 0.044" rpy="0 0 0"/>
+    <origin xyz="-0.072 -0.0068 0.044" rpy="0 3.14159 0"/>
   </joint>
   <xacro:include filename="$(find coman_urdf)/urdf/microstrain_3dmgx2_imu.gazebo.xacro" />

Commit message: Fixed error where sagittal and lateral joints and links had switched names

File: coman_urdf/urdf/coman.urdf (robot description, URDF)
Before this commit: robot COMAN, 45 links, 44 joints
Links:
- link DWL: mass 0.75398402 -> 0.54588774; geometry collision mesh filename=package://coman_urdf/meshes/collada/simple/simple_asm0001_c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 scale=0.03937 0.03937 0.03937; visual mesh filename=package://coman_urdf/meshes/collada/asm0001_collada_09_prt.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 scale=0.03937 0.03937 0.03937
- link DWS: mass 0.54588774 -> 0.75398402; geometry collision mesh filename=package://coman_urdf/meshes/collada/simple/simple_asm0001_c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 scale=0.03937 0.03937 0.03937; visual mesh filename=package://coman_urdf/meshes/collada/asm0001_collada_08_prt.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 scale=0.03937 0.03937 0.03937
Joints:
- joint WaistLat: axis 0 1 0 -> 0.939692608 0 0.3420201433; limit lower=-0.3491 upper=0.8727 effort=50 velocity=4.0 -> lower=-0.5236 upper=0.5235 effort=50 velocity=4.0; origin xyz=0 0 0 rpy=0 0 0 -> xyz=0.020281504 0 0.11912053 rpy=0 0 0; parent DWS -> Waist
- joint WaistSag: axis 0.939692608 0 0.3420201433 -> 0 1 0; limit lower=-0.5236 upper=0.5235 effort=50 velocity=4.0 -> lower=-0.3491 upper=0.8727 effort=50 velocity=4.0; origin xyz=0.020281504 0 0.11912053 rpy=0 0 0 -> xyz=0 0 0 rpy=0 0 0; parent Waist -> DWL
- joint WaistYaw: parent DWL -> DWS

File: coman_urdf/urdf/coman_base.urdf.xacro (robot description, xacro)
@@ -29,5 +29,5 @@
     </collision>
   </link>
-  <link name ="DWS">
+  <link name ="DWL">
     <inertial>
       <origin xyz="4.2999707E-4 -0.0097650317 0.033011157" rpy="0 0 0"/>
@@ -37,5 +37,5 @@
     <visual>
       <origin xyz="-0.020281504 0 -0.63912053" rpy="0 0 -3.14159265359"/>
-      <geometry name="DWS_visual">
+      <geometry name="DWL_visual">
         <mesh filename="package://coman_urdf/meshes/collada/asm0001_collada_09_prt.dae" scale="0.03937 0.03937 0.03937" />
       </geometry>
@@ -43,10 +43,10 @@
     <collision>
       <origin xyz="-0.020281504 0 -0.63912053" rpy="0 0 -3.14159265359"/>
-      <geometry name="DWS_collision">
+      <geometry name="DWL_collision">
         <mesh filename="package://coman_urdf/meshes/collada/simple/simple_asm0001_collada_09_prt.stl" scale="0.03937 0.03937 0.03937" />
       </geometry>
     </collision>
   </link>
-  <link name ="DWL">
+  <link name ="DWS">
     <inertial>
       <origin xyz="-0.0021273416 0.0033575235 -0.0010076896" rpy="0 0 0"/>
@@ -56,5 +56,5 @@
     <visual>
       <origin xyz="-0.020281504 0 -0.63912053" rpy="0 0 -3.14159265359"/>
-      <geometry name="DWL_visual">
+      <geometry name="DWS_visual">
         <mesh filename="package://coman_urdf/meshes/collada/asm0001_collada_08_prt.dae" scale="0.03937 0.03937 0.03937" />
       </geometry>
@@ -62,5 +62,5 @@
     <collision>
       <origin xyz="-0.020281504 0 -0.63912053" rpy="0 0 -3.14159265359"/>
-      <geometry name="DWL_collision">
+      <geometry name="DWS_collision">
         <mesh filename="package://coman_urdf/meshes/collada/simple/simple_asm0001_collada_08_prt.stl" scale="0.03937 0.03937 0.03937" />
       </geometry>
@@ -510,7 +510,7 @@
 </xacro:unless>
 <!-- ********************TORSO******************** -->
-  <joint name="WaistSag" type="revolute"> <!-- Wrong name! need to fix this... -->
+  <joint name="WaistLat" type="revolute"> <!-- Wrong name! need to fix this... -->
     <parent link="Waist"/>
-    <child link="DWS"/>
+    <child link="DWL"/>
     <origin xyz="0.020281504 0 0.11912053" rpy="0 0 0" />
     <axis xyz="0.939692608 0 0.3420201433" />
@@ -519,14 +519,14 @@
     <dynamics friction="0" damping="3.0"/>
   </joint>
-  <joint name="WaistLat" type="revolute"> <!-- Wrong name! need to fix this... -->
+  <joint name="WaistSag" type="revolute"> <!-- Wrong name! need to fix this... -->
+    <parent link="DWL"/>
+    <child link="DWS"/>
+    <origin xyz="0 0 0" rpy="0 0 0" />
+    <axis xyz="0 1 0" />
+    <limit velocity="4.0" effort="50" lower="-0.3491" upper="0.8727" />
+    <dynamics friction="0" damping="3.0"/>
+  </joint>
+  <joint name="WaistYaw" type="revolute">
     <parent link="DWS"/>
-    <child link="DWL"/>
-    <origin xyz="0 0 0" rpy="0 0 0" />
-    <axis xyz="0 1 0" />
-    <limit velocity="4.0" effort="50" lower="-0.3491" upper="0.8727" />
-    <dynamics friction="0" damping="3.0"/>
-  </joint>
-  <joint name="WaistYaw" type="revolute">
-    <parent link="DWL"/>
     <child link="DWYTorso"/>
     <origin xyz="0 0 0.04749999" rpy="0 0 0" />

File: coman_urdf/urdf/coman_hands.urdf (robot description, URDF)
Before this commit: robot COMAN, 45 links, 44 joints
Links:
- link DWL: mass 0.75398402 -> 0.54588774; geometry collision mesh filename=package://coman_urdf/meshes/collada/simple/simple_asm0001_c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 scale=0.03937 0.03937 0.03937; visual mesh filename=package://coman_urdf/meshes/collada/asm0001_collada_09_prt.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 scale=0.03937 0.03937 0.03937
- link DWS: mass 0.54588774 -> 0.75398402; geometry collision mesh filename=package://coman_urdf/meshes/collada/simple/simple_asm0001_c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 scale=0.03937 0.03937 0.03937; visual mesh filename=package://coman_urdf/meshes/collada/asm0001_collada_08_prt.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 scale=0.03937 0.03937 0.03937
Joints:
- joint WaistLat: axis 0 1 0 -> 0.939692608 0 0.3420201433; limit lower=-0.3491 upper=0.8727 effort=50 velocity=4.0 -> lower=-0.5236 upper=0.5235 effort=50 velocity=4.0; origin xyz=0 0 0 rpy=0 0 0 -> xyz=0.020281504 0 0.11912053 rpy=0 0 0; parent DWS -> Waist
- joint WaistSag: axis 0.939692608 0 0.3420201433 -> 0 1 0; limit lower=-0.5236 upper=0.5235 effort=50 velocity=4.0 -> lower=-0.3491 upper=0.8727 effort=50 velocity=4.0; origin xyz=0.020281504 0 0.11912053 rpy=0 0 0 -> xyz=0 0 0 rpy=0 0 0; parent Waist -> DWL
- joint WaistYaw: parent DWL -> DWS

File: coman_urdf/urdf/coman_no_forearms.urdf (robot description, URDF)
Before this commit: robot COMAN, 37 links, 36 joints
Links:
- link DWL: mass 0.75398402 -> 0.54588774; geometry collision mesh filename=package://coman_urdf/meshes/collada/simple/simple_asm0001_c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 scale=0.03937 0.03937 0.03937; visual mesh filename=package://coman_urdf/meshes/collada/asm0001_collada_09_prt.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 scale=0.03937 0.03937 0.03937
- link DWS: mass 0.54588774 -> 0.75398402; geometry collision mesh filename=package://coman_urdf/meshes/collada/simple/simple_asm0001_c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 scale=0.03937 0.03937 0.03937; visual mesh filename=package://coman_urdf/meshes/collada/asm0001_collada_08_prt.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 scale=0.03937 0.03937 0.03937
Joints:
- joint WaistLat: axis 0 1 0 -> 0.939692608 0 0.3420201433; limit lower=-0.3491 upper=0.8727 effort=50 velocity=4.0 -> lower=-0.5236 upper=0.5235 effort=50 velocity=4.0; origin xyz=0 0 0 rpy=0 0 0 -> xyz=0.020281504 0 0.11912053 rpy=0 0 0; parent DWS -> Waist
- joint WaistSag: axis 0.939692608 0 0.3420201433 -> 0 1 0; limit lower=-0.5236 upper=0.5235 effort=50 velocity=4.0 -> lower=-0.3491 upper=0.8727 effort=50 velocity=4.0; origin xyz=0.020281504 0 0.11912053 rpy=0 0 0 -> xyz=0 0 0 rpy=0 0 0; parent Waist -> DWL
- joint WaistYaw: parent DWL -> DWS
