Commit message: Added reference frames in feet to compute convex hull

File: coman_urdf/urdf/coman.urdf (robot description, URDF)
Before this commit: robot COMAN, 45 links, 44 joints
Links:
- added link l_foot_lower_left_link
- added link l_foot_lower_right_link
- added link l_foot_upper_left_link
- added link l_foot_upper_right_link
- added link r_foot_lower_left_link
- added link r_foot_lower_right_link
- added link r_foot_upper_left_link
- added link r_foot_upper_right_link
Joints:
- added joint l_foot_lower_left_joint: type fixed, parent l_sole, child l_foot_lower_left_link, origin xyz=-0.07 -0.05 0 rpy=0 0 0
- added joint l_foot_lower_right_joint: type fixed, parent l_sole, child l_foot_lower_right_link, origin xyz=-0.07 0.05 0 rpy=0 0 0
- added joint l_foot_upper_left_joint: type fixed, parent l_sole, child l_foot_upper_left_link, origin xyz=0.13 -0.05 0 rpy=0 0 0
- added joint l_foot_upper_right_joint: type fixed, parent l_sole, child l_foot_upper_right_link, origin xyz=0.13 0.05 0 rpy=0 0 0
- added joint r_foot_lower_left_joint: type fixed, parent r_sole, child r_foot_lower_left_link, origin xyz=-0.07 -0.05 0 rpy=0 0 0
- added joint r_foot_lower_right_joint: type fixed, parent r_sole, child r_foot_lower_right_link, origin xyz=-0.07 0.05 0 rpy=0 0 0
- added joint r_foot_upper_left_joint: type fixed, parent r_sole, child r_foot_upper_left_link, origin xyz=0.13 -0.05 0 rpy=0 0 0
- added joint r_foot_upper_right_joint: type fixed, parent r_sole, child r_foot_upper_right_link, origin xyz=0.13 0.05 0 rpy=0 0 0

File: coman_urdf/urdf/coman.urdf.xacro (robot description, xacro)
@@ -29,4 +29,6 @@
 <!-- The coordinate frame called torso is attached to the lowest body of the model which is a parent of l_gripper, r_gripper and gaze. -->
  <link name="torso"/>
+<!-- Reference frames in feet -->
+<xacro:include filename="$(find coman_urdf)/urdf/foot_reference_frame.urdf.xacro" />
 <!-- Head -->
 <xacro:if value="${GAZEBO_COMAN_USES_XTION}">
@@ -72,5 +74,5 @@
 <link name="gaze"/>
 <!-- ************ COMAN BASE ************** -->
-<xacro:include filename="$(find coman_urdf)//urdf/coman_base.urdf.xacro"/>
+<xacro:include filename="$(find coman_urdf)/urdf/coman_base.urdf.xacro"/>
 <!-- ************ FOREARMS ************ -->
 <xacro:if value="${GAZEBO_COMAN_USES_NO_FOREARMS}">

File: coman_urdf/urdf/coman_hands.urdf (robot description, URDF)
Before this commit: robot COMAN, 45 links, 44 joints
Links:
- added link l_foot_lower_left_link
- added link l_foot_lower_right_link
- added link l_foot_upper_left_link
- added link l_foot_upper_right_link
- added link r_foot_lower_left_link
- added link r_foot_lower_right_link
- added link r_foot_upper_left_link
- added link r_foot_upper_right_link
Joints:
- added joint l_foot_lower_left_joint: type fixed, parent l_sole, child l_foot_lower_left_link, origin xyz=-0.07 -0.05 0 rpy=0 0 0
- added joint l_foot_lower_right_joint: type fixed, parent l_sole, child l_foot_lower_right_link, origin xyz=-0.07 0.05 0 rpy=0 0 0
- added joint l_foot_upper_left_joint: type fixed, parent l_sole, child l_foot_upper_left_link, origin xyz=0.13 -0.05 0 rpy=0 0 0
- added joint l_foot_upper_right_joint: type fixed, parent l_sole, child l_foot_upper_right_link, origin xyz=0.13 0.05 0 rpy=0 0 0
- added joint r_foot_lower_left_joint: type fixed, parent r_sole, child r_foot_lower_left_link, origin xyz=-0.07 -0.05 0 rpy=0 0 0
- added joint r_foot_lower_right_joint: type fixed, parent r_sole, child r_foot_lower_right_link, origin xyz=-0.07 0.05 0 rpy=0 0 0
- added joint r_foot_upper_left_joint: type fixed, parent r_sole, child r_foot_upper_left_link, origin xyz=0.13 -0.05 0 rpy=0 0 0
- added joint r_foot_upper_right_joint: type fixed, parent r_sole, child r_foot_upper_right_link, origin xyz=0.13 0.05 0 rpy=0 0 0

File: coman_urdf/urdf/coman_no_forearms.urdf (robot description, URDF)
Before this commit: robot COMAN, 37 links, 36 joints
Links:
- added link l_foot_lower_left_link
- added link l_foot_lower_right_link
- added link l_foot_upper_left_link
- added link l_foot_upper_right_link
- added link r_foot_lower_left_link
- added link r_foot_lower_right_link
- added link r_foot_upper_left_link
- added link r_foot_upper_right_link
Joints:
- added joint l_foot_lower_left_joint: type fixed, parent l_sole, child l_foot_lower_left_link, origin xyz=-0.07 -0.05 0 rpy=0 0 0
- added joint l_foot_lower_right_joint: type fixed, parent l_sole, child l_foot_lower_right_link, origin xyz=-0.07 0.05 0 rpy=0 0 0
- added joint l_foot_upper_left_joint: type fixed, parent l_sole, child l_foot_upper_left_link, origin xyz=0.13 -0.05 0 rpy=0 0 0
- added joint l_foot_upper_right_joint: type fixed, parent l_sole, child l_foot_upper_right_link, origin xyz=0.13 0.05 0 rpy=0 0 0
- added joint r_foot_lower_left_joint: type fixed, parent r_sole, child r_foot_lower_left_link, origin xyz=-0.07 -0.05 0 rpy=0 0 0
- added joint r_foot_lower_right_joint: type fixed, parent r_sole, child r_foot_lower_right_link, origin xyz=-0.07 0.05 0 rpy=0 0 0
- added joint r_foot_upper_left_joint: type fixed, parent r_sole, child r_foot_upper_left_link, origin xyz=0.13 -0.05 0 rpy=0 0 0
- added joint r_foot_upper_right_joint: type fixed, parent r_sole, child r_foot_upper_right_link, origin xyz=0.13 0.05 0 rpy=0 0 0

Commit message: Moved IMU link and joint inside coman.urdf.xacro. Fixed names of foot reference

File: coman_urdf/urdf/coman.urdf (robot description, URDF)
Before this commit: robot COMAN, 53 links, 52 joints
Links:
- added link imu_link, mass 0.01; visual box size=0.01 0.01 0.01
Joints:
- added joint imu_joint: type fixed, parent Waist, child imu_link, origin xyz=-0.072 -0.0068 0.044 rpy=0 3.14159 0
- joint l_foot_lower_left_joint: origin xyz=-0.07 -0.05 0 rpy=0 0 0 -> xyz=-0.07 0.05 0 rpy=0 0 0
- joint l_foot_lower_right_joint: origin xyz=-0.07 0.05 0 rpy=0 0 0 -> xyz=-0.07 -0.05 0 rpy=0 0 0
- joint l_foot_upper_left_joint: origin xyz=0.13 -0.05 0 rpy=0 0 0 -> xyz=0.13 0.05 0 rpy=0 0 0
- joint l_foot_upper_right_joint: origin xyz=0.13 0.05 0 rpy=0 0 0 -> xyz=0.13 -0.05 0 rpy=0 0 0
- joint r_foot_lower_left_joint: origin xyz=-0.07 -0.05 0 rpy=0 0 0 -> xyz=-0.07 0.05 0 rpy=0 0 0
- joint r_foot_lower_right_joint: origin xyz=-0.07 0.05 0 rpy=0 0 0 -> xyz=-0.07 -0.05 0 rpy=0 0 0
- joint r_foot_upper_left_joint: origin xyz=0.13 -0.05 0 rpy=0 0 0 -> xyz=0.13 0.05 0 rpy=0 0 0
- joint r_foot_upper_right_joint: origin xyz=0.13 0.05 0 rpy=0 0 0 -> xyz=0.13 -0.05 0 rpy=0 0 0

File: coman_urdf/urdf/coman.urdf.xacro (robot description, xacro)
@@ -138,3 +138,22 @@
 	</joint>
 </xacro:if>
+<!-- IMU -->
+  <link name="imu_link">
+    <inertial>
+      <mass value="0.01"/>
+      <origin xyz="0 0 0"/>
+      <inertia ixx="1.0E-6" ixy="0" ixz="0" iyy="1.0E-6" iyz="0" izz="1.0E-6"/>
+    </inertial>
+    <visual>
+      <origin rpy="0 0 0" xyz="0 0 0"/>
+      <geometry>
+        <box size="0.01 0.01 0.01"/>
+      </geometry>
+    </visual>
+  </link>
+  <joint name="imu_joint" type="fixed">
+    <parent link="Waist"/>
+    <child link="imu_link"/>
+    <origin xyz="-0.072 -0.0068 0.044" rpy="0 3.14159 0"/>
+  </joint>
 </robot>

File: coman_urdf/urdf/coman_hands.urdf (robot description, URDF)
Before this commit: robot COMAN, 53 links, 52 joints
Links:
- added link imu_link, mass 0.01; visual box size=0.01 0.01 0.01
Joints:
- added joint imu_joint: type fixed, parent Waist, child imu_link, origin xyz=-0.072 -0.0068 0.044 rpy=0 3.14159 0
- joint l_foot_lower_left_joint: origin xyz=-0.07 -0.05 0 rpy=0 0 0 -> xyz=-0.07 0.05 0 rpy=0 0 0
- joint l_foot_lower_right_joint: origin xyz=-0.07 0.05 0 rpy=0 0 0 -> xyz=-0.07 -0.05 0 rpy=0 0 0
- joint l_foot_upper_left_joint: origin xyz=0.13 -0.05 0 rpy=0 0 0 -> xyz=0.13 0.05 0 rpy=0 0 0
- joint l_foot_upper_right_joint: origin xyz=0.13 0.05 0 rpy=0 0 0 -> xyz=0.13 -0.05 0 rpy=0 0 0
- joint r_foot_lower_left_joint: origin xyz=-0.07 -0.05 0 rpy=0 0 0 -> xyz=-0.07 0.05 0 rpy=0 0 0
- joint r_foot_lower_right_joint: origin xyz=-0.07 0.05 0 rpy=0 0 0 -> xyz=-0.07 -0.05 0 rpy=0 0 0
- joint r_foot_upper_left_joint: origin xyz=0.13 -0.05 0 rpy=0 0 0 -> xyz=0.13 0.05 0 rpy=0 0 0
- joint r_foot_upper_right_joint: origin xyz=0.13 0.05 0 rpy=0 0 0 -> xyz=0.13 -0.05 0 rpy=0 0 0

File: coman_urdf/urdf/coman_no_forearms.urdf (robot description, URDF)
Before this commit: robot COMAN, 45 links, 44 joints
Links:
- added link imu_link, mass 0.01; visual box size=0.01 0.01 0.01
Joints:
- added joint imu_joint: type fixed, parent Waist, child imu_link, origin xyz=-0.072 -0.0068 0.044 rpy=0 3.14159 0
- joint l_foot_lower_left_joint: origin xyz=-0.07 -0.05 0 rpy=0 0 0 -> xyz=-0.07 0.05 0 rpy=0 0 0
- joint l_foot_lower_right_joint: origin xyz=-0.07 0.05 0 rpy=0 0 0 -> xyz=-0.07 -0.05 0 rpy=0 0 0
- joint l_foot_upper_left_joint: origin xyz=0.13 -0.05 0 rpy=0 0 0 -> xyz=0.13 0.05 0 rpy=0 0 0
- joint l_foot_upper_right_joint: origin xyz=0.13 0.05 0 rpy=0 0 0 -> xyz=0.13 -0.05 0 rpy=0 0 0
- joint r_foot_lower_left_joint: origin xyz=-0.07 -0.05 0 rpy=0 0 0 -> xyz=-0.07 0.05 0 rpy=0 0 0
- joint r_foot_lower_right_joint: origin xyz=-0.07 0.05 0 rpy=0 0 0 -> xyz=-0.07 -0.05 0 rpy=0 0 0
- joint r_foot_upper_left_joint: origin xyz=0.13 -0.05 0 rpy=0 0 0 -> xyz=0.13 0.05 0 rpy=0 0 0
- joint r_foot_upper_right_joint: origin xyz=0.13 0.05 0 rpy=0 0 0 -> xyz=0.13 -0.05 0 rpy=0 0 0

File: coman_urdf/urdf/coman_robot.urdf.xacro (robot description, xacro)
@@ -7,23 +7,4 @@
   -->
   <xacro:include filename="$(find coman_urdf)/urdf/coman.urdf.xacro" />
-<!-- IMU -->
-  <link name="imu_link">
-    <inertial>
-      <mass value="0.01"/>
-      <origin xyz="0 0 0"/>
-      <inertia ixx="1.0E-6" ixy="0" ixz="0" iyy="1.0E-6" iyz="0" izz="1.0E-6"/>
-    </inertial>
-    <visual>
-      <origin rpy="0 0 0" xyz="0 0 0"/>
-      <geometry>
-        <box size="0.01 0.01 0.01"/>
-      </geometry>
-    </visual>
-  </link>
-  <joint name="imu_joint" type="fixed">
-    <parent link="Waist"/>
-    <child link="imu_link"/>
-    <origin xyz="-0.072 -0.0068 0.044" rpy="0 3.14159 0"/>
-  </joint>
   <xacro:include filename="$(find coman_urdf)/urdf/microstrain_3dmgx2_imu.gazebo.xacro" />
   <xacro:if value="$(optenv GAZEBO_COMAN_USES_ROS false)">

File: coman_urdf/urdf/foot_reference_frame.urdf.xacro (robot description, xacro)
@@ -16,8 +16,8 @@
 	<xacro:macro name="references_frame_foot" params="parent name">
 	<!-- macro for reference frames in foot -->
-		<xacro:reference_frame_foot parent="${parent}" name="${name}_upper_right" x="${x_positive}" y="${y_positive}" />
-		<xacro:reference_frame_foot parent="${parent}" name="${name}_upper_left" x="${x_positive}" y="${y_negative}" />
-		<xacro:reference_frame_foot parent="${parent}" name="${name}_lower_right" x="${x_negative}" y="${y_positive}" />
-		<xacro:reference_frame_foot parent="${parent}" name="${name}_lower_left" x="${x_negative}" y="${y_negative}" />
+		<xacro:reference_frame_foot parent="${parent}" name="${name}_upper_right" x="${x_positive}" y="${y_negative}" />
+		<xacro:reference_frame_foot parent="${parent}" name="${name}_upper_left" x="${x_positive}" y="${y_positive}" />
+		<xacro:reference_frame_foot parent="${parent}" name="${name}_lower_right" x="${x_negative}" y="${y_negative}" />
+		<xacro:reference_frame_foot parent="${parent}" name="${name}_lower_left" x="${x_negative}" y="${y_positive}" />
 	</xacro:macro>
 	<xacro:references_frame_foot parent="l_sole" name="l_foot"/>

Commit message: Started refactor of coman xacro. Added torso refactored.

File: coman_urdf/urdf/coman.urdf (robot description, URDF)
Before this commit: robot COMAN, 54 links, 53 joints
Joints:
- joint WaistLat: axis 0.939692608 0 0.3420201433 -> 0.93969262078 0 0.34202014332

File: coman_urdf/urdf/coman.urdf.xacro (robot description, xacro)
@@ -13,6 +13,4 @@
 <!-- This links are defined in order to be compliant with http://www.ros.org/reps/rep-0120.html#coordinate-frames
 and to define the end effectors of the robot -->
-<!-- The coordinate frame called base_link is rigidly attached to the robot root body. It is recommended to choose the robot waist as its root body. The base_link can be attached to the root in any arbitrary position or orientation; for every hardware platform there will be a different place on the base that provides an obvious point of reference. Note that REP 103 [1] specifies a preferred orientation for frames. -->
-  <link name="base_link"/>
 <!-- position and orientation of the arm regardless of the tool (grasping device for instance) attached to it -->
   <link name="l_wrist"/>

File: coman_urdf/urdf/coman_base.urdf.xacro (robot description, xacro)
@@ -10,80 +10,5 @@
 <!-- ********************TORSO******************** -->
 <!-- first real link of the robot, inertial reference frame -->
-  <link name="Waist">
-    <inertial>
-      <origin xyz="-0.026391145 -5.8216364E-4 0.052632312" rpy="0 0 0"/>
-      <mass value="1.8008695"/>
-      <inertia ixx="0.0051032982"  ixy="-5.7170981E-5"  ixz="0.0016920543" iyy="0.006241636" iyz="1.7225949E-5" izz="0.0024517762" />
-    </inertial>
-    <visual>
-      <origin xyz="0 0 -0.52" rpy="0 0 -3.14159265359"/>
-      <geometry name="Waist_visual">
-        <mesh filename="package://coman_urdf/meshes/collada/asm0001_collada_07_prt.dae" scale="0.03937 0.03937 0.03937"/>
-      </geometry>
-    </visual>
-    <collision>
-      <origin xyz="0 0 -0.52" rpy="0 0 -3.14159265359"/>
-      <geometry name="Waist_collision">
-        <mesh filename="package://coman_urdf/meshes/collada/simple/simple_asm0001_collada_07_prt.stl" scale="0.03937 0.03937 0.03937"/>
-      </geometry>
-    </collision>
-  </link>
-  <link name ="DWL">
-    <inertial>
-      <origin xyz="4.2999707E-4 -0.0097650317 0.033011157" rpy="0 0 0"/>
-      <mass value="0.54588774"/>
-      <inertia ixx="9.7126578E-4"  ixy="-7.2101244E-7"  ixz="1.1440119E-6" iyy="7.4686706E-4" iyz="-1.7450917E-4" izz="6.2196235E-4" />
-    </inertial>
-    <visual>
-      <origin xyz="-0.020281504 0 -0.63912053" rpy="0 0 -3.14159265359"/>
-      <geometry name="DWL_visual">
-        <mesh filename="package://coman_urdf/meshes/collada/asm0001_collada_09_prt.dae" scale="0.03937 0.03937 0.03937" />
-      </geometry>
-    </visual>
-    <collision>
-      <origin xyz="-0.020281504 0 -0.63912053" rpy="0 0 -3.14159265359"/>
-      <geometry name="DWL_collision">
-        <mesh filename="package://coman_urdf/meshes/collada/simple/simple_asm0001_collada_09_prt.stl" scale="0.03937 0.03937 0.03937" />
-      </geometry>
-    </collision>
-  </link>
-  <link name ="DWS">
-    <inertial>
-      <origin xyz="-0.0021273416 0.0033575235 -0.0010076896" rpy="0 0 0"/>
-      <mass value="0.75398402"/>
-      <inertia ixx="3.4093348E-4"  ixy="-6.2120042E-6"  ixz="-1.3863473E-6" iyy="3.9581916E-4" iyz="1.443019E-6" izz="3.7449753E-4" />
-    </inertial>
-    <visual>
-      <origin xyz="-0.020281504 0 -0.63912053" rpy="0 0 -3.14159265359"/>
-      <geometry name="DWS_visual">
-        <mesh filename="package://coman_urdf/meshes/collada/asm0001_collada_08_prt.dae" scale="0.03937 0.03937 0.03937" />
-      </geometry>
-    </visual>
-    <collision>
-      <origin xyz="-0.020281504 0 -0.63912053" rpy="0 0 -3.14159265359"/>
-      <geometry name="DWS_collision">
-        <mesh filename="package://coman_urdf/meshes/collada/simple/simple_asm0001_collada_08_prt.stl" scale="0.03937 0.03937 0.03937" />
-      </geometry>
-    </collision>
-  </link>
-  <link name ="DWYTorso">
-    <inertial>
-      <origin xyz="-0.0358501 1.8286043E-5 0.117557148" rpy="0 0 0"/>
-      <mass value="6.3617175"/>
-      <inertia ixx="0.034089342"  ixy="-9.8308572E-6"  ixz="-7.5649290E-4" iyy="0.030117357" iyz="6.2443771E-6" izz="0.025296582" />
-    </inertial>
-    <visual>
-      <origin xyz="-0.020281504 0.0 -0.68662053" rpy="0 0 -3.14159265359"/>
-      <geometry name="DWYTorso_visual">
-        <mesh filename="package://coman_urdf/meshes/collada/asm0001_collada_10_prt.dae" scale="0.03937 0.03937 0.03937" />
-      </geometry>
-    </visual>
-    <collision>
-      <origin xyz="-0.020281504 0.0 -0.68662053" rpy="0 0 -3.14159265359"/>
-      <geometry name="DWYTorso_collision">
-        <mesh filename="package://coman_urdf/meshes/collada/simple/simple_asm0001_collada_10_prt.stl" scale="0.03937 0.03937 0.03937" />
-      </geometry>
-    </collision>
-  </link>
+<xacro:include filename="$(find coman_urdf)/urdf/parts/torso.urdf.xacro" />
 <!-- ********************RIGHT LEG******************** -->
   <link name ="RHipMot">
@@ -441,9 +366,4 @@
   </link>
 <!-- ********************JOINTS******************** -->
-  <joint name="base_joint" type="fixed">
-    <parent link="base_link"/>
-    <child link="Waist"/>
-    <origin xyz="0 0 0" rpy="0 0 0" />
-  </joint>
     <joint name="l_ankle_joint" type="fixed">
       <parent link="LFoot"/>
@@ -515,30 +435,4 @@
   	</joint>
 </xacro:unless>
-<!-- ********************TORSO******************** -->
-  <joint name="WaistLat" type="revolute"> <!-- Wrong name! need to fix this... -->
-    <parent link="Waist"/>
-    <child link="DWL"/>
-    <origin xyz="0.020281504 0 0.11912053" rpy="0 0 0" />
-    <axis xyz="0.939692608 0 0.3420201433" />
-    <limit velocity="4.0" effort="50" lower="-0.5236" upper="0.5235" />
-    <!-- dynamics friction="0" damping="0.3"/ -->
-    <dynamics friction="0" damping="3.0"/>
-  </joint>
-  <joint name="WaistSag" type="revolute"> <!-- Wrong name! need to fix this... -->
-    <parent link="DWL"/>
-    <child link="DWS"/>
-    <origin xyz="0 0 0" rpy="0 0 0" />
-    <axis xyz="0 1 0" />
-    <limit velocity="4.0" effort="50" lower="-0.3491" upper="0.8727" />
-    <dynamics friction="0" damping="3.0"/>
-  </joint>
-  <joint name="WaistYaw" type="revolute">
-    <parent link="DWS"/>
-    <child link="DWYTorso"/>
-    <origin xyz="0 0 0.04749999" rpy="0 0 0" />
-    <axis xyz="0 0 1" />
-    <limit velocity="4.0" effort="50" lower="-1.3963" upper="1.3962" />
-    <dynamics friction="0" damping="3.0"/>
-  </joint>
 <!-- ********************RIGHT LEG******************** -->
   <joint name="RHipSag" type="revolute">

File: coman_urdf/urdf/coman_hands.urdf (robot description, URDF)
Before this commit: robot COMAN, 54 links, 53 joints
Joints:
- joint WaistLat: axis 0.939692608 0 0.3420201433 -> 0.93969262078 0 0.34202014332

File: coman_urdf/urdf/coman_no_forearms.urdf (robot description, URDF)
Before this commit: robot COMAN, 46 links, 45 joints
Joints:
- joint WaistLat: axis 0.939692608 0 0.3420201433 -> 0.93969262078 0 0.34202014332
