Commit message: Added full torso stl. Deleted old meshes.

File: coman_urdf/urdf/coman_materials.urdf.xacro (robot description, xacro)
@@ -4,3 +4,6 @@
   <color rgba="0.3 0.3 0.3 1"/>
 </material>
+<material name="red">
+  <color rgba="1.0 0.0 0.0 1"/>
+</material>
 </robot>

File: coman_urdf/urdf/gazebo/coman_materials.gazebo.xacro (robot description, xacro)
@@ -4,3 +4,12 @@
   <material>Gazebo/DarkGrey</material>
 </gazebo>
+<gazebo reference="DWL">
+  <material>Gazebo/DarkGrey</material>
+</gazebo>
+<gazebo reference="DWS">
+  <material>Gazebo/DarkGrey</material>
+</gazebo>
+<gazebo reference="DWYTorso">
+  <material>Gazebo/Red</material>
+</gazebo>
 </robot>

File: coman_urdf/urdf/parts/torso.urdf.xacro (robot description, xacro)
@@ -24,5 +24,4 @@
       <material name="dark_grey"/>
       <geometry name="Waist_visual">
-        <!--mesh filename="package://coman_urdf/meshes/collada/asm0001_collada_07_prt.dae" scale="${SF} ${SF} ${SF}"/-->
         <mesh filename="package://coman_urdf/meshes/collada/torso0.stl" scale="${SF} ${SF} ${SF}"/>
       </geometry>
@@ -43,6 +42,7 @@
     <visual>
       <origin xyz="-0.020281504 0 -0.63912053" rpy="0 0 ${PI}"/>
+      <material name="dark_grey"/>
       <geometry name="DWL_visual">
-        <mesh filename="package://coman_urdf/meshes/collada/asm0001_collada_09_prt.dae" scale="${SF} ${SF} ${SF}" />
+        <mesh filename="package://coman_urdf/meshes/collada/torso1.stl" scale="${SF} ${SF} ${SF}" />
       </geometry>
     </visual>
@@ -62,6 +62,7 @@
     <visual>
       <origin xyz="-0.020281504 0 -0.63912053" rpy="0 0 ${PI}"/>
+      <material name="dark_grey"/>
       <geometry name="DWS_visual">
-        <mesh filename="package://coman_urdf/meshes/collada/asm0001_collada_08_prt.dae" scale="${SF} ${SF} ${SF}" />
+        <mesh filename="package://coman_urdf/meshes/collada/torso2.stl" scale="${SF} ${SF} ${SF}" />
       </geometry>
     </visual>
@@ -81,6 +82,7 @@
     <visual>
       <origin xyz="-0.020281504 0.0 -0.68662053" rpy="0 0 ${PI}"/>
+      <material name="red"/>
       <geometry name="DWYTorso_visual">
-        <mesh filename="package://coman_urdf/meshes/collada/asm0001_collada_10_prt.dae" scale="${SF} ${SF} ${SF}" />
+        <mesh filename="package://coman_urdf/meshes/collada/torso3.stl" scale="${SF} ${SF} ${SF}" />
       </geometry>
     </visual>

Commit message: Added forearms.

File: coman_urdf/urdf/coman_materials.urdf.xacro (robot description, xacro)
@@ -1,4 +1,7 @@
 <?xml version="1.0"?>
 <robot xmlns:xacro="http://ros.org/wiki/xacro">
+<material name="grey">
+  <color rgba="0.5 0.5 0.5 1"/>
+</material>
 <material name="dark_grey">
   <color rgba="0.3 0.3 0.3 1"/>

File: coman_urdf/urdf/gazebo/coman_materials.gazebo.xacro (robot description, xacro)
@@ -28,4 +28,10 @@
   <material>Gazebo/DarkGrey</material>
 </gazebo>
+<gazebo reference="RWrMot2">
+  <material>Gazebo/Grey</material>
+</gazebo>
+<gazebo reference="RWrMot3">
+  <material>Gazebo/Grey</material>
+</gazebo>
 <gazebo reference="LShp">
   <material>Gazebo/DarkGrey</material>
@@ -42,4 +48,10 @@
 <gazebo reference="LForearm">
   <material>Gazebo/DarkGrey</material>
+</gazebo>
+<gazebo reference="LWrMot2">
+  <material>Gazebo/Grey</material>
+</gazebo>
+<gazebo reference="LWrMot3">
+  <material>Gazebo/Grey</material>
 </gazebo>
 <gazebo reference="RHipMot">

File: coman_urdf/urdf/parts/7DOF_forearms_DRC_14.urdf.xacro (robot description, xacro)
@@ -19,6 +19,7 @@
         <visual>
           <origin xyz="0 0 ${0.015 + Wrj1_to_FT}" rpy="3.14159265359 0 1.570796326795"/>
+          <material name="dark_grey"/>
           <geometry name="LForearm_visual">
-            <mesh filename="package://coman_urdf/meshes/collada/forearms/forearm_lowpoly.dae" scale="0.1 0.1 0.1" />
+            <mesh filename="package://coman_urdf/meshes/collada/forearms/forearm0.stl" scale="0.1 0.1 0.1" />
           </geometry>
         </visual>
@@ -40,6 +41,7 @@
         <visual>
           <origin xyz="0.025 0 0" rpy="0 1.570796326795 3.14159265359"/>
+          <material name="grey"/>
           <geometry name="LWrMot2_visual">
-            <mesh filename="package://coman_urdf/meshes/collada/forearms/fa_asm_3_right_sw0001.dae" scale="0.001 0.001 0.001" />
+            <mesh filename="package://coman_urdf/meshes/collada/forearms/forearm1.stl" scale="0.001 0.001 0.001" />
           </geometry>
         </visual>
@@ -61,6 +63,7 @@
         <visual>
           <origin xyz="0.025 -0.012 -0.02" rpy="0 3.14159265359 1.570796326795"/>
+          <material name="grey"/>
           <geometry name="LWrMot3_visual">
-            <mesh filename="package://coman_urdf/meshes/collada/forearms/fa_hand_interface_rig_sw0001.dae" scale="0.001 0.001 0.001" />
+            <mesh filename="package://coman_urdf/meshes/collada/forearms/forearm2.stl" scale="0.001 0.001 0.001" />
           </geometry>
         </visual>
@@ -83,6 +86,7 @@
         <visual>
           <origin xyz="0 0 ${0.015 + Wrj1_to_FT}" rpy="3.14159265359 0 1.570796326795"/>
+          <material name="dark_grey"/>
           <geometry name="RForearm_visual">
-            <mesh filename="package://coman_urdf/meshes/collada/forearms/forearm_lowpoly.dae" scale="0.1 0.1 0.1" />
+            <mesh filename="package://coman_urdf/meshes/collada/forearms/forearm0.stl" scale="0.1 0.1 0.1" />
           </geometry>
         </visual>
@@ -104,6 +108,7 @@
         <visual>
           <origin xyz="0.025 0 0" rpy="0 1.570796326795 3.14159265359"/>
+          <material name="grey"/>
           <geometry name="RWrMot2_visual">
-            <mesh filename="package://coman_urdf/meshes/collada/forearms/fa_asm_3_right_sw0001.dae" scale="0.001 0.001 0.001" />
+            <mesh filename="package://coman_urdf/meshes/collada/forearms/forearm1.stl" scale="0.001 0.001 0.001" />
           </geometry>
         </visual>
@@ -125,6 +130,7 @@
         <visual>
           <origin xyz="0.025 -0.012 -0.02" rpy="0 3.14159265359 1.570796326795"/>
+          <material name="grey"/>
           <geometry name="RWrMot3_visual">
-            <mesh filename="package://coman_urdf/meshes/collada/forearms/fa_hand_interface_rig_sw0001.dae" scale="0.001 0.001 0.001" />
+            <mesh filename="package://coman_urdf/meshes/collada/forearms/forearm2.stl" scale="0.001 0.001 0.001" />
           </geometry>
         </visual>
