Commit message: Corrected maximum joint torque from 30 to 50. Remember to run the script toupdate your model ingazebo!

File: coman_urdf/urdf/coman.urdf.xacro (robot description, xacro)
@@ -546,5 +546,5 @@
     <origin xyz="0.020281504 0 0.11912053" rpy="0 0 0" />
     <axis xyz="0.939692608 0 0.3420201433" />
-    <limit velocity="3.0" effort="30" lower="-0.5236" upper="0.5235" />
+    <limit velocity="3.0" effort="50" lower="-0.5236" upper="0.5235" />
   </joint>
   <joint name="WaistLat" type="revolute"> <!-- Wrong name! need to fix this... -->
@@ -553,5 +553,5 @@
     <origin xyz="0 0 0" rpy="0 0 0" />
     <axis xyz="0 1 0" />
-    <limit velocity="3.0" effort="30" lower="-0.3491" upper="0.8727" />
+    <limit velocity="3.0" effort="50" lower="-0.3491" upper="0.8727" />
   </joint>
   <joint name="WaistYaw" type="revolute">
@@ -560,5 +560,5 @@
     <origin xyz="0 0 0.04749999" rpy="0 0 0" />
     <axis xyz="0 0 1" />
-    <limit velocity="3.0" effort="30" lower="-1.3963" upper="1.3962" />
+    <limit velocity="3.0" effort="50" lower="-1.3963" upper="1.3962" />
   </joint>
 <!-- ********************RIGHT LEG******************** -->
@@ -568,5 +568,5 @@
     <origin xyz="0.0 -0.023 0.0" rpy="0 0 0" />
     <axis xyz="0 1 0" />
-    <limit velocity="3.0" effort="30" lower="-1.9199" upper="0.7854" />
+    <limit velocity="3.0" effort="50" lower="-1.9199" upper="0.7854" />
   </joint>
   <joint name="RHipLat" type="revolute">
@@ -575,5 +575,5 @@
     <origin xyz="0.0 -0.0496 0.0" rpy="0 0 0" />
     <axis xyz="1 0 0" />
-    <limit velocity="3.0" effort="30" lower="-1.0472" upper="0.4363" />
+    <limit velocity="3.0" effort="50" lower="-1.0472" upper="0.4363" />
   </joint>
   <joint name="RHipYaw" type="revolute">
@@ -582,5 +582,5 @@
     <origin xyz="0.0 0.0 -0.1024" rpy="0 0 0" />
     <axis xyz="0 0 1" />
-    <limit velocity="3.0" effort="30" lower="-0.8727" upper="0.8727" />
+    <limit velocity="3.0" effort="50" lower="-0.8727" upper="0.8727" />
   </joint>
   <joint name="RKneeSag" type="revolute">
@@ -589,5 +589,5 @@
     <origin xyz="0.0 0.0 -0.1234" rpy="0 0 0" />
     <axis xyz="0 1 0" />
-    <limit velocity="3.0" effort="30" lower="-0.1745" upper="1.9199" />
+    <limit velocity="3.0" effort="50" lower="-0.1745" upper="1.9199" />
   </joint>
   <joint name="RAnkLat" type="revolute">
@@ -596,5 +596,5 @@
     <origin xyz="0.0 0.0 -0.201" rpy="0 0 0" />
     <axis xyz="1 0 0" />
-    <limit velocity="3.0" effort="30" lower="-0.6109" upper="0.6109" />
+    <limit velocity="3.0" effort="50" lower="-0.6109" upper="0.6109" />
   </joint>
   <joint name="RAnkSag" type="revolute">
@@ -603,5 +603,5 @@
     <origin xyz="0.0 0.0 0.0" rpy="0 0 0" />
     <axis xyz="0 1 0" />
-    <limit velocity="3.0" effort="30" lower="-1.2217" upper="1.2217" />
+    <limit velocity="3.0" effort="50" lower="-1.2217" upper="1.2217" />
   </joint>
 <!-- ********************LEFT LEG******************** -->
@@ -611,5 +611,5 @@
     <origin xyz="0.0 0.023 0.0" rpy="0 0 0" />
     <axis xyz="0 1 0" />
-    <limit velocity="3.0" effort="30" lower="-1.9199" upper="0.7854" />
+    <limit velocity="3.0" effort="50" lower="-1.9199" upper="0.7854" />
   </joint>
   <joint name="LHipLat" type="revolute">
@@ -618,5 +618,5 @@
     <origin xyz="0.0 0.0496 0.0" rpy="0 0 0" />
     <axis xyz="1 0 0" />
-    <limit velocity="3.0" effort="30" lower="-0.4363" upper="1.0472" />
+    <limit velocity="3.0" effort="50" lower="-0.4363" upper="1.0472" />
   </joint>
   <joint name="LHipYaw" type="revolute">
@@ -625,5 +625,5 @@
     <origin xyz="0.0 0.0 -0.1024" rpy="0 0 0" />
     <axis xyz="0 0 1" />
-    <limit velocity="3.0" effort="30" lower="-0.8727" upper="0.8727" />
+    <limit velocity="3.0" effort="50" lower="-0.8727" upper="0.8727" />
   </joint>
   <joint name="LKneeSag" type="revolute">
@@ -632,5 +632,5 @@
     <origin xyz="0.0 0.0 -0.1234" rpy="0 0 0" />
     <axis xyz="0 1 0" />
-    <limit velocity="3.0" effort="30" lower="-0.1745" upper="1.9199" />
+    <limit velocity="3.0" effort="50" lower="-0.1745" upper="1.9199" />
   </joint>
   <joint name="LAnkLat" type="revolute">
@@ -639,5 +639,5 @@
     <origin xyz="0.0 0.0 -0.201" rpy="0 0 0" />
     <axis xyz="1 0 0" />
-    <limit velocity="3.0" effort="30" lower="-0.6109" upper="0.6109" />
+    <limit velocity="3.0" effort="50" lower="-0.6109" upper="0.6109" />
   </joint>
   <joint name="LAnkSag" type="revolute">
@@ -646,5 +646,5 @@
     <origin xyz="0.0 0.0 0.0" rpy="0 0 0" />
     <axis xyz="0 1 0" />
-    <limit velocity="3.0" effort="30" lower="-1.2217" upper="1.2217" />
+    <limit velocity="3.0" effort="50" lower="-1.2217" upper="1.2217" />
   </joint>
 <!-- ********************RIGHT ARM******************** -->
@@ -654,5 +654,5 @@
     <origin xyz="-0.014976503999999998 -0.0825 0.15770847" rpy="0 0 0" />
     <axis xyz="0 1 0" />
-    <limit velocity="3.0" effort="30" lower="-3.4034" upper="1.6581" />
+    <limit velocity="3.0" effort="50" lower="-3.4034" upper="1.6581" />
   </joint>
   <joint name="RShLat" type="revolute">
@@ -661,5 +661,5 @@
     <origin xyz="0.0 -0.07329999999999999 0.0" rpy="0 0 0" />
     <axis xyz="1 0 0" />
-    <limit velocity="3.0" effort="30" lower="-2.094" upper="0.31415" />
+    <limit velocity="3.0" effort="50" lower="-2.094" upper="0.31415" />
   </joint>
   <joint name="RShYaw" type="revolute">
@@ -668,5 +668,5 @@
     <origin xyz="0.0 0.0 -0.04480846999999999" rpy="0 0 0" />
     <axis xyz="0 0 1" />
-    <limit velocity="3.0" effort="30" lower="-1.5708" upper="1.5708" />
+    <limit velocity="3.0" effort="50" lower="-1.5708" upper="1.5708" />
   </joint>
   <joint name="RElbj" type="revolute">
@@ -675,5 +675,5 @@
     <origin xyz="0.0 0.0 -0.13519152999999998" rpy="0 0 0" />
     <axis xyz="0 1 0" />
-    <limit velocity="3.0" effort="30" lower="-2.3562" upper="0.0" />
+    <limit velocity="3.0" effort="50" lower="-2.3562" upper="0.0" />
   </joint>
 <!-- ********************LEFT ARM******************** -->
@@ -683,5 +683,5 @@
     <origin xyz="-0.014976503999999998 0.0825 0.15770847" rpy="0 0 0" />
     <axis xyz="0 1 0" />
-    <limit velocity="3.0" effort="30" lower="-3.4034" upper="1.6581" />
+    <limit velocity="3.0" effort="50" lower="-3.4034" upper="1.6581" />
   </joint>
   <joint name="LShLat" type="revolute">
@@ -690,5 +690,5 @@
     <origin xyz="0.0 0.07329999999999999 0.0" rpy="0 0 0" />
     <axis xyz="1 0 0" />
-    <limit velocity="3.0" effort="30" lower="-0.31415" upper="2.094" />
+    <limit velocity="3.0" effort="50" lower="-0.31415" upper="2.094" />
   </joint>
   <joint name="LShYaw" type="revolute">
@@ -697,5 +697,5 @@
     <origin xyz="0.0 0.0 -0.04480846999999999" rpy="0 0 0" />
     <axis xyz="0 0 1" />
-    <limit velocity="3.0" effort="30" lower="-1.5708" upper="1.5708" />
+    <limit velocity="3.0" effort="50" lower="-1.5708" upper="1.5708" />
   </joint>
   <joint name="LElbj" type="revolute">
@@ -704,5 +704,5 @@
     <origin xyz="0.0 0.0 -0.13519152999999998" rpy="0 0 0" />
     <axis xyz="0 1 0" />
-    <limit velocity="3.0" effort="30" lower="-2.3562" upper="0.0" />
+    <limit velocity="3.0" effort="50" lower="-2.3562" upper="0.0" />
   </joint>
 </robot>

Commit message: Splitted sensor and foot masses, and moved sensor frame to actual pose of sensing element. Check issue 11 for more details.

File: coman_urdf/urdf/coman.urdf.xacro (robot description, xacro)
@@ -201,23 +201,53 @@
     </collision>
   </link>
-  <link name ="RFoot">
-    <inertial>
-      <origin xyz="0.00969210464 -0.0090460227 -0.043062308" rpy="0 0 0"/>
-      <mass value="0.66646684"/>
-      <inertia ixx="0.0012944808"  ixy="-9.2387693E-5"  ixz="2.0080105E-4" iyy="0.0015851846" iyz="2.7599327E-4" izz="0.0013326766" />
-    </inertial>
-    <visual>
-      <origin xyz="0.0 0.0726 -0.0932" rpy="0 0 -3.14159265359"/>
-      <geometry name="RFoot_visual">
-        <mesh filename="package://coman_urdf/meshes/collada/asm0001_collada_15_prt.dae" scale="0.03937 0.03937 0.03937" />
-      </geometry>
-    </visual>
-    <collision>
-      <origin xyz="0.0 0.0726 -0.0932" rpy="0 0 -3.14159265359"/>
-      <geometry name="RFoot_collision">
-        <mesh filename="package://coman_urdf/meshes/collada/simple/simple_asm0001_collada_15_prt.dae" scale="0.03937 0.03937 0.03937" />
-      </geometry>
-    </collision>
-  </link>
+  <xacro:unless value="$(optenv WIP_FT_ACCURATE_POSITIONING false)">
+    <link name ="RFoot">
+      <inertial>
+        <origin xyz="0.00969210464 -0.0090460227 -0.043062308" rpy="0 0 0"/>
+        <mass value="0.66646684"/>
+        <inertia ixx="0.0012944808"  ixy="-9.2387693E-5"  ixz="2.0080105E-4" iyy="0.0015851846" iyz="2.7599327E-4" izz="0.0013326766" />
+      </inertial>
+      <visual>
+        <origin xyz="0.0 0.0726 -0.0932" rpy="0 0 -3.14159265359"/>
+        <geometry name="RFoot_visual">
+          <mesh filename="package://coman_urdf/meshes/collada/asm0001_collada_15_prt.dae" scale="0.03937 0.03937 0.03937" />
+        </geometry>
+      </visual>
+      <collision>
+        <origin xyz="0.0 0.0726 -0.0932" rpy="0 0 -3.14159265359"/>
+        <geometry name="RFoot_collision">
+          <mesh filename="package://coman_urdf/meshes/collada/simple/simple_asm0001_collada_15_prt.dae" scale="0.03937 0.03937 0.03937" />
+        </geometry>
+      </collision>
+    </link>
+  </xacro:unless>
+  <xacro:if value="$(optenv WIP_FT_ACCURATE_POSITIONING false)">
+    <link name ="RFootFTSensor">
+      <inertial>
+        <origin xyz="0.0 -0.0 -0.0325" rpy="0 0 0"/>
+        <mass value="0.280"/>
+        <inertia ixx="0.0012944808"  ixy="-9.2387693E-5"  ixz="2.0080105E-4" iyy="0.0015851846" iyz="2.7599327E-4" izz="0.0013326766" />
+      </inertial>
+    </link>
+    <link name ="RFoot">
+      <inertial>
+        <origin xyz="0.00969210464 -0.0090460227 -0.0282" rpy="0 0 0"/>
+        <mass value="0.404"/>
+        <inertia ixx="0.0012944808"  ixy="-9.2387693E-5"  ixz="2.0080105E-4" iyy="0.0015851846" iyz="2.7599327E-4" izz="0.0013326766" />
+      </inertial>
+      <visual>
+        <origin xyz="0.0 0.0726 -0.0282" rpy="0 0 -3.14159265359"/>
+        <geometry name="RFoot_visual">
+          <mesh filename="package://coman_urdf/meshes/collada/asm0001_collada_15_prt.dae" scale="0.03937 0.03937 0.03937" />
+        </geometry>
+      </visual>
+      <collision>
+        <origin xyz="0.0 0.0726 -0.0282" rpy="0 0 -3.14159265359"/>
+        <geometry name="RFoot_collision">
+          <mesh filename="package://coman_urdf/meshes/collada/simple/simple_asm0001_collada_15_prt.dae" scale="0.03937 0.03937 0.03937" />
+        </geometry>
+      </collision>
+    </link>
+  </xacro:if>
 <!-- ********************LEFT LEG******************** -->
   <link name ="LHipMot">
@@ -316,23 +346,53 @@
     </collision>
   </link>
-  <link name ="LFoot">
-    <inertial>
-      <origin xyz="0.0096921046 0.0090460227 -0.043062308" rpy="0 0 0"/>
-      <mass value="0.66646684"/>
-      <inertia ixx="0.0012944808"  ixy="9.2387693E-5"  ixz="2.0080105E-4" iyy="0.0015851846" iyz="-2.7599327E-4" izz="0.0013326766" />
-    </inertial>
-    <visual>
-      <origin xyz="0.0 -0.0726 -0.0932" rpy="0 0 -3.14159265359"/>
-      <geometry name="LFoot_visual">
-        <mesh filename="package://coman_urdf/meshes/collada/asm0001_collada_01_prt.dae" scale="0.03937 0.03937 0.03937" />
-      </geometry>
-    </visual>
-    <collision>
-      <origin xyz="0.0 -0.0726 -0.0932" rpy="0 0 -3.14159265359"/>
-      <geometry name="LFoot_collision">
-        <mesh filename="package://coman_urdf/meshes/collada/simple/simple_asm0001_collada_01_prt.dae" scale="0.03937 0.03937 0.03937" />
-      </geometry>
-    </collision>
-  </link>
+  <xacro:unless value="$(optenv WIP_FT_ACCURATE_POSITIONING false)">
+    <link name ="LFoot">
+      <inertial>
+        <origin xyz="0.0096921046 0.0090460227 -0.043062308" rpy="0 0 0"/>
+        <mass value="0.66646684"/>
+        <inertia ixx="0.0012944808"  ixy="9.2387693E-5"  ixz="2.0080105E-4" iyy="0.0015851846" iyz="-2.7599327E-4" izz="0.0013326766" />
+      </inertial>
+      <visual>
+        <origin xyz="0.0 -0.0726 -0.0932" rpy="0 0 -3.14159265359"/>
+        <geometry name="LFoot_visual">
+          <mesh filename="package://coman_urdf/meshes/collada/asm0001_collada_01_prt.dae" scale="0.03937 0.03937 0.03937" />
+        </geometry>
+      </visual>
+      <collision>
+        <origin xyz="0.0 -0.0726 -0.0932" rpy="0 0 -3.14159265359"/>
+        <geometry name="LFoot_collision">
+          <mesh filename="package://coman_urdf/meshes/collada/simple/simple_asm0001_collada_01_prt.dae" scale="0.03937 0.03937 0.03937" />
+        </geometry>
+      </collision>
+    </link>
+  </xacro:unless>
+  <xacro:if value="$(optenv WIP_FT_ACCURATE_POSITIONING false)">
+    <link name ="LFootFTSensor">
+      <inertial>
+        <origin xyz="0.0 -0.0 -0.0325" rpy="0 0 0"/>
+        <mass value="0.280"/>
+        <inertia ixx="0.0012944808"  ixy="-9.2387693E-5"  ixz="2.0080105E-4" iyy="0.0015851846" iyz="2.7599327E-4" izz="0.0013326766" />
+      </inertial>
+    </link>
+    <link name ="LFoot">
+      <inertial>
+        <origin xyz="0.0096921046 0.0090460227 -0.0282" rpy="0 0 0"/>
+        <mass value="0.404"/>
+        <inertia ixx="0.0012944808"  ixy="9.2387693E-5"  ixz="2.0080105E-4" iyy="0.0015851846" iyz="-2.7599327E-4" izz="0.0013326766" />
+      </inertial>
+      <visual>
+        <origin xyz="0.0 -0.0726 -0.0282" rpy="0 0 -3.14159265359"/>
+        <geometry name="LFoot_visual">
+          <mesh filename="package://coman_urdf/meshes/collada/asm0001_collada_01_prt.dae" scale="0.03937 0.03937 0.03937" />
+        </geometry>
+      </visual>
+      <collision>
+        <origin xyz="0.0 -0.0726 -0.0282" rpy="0 0 -3.14159265359"/>
+        <geometry name="LFoot_collision">
+          <mesh filename="package://coman_urdf/meshes/collada/simple/simple_asm0001_collada_01_prt.dae" scale="0.03937 0.03937 0.03937" />
+        </geometry>
+      </collision>
+    </link>
+  </xacro:if>
 <!-- ********************RIGHT ARM******************** -->
   <link name ="RShp">
@@ -598,11 +658,29 @@
     <limit velocity="4.0" effort="50" lower="-0.6109" upper="0.6109" />
   </joint>
-  <joint name="RAnkSag" type="revolute">
-    <parent link="RFootmot"/>
-    <child link="RFoot"/>
-    <origin xyz="0.0 0.0 0.0" rpy="0 0 0" />
-    <axis xyz="0 1 0" />
-    <limit velocity="4.0" effort="50" lower="-1.2217" upper="1.2217" />
-  </joint>
+  <xacro:unless value="$(optenv WIP_FT_ACCURATE_POSITIONING false)">
+    <joint name="RAnkSag" type="revolute">
+      <parent link="RFootmot"/>
+      <child link="RFoot"/>
+      <origin xyz="0.0 0.0 0.0" rpy="0 0 0" />
+      <axis xyz="0 1 0" />
+      <limit velocity="4.0" effort="50" lower="-1.2217" upper="1.2217" />
+    </joint>
+  </xacro:unless>
+  <xacro:if value="$(optenv WIP_FT_ACCURATE_POSITIONING false)">
+    <joint name="RAnkSag" type="revolute">
+      <parent link="RFootmot"/>
+      <child link="RFootFTSensor"/>
+      <origin xyz="0.0 0.0 0.0" rpy="0 0 0" />
+      <axis xyz="0 1 0" />
+      <limit velocity="4.0" effort="50" lower="-1.2217" upper="1.2217" />
+    </joint>
+    <joint name="RAnkSagFT" type="revolute">
+      <parent link="RFootFTSensor"/>
+      <child link="RFoot"/>
+      <origin xyz="0.0 0.0 -0.065" rpy="0 0 0" />
+      <axis xyz="0 1 0" />
+      <limit velocity="0.0" effort="0" lower="-0.0" upper="0.0" />
+    </joint>
+  </xacro:if>
 <!-- ********************LEFT LEG******************** -->
   <joint name="LHipSag" type="revolute">
@@ -641,11 +719,29 @@
     <limit velocity="4.0" effort="50" lower="-0.6109" upper="0.6109" />
   </joint>
-  <joint name="LAnkSag" type="revolute">
-    <parent link="LFootmot"/>
-    <child link="LFoot"/>
-    <origin xyz="0.0 0.0 0.0" rpy="0 0 0" />
-    <axis xyz="0 1 0" />
-    <limit velocity="4.0" effort="50" lower="-1.2217" upper="1.2217" />
-  </joint>
+  <xacro:unless value="$(optenv WIP_FT_ACCURATE_POSITIONING false)">
+    <joint name="LAnkSag" type="revolute">
+      <parent link="LFootmot"/>
+      <child link="LFoot"/>
+      <origin xyz="0.0 0.0 0.0" rpy="0 0 0" />
+      <axis xyz="0 1 0" />
+      <limit velocity="4.0" effort="50" lower="-1.2217" upper="1.2217" />
+    </joint>
+  </xacro:unless>
+  <xacro:if value="$(optenv WIP_FT_ACCURATE_POSITIONING false)">
+    <joint name="LAnkSag" type="revolute">
+      <parent link="LFootmot"/>
+      <child link="LFootFTSensor"/>
+      <origin xyz="0.0 0.0 0.0" rpy="0 0 0" />
+      <axis xyz="0 1 0" />
+      <limit velocity="4.0" effort="50" lower="-1.2217" upper="1.2217" />
+    </joint>
+    <joint name="LAnkSagFT" type="revolute">
+      <parent link="LFootFTSensor"/>
+      <child link="LFoot"/>
+      <origin xyz="0.0 0.0 -0.065" rpy="0 0 0" />
+      <axis xyz="0 1 0" />
+      <limit velocity="0.0" effort="0" lower="-0.0" upper="0.0" />
+    </joint>
+  </xacro:if>
 <!-- ********************RIGHT ARM******************** -->
   <joint name="RShSag" type="revolute">

Commit message: Added dynamics tag to joints

File: coman_urdf/urdf/coman.urdf.xacro (robot description, xacro)
@@ -607,4 +607,5 @@
     <axis xyz="0.939692608 0 0.3420201433" />
     <limit velocity="4.0" effort="50" lower="-0.5236" upper="0.5235" />
+    <dynamics friction="0" damping="0.3"/>
   </joint>
   <joint name="WaistLat" type="revolute"> <!-- Wrong name! need to fix this... -->
@@ -614,4 +615,5 @@
     <axis xyz="0 1 0" />
     <limit velocity="4.0" effort="50" lower="-0.3491" upper="0.8727" />
+    <dynamics friction="0" damping="0.3"/>
   </joint>
   <joint name="WaistYaw" type="revolute">
@@ -621,4 +623,5 @@
     <axis xyz="0 0 1" />
     <limit velocity="4.0" effort="50" lower="-1.3963" upper="1.3962" />
+    <dynamics friction="0" damping="0.3"/>
   </joint>
 <!-- ********************RIGHT LEG******************** -->
@@ -629,4 +632,5 @@
     <axis xyz="0 1 0" />
     <limit velocity="4.0" effort="50" lower="-1.9199" upper="0.7854" />
+    <dynamics friction="0" damping="0.3"/>
   </joint>
   <joint name="RHipLat" type="revolute">
@@ -636,4 +640,5 @@
     <axis xyz="1 0 0" />
     <limit velocity="4.0" effort="50" lower="-1.0472" upper="0.4363" />
+    <dynamics friction="0" damping="0.3"/>
   </joint>
   <joint name="RHipYaw" type="revolute">
@@ -643,4 +648,5 @@
     <axis xyz="0 0 1" />
     <limit velocity="4.0" effort="50" lower="-0.8727" upper="0.8727" />
+    <dynamics friction="0" damping="0.3"/>
   </joint>
   <joint name="RKneeSag" type="revolute">
@@ -650,4 +656,5 @@
     <axis xyz="0 1 0" />
     <limit velocity="4.0" effort="50" lower="-0.1745" upper="1.9199" />
+    <dynamics friction="0" damping="0.3"/>
   </joint>
   <joint name="RAnkLat" type="revolute">
@@ -657,4 +664,5 @@
     <axis xyz="1 0 0" />
     <limit velocity="4.0" effort="50" lower="-0.6109" upper="0.6109" />
+    <dynamics friction="0" damping="0.3"/>
   </joint>
   <xacro:unless value="$(optenv WIP_FT_ACCURATE_POSITIONING false)">
@@ -665,4 +673,5 @@
       <axis xyz="0 1 0" />
       <limit velocity="4.0" effort="50" lower="-1.2217" upper="1.2217" />
+      <dynamics friction="0" damping="0.3"/>
     </joint>
   </xacro:unless>
@@ -674,4 +683,5 @@
       <axis xyz="0 1 0" />
       <limit velocity="4.0" effort="50" lower="-1.2217" upper="1.2217" />
+      <dynamics friction="0" damping="0.3"/>
     </joint>
     <joint name="RAnkSagFT" type="revolute">
@@ -681,4 +691,5 @@
       <axis xyz="0 1 0" />
       <limit velocity="0.0" effort="0" lower="-0.0" upper="0.0" />
+      <dynamics friction="0" damping="0.3"/>
     </joint>
   </xacro:if>
@@ -690,4 +701,5 @@
     <axis xyz="0 1 0" />
     <limit velocity="4.0" effort="50" lower="-1.9199" upper="0.7854" />
+    <dynamics friction="0" damping="0.3"/>
   </joint>
   <joint name="LHipLat" type="revolute">
@@ -697,4 +709,5 @@
     <axis xyz="1 0 0" />
     <limit velocity="4.0" effort="50" lower="-0.4363" upper="1.0472" />
+    <dynamics friction="0" damping="0.3"/>
   </joint>
   <joint name="LHipYaw" type="revolute">
@@ -704,4 +717,5 @@
     <axis xyz="0 0 1" />
     <limit velocity="4.0" effort="50" lower="-0.8727" upper="0.8727" />
+    <dynamics friction="0" damping="0.3"/>
   </joint>
   <joint name="LKneeSag" type="revolute">
@@ -711,4 +725,5 @@
     <axis xyz="0 1 0" />
     <limit velocity="4.0" effort="50" lower="-0.1745" upper="1.9199" />
+    <dynamics friction="0" damping="0.3"/>
   </joint>
   <joint name="LAnkLat" type="revolute">
@@ -718,4 +733,5 @@
     <axis xyz="1 0 0" />
     <limit velocity="4.0" effort="50" lower="-0.6109" upper="0.6109" />
+    <dynamics friction="0" damping="0.3"/>
   </joint>
   <xacro:unless value="$(optenv WIP_FT_ACCURATE_POSITIONING false)">
@@ -726,4 +742,5 @@
       <axis xyz="0 1 0" />
       <limit velocity="4.0" effort="50" lower="-1.2217" upper="1.2217" />
+      <dynamics friction="0" damping="0.3"/>
     </joint>
   </xacro:unless>
@@ -735,4 +752,5 @@
       <axis xyz="0 1 0" />
       <limit velocity="4.0" effort="50" lower="-1.2217" upper="1.2217" />
+      <dynamics friction="0" damping="0.3"/>
     </joint>
     <joint name="LAnkSagFT" type="revolute">
@@ -742,4 +760,5 @@
       <axis xyz="0 1 0" />
       <limit velocity="0.0" effort="0" lower="-0.0" upper="0.0" />
+      <dynamics friction="0" damping="0.3"/>
     </joint>
   </xacro:if>
@@ -751,4 +770,5 @@
     <axis xyz="0 1 0" />
     <limit velocity="4.0" effort="50" lower="-3.4034" upper="1.6581" />
+    <dynamics friction="0" damping="0.3"/>
   </joint>
   <joint name="RShLat" type="revolute">
@@ -758,4 +778,5 @@
     <axis xyz="1 0 0" />
     <limit velocity="4.0" effort="50" lower="-2.094" upper="0.31415" />
+    <dynamics friction="0" damping="0.3"/>
   </joint>
   <joint name="RShYaw" type="revolute">
@@ -765,4 +786,5 @@
     <axis xyz="0 0 1" />
     <limit velocity="4.0" effort="50" lower="-1.5708" upper="1.5708" />
+    <dynamics friction="0" damping="0.3"/>
   </joint>
   <joint name="RElbj" type="revolute">
@@ -772,4 +794,5 @@
     <axis xyz="0 1 0" />
     <limit velocity="4.0" effort="50" lower="-2.3562" upper="0.0" />
+    <dynamics friction="0" damping="0.3"/>
   </joint>
 <!-- ********************LEFT ARM******************** -->
@@ -780,4 +803,5 @@
     <axis xyz="0 1 0" />
     <limit velocity="4.0" effort="50" lower="-3.4034" upper="1.6581" />
+    <dynamics friction="0" damping="0.3"/>
   </joint>
   <joint name="LShLat" type="revolute">
@@ -787,4 +811,5 @@
     <axis xyz="1 0 0" />
     <limit velocity="4.0" effort="50" lower="-0.31415" upper="2.094" />
+    <dynamics friction="0" damping="0.3"/>
   </joint>
   <joint name="LShYaw" type="revolute">
@@ -794,4 +819,5 @@
     <axis xyz="0 0 1" />
     <limit velocity="4.0" effort="50" lower="-1.5708" upper="1.5708" />
+    <dynamics friction="0" damping="0.3"/>
   </joint>
   <joint name="LElbj" type="revolute">
@@ -801,4 +827,5 @@
     <axis xyz="0 1 0" />
     <limit velocity="4.0" effort="50" lower="-2.3562" upper="0.0" />
+    <dynamics friction="0" damping="0.3"/>
   </joint>
 </robot>
