Commit message: This closes the issue https://github.com/EnricoMingo/iit-coman-ros-pkg/issues/13 Currently three modes are available for generating the sdf: by calling the generation script without any arguments, the coman sdf with yarp plugins is loaded. This version uses FT torques that are defined at underactuated joints, added specifically to put a FT sensor. The ros version includes the ros plugins, and the FT sensor is defined at actuated joints, so the reading are not accurate. The ros_accurate_ft version of the sdf contains ros plugins, and the FT sensor is placed in the correct pose by using an underactuated joint. A bare sdf is not generated, but a coman.urdf is generated instead which does not contain sensors and plugins, and is to be used by external libraries needing a urdf description of the robot.

File: coman_urdf/urdf/coman.urdf.xacro (robot description, xacro)
@@ -201,5 +201,5 @@
     </collision>
   </link>
-  <xacro:unless value="$(optenv WIP_FT_ACCURATE_POSITIONING false)">
+  <xacro:unless value="$(optenv GAZEBO_COMAN_USES_ACCURATE_FT false)">
     <link name ="RFoot">
       <inertial>
@@ -222,10 +222,10 @@
     </link>
   </xacro:unless>
-  <xacro:if value="$(optenv WIP_FT_ACCURATE_POSITIONING false)">
+  <xacro:if value="$(optenv GAZEBO_COMAN_USES_ACCURATE_FT false)">
     <link name ="RFootFTSensor">
       <inertial>
         <origin xyz="0.0 -0.0 -0.0325" rpy="0 0 0"/>
         <mass value="0.280"/>
-        <inertia ixx="0.0012944808"  ixy="-9.2387693E-5"  ixz="2.0080105E-4" iyy="0.0015851846" iyz="2.7599327E-4" izz="0.0013326766" />
+        <inertia ixx="0.0012944808"  ixy="0.0"  ixz="2.0080105E-4" iyy="0.0015851846" iyz="2.7599327E-4" izz="0.0013326766" />
       </inertial>
     </link>
@@ -346,5 +346,5 @@
     </collision>
   </link>
-  <xacro:unless value="$(optenv WIP_FT_ACCURATE_POSITIONING false)">
+  <xacro:unless value="$(optenv GAZEBO_COMAN_USES_ACCURATE_FT false)">
     <link name ="LFoot">
       <inertial>
@@ -367,5 +367,5 @@
     </link>
   </xacro:unless>
-  <xacro:if value="$(optenv WIP_FT_ACCURATE_POSITIONING false)">
+  <xacro:if value="$(optenv GAZEBO_COMAN_USES_ACCURATE_FT false)">
     <link name ="LFootFTSensor">
       <inertial>
@@ -666,5 +666,5 @@
     <dynamics friction="0" damping="0.3"/>
   </joint>
-  <xacro:unless value="$(optenv WIP_FT_ACCURATE_POSITIONING false)">
+  <xacro:unless value="$(optenv GAZEBO_COMAN_USES_ACCURATE_FT false)">
     <joint name="RAnkSag" type="revolute">
       <parent link="RFootmot"/>
@@ -676,5 +676,5 @@
     </joint>
   </xacro:unless>
-  <xacro:if value="$(optenv WIP_FT_ACCURATE_POSITIONING false)">
+  <xacro:if value="$(optenv GAZEBO_COMAN_USES_ACCURATE_FT false)">
     <joint name="RAnkSag" type="revolute">
       <parent link="RFootmot"/>
@@ -735,5 +735,5 @@
     <dynamics friction="0" damping="0.3"/>
   </joint>
-  <xacro:unless value="$(optenv WIP_FT_ACCURATE_POSITIONING false)">
+  <xacro:unless value="$(optenv GAZEBO_COMAN_USES_ACCURATE_FT false)">
     <joint name="LAnkSag" type="revolute">
       <parent link="LFootmot"/>
@@ -745,5 +745,5 @@
     </joint>
   </xacro:unless>
-  <xacro:if value="$(optenv WIP_FT_ACCURATE_POSITIONING false)">
+  <xacro:if value="$(optenv GAZEBO_COMAN_USES_ACCURATE_FT false)">
     <joint name="LAnkSag" type="revolute">
       <parent link="LFootmot"/>

Commit message: Look previous log

File: coman_urdf/urdf/coman.urdf.xacro (robot description, xacro)
@@ -472,4 +472,11 @@
     </collision>
   </link>
+  <link name ="RForearm">
+    <inertial>
+      <origin xyz="0 0 -0.085" rpy="0 0 0"/>
+      <mass value="0.263"/>
+      <inertia ixx="6.913E-4"  ixy="0.0"  ixz="0.0" iyy="6.913E-4" iyz="0.0" izz="4.0425E-5" />
+    </inertial>
+  </link>
 <!-- ********************LEFT ARM******************** -->
   <link name ="LShp">
@@ -548,4 +555,11 @@
       </geometry>
     </collision>
+  </link>
+  <link name ="LForearm">
+    <inertial>
+      <origin xyz="0 0 -0.085" rpy="0 0 0"/>
+      <mass value="0.263"/>
+      <inertia ixx="6.913E-4"  ixy="0.0"  ixz="0.0" iyy="6.913E-4" iyz="0.0" izz="4.0425E-5" />
+    </inertial>
   </link>
 <!-- ********************JOINTS******************** -->
@@ -796,4 +810,9 @@
     <dynamics friction="0" damping="0.3"/>
   </joint>
+  <joint name="RForearmPlate" type="fixed">
+    <parent link="RElb"/>
+    <child link="RForearm"/>
+    <origin xyz="-0.015 0.0 -0.05" rpy="0 0 0"/>
+  </joint>
 <!-- ********************LEFT ARM******************** -->
   <joint name="LShSag" type="revolute">
@@ -829,3 +848,8 @@
     <dynamics friction="0" damping="0.3"/>
   </joint>
+  <joint name="LForearmPlate" type="fixed">
+    <parent link="LElb"/>
+    <child link="LForearm"/>
+    <origin xyz="-0.015 0.0 -0.05" rpy="0 0 0"/>
+  </joint>
 </robot>

Commit message: Joint damping to 3.0

File: coman_urdf/urdf/coman.urdf.xacro (robot description, xacro)
@@ -621,5 +621,6 @@
     <axis xyz="0.939692608 0 0.3420201433" />
     <limit velocity="4.0" effort="50" lower="-0.5236" upper="0.5235" />
-    <dynamics friction="0" damping="0.3"/>
+    <!-- dynamics friction="0" damping="0.3"/ -->
+    <dynamics friction="0" damping="3.0"/>
   </joint>
   <joint name="WaistLat" type="revolute"> <!-- Wrong name! need to fix this... -->
@@ -629,5 +630,5 @@
     <axis xyz="0 1 0" />
     <limit velocity="4.0" effort="50" lower="-0.3491" upper="0.8727" />
-    <dynamics friction="0" damping="0.3"/>
+    <dynamics friction="0" damping="3.0"/>
   </joint>
   <joint name="WaistYaw" type="revolute">
@@ -637,5 +638,5 @@
     <axis xyz="0 0 1" />
     <limit velocity="4.0" effort="50" lower="-1.3963" upper="1.3962" />
-    <dynamics friction="0" damping="0.3"/>
+    <dynamics friction="0" damping="3.0"/>
   </joint>
 <!-- ********************RIGHT LEG******************** -->
@@ -646,5 +647,5 @@
     <axis xyz="0 1 0" />
     <limit velocity="4.0" effort="50" lower="-1.9199" upper="0.7854" />
-    <dynamics friction="0" damping="0.3"/>
+    <dynamics friction="0" damping="3.0"/>
   </joint>
   <joint name="RHipLat" type="revolute">
@@ -654,5 +655,5 @@
     <axis xyz="1 0 0" />
     <limit velocity="4.0" effort="50" lower="-1.0472" upper="0.4363" />
-    <dynamics friction="0" damping="0.3"/>
+    <dynamics friction="0" damping="3.0"/>
   </joint>
   <joint name="RHipYaw" type="revolute">
@@ -662,5 +663,5 @@
     <axis xyz="0 0 1" />
     <limit velocity="4.0" effort="50" lower="-0.8727" upper="0.8727" />
-    <dynamics friction="0" damping="0.3"/>
+    <dynamics friction="0" damping="3.0"/>
   </joint>
   <joint name="RKneeSag" type="revolute">
@@ -670,5 +671,5 @@
     <axis xyz="0 1 0" />
     <limit velocity="4.0" effort="50" lower="-0.1745" upper="1.9199" />
-    <dynamics friction="0" damping="0.3"/>
+    <dynamics friction="0" damping="3.0"/>
   </joint>
   <joint name="RAnkLat" type="revolute">
@@ -678,5 +679,5 @@
     <axis xyz="1 0 0" />
     <limit velocity="4.0" effort="50" lower="-0.6109" upper="0.6109" />
-    <dynamics friction="0" damping="0.3"/>
+    <dynamics friction="0" damping="3.0"/>
   </joint>
   <xacro:unless value="$(optenv GAZEBO_COMAN_USES_ACCURATE_FT false)">
@@ -687,5 +688,5 @@
       <axis xyz="0 1 0" />
       <limit velocity="4.0" effort="50" lower="-1.2217" upper="1.2217" />
-      <dynamics friction="0" damping="0.3"/>
+      <dynamics friction="0" damping="3.0"/>
     </joint>
   </xacro:unless>
@@ -697,5 +698,5 @@
       <axis xyz="0 1 0" />
       <limit velocity="4.0" effort="50" lower="-1.2217" upper="1.2217" />
-      <dynamics friction="0" damping="0.3"/>
+      <dynamics friction="0" damping="3.0"/>
     </joint>
     <joint name="RAnkSagFT" type="revolute">
@@ -705,5 +706,5 @@
       <axis xyz="0 1 0" />
       <limit velocity="0.0" effort="0" lower="-0.0" upper="0.0" />
-      <dynamics friction="0" damping="0.3"/>
+      <dynamics friction="0" damping="3.0"/>
     </joint>
   </xacro:if>
@@ -715,5 +716,5 @@
     <axis xyz="0 1 0" />
     <limit velocity="4.0" effort="50" lower="-1.9199" upper="0.7854" />
-    <dynamics friction="0" damping="0.3"/>
+    <dynamics friction="0" damping="3.0"/>
   </joint>
   <joint name="LHipLat" type="revolute">
@@ -723,5 +724,5 @@
     <axis xyz="1 0 0" />
     <limit velocity="4.0" effort="50" lower="-0.4363" upper="1.0472" />
-    <dynamics friction="0" damping="0.3"/>
+    <dynamics friction="0" damping="3.0"/>
   </joint>
   <joint name="LHipYaw" type="revolute">
@@ -731,5 +732,5 @@
     <axis xyz="0 0 1" />
     <limit velocity="4.0" effort="50" lower="-0.8727" upper="0.8727" />
-    <dynamics friction="0" damping="0.3"/>
+    <dynamics friction="0" damping="3.0"/>
   </joint>
   <joint name="LKneeSag" type="revolute">
@@ -739,5 +740,5 @@
     <axis xyz="0 1 0" />
     <limit velocity="4.0" effort="50" lower="-0.1745" upper="1.9199" />
-    <dynamics friction="0" damping="0.3"/>
+    <dynamics friction="0" damping="3.0"/>
   </joint>
   <joint name="LAnkLat" type="revolute">
@@ -747,5 +748,5 @@
     <axis xyz="1 0 0" />
     <limit velocity="4.0" effort="50" lower="-0.6109" upper="0.6109" />
-    <dynamics friction="0" damping="0.3"/>
+    <dynamics friction="0" damping="3.0"/>
   </joint>
   <xacro:unless value="$(optenv GAZEBO_COMAN_USES_ACCURATE_FT false)">
@@ -756,5 +757,5 @@
       <axis xyz="0 1 0" />
       <limit velocity="4.0" effort="50" lower="-1.2217" upper="1.2217" />
-      <dynamics friction="0" damping="0.3"/>
+      <dynamics friction="0" damping="3.0"/>
     </joint>
   </xacro:unless>
@@ -766,5 +767,5 @@
       <axis xyz="0 1 0" />
       <limit velocity="4.0" effort="50" lower="-1.2217" upper="1.2217" />
-      <dynamics friction="0" damping="0.3"/>
+      <dynamics friction="0" damping="3.0"/>
     </joint>
     <joint name="LAnkSagFT" type="revolute">
@@ -774,5 +775,5 @@
       <axis xyz="0 1 0" />
       <limit velocity="0.0" effort="0" lower="-0.0" upper="0.0" />
-      <dynamics friction="0" damping="0.3"/>
+      <dynamics friction="0" damping="3.0"/>
     </joint>
   </xacro:if>
@@ -784,5 +785,5 @@
     <axis xyz="0 1 0" />
     <limit velocity="4.0" effort="50" lower="-3.4034" upper="1.6581" />
-    <dynamics friction="0" damping="0.3"/>
+    <dynamics friction="0" damping="3.0"/>
   </joint>
   <joint name="RShLat" type="revolute">
@@ -792,5 +793,5 @@
     <axis xyz="1 0 0" />
     <limit velocity="4.0" effort="50" lower="-2.094" upper="0.31415" />
-    <dynamics friction="0" damping="0.3"/>
+    <dynamics friction="0" damping="3.0"/>
   </joint>
   <joint name="RShYaw" type="revolute">
@@ -800,5 +801,5 @@
     <axis xyz="0 0 1" />
     <limit velocity="4.0" effort="50" lower="-1.5708" upper="1.5708" />
-    <dynamics friction="0" damping="0.3"/>
+    <dynamics friction="0" damping="3.0"/>
   </joint>
   <joint name="RElbj" type="revolute">
@@ -808,5 +809,5 @@
     <axis xyz="0 1 0" />
     <limit velocity="4.0" effort="50" lower="-2.3562" upper="0.0" />
-    <dynamics friction="0" damping="0.3"/>
+    <dynamics friction="0" damping="3.0"/>
   </joint>
   <joint name="RForearmPlate" type="fixed">
@@ -822,5 +823,5 @@
     <axis xyz="0 1 0" />
     <limit velocity="4.0" effort="50" lower="-3.4034" upper="1.6581" />
-    <dynamics friction="0" damping="0.3"/>
+    <dynamics friction="0" damping="3.0"/>
   </joint>
   <joint name="LShLat" type="revolute">
@@ -830,5 +831,5 @@
     <axis xyz="1 0 0" />
     <limit velocity="4.0" effort="50" lower="-0.31415" upper="2.094" />
-    <dynamics friction="0" damping="0.3"/>
+    <dynamics friction="0" damping="3.0"/>
   </joint>
   <joint name="LShYaw" type="revolute">
@@ -838,5 +839,5 @@
     <axis xyz="0 0 1" />
     <limit velocity="4.0" effort="50" lower="-1.5708" upper="1.5708" />
-    <dynamics friction="0" damping="0.3"/>
+    <dynamics friction="0" damping="3.0"/>
   </joint>
   <joint name="LElbj" type="revolute">
@@ -846,5 +847,5 @@
     <axis xyz="0 1 0" />
     <limit velocity="4.0" effort="50" lower="-2.3562" upper="0.0" />
-    <dynamics friction="0" damping="0.3"/>
+    <dynamics friction="0" damping="3.0"/>
   </joint>
   <joint name="LForearmPlate" type="fixed">

Commit message: Fixed bug in urdf description

File: coman_urdf/urdf/coman.urdf.xacro (robot description, xacro)
@@ -404,8 +404,8 @@
     </collision>
   </link>
-  <xacro:if value="$(optenv GAZEBO_COMAN_USES_NO_FOREARMS true)">
+  <xacro:if value="$(optenv GAZEBO_COMAN_USES_NO_FOREARMS false)">
       <xacro:include filename="$(find coman_urdf)/urdf/forearms/no_forearms/links/no_forearms_R.urdf.xacro" />
   </xacro:if>
-  <xacro:if value="$(optenv GAZEBO_COMAN_USES_7DOF_FOREARMS_DRC_14 false)">
+  <xacro:if value="$(optenv GAZEBO_COMAN_USES_7DOF_FOREARMS_DRC_14 true)">
       <xacro:include filename="$(find coman_urdf)/urdf/forearms/7DOF_forearms_DRC_14/links/7DOF_forearms_R_DRC_14.urdf.xacro" />
   </xacro:if>
@@ -468,8 +468,8 @@
     </collision>
   </link>
-  <xacro:if value="$(optenv GAZEBO_COMAN_USES_NO_FOREARMS true)">
+  <xacro:if value="$(optenv GAZEBO_COMAN_USES_NO_FOREARMS false)">
       <xacro:include filename="$(find coman_urdf)/urdf/forearms/no_forearms/links/no_forearms_L.urdf.xacro" />
   </xacro:if>
-  <xacro:if value="$(optenv GAZEBO_COMAN_USES_7DOF_FOREARMS_DRC_14 false)">
+  <xacro:if value="$(optenv GAZEBO_COMAN_USES_7DOF_FOREARMS_DRC_14 true)">
       <xacro:include filename="$(find coman_urdf)/urdf/forearms/7DOF_forearms_DRC_14/links/7DOF_forearms_L_DRC_14.urdf.xacro" />
   </xacro:if>
@@ -480,10 +480,10 @@
     <origin xyz="0 0 0" rpy="0 0 0" />
   </joint>
-  <joint name="l_wrist_joint" type="fixed">
-    <parent link="LWrMot3"/>
-    <child link="l_wrist"/>
-    <origin xyz="0 0 0" rpy="0 0 0" />
-  </joint>
-  <xacro:if value="$(optenv GAZEBO_COMAN_USES_7DOF_FOREARMS_DRC_14 false)">
+<xacro:if value="$(optenv GAZEBO_COMAN_USES_7DOF_FOREARMS_DRC_14 true)">
+   <joint name="l_wrist_joint" type="fixed">
+     <parent link="LWrMot3"/>
+     <child link="l_wrist"/>
+     <origin xyz="0 0 0" rpy="0 0 0" />
+   </joint>
     <joint name="r_wrist_joint" type="fixed">
       <parent link="RWrMot3"/>
@@ -491,4 +491,17 @@
       <origin xyz="0 0 0" rpy="0 0 0" />
     </joint>
+</xacro:if>
+<xacro:if value="$(optenv GAZEBO_COMAN_USES_NO_FOREARMS false)">
+	<joint name="l_wrist_joint" type="fixed">
+	  <parent link="LElb"/>
+	  <child link="l_wrist"/>
+	  <origin xyz="-0.015 0 -0.22" rpy="0 0 0" />
+	</joint>
+        <joint name="r_wrist_joint" type="fixed">
+	  <parent link="RElb"/>
+	  <child link="r_wrist"/>
+	  <origin xyz="-0.015 0 -0.22" rpy="0 0 0" />
+	</joint>
+</xacro:if>
     <joint name="l_ankle_joint" type="fixed">
       <parent link="LFoot"/>
@@ -496,5 +509,4 @@
       <origin xyz="0 0 0" rpy="0 0 0" />
     </joint>
-  </xacro:if>
   <joint name="r_ankle_joint" type="fixed">
     <parent link="RFoot"/>
@@ -729,8 +741,8 @@
     <dynamics friction="0" damping="3.0"/>
   </joint>
-  <xacro:if value="$(optenv GAZEBO_COMAN_USES_NO_FOREARMS true)">
+  <xacro:if value="$(optenv GAZEBO_COMAN_USES_NO_FOREARMS false)">
       <xacro:include filename="$(find coman_urdf)/urdf/forearms/no_forearms/joints/no_forearms_R.urdf.xacro" />
   </xacro:if>
-  <xacro:if value="$(optenv GAZEBO_COMAN_USES_7DOF_FOREARMS_DRC_14 false)">
+  <xacro:if value="$(optenv GAZEBO_COMAN_USES_7DOF_FOREARMS_DRC_14 true)">
       <xacro:include filename="$(find coman_urdf)/urdf/forearms/7DOF_forearms_DRC_14/joints/7DOF_forearms_R_DRC_14.urdf.xacro" />
   </xacro:if>
@@ -768,8 +780,8 @@
     <dynamics friction="0" damping="3.0"/>
   </joint>
-  <xacro:if value="$(optenv GAZEBO_COMAN_USES_NO_FOREARMS true)">
+  <xacro:if value="$(optenv GAZEBO_COMAN_USES_NO_FOREARMS false)">
       <xacro:include filename="$(find coman_urdf)/urdf/forearms/no_forearms/joints/no_forearms_L.urdf.xacro" />
   </xacro:if>
-  <xacro:if value="$(optenv GAZEBO_COMAN_USES_7DOF_FOREARMS_DRC_14 false)">
+  <xacro:if value="$(optenv GAZEBO_COMAN_USES_7DOF_FOREARMS_DRC_14 true)">
       <xacro:include filename="$(find coman_urdf)/urdf/forearms/7DOF_forearms_DRC_14/joints/7DOF_forearms_L_DRC_14.urdf.xacro" />
   </xacro:if>

Commit message: Using a .xacro for model config instead of a .sh

File: coman_urdf/urdf/coman.urdf.xacro (robot description, xacro)
@@ -8,5 +8,6 @@
   Velocity and effort limits are fake!
 -->
-<!-- Adding macros for feet-->
+<!-- ************ MODEL CONFIGURATION ************ -->
+<xacro:include filename="$(find coman_urdf)/urdf/coman_config.urdf.xacro" />
 <!-- ********************LINKS******************** -->
 <!-- This links are defined in order to be compliant with http://www.ros.org/reps/rep-0120.html#coordinate-frames

File: coman_urdf/urdf/coman_config.urdf.xacro (robot description, xacro)
@@ -1,3 +1,5 @@
-#!/usr/bin/env bash
+<?xml version="1.0"?>
+<robot xmlns:xacro="http://ros.org/wiki/xacro" name="COMAN">
+<!--
 ####################################################
 ##
@@ -11,9 +13,10 @@
 ####################################################
 # TODO checks (must be mutually exclusive)
-#
-# 1) round feet
-export GAZEBO_COMAN_USES_ROUND_FEET_13=false
-# 2) simple feet
-export GAZEBO_COMAN_USES_SIMPLE_FEET_DRC_sw1_14=true
+-->
+<!-- 1) round feet -->
+<xacro:property name="GAZEBO_COMAN_USES_ROUND_FEET_13" value="false" />
+<!-- 2) simple feet -->
+<xacro:property name="GAZEBO_COMAN_USES_SIMPLE_FEET_DRC_sw1_14" value="true" />
+<!--
 ####################################################
 ##
@@ -31,15 +34,15 @@
 # 1) NO_FOREARMS + NO_HANDS
 #
-#export GAZEBO_COMAN_USES_NO_FOREARMS=true
-#export GAZEBO_COMAN_USES_NO_HANDS=true
-#export GAZEBO_COMAN_USES_7DOF_FOREARMS_DRC_14=false
-#export GAZEBO_COMAN_USES_SOFTHANDS_DRC_sw1_14=false
-#
+<xacro:property name="GAZEBO_COMAN_USES_NO_FOREARMS" value="true" />
+<xacro:property name="GAZEBO_COMAN_USES_NO_HANDS" value="false" />
+<xacro:property name="GAZEBO_COMAN_USES_7DOF_FOREARMS_DRC_14" value="true" />
+<xacro:property name="GAZEBO_COMAN_USES_SOFTHANDS_DRC_sw1_14" value="false" />
 # 2) 7DOFS_FOREARMS + SOFTHANDS
-#
-export GAZEBO_COMAN_USES_NO_FOREARMS=false
-export GAZEBO_COMAN_USES_NO_HANDS=false
-export GAZEBO_COMAN_USES_7DOF_FOREARMS_DRC_14=true
-export GAZEBO_COMAN_USES_SOFTHANDS_DRC_sw1_14=true
+-->
+<xacro:property name="GAZEBO_COMAN_USES_NO_FOREARMS" value="false" />
+<xacro:property name="GAZEBO_COMAN_USES_NO_HANDS" value="false" />
+<xacro:property name="GAZEBO_COMAN_USES_7DOF_FOREARMS_DRC_14" value="true" />
+<xacro:property name="GAZEBO_COMAN_USES_SOFTHANDS_DRC_sw1_14" value="true" />
+<!--
 ####################################################
 ##
@@ -67,9 +70,13 @@
 # 1) yarp
 #
-export GAZEBO_COMAN_USES_ROS=false
+-->
+<xacro:property name="GAZEBO_COMAN_USES_ROS" value="false" />
+<!--
 #
 # 2) ros
 #
-export GAZEBO_COMAN_USES_YARP=true
+-->
+<xacro:property name="GAZEBO_COMAN_USES_YARP" value="true" />
+<!--
 ####################################################
 ##
@@ -90,3 +97,5 @@
 # 1/2 (true/false)
 #
-export GAZEBO_COMAN_USES_ACCURATE_FT=false
+-->
+<xacro:property name="GAZEBO_COMAN_USES_ACCURATE_FT" value="false" />
+</robot>
