Commit message: Refactory of coman.urdf.xacro. Added hands as revolute joints.

File: coman_urdf/urdf/coman.urdf.xacro (robot description, xacro)
@@ -4,5 +4,5 @@
   ROS urdf definition of the COMAN humanoid robot by Istituto Italiano di Tecnologia
   DO NOT INCLUDE THIS FILE DIRECTLY! USE coman_robot.urdf.xacro INSTEAD!
-  Author: Enrico Mingo
+  Author: Enrico Mingo & Alessio Rocchi
   Inertial matrix has to be in CoM frame (URDF specs)
   Velocity and effort limits are fake!
@@ -10,5 +10,5 @@
 <!-- ************ MODEL CONFIGURATION ************ -->
 <xacro:include filename="$(find coman_urdf)/urdf/coman_config.urdf.xacro" />
-<!-- ********************LINKS******************** -->
+<!-- ******************** FAKE LINKS ******************** -->
 <!-- This links are defined in order to be compliant with http://www.ros.org/reps/rep-0120.html#coordinate-frames
 and to define the end effectors of the robot -->
@@ -31,461 +31,15 @@
 <!-- Head -->
  <link name="gaze"/>
-<!-- ********************TORSO******************** -->
-<!-- first real link of the robot, inertial reference frame -->
-  <link name="Waist">
-    <inertial>
-      <origin xyz="-0.026391145 -5.8216364E-4 0.052632312" rpy="0 0 0"/>
-      <mass value="1.8008695"/>
-      <inertia ixx="0.0051032982"  ixy="-5.7170981E-5"  ixz="0.0016920543" iyy="0.006241636" iyz="1.7225949E-5" izz="0.0024517762" />
-    </inertial>
-    <visual>
-      <origin xyz="0 0 -0.52" rpy="0 0 -3.14159265359"/>
-      <geometry name="Waist_visual">
-        <mesh filename="package://coman_urdf/meshes/collada/asm0001_collada_07_prt.dae" scale="0.03937 0.03937 0.03937"/>
-      </geometry>
-    </visual>
-    <collision>
-      <origin xyz="0 0 -0.52" rpy="0 0 -3.14159265359"/>
-      <geometry name="Waist_collision">
-        <mesh filename="package://coman_urdf/meshes/collada/simple/simple_asm0001_collada_07_prt.dae" scale="0.03937 0.03937 0.03937"/>
-      </geometry>
-    </collision>
-  </link>
-  <link name ="DWS">
-    <inertial>
-      <origin xyz="4.2999707E-4 -0.0097650317 0.033011157" rpy="0 0 0"/>
-      <mass value="0.54588774"/>
-      <inertia ixx="9.7126578E-4"  ixy="-7.2101244E-7"  ixz="1.1440119E-6" iyy="7.4686706E-4" iyz="-1.7450917E-4" izz="6.2196235E-4" />
-    </inertial>
-    <visual>
-      <origin xyz="-0.020281504 0 -0.63912053" rpy="0 0 -3.14159265359"/>
-      <geometry name="DWS_visual">
-        <mesh filename="package://coman_urdf/meshes/collada/asm0001_collada_09_prt.dae" scale="0.03937 0.03937 0.03937" />
-      </geometry>
-    </visual>
-    <collision>
-      <origin xyz="-0.020281504 0 -0.63912053" rpy="0 0 -3.14159265359"/>
-      <geometry name="DWS_collision">
-        <mesh filename="package://coman_urdf/meshes/collada/simple/simple_asm0001_collada_09_prt.dae" scale="0.03937 0.03937 0.03937" />
-      </geometry>
-    </collision>
-  </link>
-  <link name ="DWL">
-    <inertial>
-      <origin xyz="-0.0021273416 0.0033575235 -0.0010076896" rpy="0 0 0"/>
-      <mass value="0.75398402"/>
-      <inertia ixx="3.4093348E-4"  ixy="-6.2120042E-6"  ixz="-1.3863473E-6" iyy="3.9581916E-4" iyz="1.443019E-6" izz="3.7449753E-4" />
-    </inertial>
-    <visual>
-      <origin xyz="-0.020281504 0 -0.63912053" rpy="0 0 -3.14159265359"/>
-      <geometry name="DWL_visual">
-        <mesh filename="package://coman_urdf/meshes/collada/asm0001_collada_08_prt.dae" scale="0.03937 0.03937 0.03937" />
-      </geometry>
-    </visual>
-    <collision>
-      <origin xyz="-0.020281504 0 -0.63912053" rpy="0 0 -3.14159265359"/>
-      <geometry name="DWL_collision">
-        <mesh filename="package://coman_urdf/meshes/collada/simple/simple_asm0001_collada_08_prt.dae" scale="0.03937 0.03937 0.03937" />
-      </geometry>
-    </collision>
-  </link>
-  <link name ="DWYTorso">
-    <inertial>
-      <origin xyz="-0.0358501 1.8286043E-5 0.117557148" rpy="0 0 0"/>
-      <mass value="6.3617175"/>
-      <inertia ixx="0.034089342"  ixy="-9.8308572E-6"  ixz="-7.5649290E-4" iyy="0.030117357" iyz="6.2443771E-6" izz="0.025296582" />
-    </inertial>
-    <visual>
-      <origin xyz="-0.020281504 0.0 -0.68662053" rpy="0 0 -3.14159265359"/>
-      <geometry name="DWYTorso_visual">
-        <mesh filename="package://coman_urdf/meshes/collada/asm0001_collada_10_prt.dae" scale="0.03937 0.03937 0.03937" />
-      </geometry>
-    </visual>
-    <collision>
-      <origin xyz="-0.020281504 0.0 -0.68662053" rpy="0 0 -3.14159265359"/>
-      <geometry name="DWYTorso_collision">
-        <mesh filename="package://coman_urdf/meshes/collada/simple/simple_asm0001_collada_10_prt.dae" scale="0.03937 0.03937 0.03937" />
-      </geometry>
-    </collision>
-  </link>
-<!-- ********************RIGHT LEG******************** -->
-  <link name ="RHipMot">
-    <inertial>
-      <origin xyz="-3.269678E-4 -0.023587321 -2.6496509E-4" rpy="0 0 0"/>
-      <mass value="0.89258227"/>
-      <inertia ixx="4.7672294E-4"  ixy="-3.9936567E-6"  ixz="-2.4802574E-6" iyy="5.458038E-4" iyz="-3.3389575E-6" izz="5.126859E-4" />
-    </inertial>
-    <visual>
-      <origin xyz="0.0 0.023 -0.52" rpy="0 0 -3.14159265359"/>
-      <geometry name="RHipMot_visual">
-        <mesh filename="package://coman_urdf/meshes/collada/asm0001_collada_20_prt.dae" scale="0.03937 0.03937 0.03937" />
-      </geometry>
-    </visual>
-    <collision>
-      <origin xyz="0.0 0.023 -0.52" rpy="0 0 -3.14159265359"/>
-      <geometry name="RHipMot_collision">
-        <mesh filename="package://coman_urdf/meshes/collada/simple/simple_asm0001_collada_20_prt.dae" scale="0.03937 0.03937 0.03937" />
-      </geometry>
-    </collision>
-  </link>
-  <link name ="RThighUpLeg">
-    <inertial>
-      <origin xyz="0.0012591632 -0.016896372 -0.058903336" rpy="0 0 0"/>
-      <mass value="1.0246101"/>
-      <inertia ixx="9.165719E-4"  ixy="-1.4449904E-6"  ixz="-1.6685011E-5" iyy="0.00104849584" iyz="2.5492874E-5" izz="6.8637197E-4" />
-    </inertial>
-    <visual>
-      <origin xyz="0.0 0.0726 -0.52" rpy="0 0 -3.14159265359"/>
-      <geometry name="RThighUpLeg_visual">
-        <mesh filename="package://coman_urdf/meshes/collada/asm0001_collada_19_prt.dae" scale="0.03937 0.03937 0.03937" />
-      </geometry>
-    </visual>
-    <collision>
-      <origin xyz="0.0 0.0726 -0.52" rpy="0 0 -3.14159265359"/>
-      <geometry name="RThighUpLeg_collision">
-        <mesh filename="package://coman_urdf/meshes/collada/simple/simple_asm0001_collada_19_prt.dae" scale="0.03937 0.03937 0.03937" />
-      </geometry>
-    </collision>
-  </link>
-  <link name ="RThighLowLeg">
-    <inertial>
-      <origin xyz="9.8720058E-4 6.7037262E-4 -0.075716843" rpy="0 0 0"/>
-      <mass value="1.7001134"/>
-      <inertia ixx="0.0038979546"  ixy="1.7802399E-6"  ixz="2.6403262E-5" iyy="0.0039360845" iyz="4.522711E-5" izz="9.0218711E-4" />
-    </inertial>
-    <visual>
-      <origin xyz="0.0 0.0726 -0.4176" rpy="0 0 -3.14159265359"/>
-      <geometry name="RThighLowLeg_visual">
-        <mesh filename="package://coman_urdf/meshes/collada/asm0001_collada_18_prt.dae" scale="0.03937 0.03937 0.03937" />
-      </geometry>
-    </visual>
-    <collision>
-      <origin xyz="0.0 0.0726 -0.4176" rpy="0 0 -3.14159265359"/>
-      <geometry name="RThighLowLeg_collision">
-        <mesh filename="package://coman_urdf/meshes/collada/simple/simple_asm0001_collada_18_prt.dae" scale="0.03937 0.03937 0.03937" />
-      </geometry>
-    </collision>
-  </link>
-  <link name ="RLowLeg">
-    <inertial>
-      <origin xyz="0.0024612666 -0.0053099614 -0.08598948" rpy="0 0 0"/>
-      <mass value="1.4098179"/>
-      <inertia ixx="0.0040604004"  ixy="1.1227206E-5"  ixz="1.2260973E-5" iyy="0.004005652855" iyz="5.1899176E-4" izz="0.0012414054" />
-    </inertial>
-    <visual>
-      <origin xyz="0.0 0.0726 -0.2942" rpy="0 0 -3.14159265359"/>
-      <geometry name="RLowLeg_visual">
-        <mesh filename="package://coman_urdf/meshes/collada/asm0001_collada_17_prt.dae" scale="0.03937 0.03937 0.03937" />
-      </geometry>
-    </visual>
-    <collision>
-      <origin xyz="0.0 0.0726 -0.2942" rpy="0 0 -3.14159265359"/>
-      <geometry name="RLowLeg_collision">
-        <mesh filename="package://coman_urdf/meshes/collada/simple/simple_asm0001_collada_17_prt.dae" scale="0.03937 0.03937 0.03937" />
-      </geometry>
-    </collision>
-  </link>
-  <link name ="RFootmot">
-    <inertial>
-      <origin xyz="8.8067281E-4 -9.2224881E-4 2.3038476E-4" rpy="0 0 0"/>
-      <mass value="0.72992131"/>
-      <inertia ixx="3.2034425E-4"  ixy="7.6346303E-6"  ixz="2.5430158E-7" iyy="3.6584358E-4" iyz="-3.6889276E-6" izz="3.6065156E-4" />
-    </inertial>
-    <visual>
-      <origin xyz="0.0 0.0726 -0.0932" rpy="0 0 -3.14159265359"/>
-      <geometry name="RFootmot_visual">
-        <mesh filename="package://coman_urdf/meshes/collada/asm0001_collada_16_prt.dae" scale="0.03937 0.03937 0.03937" />
-      </geometry>
-    </visual>
-    <collision>
-      <origin xyz="0.0 0.0726 -0.0932" rpy="0 0 -3.14159265359"/>
-      <geometry name="RFootmot_collision">
-        <mesh filename="package://coman_urdf/meshes/collada/simple/simple_asm0001_collada_16_prt.dae" scale="0.03937 0.03937 0.03937" />
-      </geometry>
-    </collision>
-  </link>
-  <xacro:unless value="${GAZEBO_COMAN_USES_ACCURATE_FT}">
-    <xacro:if value="${GAZEBO_COMAN_USES_ROUND_FEET_13}">
-      <xacro:include filename="$(find coman_urdf)/urdf/feet/round_feet_13/round_foot_R_13.urdf.xacro" />
-    </xacro:if>
-    <xacro:if value="${GAZEBO_COMAN_USES_SIMPLE_FEET_DRC_sw1_14}">
-      <xacro:include filename="$(find coman_urdf)/urdf/feet/simple_feet_DRC_sw1_14/simple_foot_R_DRC_sw1_14.urdf.xacro" />
-    </xacro:if>
-  </xacro:unless>
-  <xacro:if value="${GAZEBO_COMAN_USES_ACCURATE_FT}">
-    <link name ="RFootFTSensor">
-      <inertial>
-        <origin xyz="0.0 -0.0 -0.0325" rpy="0 0 0"/>
-        <mass value="0.280"/>
-        <inertia ixx="0.0012944808"  ixy="0.0"  ixz="2.0080105E-4" iyy="0.0015851846" iyz="2.7599327E-4" izz="0.0013326766" />
-      </inertial>
-    </link>
-    <xacro:if value="${GAZEBO_COMAN_USES_ROUND_FEET_13}">
-      <xacro:include filename="$(find coman_urdf)/urdf/feet/round_feet_13/accurate_FT_round_foot_R_13.urdf.xacro" />
-    </xacro:if>
-    <xacro:if value="${GAZEBO_COMAN_USES_SIMPLE_FEET_DRC_sw1_14}">
-      <xacro:include filename="$(find coman_urdf)/urdf/feet/simple_feet_DRC_sw1_14/accurate_FT_simple_foot_R_DRC_sw1_14.urdf.xacro" />
-    </xacro:if>
-  </xacro:if>
-<!-- ********************LEFT LEG******************** -->
-  <link name ="LHipMot">
-    <inertial>
-      <origin xyz="-3.269678E-4 0.023587321 -2.6496509E-4" rpy="0 0 0"/>
-      <mass value="0.89258227"/>
-      <inertia ixx="4.7672294E-4"  ixy="3.9936567E-6"  ixz="-2.4802574E-6" iyy="5.458038E-4" iyz="3.3389575E-6" izz="5.126859E-4" />
-    </inertial>
-    <visual>
-      <origin xyz="0.0 -0.023 -0.52" rpy="0 0 -3.14159265359"/>
-      <geometry name="RHipMot_visual">
-        <mesh filename="package://coman_urdf/meshes/collada/asm0001_collada_06_prt.dae" scale="0.03937 0.03937 0.03937" />
-      </geometry>
-    </visual>
-    <collision>
-      <origin xyz="0.0 -0.023 -0.52" rpy="0 0 -3.14159265359"/>
-      <geometry name="RHipMot_collision">
-        <mesh filename="package://coman_urdf/meshes/collada/simple/simple_asm0001_collada_06_prt.dae" scale="0.03937 0.03937 0.03937" />
-      </geometry>
-    </collision>
-  </link>
-  <link name ="LThighUpLeg">
-    <inertial>
-      <origin xyz="0.0012591632 0.016896372 -0.058903336" rpy="0 0 0"/>
-      <mass value="1.0246101"/>
-      <inertia ixx="9.165719E-4"  ixy="1.4449904E-6"  ixz="-1.6685011E-5" iyy="0.00104849584" iyz="-2.5492874E-5" izz="6.8637197E-4" />
-    </inertial>
-    <visual>
-      <origin xyz="0.0 -0.0726 -0.52" rpy="0 0 -3.14159265359"/>
-      <geometry name="LThighUpLeg_visual">
-        <mesh filename="package://coman_urdf/meshes/collada/asm0001_collada_05_prt.dae" scale="0.03937 0.03937 0.03937" />
-      </geometry>
-    </visual>
-    <collision>
-      <origin xyz="0.0 -0.0726 -0.52" rpy="0 0 -3.14159265359"/>
-      <geometry name="LThighUpLeg_collision">
-        <mesh filename="package://coman_urdf/meshes/collada/simple/simple_asm0001_collada_05_prt.dae" scale="0.03937 0.03937 0.03937" />
-      </geometry>
-    </collision>
-  </link>
-  <link name ="LThighLowLeg">
-    <inertial>
-      <origin xyz="9.8720058E-4 -6.7037262E-4 -0.075716843" rpy="0 0 0"/>
-      <mass value="1.7001134"/>
-      <inertia ixx="0.0038979546"  ixy="-1.7802399E-6"  ixz="2.6403262E-5" iyy="0.0039360845" iyz="-4.5227110E-5" izz="9.0218711E-4" />
-    </inertial>
-    <visual>
-      <origin xyz="0.0 -0.0726 -0.4176" rpy="0 0 -3.14159265359"/>
-      <geometry name="LThighLowLeg_visual">
-        <mesh filename="package://coman_urdf/meshes/collada/asm0001_collada_04_prt.dae" scale="0.03937 0.03937 0.03937" />
-      </geometry>
-    </visual>
-    <collision>
-      <origin xyz="0.0 -0.0726 -0.4176" rpy="0 0 -3.14159265359"/>
-      <geometry name="LThighLowLeg_collision">
-        <mesh filename="package://coman_urdf/meshes/collada/simple/simple_asm0001_collada_04_prt.dae" scale="0.03937 0.03937 0.03937" />
-      </geometry>
-    </collision>
-  </link>
-  <link name ="LLowLeg">
-    <inertial>
-      <origin xyz="0.0024612666 0.0053099614 -0.085989484" rpy="0 0 0"/>
-      <mass value="1.4098179"/>
-      <inertia ixx="0.0040604004"  ixy="-1.1227206E-5"  ixz="1.2260973E-5" iyy="0.004005652855" iyz="-5.1899176E-4" izz="0.0012414054" />
-    </inertial>
-    <visual>
-      <origin xyz="0.0 -0.0726 -0.2942" rpy="0 0 -3.14159265359"/>
-      <geometry name="LLowLeg_visual">
-        <mesh filename="package://coman_urdf/meshes/collada/asm0001_collada_03_prt.dae" scale="0.03937 0.03937 0.03937" />
-      </geometry>
-    </visual>
-    <collision>
-      <origin xyz="0.0 -0.0726 -0.2942" rpy="0 0 -3.14159265359"/>
-      <geometry name="LLowLeg_collision">
-        <mesh filename="package://coman_urdf/meshes/collada/simple/simple_asm0001_collada_03_prt.dae" scale="0.03937 0.03937 0.03937" />
-      </geometry>
-    </collision>
-  </link>
-  <link name ="LFootmot">
-    <inertial>
-      <origin xyz="8.8067281E-4 9.2224881E-4 2.3038476E-4" rpy="0 0 0"/>
-      <mass value="0.72992131"/>
-      <inertia ixx="3.2034425E-4"  ixy="-7.6346303E-6"  ixz="2.5430158E-7" iyy="3.6584358E-4" iyz="3.6889276E-6" izz="3.6065156E-4" />
-    </inertial>
-    <visual>
-      <origin xyz="0.0 -0.0726 -0.0932" rpy="0 0 -3.14159265359"/>
-      <geometry name="LFootmot_visual">
-        <mesh filename="package://coman_urdf/meshes/collada/asm0001_collada_02_prt.dae" scale="0.03937 0.03937 0.03937" />
-      </geometry>
-    </visual>
-    <collision>
-      <origin xyz="0.0 -0.0726 -0.0932" rpy="0 0 -3.14159265359"/>
-      <geometry name="LFootmot_collision">
-        <mesh filename="package://coman_urdf/meshes/collada/simple/simple_asm0001_collada_02_prt.dae" scale="0.03937 0.03937 0.03937" />
-      </geometry>
-    </collision>
-  </link>
-  <xacro:unless value="${GAZEBO_COMAN_USES_ACCURATE_FT}">
-    <xacro:if value="${GAZEBO_COMAN_USES_ROUND_FEET_13}">
-      <xacro:include filename="$(find coman_urdf)/urdf/feet/round_feet_13/round_foot_L_13.urdf.xacro" />
-    </xacro:if>
-    <xacro:if value="${GAZEBO_COMAN_USES_SIMPLE_FEET_DRC_sw1_14}">
-      <xacro:include filename="$(find coman_urdf)/urdf/feet/simple_feet_DRC_sw1_14/simple_foot_L_DRC_sw1_14.urdf.xacro" />
-    </xacro:if>
-  </xacro:unless>
-  <xacro:if value="${GAZEBO_COMAN_USES_ACCURATE_FT}">
-    <link name ="LFootFTSensor">
-      <inertial>
-        <origin xyz="0.0 -0.0 -0.0325" rpy="0 0 0"/>
-        <mass value="0.280"/>
-        <inertia ixx="0.0012944808"  ixy="-9.2387693E-5"  ixz="2.0080105E-4" iyy="0.0015851846" iyz="2.7599327E-4" izz="0.0013326766" />
-      </inertial>
-    </link>
-    <xacro:if value="${GAZEBO_COMAN_USES_ROUND_FEET_13}">
-      <xacro:include filename="$(find coman_urdf)/urdf/feet/round_feet_13/accurate_FT_round_foot_L_13.urdf.xacro" />
-    </xacro:if>
-    <xacro:if value="${GAZEBO_COMAN_USES_SIMPLE_FEET_DRC_sw1_14}">
-      <xacro:include filename="$(find coman_urdf)/urdf/feet/simple_feet_DRC_sw1_14/accurate_FT_simple_foot_L_DRC_sw1_14.urdf.xacro" />
-    </xacro:if>
-  </xacro:if>
-<!-- ********************RIGHT ARM******************** -->
-  <link name ="RShp">
-    <inertial>
-      <origin xyz="0.0099500565 -0.038682024 1.6446924E-4" rpy="0 0 0"/>
-      <mass value="0.56782202"/>
-      <inertia ixx="7.8337456E-4"  ixy="1.9035768E-4"  ixz="-3.0037676E-6" iyy="6.3399921E-4" iyz="4.3840774E-6" izz="0.001008054" />
-    </inertial>
-    <visual>
-      <origin xyz="-0.005305 0.0825 -0.844329" rpy="0 0 -3.14159265359"/>
-      <geometry name="RShp_visual">
-        <mesh filename="package://coman_urdf/meshes/collada/asm0001_collada_24_prt.dae" scale="0.03937 0.03937 0.03937" />
-      </geometry>
-    </visual>
-    <collision>
-      <origin xyz="-0.005305 0.0825 -0.844329" rpy="0 0 -3.14159265359"/>
-      <geometry name="RShp_collision">
-        <mesh filename="package://coman_urdf/meshes/collada/simple/simple_asm0001_collada_24_prt.dae" scale="0.03937 0.03937 0.03937" />
-      </geometry>
-    </collision>
-  </link>
-  <link name ="RShr">
-    <inertial>
-      <origin xyz="-0.0038936743 2.2022151E-6 -0.0048616005" rpy="0 0 0"/>
-      <mass value="0.77683752"/>
-      <inertia ixx="4.5812904E-4"  ixy="-2.4111086E-7"  ixz="9.2521185E-6" iyy="4.3089204E-4" iyz="-4.7216950E-7" izz="3.4174855E-4" />
-    </inertial>
-    <visual>
-      <origin xyz="-0.005305 0.1558 -0.844329" rpy="0 0 -3.14159265359"/>
-      <geometry name="RShr_visual">
-        <mesh filename="package://coman_urdf/meshes/collada/asm0001_collada_23_prt.dae" scale="0.03937 0.03937 0.03937" />
-      </geometry>
-    </visual>
-    <collision>
-      <origin xyz="-0.005305 0.1558 -0.844329" rpy="0 0 -3.14159265359"/>
-      <geometry name="RShr_collision">
-        <mesh filename="package://coman_urdf/meshes/collada/simple/simple_asm0001_collada_23_prt.dae" scale="0.03937 0.03937 0.03937" />
-      </geometry>
-    </collision>
-  </link>
-  <link name ="RShy">
-    <inertial>
-      <origin xyz="0.0022714213 -0.0071091517 -0.057455221" rpy="0 0 0"/>
-      <mass value="1.0462304"/>
-      <inertia ixx="0.0030934574"  ixy="6.6702837E-5"  ixz="3.0222291E-4" iyy="0.0029181573" iyz="-5.2663661E-4" izz="8.0830389E-4" />
-    </inertial>
-    <visual>
-      <origin xyz="-0.005305 0.1558 -0.79952053" rpy="0 0 -3.14159265359"/>
-      <geometry name="RShy_visual">
-        <mesh filename="package://coman_urdf/meshes/collada/asm0001_collada_22_prt.dae" scale="0.03937 0.03937 0.03937" />
-      </geometry>
-    </visual>
-    <collision>
-      <origin xyz="-0.005305 0.1558 -0.79952053" rpy="0 0 -3.14159265359"/>
-      <geometry name="RShy_collision">
-        <mesh filename="package://coman_urdf/meshes/collada/simple/simple_asm0001_collada_22_prt.dae" scale="0.03937 0.03937 0.03937" />
-      </geometry>
-    </collision>
-  </link>
-  <xacro:if value="${GAZEBO_COMAN_USES_NO_FOREARMS}">
-      <xacro:include filename="$(find coman_urdf)/urdf/forearms/no_forearms/links/no_forearms_R.urdf.xacro" />
+<!-- ************ COMAN BASE ************** -->
+<xacro:include filename="$(find coman_urdf)//urdf/coman_base.urdf.xacro"/>
+<!-- ************ FOREARMS ************ -->
+<xacro:if value="${GAZEBO_COMAN_USES_NO_FOREARMS}">
+      <xacro:include filename="$(find coman_urdf)/urdf/forearms/no_forearms/no_forearms.urdf.xacro" />
   </xacro:if>
   <xacro:if value="${GAZEBO_COMAN_USES_7DOF_FOREARMS_DRC_14}">
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