Commit message: self-collision detection fixed...
...the secret is .stl instead of .dae for collision geometries :O

File: coman_urdf/urdf/coman.urdf.xacro (robot description, xacro)
@@ -46,5 +46,5 @@
       <origin xyz="-0.020281504 0.0 -0.68662053" rpy="0 0 -3.14159265359"/>
       <geometry name="Xtion_body_collision">
-        <mesh filename="package://coman_urdf/meshes/collada/simple/Xtion/xtion_base.dae" scale="0.03937 0.03937 0.03937" />
+        <mesh filename="package://coman_urdf/meshes/collada/simple/Xtion/xtion_base.stl" scale="0.03937 0.03937 0.03937" />
       </geometry>
     </collision>
@@ -65,5 +65,5 @@
       <origin xyz="-0.0915 0.0 -1.2778" rpy="0 0 -3.14159265359"/>
       <geometry name="Xtion_cam_body_collision">
-        <mesh filename="package://coman_urdf/meshes/collada/Xtion/xtion_cam_body.dae" scale="0.001 0.001 0.001" />
+        <mesh filename="package://coman_urdf/meshes/collada/simple/Xtion/xtion_cam_body.stl" scale="0.001 0.001 0.001" />
       </geometry>
     </collision>

File: coman_urdf/urdf/coman_base.urdf.xacro (robot description, xacro)
@@ -25,5 +25,5 @@
       <origin xyz="0 0 -0.52" rpy="0 0 -3.14159265359"/>
       <geometry name="Waist_collision">
-        <mesh filename="package://coman_urdf/meshes/collada/simple/simple_asm0001_collada_07_prt.dae" scale="0.03937 0.03937 0.03937"/>
+        <mesh filename="package://coman_urdf/meshes/collada/simple/simple_asm0001_collada_07_prt.stl" scale="0.03937 0.03937 0.03937"/>
       </geometry>
     </collision>
@@ -44,5 +44,5 @@
       <origin xyz="-0.020281504 0 -0.63912053" rpy="0 0 -3.14159265359"/>
       <geometry name="DWS_collision">
-        <mesh filename="package://coman_urdf/meshes/collada/simple/simple_asm0001_collada_09_prt.dae" scale="0.03937 0.03937 0.03937" />
+        <mesh filename="package://coman_urdf/meshes/collada/simple/simple_asm0001_collada_09_prt.stl" scale="0.03937 0.03937 0.03937" />
       </geometry>
     </collision>
@@ -63,5 +63,5 @@
       <origin xyz="-0.020281504 0 -0.63912053" rpy="0 0 -3.14159265359"/>
       <geometry name="DWL_collision">
-        <mesh filename="package://coman_urdf/meshes/collada/simple/simple_asm0001_collada_08_prt.dae" scale="0.03937 0.03937 0.03937" />
+        <mesh filename="package://coman_urdf/meshes/collada/simple/simple_asm0001_collada_08_prt.stl" scale="0.03937 0.03937 0.03937" />
       </geometry>
     </collision>
@@ -82,5 +82,5 @@
       <origin xyz="-0.020281504 0.0 -0.68662053" rpy="0 0 -3.14159265359"/>
       <geometry name="DWYTorso_collision">
-        <mesh filename="package://coman_urdf/meshes/collada/simple/simple_asm0001_collada_10_prt.dae" scale="0.03937 0.03937 0.03937" />
+        <mesh filename="package://coman_urdf/meshes/collada/simple/simple_asm0001_collada_10_prt.stl" scale="0.03937 0.03937 0.03937" />
       </geometry>
     </collision>
@@ -102,5 +102,5 @@
       <origin xyz="0.0 0.023 -0.52" rpy="0 0 -3.14159265359"/>
       <geometry name="RHipMot_collision">
-        <mesh filename="package://coman_urdf/meshes/collada/simple/simple_asm0001_collada_20_prt.dae" scale="0.03937 0.03937 0.03937" />
+        <mesh filename="package://coman_urdf/meshes/collada/simple/simple_asm0001_collada_20_prt.stl" scale="0.03937 0.03937 0.03937" />
       </geometry>
     </collision>
@@ -121,5 +121,5 @@
       <origin xyz="0.0 0.0726 -0.52" rpy="0 0 -3.14159265359"/>
       <geometry name="RThighUpLeg_collision">
-        <mesh filename="package://coman_urdf/meshes/collada/simple/simple_asm0001_collada_19_prt.dae" scale="0.03937 0.03937 0.03937" />
+        <mesh filename="package://coman_urdf/meshes/collada/simple/simple_asm0001_collada_19_prt.stl" scale="0.03937 0.03937 0.03937" />
       </geometry>
     </collision>
@@ -140,5 +140,5 @@
       <origin xyz="0.0 0.0726 -0.4176" rpy="0 0 -3.14159265359"/>
       <geometry name="RThighLowLeg_collision">
-        <mesh filename="package://coman_urdf/meshes/collada/simple/simple_asm0001_collada_18_prt.dae" scale="0.03937 0.03937 0.03937" />
+        <mesh filename="package://coman_urdf/meshes/collada/simple/simple_asm0001_collada_18_prt.stl" scale="0.03937 0.03937 0.03937" />
       </geometry>
     </collision>
@@ -159,5 +159,5 @@
       <origin xyz="0.0 0.0726 -0.2942" rpy="0 0 -3.14159265359"/>
       <geometry name="RLowLeg_collision">
-        <mesh filename="package://coman_urdf/meshes/collada/simple/simple_asm0001_collada_17_prt.dae" scale="0.03937 0.03937 0.03937" />
+        <mesh filename="package://coman_urdf/meshes/collada/simple/simple_asm0001_collada_17_prt.stl" scale="0.03937 0.03937 0.03937" />
       </geometry>
     </collision>
@@ -178,5 +178,5 @@
       <origin xyz="0.0 0.0726 -0.0932" rpy="0 0 -3.14159265359"/>
       <geometry name="RFootmot_collision">
-        <mesh filename="package://coman_urdf/meshes/collada/simple/simple_asm0001_collada_16_prt.dae" scale="0.03937 0.03937 0.03937" />
+        <mesh filename="package://coman_urdf/meshes/collada/simple/simple_asm0001_collada_16_prt.stl" scale="0.03937 0.03937 0.03937" />
       </geometry>
     </collision>
@@ -221,5 +221,5 @@
       <origin xyz="0.0 -0.023 -0.52" rpy="0 0 -3.14159265359"/>
       <geometry name="RHipMot_collision">
-        <mesh filename="package://coman_urdf/meshes/collada/simple/simple_asm0001_collada_06_prt.dae" scale="0.03937 0.03937 0.03937" />
+        <mesh filename="package://coman_urdf/meshes/collada/simple/simple_asm0001_collada_06_prt.stl" scale="0.03937 0.03937 0.03937" />
       </geometry>
     </collision>
@@ -240,5 +240,5 @@
       <origin xyz="0.0 -0.0726 -0.52" rpy="0 0 -3.14159265359"/>
       <geometry name="LThighUpLeg_collision">
-        <mesh filename="package://coman_urdf/meshes/collada/simple/simple_asm0001_collada_05_prt.dae" scale="0.03937 0.03937 0.03937" />
+        <mesh filename="package://coman_urdf/meshes/collada/simple/simple_asm0001_collada_05_prt.stl" scale="0.03937 0.03937 0.03937" />
       </geometry>
     </collision>
@@ -259,5 +259,5 @@
       <origin xyz="0.0 -0.0726 -0.4176" rpy="0 0 -3.14159265359"/>
       <geometry name="LThighLowLeg_collision">
-        <mesh filename="package://coman_urdf/meshes/collada/simple/simple_asm0001_collada_04_prt.dae" scale="0.03937 0.03937 0.03937" />
+        <mesh filename="package://coman_urdf/meshes/collada/simple/simple_asm0001_collada_04_prt.stl" scale="0.03937 0.03937 0.03937" />
       </geometry>
     </collision>
@@ -278,5 +278,5 @@
       <origin xyz="0.0 -0.0726 -0.2942" rpy="0 0 -3.14159265359"/>
       <geometry name="LLowLeg_collision">
-        <mesh filename="package://coman_urdf/meshes/collada/simple/simple_asm0001_collada_03_prt.dae" scale="0.03937 0.03937 0.03937" />
+        <mesh filename="package://coman_urdf/meshes/collada/simple/simple_asm0001_collada_03_prt.stl" scale="0.03937 0.03937 0.03937" />
       </geometry>
     </collision>
@@ -297,5 +297,5 @@
       <origin xyz="0.0 -0.0726 -0.0932" rpy="0 0 -3.14159265359"/>
       <geometry name="LFootmot_collision">
-        <mesh filename="package://coman_urdf/meshes/collada/simple/simple_asm0001_collada_02_prt.dae" scale="0.03937 0.03937 0.03937" />
+        <mesh filename="package://coman_urdf/meshes/collada/simple/simple_asm0001_collada_02_prt.stl" scale="0.03937 0.03937 0.03937" />
       </geometry>
     </collision>
@@ -340,5 +340,5 @@
       <origin xyz="-0.005305 0.0825 -0.844329" rpy="0 0 -3.14159265359"/>
       <geometry name="RShp_collision">
-        <mesh filename="package://coman_urdf/meshes/collada/simple/simple_asm0001_collada_24_prt.dae" scale="0.03937 0.03937 0.03937" />
+        <mesh filename="package://coman_urdf/meshes/collada/simple/simple_asm0001_collada_24_prt.stl" scale="0.03937 0.03937 0.03937" />
       </geometry>
     </collision>
@@ -359,5 +359,5 @@
       <origin xyz="-0.005305 0.1558 -0.844329" rpy="0 0 -3.14159265359"/>
       <geometry name="RShr_collision">
-        <mesh filename="package://coman_urdf/meshes/collada/simple/simple_asm0001_collada_23_prt.dae" scale="0.03937 0.03937 0.03937" />
+        <mesh filename="package://coman_urdf/meshes/collada/simple/simple_asm0001_collada_23_prt.stl" scale="0.03937 0.03937 0.03937" />
       </geometry>
     </collision>
@@ -378,5 +378,5 @@
       <origin xyz="-0.005305 0.1558 -0.79952053" rpy="0 0 -3.14159265359"/>
       <geometry name="RShy_collision">
-        <mesh filename="package://coman_urdf/meshes/collada/simple/simple_asm0001_collada_22_prt.dae" scale="0.03937 0.03937 0.03937" />
+        <mesh filename="package://coman_urdf/meshes/collada/simple/simple_asm0001_collada_22_prt.stl" scale="0.03937 0.03937 0.03937" />
       </geometry>
     </collision>
@@ -398,5 +398,5 @@
       <origin xyz="-0.005305 -0.0825 -0.844329" rpy="0 0 -3.14159265359"/>
       <geometry name="LShp_collision">
-        <mesh filename="package://coman_urdf/meshes/collada/simple/simple_asm0001_collada_14_prt.dae" scale="0.03937 0.03937 0.03937" />
+        <mesh filename="package://coman_urdf/meshes/collada/simple/simple_asm0001_collada_14_prt.stl" scale="0.03937 0.03937 0.03937" />
       </geometry>
     </collision>
@@ -417,5 +417,5 @@
       <origin xyz="-0.005305 -0.1558 -0.844329" rpy="0 0 -3.14159265359"/>
       <geometry name="LShr_collision">
-        <mesh filename="package://coman_urdf/meshes/collada/simple/simple_asm0001_collada_13_prt.dae" scale="0.03937 0.03937 0.03937" />
+        <mesh filename="package://coman_urdf/meshes/collada/simple/simple_asm0001_collada_13_prt.stl" scale="0.03937 0.03937 0.03937" />
       </geometry>
     </collision>
@@ -436,5 +436,5 @@
       <origin xyz="-0.005305 -0.1558 -0.79952053" rpy="0 0 -3.14159265359"/>
       <geometry name="LShy_collision">
-        <mesh filename="package://coman_urdf/meshes/collada/simple/simple_asm0001_collada_12_prt.dae" scale="0.03937 0.03937 0.03937" />
+        <mesh filename="package://coman_urdf/meshes/collada/simple/simple_asm0001_collada_12_prt.stl" scale="0.03937 0.03937 0.03937" />
       </geometry>
     </collision>

File: coman_urdf/urdf/feet/round_feet_13/accurate_FT_round_foot_L_13.urdf.xacro (robot description, xacro)
@@ -16,5 +16,5 @@
         <origin xyz="0.0 -0.0726 -0.0282" rpy="0 0 -3.14159265359"/>
         <geometry name="LFoot_collision">
-          <mesh filename="package://coman_urdf/meshes/collada/simple/simple_asm0001_collada_01_prt.dae" scale="0.03937 0.03937 0.03937" />
+          <mesh filename="package://coman_urdf/meshes/collada/simple/simple_asm0001_collada_01_prt.stl" scale="0.03937 0.03937 0.03937" />
         </geometry>
       </collision>

File: coman_urdf/urdf/feet/round_feet_13/accurate_FT_round_foot_R_13.urdf.xacro (robot description, xacro)
@@ -16,5 +16,5 @@
         <origin xyz="0.0 0.0726 -0.0282" rpy="0 0 -3.14159265359"/>
         <geometry name="RFoot_collision">
-          <mesh filename="package://coman_urdf/meshes/collada/simple/simple_asm0001_collada_15_prt.dae" scale="0.03937 0.03937 0.03937" />
+          <mesh filename="package://coman_urdf/meshes/collada/simple/simple_asm0001_collada_15_prt.stl" scale="0.03937 0.03937 0.03937" />
         </geometry>
       </collision>

File: coman_urdf/urdf/feet/round_feet_13/round_foot_L_13.urdf.xacro (robot description, xacro)
@@ -16,5 +16,5 @@
         <origin xyz="0.0 -0.0726 -0.0932" rpy="0 0 -3.14159265359"/>
         <geometry name="LFoot_collision">
-          <mesh filename="package://coman_urdf/meshes/collada/simple/simple_asm0001_collada_01_prt.dae" scale="0.03937 0.03937 0.03937" />
+          <mesh filename="package://coman_urdf/meshes/collada/simple/simple_asm0001_collada_01_prt.stl" scale="0.03937 0.03937 0.03937" />
         </geometry>
       </collision>

File: coman_urdf/urdf/feet/round_feet_13/round_foot_R_13.urdf.xacro (robot description, xacro)
@@ -16,5 +16,5 @@
         <origin xyz="0.0 0.0726 -0.0932" rpy="0 0 -3.14159265359"/>
         <geometry name="RFoot_collision">
-          <mesh filename="package://coman_urdf/meshes/collada/simple/simple_asm0001_collada_15_prt.dae" scale="0.03937 0.03937 0.03937" />
+          <mesh filename="package://coman_urdf/meshes/collada/simple/simple_asm0001_collada_15_prt.stl" scale="0.03937 0.03937 0.03937" />
         </geometry>
       </collision>

File: coman_urdf/urdf/forearms/7DOF_forearms_DRC_14/7DOF_forearms_DRC_14.urdf.xacro (robot description, xacro)
@@ -24,5 +24,5 @@
           <origin xyz="0 0 0" rpy="-1.570796326795 1.570796326795 0"/>
           <geometry name="LElb_collision">
-            <mesh filename="package://coman_urdf/meshes/collada/simple/forearms/elbow.dae" scale="1.0 1.0 1.0" />
+            <mesh filename="package://coman_urdf/meshes/collada/simple/forearms/elbow.stl" scale="1.0 1.0 1.0" />
           </geometry>
         </collision>
@@ -45,5 +45,5 @@
           <origin xyz="0 0 ${0.015 + Wrj1_to_FT}" rpy="0 3.14159265359 1.570796326795"/>
           <geometry name="LForearm_collision">
-            <mesh filename="package://coman_urdf/meshes/collada/simple/forearms/forearm.dae" scale="1.0 1.0 1.0" />
+            <mesh filename="package://coman_urdf/meshes/collada/simple/forearms/forearm.stl" scale="1.0 1.0 1.0" />
           </geometry>
         </collision>
@@ -66,5 +66,5 @@
           <origin xyz="0.025 0 0" rpy="0 1.570796326795 3.14159265359"/>
           <geometry name="LWrMot2_collision">
-            <mesh filename="package://coman_urdf/meshes/collada/simple/forearms/simple_fa_asm_3_right_sw0001.dae" scale="0.001 0.001 0.001" />
+            <mesh filename="package://coman_urdf/meshes/collada/simple/forearms/simple_fa_asm_3_right_sw0001.stl" scale="0.001 0.001 0.001" />
           </geometry>
         </collision>
@@ -87,5 +87,5 @@
           <origin xyz="0.025 -0.012 -0.02" rpy="0 3.14159265359 1.570796326795"/>
           <geometry name="LWrMot3_collision">
-            <mesh filename="package://coman_urdf/meshes/collada/simple/forearms/simple_fa_hand_interface_rig_sw0001.dae" scale="0.001 0.001 0.001" />
+            <mesh filename="package://coman_urdf/meshes/collada/simple/forearms/simple_fa_hand_interface_rig_sw0001.stl" scale="0.001 0.001 0.001" />
           </geometry>
         </collision>
@@ -107,5 +107,5 @@
           <origin xyz="0 0 0" rpy="-1.570796326795 1.570796326795 0"/>
           <geometry name="RElb_collision">
-            <mesh filename="package://coman_urdf/meshes/collada/simple/forearms/elbow.dae" scale="1.0 1.0 1.0" />
+            <mesh filename="package://coman_urdf/meshes/collada/simple/forearms/elbow.stl" scale="1.0 1.0 1.0" />
           </geometry>
         </collision>
@@ -128,5 +128,5 @@
           <origin xyz="0 0 ${0.015 + Wrj1_to_FT}" rpy="0 3.14159265359 1.570796326795"/>
           <geometry name="RForearm_collision">
-            <mesh filename="package://coman_urdf/meshes/collada/simple/forearms/forearm.dae" scale="1.0 1.0 1.0" />
+            <mesh filename="package://coman_urdf/meshes/collada/simple/forearms/forearm.stl" scale="1.0 1.0 1.0" />
           </geometry>
         </collision>
@@ -149,5 +149,5 @@
           <origin xyz="0.025 0 0" rpy="0 1.570796326795 3.14159265359"/>
           <geometry name="RWrMot2_collision">
-            <mesh filename="package://coman_urdf/meshes/collada/simple/forearms/simple_fa_asm_3_right_sw0001.dae" scale="0.001 0.001 0.001" />
+            <mesh filename="package://coman_urdf/meshes/collada/simple/forearms/simple_fa_asm_3_right_sw0001.stl" scale="0.001 0.001 0.001" />
           </geometry>
         </collision>
@@ -170,5 +170,5 @@
           <origin xyz="0.025 -0.012 -0.02" rpy="0 3.14159265359 1.570796326795"/>
           <geometry name="RWrMot3_collision">
-            <mesh filename="package://coman_urdf/meshes/collada/simple/forearms/simple_fa_hand_interface_rig_sw0001.dae" scale="0.001 0.001 0.001" />
+            <mesh filename="package://coman_urdf/meshes/collada/simple/forearms/simple_fa_hand_interface_rig_sw0001.stl" scale="0.001 0.001 0.001" />
           </geometry>
         </collision>

File: coman_urdf/urdf/forearms/no_forearms/no_forearms.urdf.xacro (robot description, xacro)
@@ -18,5 +18,5 @@
         <origin xyz="-0.020305 -0.1558 -0.664329" rpy="0 0 -3.14159265359"/>
         <geometry name="LElb_collision">
-          <mesh filename="package://coman_urdf/meshes/collada/simple/simple_asm0001_collada_11_prt.dae" scale="0.03937 0.03937 0.03937" />
+          <mesh filename="package://coman_urdf/meshes/collada/simple/simple_asm0001_collada_11_prt.stl" scale="0.03937 0.03937 0.03937" />
         </geometry>
       </collision>
@@ -45,5 +45,5 @@
       <origin xyz="-0.020305 -0.1558 -0.664329" rpy="0 0 -3.14159265359"/>
       <geometry name="RElb_collision">
-        <mesh filename="package://coman_urdf/meshes/collada/simple/simple_asm0001_collada_11_prt.dae" scale="0.03937 0.03937 0.03937" />
+        <mesh filename="package://coman_urdf/meshes/collada/simple/simple_asm0001_collada_11_prt.stl" scale="0.03937 0.03937 0.03937" />
       </geometry>
     </collision>

File: coman_urdf/urdf/soft_hand.urdf.xacro (robot description, xacro)
@@ -17,5 +17,5 @@
       <origin xyz="0 0.01 -0.04" rpy="0 0 3.14159265359"/>
       <geometry name="RSoftHand_collision">
-        <mesh filename="package://coman_urdf/meshes/collada/simple/forearms/R_soft_hand_open.dae" scale="1E-3 1E-3 1E-3" />
+        <mesh filename="package://coman_urdf/meshes/collada/simple/forearms/R_soft_hand_open.stl" scale="1E-3 1E-3 1E-3" />
       </geometry>
    </collision>
@@ -36,5 +36,5 @@
      <origin xyz="0.007 -0.012 -0.04" rpy="0 0 ${3.14159265359/2}"/>
       <geometry name="LSoftHand_collision">
-        <mesh filename="package://coman_urdf/meshes/collada/simple/forearms/L_soft_hand_open.dae" scale="1E-3 1E-3 1E-3" />
+        <mesh filename="package://coman_urdf/meshes/collada/simple/forearms/L_soft_hand_open.stl" scale="1E-3 1E-3 1E-3" />
       </geometry>
    </collision>
