Commit message: File to add actuated soft hand to coman

File: coman_urdf/urdf/coman.urdf.xacro (robot description, xacro)
@@ -106,8 +106,8 @@
     </xacro:if>
     <xacro:unless value="${GAZEBO_COMAN_USES_SOFTHANDS_DRC_sw1_14}">
-      <joint name="r_handj" type="revolute">
+      <joint name="r_handj" type="fixed">
         <parent link="RWrMot3"/>
         <child link="RSoftHand"/>
-        <origin xyz="0 0 -0.04" rpy="0 0 0"/>
+        <origin xyz="0 0 -0.04" rpy="-3.1415 0 0"/>
         <axis xyz="1 0 0" />
         <limit velocity="4.0" effort="5" lower="0.0" upper="1.57075" />

File: coman_urdf/urdf/coman_hands.urdf (robot description, URDF)
Before this commit: robot COMAN, 45 links, 44 joints
Links:
- added link Rhand_index_distal_link; visual mesh filename=package://complete_soft_hand/meshes/phalanx_distal_out_no_a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 scale=.001 .001 .001
- added link Rhand_index_fake_link2
- added link Rhand_index_fake_link3
- added link Rhand_index_inner_link  
- added link Rhand_index_knuckle_link; visual mesh filename=package://complete_soft_hand/meshes/phalanx_prossimal_injec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 scale=.001 .001 .001
- added link Rhand_index_middle_link; visual mesh filename=package://complete_soft_hand/meshes/phalanx_short_injection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 scale=.001 .001 .001
- added link Rhand_index_proximal_link; visual mesh filename=package://complete_soft_hand/meshes/phalanx_short_injection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 scale=.001 .001 .001
- added link Rhand_little_distal_link; visual mesh filename=package://complete_soft_hand/meshes/phalanx_distal_out_no_a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 scale=.001 .001 .001
- added link Rhand_little_fake_link2
- added link Rhand_little_fake_link3
- added link Rhand_little_inner_link  
- added link Rhand_little_knuckle_link; visual mesh filename=package://complete_soft_hand/meshes/phalanx_prossimal_injec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 scale=.001 .001 .001
- added link Rhand_little_middle_link; visual mesh filename=package://complete_soft_hand/meshes/phalanx_short_injection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 scale=.001 .001 .001
- added link Rhand_little_proximal_link; visual mesh filename=package://complete_soft_hand/meshes/phalanx_short_injection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 scale=.001 .001 .001
- added link Rhand_middle_distal_link; visual mesh filename=package://complete_soft_hand/meshes/phalanx_distal_out_no_a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 scale=.001 .001 .001
- added link Rhand_middle_fake_link2
- added link Rhand_middle_fake_link3
- added link Rhand_middle_inner_link  
- added link Rhand_middle_knuckle_link; visual mesh filename=package://complete_soft_hand/meshes/phalanx_prossimal_injec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 scale=.001 .001 .001
- added link Rhand_middle_middle_link; visual mesh filename=package://complete_soft_hand/meshes/phalanx_short_injection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 scale=.001 .001 .001
- added link Rhand_middle_proximal_link; visual mesh filename=package://complete_soft_hand/meshes/phalanx_short_injection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 scale=.001 .001 .001
- added link Rhand_palm_link; visual mesh filename=package://complete_soft_hand/meshes/palm_hand2.stl scale=.001 .001 .001
- added link Rhand_ring_distal_link; visual mesh filename=package://complete_soft_hand/meshes/phalanx_distal_out_no_a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 scale=.001 .001 .001
- added link Rhand_ring_fake_link2
- added link Rhand_ring_fake_link3
- added link Rhand_ring_inner_link  
- added link Rhand_ring_knuckle_link; visual mesh filename=package://complete_soft_hand/meshes/phalanx_prossimal_injec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 scale=.001 .001 .001
- added link Rhand_ring_middle_link; visual mesh filename=package://complete_soft_hand/meshes/phalanx_short_injection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 scale=.001 .001 .001
- added link Rhand_ring_proximal_link; visual mesh filename=package://complete_soft_hand/meshes/phalanx_short_injection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 scale=.001 .001 .001
- added link Rhand_thumb_distal_link; visual mesh filename=package://complete_soft_hand/meshes/phalanx_distal_out_no_a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 scale=.001 .001 .001
- added link Rhand_thumb_fake_link2
- added link Rhand_thumb_fake_link3
- added link Rhand_thumb_inner_link  
- added link Rhand_thumb_knuckle_link; visual mesh filename=package://complete_soft_hand/meshes/phalanx_thumb_injection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 scale=.001 .001 .001
- added link Rhand_thumb_middle_link; visual mesh filename=package://complete_soft_hand/meshes/phalanx_short_injection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 scale=.001 .001 .001
- added link Rhand_thumb_proximal_link; visual mesh filename=package://complete_soft_hand/meshes/phalanx_short_injection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 scale=.001 .001 .001
- link RSoftHand: mass 0.3 -> 0.001; geometry collision box size=0.001 0.001 0.001; visual box size=0.001 0.001 0.001
Joints:
- added joint Rhand_index_abd_joint: type revolute, parent Rhand_palm_link, child Rhand_index_knuckle_link, origin xyz=-0.0285 0.0943918 0.00205 rpy=3.14159265359 0 -1.2217304764, axis 0 0 1, limit lower=-0.523598775598 upper=0.785398163397 effort=100 velocity=100
- added joint Rhand_index_inner_joint: type revolute, parent Rhand_index_inner_link  , child Rhand_index_proximal_link, origin xyz=-0.013 0 0 rpy=0 0 0, axis 0 1 0, limit lower=0.0 upper=0.785398163397 effort=100 velocity=100, mimic joint=Rhand_index_inner_joint  multiplier=1
- added joint Rhand_index_inner_joint : type revolute, parent Rhand_index_knuckle_link, child Rhand_index_inner_link  , origin xyz=-0.009 0 0 rpy=0 0 0, axis 0 1 0, limit lower=0.0 upper=0.785398163397 effort=100 velocity=100
- added joint Rhand_index_middle_joint: type revolute, parent Rhand_index_fake_link2, child Rhand_index_middle_link, origin xyz=-0.013 0 0 rpy=0 0 0, axis 0 1 0, limit lower=0.0 upper=0.785398163397 effort=100 velocity=100, mimic joint=Rhand_index_middle_joint   multiplier=1
- added joint Rhand_index_middle_joint  : type revolute, parent Rhand_index_proximal_link, child Rhand_index_fake_link2, origin xyz=-0.009 0 0 rpy=0 0 0, axis 0 1 0, limit lower=0.0 upper=0.785398163397 effort=100 velocity=100
- added joint Rhand_index_outer_joint: type revolute, parent Rhand_index_fake_link3, child Rhand_index_distal_link, origin xyz=-0.013 0 0 rpy=0 0 0, axis 0 1 0, limit lower=0.0 upper=0.785398163397 effort=100 velocity=100, mimic joint=Rhand_index_outer_joint  multiplier=1
- added joint Rhand_index_outer_joint : type revolute, parent Rhand_index_middle_link, child Rhand_index_fake_link3, origin xyz=-0.009 0 0 rpy=0 0 0, axis 0 1 0, limit lower=0.0 upper=0.785398163397 effort=100 velocity=100
- added joint Rhand_little_abd_joint: type revolute, parent Rhand_palm_link, child Rhand_little_knuckle_link, origin xyz=0.030 0.0808918 0.00205 rpy=3.14159265359 0 -1.91986217719, axis 0 0 1, limit lower=-0.523598775598 upper=0.785398163397 effort=100 velocity=100
- added joint Rhand_little_inner_joint: type revolute, parent Rhand_little_inner_link  , child Rhand_little_proximal_link, origin xyz=-0.013 0 0 rpy=0 0 0, axis 0 1 0, limit lower=0.0 upper=0.785398163397 effort=100 velocity=100, mimic joint=Rhand_little_inner_joint  multiplier=1
- added joint Rhand_little_inner_joint : type revolute, parent Rhand_little_knuckle_link, child Rhand_little_inner_link  , origin xyz=-0.009 0 0 rpy=0 0 0, axis 0 1 0, limit lower=0.0 upper=0.785398163397 effort=100 velocity=100
- added joint Rhand_little_middle_joint: type revolute, parent Rhand_little_fake_link2, child Rhand_little_middle_link, origin xyz=-0.013 0 0 rpy=0 0 0, axis 0 1 0, limit lower=0.0 upper=0.785398163397 effort=100 velocity=100, mimic joint=Rhand_little_middle_joint   multiplier=1
- added joint Rhand_little_middle_joint  : type revolute, parent Rhand_little_proximal_link, child Rhand_little_fake_link2, origin xyz=-0.009 0 0 rpy=0 0 0, axis 0 1 0, limit lower=0.0 upper=0.785398163397 effort=100 velocity=100
- added joint Rhand_little_outer_joint: type revolute, parent Rhand_little_fake_link3, child Rhand_little_distal_link, origin xyz=-0.013 0 0 rpy=0 0 0, axis 0 1 0, limit lower=0.0 upper=0.785398163397 effort=100 velocity=100, mimic joint=Rhand_little_outer_joint  multiplier=1
- added joint Rhand_little_outer_joint : type revolute, parent Rhand_little_middle_link, child Rhand_little_fake_link3, origin xyz=-0.009 0 0 rpy=0 0 0, axis 0 1 0, limit lower=0.0 upper=0.785398163397 effort=100 velocity=100
- added joint Rhand_middle_abd_joint: type revolute, parent Rhand_palm_link, child Rhand_middle_knuckle_link, origin xyz=-0.009 0.107892 0.00205 rpy=3.14159265359 0 -1.57079632679, axis 0 0 1, limit lower=-0.523598775598 upper=0.785398163397 effort=100 velocity=100
- added joint Rhand_middle_inner_joint: type revolute, parent Rhand_middle_inner_link  , child Rhand_middle_proximal_link, origin xyz=-0.013 0 0 rpy=0 0 0, axis 0 1 0, limit lower=0.0 upper=0.785398163397 effort=100 velocity=100, mimic joint=Rhand_middle_inner_joint  multiplier=1
- added joint Rhand_middle_inner_joint : type revolute, parent Rhand_middle_knuckle_link, child Rhand_middle_inner_link  , origin xyz=-0.009 0 0 rpy=0 0 0, axis 0 1 0, limit lower=0.0 upper=0.785398163397 effort=100 velocity=100
- added joint Rhand_middle_middle_joint: type revolute, parent Rhand_middle_fake_link2, child Rhand_middle_middle_link, origin xyz=-0.013 0 0 rpy=0 0 0, axis 0 1 0, limit lower=0.0 upper=0.785398163397 effort=100 velocity=100, mimic joint=Rhand_middle_middle_joint   multiplier=1
- added joint Rhand_middle_middle_joint  : type revolute, parent Rhand_middle_proximal_link, child Rhand_middle_fake_link2, origin xyz=-0.009 0 0 rpy=0 0 0, axis 0 1 0, limit lower=0.0 upper=0.785398163397 effort=100 velocity=100
- added joint Rhand_middle_outer_joint: type revolute, parent Rhand_middle_fake_link3, child Rhand_middle_distal_link, origin xyz=-0.013 0 0 rpy=0 0 0, axis 0 1 0, limit lower=0.0 upper=0.785398163397 effort=100 velocity=100, mimic joint=Rhand_middle_outer_joint  multiplier=1
- added joint Rhand_middle_outer_joint : type revolute, parent Rhand_middle_middle_link, child Rhand_middle_fake_link3, origin xyz=-0.009 0 0 rpy=0 0 0, axis 0 1 0, limit lower=0.0 upper=0.785398163397 effort=100 velocity=100
- added joint Rhand_palm_joint: type fixed, parent RSoftHand, child Rhand_palm_link, origin xyz=0 0 0 rpy=0 0 0
- added joint Rhand_ring_abd_joint: type revolute, parent Rhand_palm_link, child Rhand_ring_knuckle_link, origin xyz=0.0105 0.0943918 0.00205 rpy=3.14159265359 0 -1.74532925199, axis 0 0 1, limit lower=-0.523598775598 upper=0.785398163397 effort=100 velocity=100
- added joint Rhand_ring_inner_joint: type revolute, parent Rhand_ring_inner_link  , child Rhand_ring_proximal_link, origin xyz=-0.013 0 0 rpy=0 0 0, axis 0 1 0, limit lower=0.0 upper=0.785398163397 effort=100 velocity=100, mimic joint=Rhand_ring_inner_joint  multiplier=1
- added joint Rhand_ring_inner_joint : type revolute, parent Rhand_ring_knuckle_link, child Rhand_ring_inner_link  , origin xyz=-0.009 0 0 rpy=0 0 0, axis 0 1 0, limit lower=0.0 upper=0.785398163397 effort=100 velocity=100
- added joint Rhand_ring_middle_joint: type revolute, parent Rhand_ring_fake_link2, child Rhand_ring_middle_link, origin xyz=-0.013 0 0 rpy=0 0 0, axis 0 1 0, limit lower=0.0 upper=0.785398163397 effort=100 velocity=100, mimic joint=Rhand_ring_middle_joint   multiplier=1
- added joint Rhand_ring_middle_joint  : type revolute, parent Rhand_ring_proximal_link, child Rhand_ring_fake_link2, origin xyz=-0.009 0 0 rpy=0 0 0, axis 0 1 0, limit lower=0.0 upper=0.785398163397 effort=100 velocity=100
- added joint Rhand_ring_outer_joint: type revolute, parent Rhand_ring_fake_link3, child Rhand_ring_distal_link, origin xyz=-0.013 0 0 rpy=0 0 0, axis 0 1 0, limit lower=0.0 upper=0.785398163397 effort=100 velocity=100, mimic joint=Rhand_ring_outer_joint  multiplier=1
- added joint Rhand_ring_outer_joint : type revolute, parent Rhand_ring_middle_link, child Rhand_ring_fake_link3, origin xyz=-0.009 0 0 rpy=0 0 0, axis 0 1 0, limit lower=0.0 upper=0.785398163397 effort=100 velocity=100
- added joint Rhand_thumb_abd_joint: type revolute, parent Rhand_palm_link, child Rhand_thumb_knuckle_link, origin xyz=-0.0418769 0.0538740 -0.00691972  rpy=0 0 -0.43633181, axis 0 1 0, limit lower=-1.57079632679 upper=0.0 effort=100 velocity=100
- added joint Rhand_thumb_inner_joint: type revolute, parent Rhand_thumb_inner_link  , child Rhand_thumb_proximal_link, origin xyz=-0.013 0 0 rpy=0 0 0, axis 0 1 0, limit lower=0.0 upper=0.785398163397 effort=100 velocity=100, mimic joint=Rhand_thumb_inner_joint  multiplier=1
- added joint Rhand_thumb_inner_joint : type revolute, parent Rhand_thumb_knuckle_link, child Rhand_thumb_inner_link  , origin xyz=-0.0225 0 -0.0033 rpy=-1.9974238811 0 0, axis 0 1 0, limit lower=0.0 upper=0.785398163397 effort=100 velocity=100
- added joint Rhand_thumb_middle_joint: type revolute, parent Rhand_thumb_fake_link2, child Rhand_thumb_middle_link, origin xyz=-0.013 0 0 rpy=0 0 0, axis 0 1 0, limit lower=0.0 upper=0.785398163397 effort=100 velocity=100, mimic joint=Rhand_thumb_middle_joint   multiplier=1
- added joint Rhand_thumb_middle_joint  : type revolute, parent Rhand_thumb_proximal_link, child Rhand_thumb_fake_link2, origin xyz=-0.009 0 0 rpy=0 0 0, axis 0 1 0, limit lower=0.0 upper=0.785398163397 effort=100 velocity=100
- added joint Rhand_thumb_outer_joint: type revolute, parent Rhand_thumb_fake_link3, child Rhand_thumb_distal_link, origin xyz=-0.013 0 0 rpy=0 0 0, axis 0 1 0, limit lower=0.0 upper=0.785398163397 effort=100 velocity=100, mimic joint=Rhand_thumb_outer_joint  multiplier=1
- added joint Rhand_thumb_outer_joint : type revolute, parent Rhand_thumb_middle_link, child Rhand_thumb_fake_link3, origin xyz=-0.009 0 0.0 rpy=0 0 0, axis 0 1 0, limit lower=0.0 upper=0.785398163397 effort=100 velocity=100
- joint r_handj: origin xyz=0 0 -0.04 rpy=0 0 0 -> xyz=0 0 -0.04 rpy=-3.1415 0 0; type revolute -> fixed

File: coman_urdf/urdf/soft_hand.urdf.xacro (robot description, xacro)
@@ -46,14 +46,14 @@
     <inertial>
       <origin xyz="0 0 0" rpy="0 0 0"/>
-      <mass value="0.3"/>
-      <inertia ixx="0.001"  ixy="0"  ixz="0" iyy="0.001" iyz="0" izz="0.001" />
+      <mass value="0.001"/>
+      <inertia ixx="0.0001"  ixy="0"  ixz="0" iyy="0.0001" iyz="0" izz="0.0001" />
     </inertial>
     <visual>
      <origin xyz="0 0 0" rpy="0 0 0" />
      <geometry>
-        <box size="0.07 0.07 0.07" />
+        <box size="0.001 0.001 0.001" />
      </geometry>
      <material name="Cyan">
-       <color rgba="0 1.0 1.0 1.0"/>
+       <color rgba="0 0.0 0.0 0.0"/>
      </material>
    </visual>
@@ -61,5 +61,5 @@
      <origin xyz="0 0 0" rpy="0 0 0"/>
      <geometry>
-       <box size="0.07 0.07 0.07" />
+       <box size="0.001 0.001 0.001" />
      </geometry>
    </collision>
@@ -87,4 +87,8 @@
    </collision>
   </link>
+    <xacro:include filename="$(find complete_soft_hand)/model/complete_soft_hand.urdf.xacro"/>
+  <xacro:complete_soft_hand parent="RSoftHand" name="Rhand">
+    <origin xyz="0 0 0" rpy="0 0 0"/>
+  </xacro:complete_soft_hand>
 </xacro:unless>
 </robot>

Commit message: urdf based camera transform

File: coman_urdf/urdf/coman.urdf.xacro (robot description, xacro)
@@ -109,5 +109,5 @@
             <updateRate>10.0</updateRate>
             <cameraName>camera</cameraName>
-            <frameName>camera_link</frameName>
+            <frameName>gaze</frameName>
             <imageTopicName>rgb/image_raw</imageTopicName>
             <depthImageTopicName>depth/image_raw</depthImageTopicName>

File: coman_urdf/urdf/coman_base.urdf.xacro (robot description, xacro)
@@ -499,5 +499,5 @@
     		<parent link="Xtion_cam_body"/>
     		<child link="gaze"/>
-    		<origin xyz="0.015 0 0.022" rpy="0 0 0" />
+    		<origin xyz="0.015 0 0.022" rpy="-1.57075 0 -1.57075" />
   	</joint>
 </xacro:if>

Commit message: Added gaze_sim link specifically for simulation

File: coman_urdf/urdf/coman.urdf.xacro (robot description, xacro)
@@ -109,5 +109,5 @@
             <updateRate>10.0</updateRate>
             <cameraName>camera</cameraName>
-            <frameName>gaze</frameName>
+            <frameName>camera_link_sim</frameName>
             <imageTopicName>rgb/image_raw</imageTopicName>
             <depthImageTopicName>depth/image_raw</depthImageTopicName>
@@ -139,4 +139,5 @@
 </xacro:if>
 <link name="gaze"/>
+<link name="gaze_sim"/>
 <!-- ************ COMAN BASE ************** -->
 <xacro:include filename="$(find coman_urdf)/urdf/coman_base.urdf.xacro"/>

File: coman_urdf/urdf/coman_base.urdf.xacro (robot description, xacro)
@@ -499,4 +499,9 @@
     		<parent link="Xtion_cam_body"/>
     		<child link="gaze"/>
+    		<origin xyz="0.015 0 0.022" rpy="0 0 0" />
+  	</joint>
+ 	<joint name="gaze_joint_sim" type="fixed">
+    		<parent link="Xtion_cam_body"/>
+    		<child link="gaze_sim"/>
     		<origin xyz="0.015 0 0.022" rpy="-1.57075 0 -1.57075" />
   	</joint>

Commit message: Removed useless things and camera_link frame from urdf...
...it should be published outside depending on WALKMAN_PROFILE

File: coman_urdf/urdf/coman.urdf.xacro (robot description, xacro)
@@ -71,20 +71,7 @@
     </collision>
   </link>
-    <gazebo reference="Xtion_cam_body">
-        <sensor name="camera" type="depth">
-          <update_rate>20</update_rate>
-          <camera name="__default__">
-            <horizontal_fov>1.0472</horizontal_fov>
-            <image>
-              <width>640</width>
-              <height>480</height>
-              <format>R8G8B8</format>
-            </image>
-            <clip>
-              <near>0.05</near>
-              <far>3</far>
-            </clip>
-          </camera>
-        </sensor>
+  <link name="gaze"/>
+  <!--link name="camera_link"/-->
+    <gazebo reference="gaze">
         <sensor name="openni_camera_camera" type="depth">
           <always_on>1</always_on>
@@ -109,5 +96,5 @@
             <updateRate>10.0</updateRate>
             <cameraName>camera</cameraName>
-            <frameName>camera_link_sim</frameName>
+            <frameName>camera_link</frameName>
             <imageTopicName>rgb/image_raw</imageTopicName>
             <depthImageTopicName>depth/image_raw</depthImageTopicName>
@@ -128,16 +115,6 @@
           </plugin>
         </sensor>
-        <velocity_decay>
-          <linear>0</linear>
-          <angular>0</angular>
-        </velocity_decay>
-        <pose>0.1 0 0.8 0 -0 0</pose>
-        <self_collide>0</self_collide>
-        <kinematic>0</kinematic>
-        <gravity>1</gravity>
     </gazebo>
 </xacro:if>
-<link name="gaze"/>
-<link name="gaze_sim"/>
 <!-- ************ COMAN BASE ************** -->
 <xacro:include filename="$(find coman_urdf)/urdf/coman_base.urdf.xacro"/>

File: coman_urdf/urdf/coman_base.urdf.xacro (robot description, xacro)
@@ -501,9 +501,10 @@
     		<origin xyz="0.015 0 0.022" rpy="0 0 0" />
   	</joint>
- 	<joint name="gaze_joint_sim" type="fixed">
-    		<parent link="Xtion_cam_body"/>
-    		<child link="gaze_sim"/>
-    		<origin xyz="0.015 0 0.022" rpy="-1.57075 0 -1.57075" />
-  	</joint>
+    <!--joint name="camera_link_joint" type="fixed">
+    		<parent link="gaze"/>
+    		<child link="camera_link"/-->
+    		<!--origin xyz="0.004 0.06 0.019" rpy="0.00 0.003 0.0" /--> <!--Real xtion pro live-->
+        <!--origin xyz="0.0 0.0 0.0" rpy="-1.57 0.0 -1.57" /--> <!--Simulated xtion pro live-->
+  	<!--/joint-->
 </xacro:if>
 <xacro:unless value="${GAZEBO_COMAN_USES_XTION}">

Commit message: bug solved: Gaze frame should be defined also when XTION is not used

File: coman_urdf/urdf/coman.urdf.xacro (robot description, xacro)
@@ -32,4 +32,5 @@
 <xacro:include filename="$(find coman_urdf)/urdf/foot_reference_frame.urdf.xacro" />
 <!-- Head -->
+<link name="gaze"/>
 <xacro:if value="${GAZEBO_COMAN_USES_XTION}">
 	<link name ="Xtion_body">
@@ -52,5 +53,5 @@
     </collision>
   </link>
-  <link name ="Xtion_cam_body">
+  <link name="Xtion_cam_body">
     <inertial>
       <origin xyz="0.0 0.0 0.0225" rpy="0 0 0"/>
@@ -71,6 +72,4 @@
     </collision>
   </link>
-  <link name="gaze"/>
-  <!--link name="camera_link"/-->
     <gazebo reference="gaze">
         <sensor name="openni_camera_camera" type="depth">

Commit message: Added torso link in torso.urdf.xacro

File: coman_urdf/urdf/coman.urdf.xacro (robot description, xacro)
@@ -25,6 +25,4 @@
   <link name="l_toe"/>
   <link name="r_toe"/>
-<!-- The coordinate frame called torso is attached to the lowest body of the model which is a parent of l_gripper, r_gripper and gaze. -->
- <link name="torso"/>
 <!-- Reference frames in feet -->
 <xacro:include filename="$(find coman_urdf)/urdf/foot_reference_frame.urdf.xacro" />

File: coman_urdf/urdf/coman_base.urdf.xacro (robot description, xacro)
@@ -395,9 +395,4 @@
     <child link="r_toe"/>
     <origin xyz="0.13 0 0" rpy="0 0 0" />
-  </joint>
-  <joint name="torso_joint" type="fixed">
-    <parent link="DWYTorso"/>
-    <child link="torso"/>
-    <origin xyz="-0.014976503999999998 0 0.15770847" rpy="0 0 0" />
   </joint>
 <xacro:if value="${GAZEBO_COMAN_USES_XTION}">

File: coman_urdf/urdf/parts/torso.urdf.xacro (robot description, xacro)
@@ -12,4 +12,6 @@
 The coordinate frame called base_link is rigidly attached to the robot root body. It is recommended to choose the robot waist as its root body. The base_link can be attached to the root in any arbitrary position or orientation; for every hardware platform there will be a different place on the base that provides an obvious point of reference. Note that REP 103 [1] specifies a preferred orientation for frames. -->
 <link name="base_link"/>
+<!-- The coordinate frame called torso is attached to the lowest body of the model which is a parent of l_gripper, r_gripper and gaze. -->
+ <link name="torso"/>
 <link name="Waist">
     <inertial>
@@ -94,4 +96,9 @@
     <origin xyz="0 0 0" rpy="0 0 0" />
 </joint>
+<joint name="torso_joint" type="fixed">
+    <parent link="DWYTorso"/>
+    <child link="torso"/>
+    <origin xyz="-0.014976503999999998 0 0.15770847" rpy="0 0 0" />
+</joint>
 <joint name="WaistLat" type="revolute">
     <parent link="Waist"/>
