Commit message: Moved fake joints for forearms inside parts/forearms.urdf.xacro

File: coman_urdf/urdf/coman.urdf.xacro (robot description, xacro)
@@ -13,7 +13,4 @@
 <!-- This links are defined in order to be compliant with http://www.ros.org/reps/rep-0120.html#coordinate-frames
 and to define the end effectors of the robot -->
-<!-- position and orientation of the arm regardless of the tool (grasping device for instance) attached to it -->
-  <link name="l_wrist"/>
-  <link name="r_wrist"/>
 <!--  position and orientation of the leg regardless of the support body geometry -->
   <link name="l_ankle"/>
@@ -115,22 +112,17 @@
 <xacro:include filename="$(find coman_urdf)/urdf/coman_base.urdf.xacro"/>
 <!-- ************ FOREARMS ************ -->
+<!-- This links are defined in order to be compliant with http://www.ros.org/reps/rep-0120.html#coordinate-frames
+and to define the end effectors of the robot -->
+<!-- position and orientation of the arm regardless of the tool (grasping device for instance) attached to it -->
+<link name="l_wrist"/>
+<link name="r_wrist"/>
 <xacro:if value="${GAZEBO_COMAN_USES_NO_FOREARMS}">
-      <xacro:include filename="$(find coman_urdf)/urdf/parts/no_forearms.urdf.xacro" />
-  </xacro:if>
-  <xacro:if value="${GAZEBO_COMAN_USES_7DOF_FOREARMS_DRC_14}">
-      <xacro:include filename="$(find coman_urdf)/urdf/parts/7DOF_forearms_DRC_14.urdf.xacro" />
-  </xacro:if>
+    <xacro:include filename="$(find coman_urdf)/urdf/parts/no_forearms.urdf.xacro" />
+</xacro:if>
+<xacro:if value="${GAZEBO_COMAN_USES_7DOF_FOREARMS_DRC_14}">
+    <xacro:include filename="$(find coman_urdf)/urdf/parts/7DOF_forearms_DRC_14.urdf.xacro" />
+</xacro:if>
 <!-- ************ HANDS ************ -->
   <xacro:if value="${GAZEBO_COMAN_USES_7DOF_FOREARMS_DRC_14}">
-   <joint name="l_wrist_joint" type="fixed">
-     <parent link="LWrMot3"/>
-     <child link="l_wrist"/>
-     <origin xyz="0 0 0" rpy="0 0 0" />
-   </joint>
-    <joint name="r_wrist_joint" type="fixed">
-      <parent link="RWrMot3"/>
-      <child link="r_wrist"/>
-      <origin xyz="0 0 0" rpy="0 0 0" />
-    </joint>
     <xacro:include filename="$(find coman_urdf)/urdf/soft_hand.urdf.xacro" />
     <xacro:if value="${GAZEBO_COMAN_USES_SOFTHANDS_DRC_sw1_14}">
@@ -165,16 +157,4 @@
     </xacro:unless>
   </xacro:if>
-<xacro:if value="${GAZEBO_COMAN_USES_NO_FOREARMS}">
-	<joint name="l_wrist_joint" type="fixed">
-	  <parent link="LElb"/>
-	  <child link="l_wrist"/>
-	  <origin xyz="-0.015 0 -0.22" rpy="0 0 0" />
-	</joint>
-        <joint name="r_wrist_joint" type="fixed">
-	  <parent link="RElb"/>
-	  <child link="r_wrist"/>
-	  <origin xyz="-0.015 0 -0.22" rpy="0 0 0" />
-	</joint>
-</xacro:if>
 <!-- IMU -->
   <link name="imu_link">

File: coman_urdf/urdf/parts/7DOF_forearms_DRC_14.urdf.xacro (robot description, xacro)
@@ -162,4 +162,9 @@
     <dynamics friction="0" damping="0.03"/>
   </joint>
+  <joint name="l_wrist_joint" type="fixed">
+     <parent link="LWrMot3"/>
+     <child link="l_wrist"/>
+     <origin xyz="0 0 0" rpy="0 0 0" />
+   </joint>
 <!-- ****************RIGHT FOREARM**************** -->
 <joint name="RForearmPlate" type="revolute">
@@ -187,3 +192,8 @@
     <dynamics friction="0" damping="0.03"/>
   </joint>
+  <joint name="r_wrist_joint" type="fixed">
+      <parent link="RWrMot3"/>
+      <child link="r_wrist"/>
+      <origin xyz="0 0 0" rpy="0 0 0" />
+  </joint>
 </robot>

File: coman_urdf/urdf/parts/no_forearms.urdf.xacro (robot description, xacro)
@@ -49,5 +49,10 @@
         <child link="LForearm"/>
         <origin xyz="-0.015 0.0 -0.05" rpy="0 0 0"/>
-      </joint>
+</joint>
+<joint name="l_wrist_joint" type="fixed">
+	  <parent link="LElb"/>
+	  <child link="l_wrist"/>
+	  <origin xyz="-0.015 0 -0.22" rpy="0 0 0" />
+</joint>
 <!-- ***********RIGHT FOREARM***********-->
 <joint name="RForearmPlate" type="fixed">
@@ -55,4 +60,9 @@
       <child link="RForearm"/>
       <origin xyz="-0.015 0.0 -0.05" rpy="0 0 0"/>
-    </joint>
+</joint>
+<joint name="r_wrist_joint" type="fixed">
+	<parent link="RElb"/>
+	<child link="r_wrist"/>
+	<origin xyz="-0.015 0 -0.22" rpy="0 0 0" />
+</joint>
 </robot>

Commit message: Added sensor folder. Moved imu links and joints in sensors/imu.urdf.xacro

File: coman_urdf/urdf/coman.urdf.xacro (robot description, xacro)
@@ -158,21 +158,4 @@
   </xacro:if>
 <!-- IMU -->
-  <link name="imu_link">
-    <inertial>
-      <mass value="0.01"/>
-      <origin xyz="0 0 0"/>
-      <inertia ixx="1.0E-6" ixy="0" ixz="0" iyy="1.0E-6" iyz="0" izz="1.0E-6"/>
-    </inertial>
-    <visual>
-      <origin rpy="0 0 0" xyz="0 0 0"/>
-      <geometry>
-        <box size="0.01 0.01 0.01"/>
-      </geometry>
-    </visual>
-  </link>
-  <joint name="imu_joint" type="fixed">
-    <parent link="Waist"/>
-    <child link="imu_link"/>
-    <origin xyz="-0.072 -0.0068 0.044" rpy="0 3.14159 0"/>
-  </joint>
+<xacro:include filename="$(find coman_urdf)/urdf/sensors/imu.urdf.xacro"/>
 </robot>

Commit message: Moved all feet logic in legs. Moved fake joints in legs

File: coman_urdf/urdf/coman.urdf.xacro (robot description, xacro)
@@ -10,18 +10,4 @@
 <!-- ************ MODEL CONFIGURATION ************ -->
 <xacro:include filename="$(find coman_urdf)/urdf/coman_config.urdf.xacro" />
-<!-- ******************** FAKE LINKS ******************** -->
-<!-- This links are defined in order to be compliant with http://www.ros.org/reps/rep-0120.html#coordinate-frames
-and to define the end effectors of the robot -->
-<!--  position and orientation of the leg regardless of the support body geometry -->
-  <link name="l_ankle"/>
-  <link name="r_ankle"/>
-<!-- position and orientation of the left leg support body. The (X,Y) plane of this frame must be coplanar with the support body contact surface. It is recommended to choose the origin as the projection of the support body origin on the contact surface. The Z coordinate of this frame should be on the ground level when standing. -->
-  <link name="l_sole"/>
-  <link name="r_sole"/>
-<!--  position and orientation of the leg toe body. The (X,Y) plan of this frame must be coplanar with the toe body contact surface. It is recommended to choose the origin as the projection of the body center on the contact surface. -->
-  <link name="l_toe"/>
-  <link name="r_toe"/>
-<!-- Reference frames in feet -->
-<xacro:include filename="$(find coman_urdf)/urdf/foot_reference_frame.urdf.xacro" />
 <!-- Head -->
 <link name="gaze"/>

File: coman_urdf/urdf/coman_base.urdf.xacro (robot description, xacro)
@@ -12,13 +12,21 @@
 <xacro:include filename="$(find coman_urdf)/urdf/parts/torso.urdf.xacro" />
 <!-- ********************LEGS******************** -->
+<!-- This links are defined in order to be compliant with http://www.ros.org/reps/rep-0120.html#coordinate-frames
+and to define the end effectors of the robot -->
+<!--  position and orientation of the leg regardless of the support body geometry -->
+  <link name="l_ankle"/>
+  <link name="r_ankle"/>
+<!-- position and orientation of the left leg support body. The (X,Y) plane of this frame must be coplanar with the support body contact surface. It is recommended to choose the origin as the projection of the support body origin on the contact surface. The Z coordinate of this frame should be on the ground level when standing. -->
+  <link name="l_sole"/>
+  <link name="r_sole"/>
+<!--  position and orientation of the leg toe body. The (X,Y) plan of this frame must be coplanar with the toe body contact surface. It is recommended to choose the origin as the projection of the body center on the contact surface. -->
+  <link name="l_toe"/>
+  <link name="r_toe"/>
 <xacro:include filename="$(find coman_urdf)/urdf/parts/legs.urdf.xacro" />
-<!-- ********************ARMS******************** -->
-<xacro:include filename="$(find coman_urdf)/urdf/parts/arms.urdf.xacro" />
-<!-- ********************JOINTS******************** -->
-    <joint name="l_ankle_joint" type="fixed">
-      <parent link="LFoot"/>
-      <child link="l_ankle"/>
-      <origin xyz="0 0 0" rpy="0 0 0" />
-    </joint>
+  <joint name="l_ankle_joint" type="fixed">
+     <parent link="LFoot"/>
+     <child link="l_ankle"/>
+     <origin xyz="0 0 0" rpy="0 0 0" />
+  </joint>
   <joint name="r_ankle_joint" type="fixed">
     <parent link="RFoot"/>
@@ -46,4 +54,9 @@
     <origin xyz="0.13 0 0" rpy="0 0 0" />
   </joint>
+<!-- Reference frames in feet -->
+<xacro:include filename="$(find coman_urdf)/urdf/parts/foot_reference_frame.urdf.xacro" />
+<!-- ********************ARMS******************** -->
+<xacro:include filename="$(find coman_urdf)/urdf/parts/arms.urdf.xacro" />
+<!-- ********************JOINTS******************** -->
 <xacro:if value="${GAZEBO_COMAN_USES_XTION}">
         <joint name="Xtion_body_joint" type="fixed">

File: coman_urdf/urdf/parts/legs.urdf.xacro (robot description, xacro)
@@ -103,8 +103,8 @@
 <xacro:unless value="${GAZEBO_COMAN_USES_ACCURATE_FT}">
     <xacro:if value="${GAZEBO_COMAN_USES_ROUND_FEET_13}">
-      <xacro:include filename="$(find coman_urdf)/urdf/feet/round_feet_13/round_foot_R_13.urdf.xacro" />
+      <xacro:include filename="$(find coman_urdf)/urdf/parts/subparts/round_feet_13/round_foot_R_13.urdf.xacro" />
     </xacro:if>
     <xacro:if value="${GAZEBO_COMAN_USES_SIMPLE_FEET_DRC_sw1_14}">
-      <xacro:include filename="$(find coman_urdf)/urdf/feet/simple_feet_DRC_sw1_14/simple_foot_R_DRC_sw1_14.urdf.xacro" />
+      <xacro:include filename="$(find coman_urdf)/urdf/parts/subparts/simple_feet_DRC_sw1_14/simple_foot_R_DRC_sw1_14.urdf.xacro" />
     </xacro:if>
   </xacro:unless>
@@ -118,8 +118,8 @@
     </link>
     <xacro:if value="${GAZEBO_COMAN_USES_ROUND_FEET_13}">
-      <xacro:include filename="$(find coman_urdf)/urdf/feet/round_feet_13/accurate_FT_round_foot_R_13.urdf.xacro" />
+      <xacro:include filename="$(find coman_urdf)/urdf/parts/subparts/round_feet_13/accurate_FT_round_foot_R_13.urdf.xacro" />
     </xacro:if>
     <xacro:if value="${GAZEBO_COMAN_USES_SIMPLE_FEET_DRC_sw1_14}">
-      <xacro:include filename="$(find coman_urdf)/urdf/feet/simple_feet_DRC_sw1_14/accurate_FT_simple_foot_R_DRC_sw1_14.urdf.xacro" />
+      <xacro:include filename="$(find coman_urdf)/urdf/parts/subparts/simple_feet_DRC_sw1_14/accurate_FT_simple_foot_R_DRC_sw1_14.urdf.xacro" />
     </xacro:if>
   </xacro:if>
@@ -222,8 +222,8 @@
   <xacro:unless value="${GAZEBO_COMAN_USES_ACCURATE_FT}">
     <xacro:if value="${GAZEBO_COMAN_USES_ROUND_FEET_13}">
-      <xacro:include filename="$(find coman_urdf)/urdf/feet/round_feet_13/round_foot_L_13.urdf.xacro" />
+      <xacro:include filename="$(find coman_urdf)/urdf/parts/subparts/round_feet_13/round_foot_L_13.urdf.xacro" />
     </xacro:if>
     <xacro:if value="${GAZEBO_COMAN_USES_SIMPLE_FEET_DRC_sw1_14}">
-      <xacro:include filename="$(find coman_urdf)/urdf/feet/simple_feet_DRC_sw1_14/simple_foot_L_DRC_sw1_14.urdf.xacro" />
+      <xacro:include filename="$(find coman_urdf)/urdf/parts/subparts/simple_feet_DRC_sw1_14/simple_foot_L_DRC_sw1_14.urdf.xacro" />
     </xacro:if>
   </xacro:unless>
@@ -237,8 +237,8 @@
     </link>
     <xacro:if value="${GAZEBO_COMAN_USES_ROUND_FEET_13}">
-      <xacro:include filename="$(find coman_urdf)/urdf/feet/round_feet_13/accurate_FT_round_foot_L_13.urdf.xacro" />
+      <xacro:include filename="$(find coman_urdf)/urdf/parts/subparts/round_feet_13/accurate_FT_round_foot_L_13.urdf.xacro" />
     </xacro:if>
     <xacro:if value="${GAZEBO_COMAN_USES_SIMPLE_FEET_DRC_sw1_14}">
-      <xacro:include filename="$(find coman_urdf)/urdf/feet/simple_feet_DRC_sw1_14/accurate_FT_simple_foot_L_DRC_sw1_14.urdf.xacro" />
+      <xacro:include filename="$(find coman_urdf)/urdf/parts/subparts/simple_feet_DRC_sw1_14/accurate_FT_simple_foot_L_DRC_sw1_14.urdf.xacro" />
     </xacro:if>
   </xacro:if>

Commit message: Moved xtion stuffs in sensors/xtion.urdf.xacro

File: coman_urdf/urdf/coman.urdf.xacro (robot description, xacro)
@@ -11,44 +11,10 @@
 <xacro:include filename="$(find coman_urdf)/urdf/coman_config.urdf.xacro" />
 <!-- Head -->
+<!-- This links are defined in order to be compliant with http://www.ros.org/reps/rep-0120.html#coordinate-frames
+and to define the end effectors of the robot.
+The coordinate frame called gaze defines the head position and orientation. The orientation indicates in which direction the head appears to be looking regardless of any sensors (camera for instance). -->
 <link name="gaze"/>
 <xacro:if value="${GAZEBO_COMAN_USES_XTION}">
-	<link name ="Xtion_body">
-    <inertial>
-      <origin xyz="0.047 0.0 0.40" rpy="0 0 0"/>
-      <mass value="0.39"/>
-      <inertia ixx="0.01"  ixy="3.34E-7"  ixz="-2.66E-4" iyy="0.009" iyz="1.97E-6" izz="5.1E-4" />
-    </inertial>
-    <visual>
-      <origin xyz="-0.020281504 0.0 -0.68662053" rpy="0 0 -3.14159265359"/>
-      <geometry name="Xtion_body_visual">
-        <mesh filename="package://coman_urdf/meshes/collada/Xtion/xtion_base.dae" scale="0.03937 0.03937 0.03937" />
-      </geometry>
-    </visual>
-    <collision>
-      <origin xyz="-0.020281504 0.0 -0.68662053" rpy="0 0 -3.14159265359"/>
-      <geometry name="Xtion_body_collision">
-        <mesh filename="package://coman_urdf/meshes/collada/simple/Xtion/xtion_base.stl" scale="0.03937 0.03937 0.03937" />
-      </geometry>
-    </collision>
-  </link>
-  <link name="Xtion_cam_body">
-    <inertial>
-      <origin xyz="0.0 0.0 0.0225" rpy="0 0 0"/>
-      <mass value="0.2"/>
-      <inertia ixx="0.00053"  ixy="0.0"  ixz="0.0" iyy="0.00008" iyz="0.0" izz="0.00053" />
-    </inertial>
-    <visual>
-      <origin xyz="-0.0915 0.0 -1.2778" rpy="0 0 -3.14159265359"/>
-      <geometry name="Xtion_cam_body_visual">
-        <mesh filename="package://coman_urdf/meshes/collada/Xtion/xtion_cam_body.dae" scale="0.001 0.001 0.001" />
-      </geometry>
-    </visual>
-    <collision>
-      <origin xyz="-0.0915 0.0 -1.2778" rpy="0 0 -3.14159265359"/>
-      <geometry name="Xtion_cam_body_collision">
-        <mesh filename="package://coman_urdf/meshes/collada/simple/Xtion/xtion_cam_body.stl" scale="0.001 0.001 0.001" />
-      </geometry>
-    </collision>
-  </link>
+<xacro:include filename="$(find coman_urdf)/urdf/sensors/xtion.urdf.xacro" />
     <gazebo reference="gaze">
         <sensor name="openni_camera_camera" type="depth">
@@ -95,4 +61,11 @@
     </gazebo>
 </xacro:if>
+<xacro:unless value="${GAZEBO_COMAN_USES_XTION}">
+<joint name="gaze_joint" type="fixed">
+	<parent link="torso"/>
+	<child link="gaze"/>
+	<origin xyz="0 0 0.1" rpy="0 0 0" />
+</joint>
+</xacro:unless>
 <!-- ************ COMAN BASE ************** -->
 <xacro:include filename="$(find coman_urdf)/urdf/coman_base.urdf.xacro"/>

File: coman_urdf/urdf/coman_base.urdf.xacro (robot description, xacro)
@@ -58,38 +58,3 @@
 <!-- ********************ARMS******************** -->
 <xacro:include filename="$(find coman_urdf)/urdf/parts/arms.urdf.xacro" />
-<!-- ********************JOINTS******************** -->
-<xacro:if value="${GAZEBO_COMAN_USES_XTION}">
-        <joint name="Xtion_body_joint" type="fixed">
-    		<parent link="DWYTorso"/>
-    		<child link="Xtion_body"/>
-    		<origin xyz="0 0 0" rpy="0 0 0" />
-  	</joint>
-        <joint name="Xtion_cam_body_joint" type="fixed">
-    		<parent link="Xtion_body"/>
-    		<child link="Xtion_cam_body"/>
-		<!-- origin xyz="0.071 0 0.591" rpy="0 1.396 0" / -->
-                <origin xyz="0.071 0 0.591" rpy="0 0 0" />
-		<!--axis xyz="0 1 0" />
-    		<limit velocity="4.0" effort="5" lower="-0.4145" upper="1.57075" />
-    		<dynamics friction="0" damping="3.0"/-->
-  	</joint>
-        <joint name="gaze_joint" type="fixed">
-    		<parent link="Xtion_cam_body"/>
-    		<child link="gaze"/>
-    		<origin xyz="0.015 0 0.022" rpy="0 0 0" />
-  	</joint>
-    <!--joint name="camera_link_joint" type="fixed">
-    		<parent link="gaze"/>
-    		<child link="camera_link"/-->
-    		<!--origin xyz="0.004 0.06 0.019" rpy="0.00 0.003 0.0" /--> <!--Real xtion pro live-->
-        <!--origin xyz="0.0 0.0 0.0" rpy="-1.57 0.0 -1.57" /--> <!--Simulated xtion pro live-->
-  	<!--/joint-->
-</xacro:if>
-<xacro:unless value="${GAZEBO_COMAN_USES_XTION}">
- 	<joint name="gaze_joint" type="fixed">
-    		<parent link="torso"/>
-    		<child link="gaze"/>
-    		<origin xyz="0 0 0.1" rpy="0 0 0" />
-  	</joint>
-</xacro:unless>
 </robot>

Commit message: Moved kinect plugin in gazebo/openni_kinect_gazebo.xacro

File: coman_urdf/urdf/coman.urdf.xacro (robot description, xacro)
@@ -16,55 +16,12 @@
 <link name="gaze"/>
 <xacro:if value="${GAZEBO_COMAN_USES_XTION}">
-<xacro:include filename="$(find coman_urdf)/urdf/sensors/xtion.urdf.xacro" />
-    <gazebo reference="gaze">
-        <sensor name="openni_camera_camera" type="depth">
-          <always_on>1</always_on>
-          <visualize>1</visualize>
-          <camera name="__default__">
-            <horizontal_fov>1.047</horizontal_fov>
-            <image>
-              <width>640</width>
-              <height>480</height>
-              <format>R8G8B8</format>
-            </image>
-            <depth_camera>
-              <output>depths</output>
-            </depth_camera>
-            <clip>
-              <near>0.1</near>
-              <far>100</far>
-            </clip>
-          </camera>
-          <plugin name="camera_controller" filename="libgazebo_ros_openni_kinect.so">
-            <alwaysOn>true</alwaysOn>
-            <updateRate>10.0</updateRate>
-            <cameraName>camera</cameraName>
-            <frameName>camera_link</frameName>
-            <imageTopicName>rgb/image_raw</imageTopicName>
-            <depthImageTopicName>depth/image_raw</depthImageTopicName>
-            <pointCloudTopicName>depth/points</pointCloudTopicName>
-            <cameraInfoTopicName>rgb/camera_info</cameraInfoTopicName>
-            <depthImageCameraInfoTopicName>depth/camera_info</depthImageCameraInfoTopicName>
-            <pointCloudCutoff>0.4</pointCloudCutoff>
-            <hackBaseline>0.07</hackBaseline>
-            <distortionK1>0.0</distortionK1>
-            <distortionK2>0.0</distortionK2>
-            <distortionK3>0.0</distortionK3>
-            <distortionT1>0.0</distortionT1>
-            <distortionT2>0.0</distortionT2>
-            <CxPrime>0.0</CxPrime>
-            <Cx>0.0</Cx>
-            <Cy>0.0</Cy>
-            <focalLength>0.0</focalLength>
-          </plugin>
-        </sensor>
-    </gazebo>
+	<xacro:include filename="$(find coman_urdf)/urdf/sensors/xtion.urdf.xacro" />
 </xacro:if>
 <xacro:unless value="${GAZEBO_COMAN_USES_XTION}">
-<joint name="gaze_joint" type="fixed">
-	<parent link="torso"/>
-	<child link="gaze"/>
-	<origin xyz="0 0 0.1" rpy="0 0 0" />
-</joint>
+	<joint name="gaze_joint" type="fixed">
+		<parent link="torso"/>
+		<child link="gaze"/>
+		<origin xyz="0 0 0.1" rpy="0 0 0" />
+	</joint>
 </xacro:unless>
 <!-- ************ COMAN BASE ************** -->

File: coman_urdf/urdf/coman_robot.urdf.xacro (robot description, xacro)
@@ -9,4 +9,7 @@
   <xacro:include filename="$(find coman_urdf)/urdf/gazebo/microstrain_3dmgx2_imu.gazebo.xacro" />
   <xacro:include filename="$(find coman_urdf)/urdf/gazebo/coman.gazebo.xacro" />
+  <xacro:if value="${GAZEBO_COMAN_USES_XTION}">
+	<xacro:include filename="$(find coman_urdf)/urdf/gazebo/openni_kinect.gazebo.xacro" />
+  </xacro:if>
 <!-- YARP PLUGINS for GAZEBO SIMULATION -->
   <xacro:include filename="$(find coman_urdf)/urdf/gazebo/yarp_control.gazebo.xacro" />

Commit message: Moved hands in parts.

File: coman_urdf/urdf/coman.urdf.xacro (robot description, xacro)
@@ -40,37 +40,7 @@
 </xacro:if>
 <!-- ************ HANDS ************ -->
-  <xacro:if value="${GAZEBO_COMAN_USES_7DOF_FOREARMS_DRC_14}">
-    <xacro:include filename="$(find coman_urdf)/urdf/soft_hand.urdf.xacro" />
-    <xacro:if value="${GAZEBO_COMAN_USES_SOFTHANDS_DRC_sw1_14}">
-      <joint name="r_handj" type="fixed">
-        <parent link="RWrMot3"/>
-        <child link="RSoftHand"/>
-        <origin xyz="0 0 -0.07" rpy="0 0 0"/>
-      </joint>
-      <joint name="l_handj" type="fixed">
-        <parent link="LWrMot3"/>
-        <child link="LSoftHand"/>
-        <origin xyz="0 0 -0.07" rpy="0 0 0"/>
-      </joint>
-    </xacro:if>
-    <xacro:unless value="${GAZEBO_COMAN_USES_SOFTHANDS_DRC_sw1_14}">
-      <joint name="r_handj" type="revolute">
-        <parent link="RWrMot3"/>
-        <child link="RSoftHand"/>
-        <origin xyz="0 0 -0.04" rpy="0 0 0"/>
-        <axis xyz="1 0 0" />
-        <limit velocity="4.0" effort="5" lower="0.0" upper="1.57075" />
-        <dynamics friction="0" damping="3.0"/>
-      </joint>
-      <joint name="l_handj" type="revolute">
-        <parent link="LWrMot3"/>
-        <child link="LSoftHand"/>
-        <origin xyz="0 0 -0.04" rpy="0 0 0"/>
-        <axis xyz="1 0 0" />
-        <limit velocity="4.0" effort="5" lower="-1.57075" upper="0.0" />
-        <dynamics friction="0" damping="3.0"/>
-      </joint>
-    </xacro:unless>
-  </xacro:if>
+<xacro:if value="${GAZEBO_COMAN_USES_7DOF_FOREARMS_DRC_14}">
+    <xacro:include filename="$(find coman_urdf)/urdf/parts/soft_hand.urdf.xacro" />
+</xacro:if>
 <!-- IMU -->
 <xacro:include filename="$(find coman_urdf)/urdf/sensors/imu.urdf.xacro"/>

File: coman_urdf/urdf/parts/soft_hand.urdf.xacro (robot description, xacro)
@@ -2,4 +2,5 @@
 <robot xmlns:xacro="http://ros.org/wiki/xacro" name="SoftHand">
 <xacro:if value="${GAZEBO_COMAN_USES_SOFTHANDS_DRC_sw1_14}">
+<!-- LINKS -->
 <link name="RSoftHand">
     <inertial>
@@ -40,6 +41,18 @@
    </collision>
   </link>
+<!-- JOINTS -->
+  <joint name="r_handj" type="fixed">
+        <parent link="RWrMot3"/>
+        <child link="RSoftHand"/>
+        <origin xyz="0 0 -0.07" rpy="0 0 0"/>
+  </joint>
+  <joint name="l_handj" type="fixed">
+        <parent link="LWrMot3"/>
+        <child link="LSoftHand"/>
+        <origin xyz="0 0 -0.07" rpy="0 0 0"/>
+  </joint>
 </xacro:if>
 <xacro:unless value="${GAZEBO_COMAN_USES_SOFTHANDS_DRC_sw1_14}">
+<!-- LINKS -->
 <!-- ## WRONG NUMBERS FOR... ok lasciamo perde... FIX THEM!! ## -->
   <link name="RSoftHand">
@@ -87,4 +100,21 @@
    </collision>
   </link>
+<!-- JOINTS -->
+<joint name="r_handj" type="revolute">
+        <parent link="RWrMot3"/>
+        <child link="RSoftHand"/>
+        <origin xyz="0 0 -0.04" rpy="0 0 0"/>
+        <axis xyz="1 0 0" />
+        <limit velocity="4.0" effort="5" lower="0.0" upper="1.57075" />
+        <dynamics friction="0" damping="3.0"/>
+</joint>
+<joint name="l_handj" type="revolute">
+        <parent link="LWrMot3"/>
+        <child link="LSoftHand"/>
+        <origin xyz="0 0 -0.04" rpy="0 0 0"/>
+        <axis xyz="1 0 0" />
+        <limit velocity="4.0" effort="5" lower="-1.57075" upper="0.0" />
+        <dynamics friction="0" damping="3.0"/>
+</joint>
 </xacro:unless>
 </robot>
