Commit message: Added material file for urdf and sdf.

File: coman_urdf/urdf/coman.urdf.xacro (robot description, xacro)
@@ -10,4 +10,6 @@
 <!-- ************ MODEL CONFIGURATION ************ -->
 <xacro:include filename="$(find coman_urdf)/urdf/coman_config.urdf.xacro" />
+<!-- ***********  MODEL COLORS *********** -->
+<xacro:include filename="$(find coman_urdf)/urdf/coman_materials.urdf.xacro" />
 <!-- Head -->
 <!-- This links are defined in order to be compliant with http://www.ros.org/reps/rep-0120.html#coordinate-frames

File: coman_urdf/urdf/coman_robot.urdf.xacro (robot description, xacro)
@@ -14,4 +14,5 @@
 <!-- YARP PLUGINS for GAZEBO SIMULATION -->
   <xacro:include filename="$(find coman_urdf)/urdf/gazebo/yarp_control.gazebo.xacro" />
+  <xacro:include filename="$(find coman_urdf)/urdf/gazebo/coman_materials.gazebo.xacro" />
   <origin xyz="0.0 0.0 0.521" rpy="0 0 0" />
 </robot>

File: coman_urdf/urdf/parts/torso.urdf.xacro (robot description, xacro)
@@ -22,6 +22,8 @@
     <visual>
       <origin xyz="0 0 ${base_link_z_translation}" rpy="0 0 ${PI}"/>
+      <material name="dark_grey"/>
       <geometry name="Waist_visual">
-        <mesh filename="package://coman_urdf/meshes/collada/asm0001_collada_07_prt.dae" scale="${SF} ${SF} ${SF}"/>
+        <!--mesh filename="package://coman_urdf/meshes/collada/asm0001_collada_07_prt.dae" scale="${SF} ${SF} ${SF}"/-->
+        <mesh filename="package://coman_urdf/meshes/collada/torso0.stl" scale="${SF} ${SF} ${SF}"/>
       </geometry>
     </visual>

Commit message: Added fixed reference frame in arms for the force torque sensors.

File: coman_urdf/urdf/coman.urdf.xacro (robot description, xacro)
@@ -36,5 +36,17 @@
 <link name="r_wrist"/>
 <xacro:if value="${GAZEBO_COMAN_USES_FOREARMS}">
-    <xacro:include filename="$(find coman_urdf)/urdf/parts/7DOF_forearms_DRC_14.urdf.xacro" />
+    <xacro:include filename="$(find coman_urdf)/urdf/parts/forearms.urdf.xacro" />
+    <link name="l_arm_ft"/>
+    <link name="r_arm_ft"/>
+    <joint name="l_arm_ft_joint" type="fixed">
+      <parent link="LForearm"/>
+      <child link="l_arm_ft"/>
+      <origin xyz="0 0 0" rpy="0 0 0" />
+    </joint>
+    <joint name="r_arm_ft_joint" type="fixed">
+      <parent link="RForearm"/>
+      <child link="r_arm_ft"/>
+      <origin xyz="0 0 0" rpy="0 0 0" />
+    </joint>
 </xacro:if>
 <xacro:unless value="${GAZEBO_COMAN_USES_FOREARMS}">
