Commit message: Added part for arms. Added first three joints of each arm.

File: coman_urdf/urdf/coman_base.urdf.xacro (robot description, xacro)
@@ -249,120 +249,6 @@
     </xacro:if>
   </xacro:if>
-<!-- ********************RIGHT ARM******************** -->
-  <link name ="RShp">
-    <inertial>
-      <origin xyz="0.0099500565 -0.038682024 1.6446924E-4" rpy="0 0 0"/>
-      <mass value="0.56782202"/>
-      <inertia ixx="7.8337456E-4"  ixy="1.9035768E-4"  ixz="-3.0037676E-6" iyy="6.3399921E-4" iyz="4.3840774E-6" izz="0.001008054" />
-    </inertial>
-    <visual>
-      <origin xyz="-0.005305 0.0825 -0.844329" rpy="0 0 -3.14159265359"/>
-      <geometry name="RShp_visual">
-        <mesh filename="package://coman_urdf/meshes/collada/asm0001_collada_24_prt.dae" scale="0.03937 0.03937 0.03937" />
-      </geometry>
-    </visual>
-    <collision>
-      <origin xyz="-0.005305 0.0825 -0.844329" rpy="0 0 -3.14159265359"/>
-      <geometry name="RShp_collision">
-        <mesh filename="package://coman_urdf/meshes/collada/simple/simple_asm0001_collada_24_prt.stl" scale="0.03937 0.03937 0.03937" />
-      </geometry>
-    </collision>
-  </link>
-  <link name ="RShr">
-    <inertial>
-      <origin xyz="-0.0038936743 2.2022151E-6 -0.0048616005" rpy="0 0 0"/>
-      <mass value="0.77683752"/>
-      <inertia ixx="4.5812904E-4"  ixy="-2.4111086E-7"  ixz="9.2521185E-6" iyy="4.3089204E-4" iyz="-4.7216950E-7" izz="3.4174855E-4" />
-    </inertial>
-    <visual>
-      <origin xyz="-0.005305 0.1558 -0.844329" rpy="0 0 -3.14159265359"/>
-      <geometry name="RShr_visual">
-        <mesh filename="package://coman_urdf/meshes/collada/asm0001_collada_23_prt.dae" scale="0.03937 0.03937 0.03937" />
-      </geometry>
-    </visual>
-    <collision>
-      <origin xyz="-0.005305 0.1558 -0.844329" rpy="0 0 -3.14159265359"/>
-      <geometry name="RShr_collision">
-        <mesh filename="package://coman_urdf/meshes/collada/simple/simple_asm0001_collada_23_prt.stl" scale="0.03937 0.03937 0.03937" />
-      </geometry>
-    </collision>
-  </link>
-  <link name ="RShy">
-    <inertial>
-      <origin xyz="0.0022714213 -0.0071091517 -0.057455221" rpy="0 0 0"/>
-      <mass value="1.0462304"/>
-      <inertia ixx="0.0030934574"  ixy="6.6702837E-5"  ixz="3.0222291E-4" iyy="0.0029181573" iyz="-5.2663661E-4" izz="8.0830389E-4" />
-    </inertial>
-    <visual>
-      <origin xyz="-0.005305 0.1558 -0.79952053" rpy="0 0 -3.14159265359"/>
-      <geometry name="RShy_visual">
-        <mesh filename="package://coman_urdf/meshes/collada/asm0001_collada_22_prt.dae" scale="0.03937 0.03937 0.03937" />
-      </geometry>
-    </visual>
-    <collision>
-      <origin xyz="-0.005305 0.1558 -0.79952053" rpy="0 0 -3.14159265359"/>
-      <geometry name="RShy_collision">
-        <mesh filename="package://coman_urdf/meshes/collada/simple/simple_asm0001_collada_22_prt.stl" scale="0.03937 0.03937 0.03937" />
-      </geometry>
-    </collision>
-  </link>
-<!-- ********************LEFT ARM******************** -->
-  <link name ="LShp">
-    <inertial>
-      <origin xyz="0.0099500565 0.038682024 1.6446924E-4" rpy="0 0 0"/>
-      <mass value="0.56782202"/>
-      <inertia ixx="7.8337456E-4"  ixy="-1.9035768E-4"  ixz="-3.0037676E-6" iyy="6.3399921E-4" iyz="-4.3840774E-6" izz="0.001008054" />
-    </inertial>
-    <visual>
-      <origin xyz="-0.005305 -0.0825 -0.844329" rpy="0 0 -3.14159265359"/>
-      <geometry name="LShp_visual">
-        <mesh filename="package://coman_urdf/meshes/collada/asm0001_collada_14_prt.dae" scale="0.03937 0.03937 0.03937" />
-      </geometry>
-    </visual>
-    <collision>
-      <origin xyz="-0.005305 -0.0825 -0.844329" rpy="0 0 -3.14159265359"/>
-      <geometry name="LShp_collision">
-        <mesh filename="package://coman_urdf/meshes/collada/simple/simple_asm0001_collada_14_prt.stl" scale="0.03937 0.03937 0.03937" />
-      </geometry>
-    </collision>
-  </link>
-  <link name ="LShr">
-    <inertial>
-      <origin xyz="-0.0038936743 -2.2022151E-6 -0.0048616005" rpy="0 0 0"/>
-      <mass value="0.77683752"/>
-      <inertia ixx="4.5812904E-4"  ixy="2.4111086E-7"  ixz="9.2521185E-6" iyy="4.3089204E-4" iyz="4.721695E-7" izz="3.4174855E-4" />
-    </inertial>
-    <visual>
-      <origin xyz="-0.005305 -0.1558 -0.844329" rpy="0 0 -3.14159265359"/>
-      <geometry name="LShr_visual">
-        <mesh filename="package://coman_urdf/meshes/collada/asm0001_collada_13_prt.dae" scale="0.03937 0.03937 0.03937" />
-      </geometry>
-    </visual>
-    <collision>
-      <origin xyz="-0.005305 -0.1558 -0.844329" rpy="0 0 -3.14159265359"/>
-      <geometry name="LShr_collision">
-        <mesh filename="package://coman_urdf/meshes/collada/simple/simple_asm0001_collada_13_prt.stl" scale="0.03937 0.03937 0.03937" />
-      </geometry>
-    </collision>
-  </link>
-  <link name ="LShy">
-    <inertial>
-      <origin xyz="0.0022714213 0.0071091517 -0.057455221" rpy="0 0 0"/>
-      <mass value="1.0462304"/>
-      <inertia ixx="0.0030934574"  ixy="-6.6702837E-5"  ixz="3.0222291E-4" iyy="0.0029181573" iyz="5.2663661E-4" izz="8.0830389E-4" />
-    </inertial>
-    <visual>
-      <origin xyz="-0.005305 -0.1558 -0.79952053" rpy="0 0 -3.14159265359"/>
-      <geometry name="LShy_visual">
-        <mesh filename="package://coman_urdf/meshes/collada/asm0001_collada_12_prt.dae" scale="0.03937 0.03937 0.03937" />
-      </geometry>
-    </visual>
-    <collision>
-      <origin xyz="-0.005305 -0.1558 -0.79952053" rpy="0 0 -3.14159265359"/>
-      <geometry name="LShy_collision">
-        <mesh filename="package://coman_urdf/meshes/collada/simple/simple_asm0001_collada_12_prt.stl" scale="0.03937 0.03937 0.03937" />
-      </geometry>
-    </collision>
-  </link>
+<!-- ********************ARMS******************** -->
+<xacro:include filename="$(find coman_urdf)/urdf/parts/arms.urdf.xacro" />
 <!-- ********************JOINTS******************** -->
     <joint name="l_ankle_joint" type="fixed">
@@ -569,28 +455,4 @@
   </xacro:if>
 <!-- ********************RIGHT ARM******************** -->
-  <joint name="RShSag" type="revolute">
-    <parent link="DWYTorso"/>
-    <child link="RShp"/>
-    <origin xyz="-0.014976503999999998 -0.0825 0.15770847" rpy="0 0 0" />
-    <axis xyz="0 1 0" />
-    <limit velocity="4.0" effort="50" lower="-3.4034" upper="1.6581" />
-    <dynamics friction="0" damping="3.0"/>
-  </joint>
-  <joint name="RShLat" type="revolute">
-    <parent link="RShp"/>
-    <child link="RShr"/>
-    <origin xyz="0.0 -0.07329999999999999 0.0" rpy="0 0 0" />
-    <axis xyz="1 0 0" />
-    <limit velocity="4.0" effort="50" lower="-2.094" upper="0.31415" />
-    <dynamics friction="0" damping="3.0"/>
-  </joint>
-  <joint name="RShYaw" type="revolute">
-    <parent link="RShr"/>
-    <child link="RShy"/>
-    <origin xyz="0.0 0.0 -0.04480846999999999" rpy="0 0 0" />
-    <axis xyz="0 0 1" />
-    <limit velocity="4.0" effort="50" lower="-1.5708" upper="1.5708" />
-    <dynamics friction="0" damping="3.0"/>
-  </joint>
   <joint name="RElbj" type="revolute">
     <parent link="RShy"/>
@@ -602,28 +464,4 @@
   </joint>
 <!-- ********************LEFT ARM******************** -->
-  <joint name="LShSag" type="revolute">
-    <parent link="DWYTorso"/>
-    <child link="LShp"/>
-    <origin xyz="-0.014976503999999998 0.0825 0.15770847" rpy="0 0 0" />
-    <axis xyz="0 1 0" />
-    <limit velocity="4.0" effort="50" lower="-3.4034" upper="1.6581" />
-    <dynamics friction="0" damping="3.0"/>
-  </joint>
-  <joint name="LShLat" type="revolute">
-    <parent link="LShp"/>
-    <child link="LShr"/>
-    <origin xyz="0.0 0.07329999999999999 0.0" rpy="0 0 0" />
-    <axis xyz="1 0 0" />
-    <limit velocity="4.0" effort="50" lower="-0.31415" upper="2.094" />
-    <dynamics friction="0" damping="3.0"/>
-  </joint>
-  <joint name="LShYaw" type="revolute">
-    <parent link="LShr"/>
-    <child link="LShy"/>
-    <origin xyz="0.0 0.0 -0.04480846999999999" rpy="0 0 0" />
-    <axis xyz="0 0 1" />
-    <limit velocity="4.0" effort="50" lower="-1.5708" upper="1.5708" />
-    <dynamics friction="0" damping="3.0"/>
-  </joint>
   <joint name="LElbj" type="revolute">
     <parent link="LShy"/>

Commit message: Deleted form old forearm mesh the elbow. Added elbow joint and link in arm.

File: coman_urdf/urdf/coman_base.urdf.xacro (robot description, xacro)
@@ -454,21 +454,3 @@
     </joint>
   </xacro:if>
-<!-- ********************RIGHT ARM******************** -->
-  <joint name="RElbj" type="revolute">
-    <parent link="RShy"/>
-    <child link="RElb"/>
-    <origin xyz="0.015 0.0 -0.13519152999999998" rpy="0 0 0" />
-    <axis xyz="0 1 0" />
-    <limit velocity="4.0" effort="50" lower="-2.3562" upper="0.0" />
-    <dynamics friction="0" damping="3.0"/>
-  </joint>
-<!-- ********************LEFT ARM******************** -->
-  <joint name="LElbj" type="revolute">
-    <parent link="LShy"/>
-    <child link="LElb"/>
-    <origin xyz="0.015 0.0 -0.13519152999999998" rpy="0 0 0" />
-    <axis xyz="0 1 0" />
-    <limit velocity="4.0" effort="50" lower="-2.3562" upper="0.0" />
-    <dynamics friction="0" damping="3.0"/>
-  </joint>
 </robot>

File: coman_urdf/urdf/coman_no_forearms.urdf (robot description, URDF)
Before this commit: robot COMAN, 46 links, 45 joints
Links:
- link LElb: geometry collision mesh filename=package://coman_urdf/meshes/collada/simple/forearms/elbow.s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 scale=1.0 1.0 1.0; visual mesh filename=package://coman_urdf/meshes/collada/forearms/elbow.dae scale=1.0 1.0 1.0
- link LForearm: geometry collision mesh filename=package://coman_urdf/meshes/collada/simple/forearm_old.dae scale=0.03937 0.03937 0.03937; visual mesh filename=package://coman_urdf/meshes/collada/forearm_old.dae scale=0.03937 0.03937 0.03937
- link RElb: geometry collision mesh filename=package://coman_urdf/meshes/collada/simple/forearms/elbow.s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 scale=1.0 1.0 1.0; visual mesh filename=package://coman_urdf/meshes/collada/forearms/elbow.dae scale=1.0 1.0 1.0
- link RForearm: geometry collision mesh filename=package://coman_urdf/meshes/collada/simple/forearm_old.dae scale=0.03937 0.03937 0.03937; visual mesh filename=package://coman_urdf/meshes/collada/forearm_old.dae scale=0.03937 0.03937 0.03937

File: coman_urdf/urdf/forearms/7DOF_forearms_DRC_14/7DOF_forearms_DRC_14.urdf.xacro (robot description, xacro)
@@ -9,23 +9,4 @@
 <!-- ****************LINKS**************** -->
 <!-- ****************LEFT FOREARM**************** -->
-    <link name ="LElb">
-        <inertial>
-          <origin xyz="-6.5553403E-4 9.3464748E-4 -9.3101289E-4" rpy="0 0 0"/>
-          <mass value="0.63306933"/>
-          <inertia ixx="2.2599075E-4"  ixy="2.6376470E-7"  ixz="-9.8007285E-6" iyy="2.7781302E-4" iyz="2.0435288E-6" izz="2.1878992E-4" />
-        </inertial>
-        <visual>
-          <origin xyz="0 0 0" rpy="-1.570796326795 1.570796326795 0"/>
-          <geometry name="LElb_visual">
-            <mesh filename="package://coman_urdf/meshes/collada/forearms/elbow.dae" scale="1.0 1.0 1.0" />
-          </geometry>
-        </visual>
-        <collision>
-          <origin xyz="0 0 0" rpy="-1.570796326795 1.570796326795 0"/>
-          <geometry name="LElb_collision">
-            <mesh filename="package://coman_urdf/meshes/collada/simple/forearms/elbow.stl" scale="1.0 1.0 1.0" />
-          </geometry>
-        </collision>
-      </link>
       <!-- ## WRONG NUMBERS FOR INERTIAL!!! FIX THEM!! ## -->
       <!-- In ROBOTRAN this link is named LFARM -->
@@ -92,23 +73,4 @@
       </link>
 <!-- ****************RIGHT FOREARM**************** -->
-<link name ="RElb">
-        <inertial>
-          <origin xyz="-6.5553403E-4 -9.3464748E-4 -9.3101289E-4" rpy="0 0 0"/>
-          <mass value="0.63306933"/>
-          <inertia ixx="2.2599075E-4"  ixy="-2.6376470E-7"  ixz="-9.8007285E-6" iyy="2.7781302E-4" iyz="-2.0435288E-6" izz="2.1878992E-4" />
-        </inertial>
-        <visual>
-          <origin xyz="0 0 0" rpy="-1.570796326795 1.570796326795 0"/>
-          <geometry name="RElb_visual">
-            <mesh filename="package://coman_urdf/meshes/collada/forearms/elbow.dae" scale="1.0 1.0 1.0" />
-          </geometry>
-        </visual>
-        <collision>
-          <origin xyz="0 0 0" rpy="-1.570796326795 1.570796326795 0"/>
-          <geometry name="RElb_collision">
-            <mesh filename="package://coman_urdf/meshes/collada/simple/forearms/elbow.stl" scale="1.0 1.0 1.0" />
-          </geometry>
-        </collision>
-      </link>
       <!-- ## WRONG NUMBERS FOR INERTIAL!!! FIX THEM!! ## -->
       <!-- In ROBOTRAN this link is named RFArm -->

File: coman_urdf/urdf/forearms/no_forearms/no_forearms.urdf.xacro (robot description, xacro)
@@ -1,25 +1,7 @@
 <?xml version="1.0"?>
 <robot xmlns:xacro="http://ros.org/wiki/xacro">
+<xacro:property name="Wrj1_to_FT" value="0.0568" />
 <!-- ***********LINKS*********** -->
 <!-- ***********LEFT FOREARM***********-->
-<link name ="LElb">
-      <inertial>
-        <origin xyz="-6.5553403E-4 9.3464748E-4 -9.3101289E-4" rpy="0 0 0"/>
-        <mass value="0.63306933"/>
-        <inertia ixx="2.2599075E-4"  ixy="2.637647E-7"  ixz="-9.8007285E-6" iyy="2.7781302E-4" iyz="2.0435288E-6" izz="2.1878992E-4" />
-      </inertial>
-      <visual>
-        <origin xyz="-0.020305 -0.1558 -0.664329" rpy="0 0 -3.14159265359"/>
-        <geometry name="LElb_visual">
-          <mesh filename="package://coman_urdf/meshes/collada/asm0001_collada_11_prt.dae" scale="0.03937 0.03937 0.03937" />
-        </geometry>
-      </visual>
-      <collision>
-        <origin xyz="-0.020305 -0.1558 -0.664329" rpy="0 0 -3.14159265359"/>
-        <geometry name="LElb_collision">
-          <mesh filename="package://coman_urdf/meshes/collada/simple/simple_asm0001_collada_11_prt.stl" scale="0.03937 0.03937 0.03937" />
-        </geometry>
-      </collision>
-    </link>
     <link name ="LForearm">
       <inertial>
@@ -28,32 +10,37 @@
         <inertia ixx="6.913E-4"  ixy="0.0"  ixz="0.0" iyy="6.913E-4" iyz="0.0" izz="4.0425E-5" />
       </inertial>
+      <visual>
+        <origin xyz="-0.0055 -0.1558 -0.6175" rpy="0 0 3.14159265359"/>
+        <geometry name="LForearm_visual">
+          <mesh filename="package://coman_urdf/meshes/collada/forearm_old.dae" scale="0.03937 0.03937 0.03937" />
+        </geometry>
+      </visual>
+      <collision>
+        <origin xyz="-0.0055 -0.1558 -0.6175" rpy="0 0 3.14159265359"/>
+        <geometry name="LForearm_collision">
+          <mesh filename="package://coman_urdf/meshes/collada/simple/forearm_old.dae" scale="0.03937 0.03937 0.03937" />
+        </geometry>
+      </collision>
     </link>
 <!-- ***********RIGHT FOREARM***********-->
- <link name ="RElb">
-    <inertial>
-      <origin xyz="-6.5553403E-4 -9.3464748E-4 -9.3101289E-4" rpy="0 0 0"/>
-      <mass value="0.63306933"/>
-      <inertia ixx="2.2599075E-4"  ixy="-2.6376470E-7"  ixz="-9.8007285E-6" iyy="2.7781302E-4" iyz="-2.0435288E-6" izz="2.1878992E-4" />
-    </inertial>
-    <visual>
-      <origin xyz="-0.020305 -0.1558 -0.664329" rpy="0 0 -3.14159265359"/>
-      <geometry name="RElb_visual">
-        <mesh filename="package://coman_urdf/meshes/collada/asm0001_collada_11_prt.dae" scale="0.03937 0.03937 0.03937" />
-      </geometry>
-    </visual>
-    <collision>
-      <origin xyz="-0.020305 -0.1558 -0.664329" rpy="0 0 -3.14159265359"/>
-      <geometry name="RElb_collision">
-        <mesh filename="package://coman_urdf/meshes/collada/simple/simple_asm0001_collada_11_prt.stl" scale="0.03937 0.03937 0.03937" />
-      </geometry>
-    </collision>
-  </link>
-  <link name ="RForearm">
-    <inertial>
-      <origin xyz="0 0 -0.085" rpy="0 0 0"/>
-      <mass value="0.263"/>
+<link name ="RForearm">
+      <inertial>
+      	<origin xyz="0 0 -0.085" rpy="0 0 0"/>
+      	<mass value="0.263"/>
       <inertia ixx="6.913E-4"  ixy="0.0"  ixz="0.0" iyy="6.913E-4" iyz="0.0" izz="4.0425E-5" />
     </inertial>
-  </link>
+      <visual>
+        <origin xyz="-0.0055 -0.1558 -0.6175" rpy="0 0 3.14159265359"/>
+        <geometry name="RForearm_visual">
+          <mesh filename="package://coman_urdf/meshes/collada/forearm_old.dae" scale="0.03937 0.03937 0.03937" />
+        </geometry>
+      </visual>
+      <collision>
+        <origin xyz="-0.0055 -0.1558 -0.6175" rpy="0 0 3.14159265359"/>
+        <geometry name="RForearm_collision">
+          <mesh filename="package://coman_urdf/meshes/collada/simple/forearm_old.dae" scale="0.03937 0.03937 0.03937" />
+        </geometry>
+      </collision>
+    </link>
 <!-- ***********JOINTS*********** -->
 <!-- ***********LEFT FOREARM***********-->

File: coman_urdf/urdf/parts/arms.urdf.xacro (robot description, xacro)
@@ -62,4 +62,23 @@
     </collision>
 </link>
+<link name ="RElb">
+        <inertial>
+          <origin xyz="-6.5553403E-4 -9.3464748E-4 -9.3101289E-4" rpy="0 0 0"/>
+          <mass value="0.63306933"/>
+          <inertia ixx="2.2599075E-4"  ixy="-2.6376470E-7"  ixz="-9.8007285E-6" iyy="2.7781302E-4" iyz="-2.0435288E-6" izz="2.1878992E-4" />
+        </inertial>
+        <visual>
+          <origin xyz="0 0 0" rpy="-1.570796326795 1.570796326795 0"/>
+          <geometry name="RElb_visual">
+            <mesh filename="package://coman_urdf/meshes/collada/forearms/elbow.dae" scale="1.0 1.0 1.0" />
+          </geometry>
+        </visual>
+        <collision>
+          <origin xyz="0 0 0" rpy="-1.570796326795 1.570796326795 0"/>
+          <geometry name="RElb_collision">
+            <mesh filename="package://coman_urdf/meshes/collada/simple/forearms/elbow.stl" scale="1.0 1.0 1.0" />
+          </geometry>
+        </collision>
+</link>
 <!-- LEFT ARM -->
 <link name ="LShp">
@@ -120,4 +139,23 @@
     </collision>
   </link>
+    <link name ="LElb">
+        <inertial>
+          <origin xyz="-6.5553403E-4 9.3464748E-4 -9.3101289E-4" rpy="0 0 0"/>
+          <mass value="0.63306933"/>
+          <inertia ixx="2.2599075E-4"  ixy="2.6376470E-7"  ixz="-9.8007285E-6" iyy="2.7781302E-4" iyz="2.0435288E-6" izz="2.1878992E-4" />
+        </inertial>
+        <visual>
+          <origin xyz="0 0 0" rpy="-1.570796326795 1.570796326795 0"/>
+          <geometry name="LElb_visual">
+            <mesh filename="package://coman_urdf/meshes/collada/forearms/elbow.dae" scale="1.0 1.0 1.0" />
+          </geometry>
+        </visual>
+        <collision>
+          <origin xyz="0 0 0" rpy="-1.570796326795 1.570796326795 0"/>
+          <geometry name="LElb_collision">
+            <mesh filename="package://coman_urdf/meshes/collada/simple/forearms/elbow.stl" scale="1.0 1.0 1.0" />
+          </geometry>
+        </collision>
+      </link>
 <!-- JOINTS -->
 <!-- RIGHT ARM -->
@@ -146,4 +184,12 @@
     <dynamics friction="0" damping="3.0"/>
 </joint>
+  <joint name="RElbj" type="revolute">
+    <parent link="RShy"/>
+    <child link="RElb"/>
+    <origin xyz="0.015 0.0 -0.13519152999999998" rpy="0 0 0" />
+    <axis xyz="0 1 0" />
+    <limit velocity="4.0" effort="50" lower="-2.3562" upper="0.0" />
+    <dynamics friction="0" damping="3.0"/>
+  </joint>
 <!-- LEFT ARM -->
 <joint name="LShSag" type="revolute">
@@ -171,3 +217,11 @@
     <dynamics friction="0" damping="3.0"/>
 </joint>
+  <joint name="LElbj" type="revolute">
+    <parent link="LShy"/>
+    <child link="LElb"/>
+    <origin xyz="0.015 0.0 -0.13519152999999998" rpy="0 0 0" />
+    <axis xyz="0 1 0" />
+    <limit velocity="4.0" effort="50" lower="-2.3562" upper="0.0" />
+    <dynamics friction="0" damping="3.0"/>
+  </joint>
 </robot>
