Commit message: Added legs part. Moved part of the legs in legs.urdf.xacro.

File: coman_urdf/urdf/coman_base.urdf.xacro (robot description, xacro)
@@ -11,242 +11,6 @@
 <!-- first real link of the robot, inertial reference frame -->
 <xacro:include filename="$(find coman_urdf)/urdf/parts/torso.urdf.xacro" />
-<!-- ********************RIGHT LEG******************** -->
-  <link name ="RHipMot">
-    <inertial>
-      <origin xyz="-3.269678E-4 -0.023587321 -2.6496509E-4" rpy="0 0 0"/>
-      <mass value="0.89258227"/>
-      <inertia ixx="4.7672294E-4"  ixy="-3.9936567E-6"  ixz="-2.4802574E-6" iyy="5.458038E-4" iyz="-3.3389575E-6" izz="5.126859E-4" />
-    </inertial>
-    <visual>
-      <origin xyz="0.0 0.023 -0.52" rpy="0 0 -3.14159265359"/>
-      <geometry name="RHipMot_visual">
-        <mesh filename="package://coman_urdf/meshes/collada/asm0001_collada_20_prt.dae" scale="0.03937 0.03937 0.03937" />
-      </geometry>
-    </visual>
-    <collision>
-      <origin xyz="0.0 0.023 -0.52" rpy="0 0 -3.14159265359"/>
-      <geometry name="RHipMot_collision">
-        <mesh filename="package://coman_urdf/meshes/collada/simple/simple_asm0001_collada_20_prt.stl" scale="0.03937 0.03937 0.03937" />
-      </geometry>
-    </collision>
-  </link>
-  <link name ="RThighUpLeg">
-    <inertial>
-      <origin xyz="0.0012591632 -0.016896372 -0.058903336" rpy="0 0 0"/>
-      <mass value="1.0246101"/>
-      <inertia ixx="9.165719E-4"  ixy="-1.4449904E-6"  ixz="-1.6685011E-5" iyy="0.00104849584" iyz="2.5492874E-5" izz="6.8637197E-4" />
-    </inertial>
-    <visual>
-      <origin xyz="0.0 0.0726 -0.52" rpy="0 0 -3.14159265359"/>
-      <geometry name="RThighUpLeg_visual">
-        <mesh filename="package://coman_urdf/meshes/collada/asm0001_collada_19_prt.dae" scale="0.03937 0.03937 0.03937" />
-      </geometry>
-    </visual>
-    <collision>
-      <origin xyz="0.0 0.0726 -0.52" rpy="0 0 -3.14159265359"/>
-      <geometry name="RThighUpLeg_collision">
-        <mesh filename="package://coman_urdf/meshes/collada/simple/simple_asm0001_collada_19_prt.stl" scale="0.03937 0.03937 0.03937" />
-      </geometry>
-    </collision>
-  </link>
-  <link name ="RThighLowLeg">
-    <inertial>
-      <origin xyz="9.8720058E-4 6.7037262E-4 -0.075716843" rpy="0 0 0"/>
-      <mass value="1.7001134"/>
-      <inertia ixx="0.0038979546"  ixy="1.7802399E-6"  ixz="2.6403262E-5" iyy="0.0039360845" iyz="4.522711E-5" izz="9.0218711E-4" />
-    </inertial>
-    <visual>
-      <origin xyz="0.0 0.0726 -0.4176" rpy="0 0 -3.14159265359"/>
-      <geometry name="RThighLowLeg_visual">
-        <mesh filename="package://coman_urdf/meshes/collada/asm0001_collada_18_prt.dae" scale="0.03937 0.03937 0.03937" />
-      </geometry>
-    </visual>
-    <collision>
-      <origin xyz="0.0 0.0726 -0.4176" rpy="0 0 -3.14159265359"/>
-      <geometry name="RThighLowLeg_collision">
-        <mesh filename="package://coman_urdf/meshes/collada/simple/simple_asm0001_collada_18_prt.stl" scale="0.03937 0.03937 0.03937" />
-      </geometry>
-    </collision>
-  </link>
-  <link name ="RLowLeg">
-    <inertial>
-      <origin xyz="0.0024612666 -0.0053099614 -0.08598948" rpy="0 0 0"/>
-      <mass value="1.4098179"/>
-      <inertia ixx="0.0040604004"  ixy="1.1227206E-5"  ixz="1.2260973E-5" iyy="0.004005652855" iyz="5.1899176E-4" izz="0.0012414054" />
-    </inertial>
-    <visual>
-      <origin xyz="0.0 0.0726 -0.2942" rpy="0 0 -3.14159265359"/>
-      <geometry name="RLowLeg_visual">
-        <mesh filename="package://coman_urdf/meshes/collada/asm0001_collada_17_prt.dae" scale="0.03937 0.03937 0.03937" />
-      </geometry>
-    </visual>
-    <collision>
-      <origin xyz="0.0 0.0726 -0.2942" rpy="0 0 -3.14159265359"/>
-      <geometry name="RLowLeg_collision">
-        <mesh filename="package://coman_urdf/meshes/collada/simple/simple_asm0001_collada_17_prt.stl" scale="0.03937 0.03937 0.03937" />
-      </geometry>
-    </collision>
-  </link>
-  <link name ="RFootmot">
-    <inertial>
-      <origin xyz="8.8067281E-4 -9.2224881E-4 2.3038476E-4" rpy="0 0 0"/>
-      <mass value="0.72992131"/>
-      <inertia ixx="3.2034425E-4"  ixy="7.6346303E-6"  ixz="2.5430158E-7" iyy="3.6584358E-4" iyz="-3.6889276E-6" izz="3.6065156E-4" />
-    </inertial>
-    <visual>
-      <origin xyz="0.0 0.0726 -0.0932" rpy="0 0 -3.14159265359"/>
-      <geometry name="RFootmot_visual">
-        <mesh filename="package://coman_urdf/meshes/collada/asm0001_collada_16_prt.dae" scale="0.03937 0.03937 0.03937" />
-      </geometry>
-    </visual>
-    <collision>
-      <origin xyz="0.0 0.0726 -0.0932" rpy="0 0 -3.14159265359"/>
-      <geometry name="RFootmot_collision">
-        <mesh filename="package://coman_urdf/meshes/collada/simple/simple_asm0001_collada_16_prt.stl" scale="0.03937 0.03937 0.03937" />
-      </geometry>
-    </collision>
-  </link>
-  <xacro:unless value="${GAZEBO_COMAN_USES_ACCURATE_FT}">
-    <xacro:if value="${GAZEBO_COMAN_USES_ROUND_FEET_13}">
-      <xacro:include filename="$(find coman_urdf)/urdf/feet/round_feet_13/round_foot_R_13.urdf.xacro" />
-    </xacro:if>
-    <xacro:if value="${GAZEBO_COMAN_USES_SIMPLE_FEET_DRC_sw1_14}">
-      <xacro:include filename="$(find coman_urdf)/urdf/feet/simple_feet_DRC_sw1_14/simple_foot_R_DRC_sw1_14.urdf.xacro" />
-    </xacro:if>
-  </xacro:unless>
-  <xacro:if value="${GAZEBO_COMAN_USES_ACCURATE_FT}">
-    <link name ="RFootFTSensor">
-      <inertial>
-        <origin xyz="0.0 -0.0 -0.0325" rpy="0 0 0"/>
-        <mass value="0.280"/>
-        <inertia ixx="0.0012944808"  ixy="0.0"  ixz="2.0080105E-4" iyy="0.0015851846" iyz="2.7599327E-4" izz="0.0013326766" />
-      </inertial>
-    </link>
-    <xacro:if value="${GAZEBO_COMAN_USES_ROUND_FEET_13}">
-      <xacro:include filename="$(find coman_urdf)/urdf/feet/round_feet_13/accurate_FT_round_foot_R_13.urdf.xacro" />
-    </xacro:if>
-    <xacro:if value="${GAZEBO_COMAN_USES_SIMPLE_FEET_DRC_sw1_14}">
-      <xacro:include filename="$(find coman_urdf)/urdf/feet/simple_feet_DRC_sw1_14/accurate_FT_simple_foot_R_DRC_sw1_14.urdf.xacro" />
-    </xacro:if>
-  </xacro:if>
-<!-- ********************LEFT LEG******************** -->
-  <link name ="LHipMot">
-    <inertial>
-      <origin xyz="-3.269678E-4 0.023587321 -2.6496509E-4" rpy="0 0 0"/>
-      <mass value="0.89258227"/>
-      <inertia ixx="4.7672294E-4"  ixy="3.9936567E-6"  ixz="-2.4802574E-6" iyy="5.458038E-4" iyz="3.3389575E-6" izz="5.126859E-4" />
-    </inertial>
-    <visual>
-      <origin xyz="0.0 -0.023 -0.52" rpy="0 0 -3.14159265359"/>
-      <geometry name="RHipMot_visual">
-        <mesh filename="package://coman_urdf/meshes/collada/asm0001_collada_06_prt.dae" scale="0.03937 0.03937 0.03937" />
-      </geometry>
-    </visual>
-    <collision>
-      <origin xyz="0.0 -0.023 -0.52" rpy="0 0 -3.14159265359"/>
-      <geometry name="RHipMot_collision">
-        <mesh filename="package://coman_urdf/meshes/collada/simple/simple_asm0001_collada_06_prt.stl" scale="0.03937 0.03937 0.03937" />
-      </geometry>
-    </collision>
-  </link>
-  <link name ="LThighUpLeg">
-    <inertial>
-      <origin xyz="0.0012591632 0.016896372 -0.058903336" rpy="0 0 0"/>
-      <mass value="1.0246101"/>
-      <inertia ixx="9.165719E-4"  ixy="1.4449904E-6"  ixz="-1.6685011E-5" iyy="0.00104849584" iyz="-2.5492874E-5" izz="6.8637197E-4" />
-    </inertial>
-    <visual>
-      <origin xyz="0.0 -0.0726 -0.52" rpy="0 0 -3.14159265359"/>
-      <geometry name="LThighUpLeg_visual">
-        <mesh filename="package://coman_urdf/meshes/collada/asm0001_collada_05_prt.dae" scale="0.03937 0.03937 0.03937" />
-      </geometry>
-    </visual>
-    <collision>
-      <origin xyz="0.0 -0.0726 -0.52" rpy="0 0 -3.14159265359"/>
-      <geometry name="LThighUpLeg_collision">
-        <mesh filename="package://coman_urdf/meshes/collada/simple/simple_asm0001_collada_05_prt.stl" scale="0.03937 0.03937 0.03937" />
-      </geometry>
-    </collision>
-  </link>
-  <link name ="LThighLowLeg">
-    <inertial>
-      <origin xyz="9.8720058E-4 -6.7037262E-4 -0.075716843" rpy="0 0 0"/>
-      <mass value="1.7001134"/>
-      <inertia ixx="0.0038979546"  ixy="-1.7802399E-6"  ixz="2.6403262E-5" iyy="0.0039360845" iyz="-4.5227110E-5" izz="9.0218711E-4" />
-    </inertial>
-    <visual>
-      <origin xyz="0.0 -0.0726 -0.4176" rpy="0 0 -3.14159265359"/>
-      <geometry name="LThighLowLeg_visual">
-        <mesh filename="package://coman_urdf/meshes/collada/asm0001_collada_04_prt.dae" scale="0.03937 0.03937 0.03937" />
-      </geometry>
-    </visual>
-    <collision>
-      <origin xyz="0.0 -0.0726 -0.4176" rpy="0 0 -3.14159265359"/>
-      <geometry name="LThighLowLeg_collision">
-        <mesh filename="package://coman_urdf/meshes/collada/simple/simple_asm0001_collada_04_prt.stl" scale="0.03937 0.03937 0.03937" />
-      </geometry>
-    </collision>
-  </link>
-  <link name ="LLowLeg">
-    <inertial>
-      <origin xyz="0.0024612666 0.0053099614 -0.085989484" rpy="0 0 0"/>
-      <mass value="1.4098179"/>
-      <inertia ixx="0.0040604004"  ixy="-1.1227206E-5"  ixz="1.2260973E-5" iyy="0.004005652855" iyz="-5.1899176E-4" izz="0.0012414054" />
-    </inertial>
-    <visual>
-      <origin xyz="0.0 -0.0726 -0.2942" rpy="0 0 -3.14159265359"/>
-      <geometry name="LLowLeg_visual">
-        <mesh filename="package://coman_urdf/meshes/collada/asm0001_collada_03_prt.dae" scale="0.03937 0.03937 0.03937" />
-      </geometry>
-    </visual>
-    <collision>
-      <origin xyz="0.0 -0.0726 -0.2942" rpy="0 0 -3.14159265359"/>
-      <geometry name="LLowLeg_collision">
-        <mesh filename="package://coman_urdf/meshes/collada/simple/simple_asm0001_collada_03_prt.stl" scale="0.03937 0.03937 0.03937" />
-      </geometry>
-    </collision>
-  </link>
-  <link name ="LFootmot">
-    <inertial>
-      <origin xyz="8.8067281E-4 9.2224881E-4 2.3038476E-4" rpy="0 0 0"/>
-      <mass value="0.72992131"/>
-      <inertia ixx="3.2034425E-4"  ixy="-7.6346303E-6"  ixz="2.5430158E-7" iyy="3.6584358E-4" iyz="3.6889276E-6" izz="3.6065156E-4" />
-    </inertial>
-    <visual>
-      <origin xyz="0.0 -0.0726 -0.0932" rpy="0 0 -3.14159265359"/>
-      <geometry name="LFootmot_visual">
-        <mesh filename="package://coman_urdf/meshes/collada/asm0001_collada_02_prt.dae" scale="0.03937 0.03937 0.03937" />
-      </geometry>
-    </visual>
-    <collision>
-      <origin xyz="0.0 -0.0726 -0.0932" rpy="0 0 -3.14159265359"/>
-      <geometry name="LFootmot_collision">
-        <mesh filename="package://coman_urdf/meshes/collada/simple/simple_asm0001_collada_02_prt.stl" scale="0.03937 0.03937 0.03937" />
-      </geometry>
-    </collision>
-  </link>
-  <xacro:unless value="${GAZEBO_COMAN_USES_ACCURATE_FT}">
-    <xacro:if value="${GAZEBO_COMAN_USES_ROUND_FEET_13}">
-      <xacro:include filename="$(find coman_urdf)/urdf/feet/round_feet_13/round_foot_L_13.urdf.xacro" />
-    </xacro:if>
-    <xacro:if value="${GAZEBO_COMAN_USES_SIMPLE_FEET_DRC_sw1_14}">
-      <xacro:include filename="$(find coman_urdf)/urdf/feet/simple_feet_DRC_sw1_14/simple_foot_L_DRC_sw1_14.urdf.xacro" />
-    </xacro:if>
-  </xacro:unless>
-  <xacro:if value="${GAZEBO_COMAN_USES_ACCURATE_FT}">
-    <link name ="LFootFTSensor">
-      <inertial>
-        <origin xyz="0.0 -0.0 -0.0325" rpy="0 0 0"/>
-        <mass value="0.280"/>
-        <inertia ixx="0.0012944808"  ixy="-9.2387693E-5"  ixz="2.0080105E-4" iyy="0.0015851846" iyz="2.7599327E-4" izz="0.0013326766" />
-      </inertial>
-    </link>
-    <xacro:if value="${GAZEBO_COMAN_USES_ROUND_FEET_13}">
-      <xacro:include filename="$(find coman_urdf)/urdf/feet/round_feet_13/accurate_FT_round_foot_L_13.urdf.xacro" />
-    </xacro:if>
-    <xacro:if value="${GAZEBO_COMAN_USES_SIMPLE_FEET_DRC_sw1_14}">
-      <xacro:include filename="$(find coman_urdf)/urdf/feet/simple_feet_DRC_sw1_14/accurate_FT_simple_foot_L_DRC_sw1_14.urdf.xacro" />
-    </xacro:if>
-  </xacro:if>
+<!-- ********************LEGS******************** -->
+<xacro:include filename="$(find coman_urdf)/urdf/parts/legs.urdf.xacro" />
 <!-- ********************ARMS******************** -->
 <xacro:include filename="$(find coman_urdf)/urdf/parts/arms.urdf.xacro" />
@@ -316,141 +80,3 @@
   	</joint>
 </xacro:unless>
-<!-- ********************RIGHT LEG******************** -->
-  <joint name="RHipSag" type="revolute">
-    <parent link="Waist"/>
-    <child link="RHipMot"/>
-    <origin xyz="0.0 -0.023 0.0" rpy="0 0 0" />
-    <axis xyz="0 1 0" />
-    <limit velocity="4.0" effort="50" lower="-1.9199" upper="0.7854" />
-    <dynamics friction="0" damping="3.0"/>
-  </joint>
-  <joint name="RHipLat" type="revolute">
-    <parent link="RHipMot"/>
-    <child link="RThighUpLeg"/>
-    <origin xyz="0.0 -0.0496 0.0" rpy="0 0 0" />
-    <axis xyz="1 0 0" />
-    <limit velocity="4.0" effort="50" lower="-1.0472" upper="0.4363" />
-    <dynamics friction="0" damping="3.0"/>
-  </joint>
-  <joint name="RHipYaw" type="revolute">
-    <parent link="RThighUpLeg"/>
-    <child link="RThighLowLeg"/>
-    <origin xyz="0.0 0.0 -0.1024" rpy="0 0 0" />
-    <axis xyz="0 0 1" />
-    <limit velocity="4.0" effort="50" lower="-0.8727" upper="0.8727" />
-    <dynamics friction="0" damping="3.0"/>
-  </joint>
-  <joint name="RKneeSag" type="revolute">
-    <parent link="RThighLowLeg"/>
-    <child link="RLowLeg"/>
-    <origin xyz="0.0 0.0 -0.1234" rpy="0 0 0" />
-    <axis xyz="0 1 0" />
-    <limit velocity="4.0" effort="50" lower="-0.1745" upper="1.9199" />
-    <dynamics friction="0" damping="3.0"/>
-  </joint>
-  <joint name="RAnkLat" type="revolute">
-    <parent link="RLowLeg"/>
-    <child link="RFootmot"/>
-    <origin xyz="0.0 0.0 -0.201" rpy="0 0 0" />
-    <axis xyz="1 0 0" />
-    <limit velocity="4.0" effort="50" lower="-0.6109" upper="0.6109" />
-    <dynamics friction="0" damping="3.0"/>
-  </joint>
-  <xacro:unless value="${GAZEBO_COMAN_USES_ACCURATE_FT}">
-    <joint name="RAnkSag" type="revolute">
-      <parent link="RFootmot"/>
-      <child link="RFoot"/>
-      <origin xyz="0.0 0.0 0.0" rpy="0 0 0" />
-      <axis xyz="0 1 0" />
-      <limit velocity="4.0" effort="50" lower="-1.2217" upper="1.2217" />
-      <dynamics friction="0" damping="3.0"/>
-    </joint>
-  </xacro:unless>
-  <xacro:if value="${GAZEBO_COMAN_USES_ACCURATE_FT}">
-    <joint name="RAnkSag" type="revolute">
-      <parent link="RFootmot"/>
-      <child link="RFootFTSensor"/>
-      <origin xyz="0.0 0.0 0.0" rpy="0 0 0" />
-      <axis xyz="0 1 0" />
-      <limit velocity="4.0" effort="50" lower="-1.2217" upper="1.2217" />
-      <dynamics friction="0" damping="3.0"/>
-    </joint>
-    <joint name="RAnkSagFT" type="revolute">
-      <parent link="RFootFTSensor"/>
-      <child link="RFoot"/>
-      <origin xyz="0.0 0.0 -0.065" rpy="0 0 0" />
-      <axis xyz="0 1 0" />
-      <limit velocity="0.0" effort="0" lower="-0.0" upper="0.0" />
-      <dynamics friction="0" damping="3.0"/>
-    </joint>
-  </xacro:if>
-<!-- ********************LEFT LEG******************** -->
-  <joint name="LHipSag" type="revolute">
-    <parent link="Waist"/>
-    <child link="LHipMot"/>
-    <origin xyz="0.0 0.023 0.0" rpy="0 0 0" />
-    <axis xyz="0 1 0" />
-    <limit velocity="4.0" effort="50" lower="-1.9199" upper="0.7854" />
-    <dynamics friction="0" damping="3.0"/>
-  </joint>
-  <joint name="LHipLat" type="revolute">
-    <parent link="LHipMot"/>
-    <child link="LThighUpLeg"/>
-    <origin xyz="0.0 0.0496 0.0" rpy="0 0 0" />
-    <axis xyz="1 0 0" />
-    <limit velocity="4.0" effort="50" lower="-0.4363" upper="1.0472" />
-    <dynamics friction="0" damping="3.0"/>
-  </joint>
-  <joint name="LHipYaw" type="revolute">
-    <parent link="LThighUpLeg"/>
-    <child link="LThighLowLeg"/>
-    <origin xyz="0.0 0.0 -0.1024" rpy="0 0 0" />
-    <axis xyz="0 0 1" />
-    <limit velocity="4.0" effort="50" lower="-0.8727" upper="0.8727" />
-    <dynamics friction="0" damping="3.0"/>
-  </joint>
-  <joint name="LKneeSag" type="revolute">
-    <parent link="LThighLowLeg"/>
-    <child link="LLowLeg"/>
-    <origin xyz="0.0 0.0 -0.1234" rpy="0 0 0" />
-    <axis xyz="0 1 0" />
-    <limit velocity="4.0" effort="50" lower="-0.1745" upper="1.9199" />
-    <dynamics friction="0" damping="3.0"/>
-  </joint>
-  <joint name="LAnkLat" type="revolute">
-    <parent link="LLowLeg"/>
-    <child link="LFootmot"/>
-    <origin xyz="0.0 0.0 -0.201" rpy="0 0 0" />
-    <axis xyz="1 0 0" />
-    <limit velocity="4.0" effort="50" lower="-0.6109" upper="0.6109" />
-    <dynamics friction="0" damping="3.0"/>
-  </joint>
-  <xacro:unless value="${GAZEBO_COMAN_USES_ACCURATE_FT}">
-    <joint name="LAnkSag" type="revolute">
-      <parent link="LFootmot"/>
-      <child link="LFoot"/>
-      <origin xyz="0.0 0.0 0.0" rpy="0 0 0" />
-      <axis xyz="0 1 0" />
-      <limit velocity="4.0" effort="50" lower="-1.2217" upper="1.2217" />
-      <dynamics friction="0" damping="3.0"/>
-    </joint>
-  </xacro:unless>
-  <xacro:if value="${GAZEBO_COMAN_USES_ACCURATE_FT}">
-    <joint name="LAnkSag" type="revolute">
-      <parent link="LFootmot"/>
-      <child link="LFootFTSensor"/>
-      <origin xyz="0.0 0.0 0.0" rpy="0 0 0" />
-      <axis xyz="0 1 0" />
-      <limit velocity="4.0" effort="50" lower="-1.2217" upper="1.2217" />
-      <dynamics friction="0" damping="3.0"/>
-    </joint>
-    <joint name="LAnkSagFT" type="revolute">
-      <parent link="LFootFTSensor"/>
-      <child link="LFoot"/>
-      <origin xyz="0.0 0.0 -0.065" rpy="0 0 0" />
-      <axis xyz="0 1 0" />
-      <limit velocity="0.0" effort="0" lower="-0.0" upper="0.0" />
-      <dynamics friction="0" damping="3.0"/>
-    </joint>
-  </xacro:if>
 </robot>

Commit message: Start refactor of urdf for coman.

File: coman_urdf/urdf/coman_base.urdf.xacro (robot description, xacro)
@@ -8,4 +8,34 @@
   Velocity and effort limits are fake!
 -->
+<xacro:property name="PI" value="3.14159265359" />
+<!-- This links are defined in order to be compliant with http://www.ros.org/reps/rep-0120.html#coordinate-frames
+and to define the end effectors of the robot
+The coordinate frame called base_link is rigidly attached to the robot root body. It is recommended to choose the robot waist as its root body. The base_link can be attached to the root in any arbitrary position or orientation; for every hardware platform there will be a different place on the base that provides an obvious point of reference. Note that REP 103 [1] specifies a preferred orientation for frames. -->
+<link name="base_link"/>
+<link name="Waist">
+    <inertial>
+      <origin xyz="-0.026391145 -5.8216364E-4 0.052632312" rpy="0.0 0.0 0.0"/>
+      <mass value="1.8008695"/>
+      <inertia ixx="0.0051032982"  ixy="-5.7170981E-5"  ixz="0.0016920543" iyy="0.006241636" iyz="1.7225949E-5" izz="0.0024517762" />
+    </inertial>
+    <visual>
+      <origin xyz="0 0 -0.52" rpy="0 0 ${PI}"/>
+      <material name="dark_grey"/>
+      <geometry name="Waist_visual">
+        <mesh filename="package://coman_urdf/meshes/Waist.STL" scale="0.03937 0.03937 0.03937"/>
+      </geometry>
+    </visual>
+    <collision>
+      <origin xyz="0 0 -0.52" rpy="0 0 ${PI}"/>
+      <geometry name="Waist_collision">
+        <mesh filename="package://coman_urdf/meshes/simple/Waist.STL" scale="0.03937 0.03937 0.03937"/>
+      </geometry>
+    </collision>
+</link>
+<joint name="base_joint" type="fixed">
+    <parent link="base_link"/>
+    <child link="Waist"/>
+    <origin xyz="0 0 0" rpy="0 0 0" />
+</joint>
 <!-- ********************TORSO******************** -->
 <!-- first real link of the robot, inertial reference frame -->

File: coman_urdf/urdf/parts/torso.urdf.xacro (robot description, xacro)
@@ -4,34 +4,9 @@
 <xacro:property name="PI_2" value="1.57079632679" />
 <xacro:property name="SF" value="0.03937" /> <!-- Scale factor for meshes -->
-<xacro:property name="base_link_z_translation" value="-0.52" />
 <xacro:property name="cos_20" value="0.93969262078" />
 <xacro:property name="sin_20" value="0.34202014332" />
 <!-- LINKS -->
-<!-- This links are defined in order to be compliant with http://www.ros.org/reps/rep-0120.html#coordinate-frames
-and to define the end effectors of the robot
-The coordinate frame called base_link is rigidly attached to the robot root body. It is recommended to choose the robot waist as its root body. The base_link can be attached to the root in any arbitrary position or orientation; for every hardware platform there will be a different place on the base that provides an obvious point of reference. Note that REP 103 [1] specifies a preferred orientation for frames. -->
-<link name="base_link"/>
 <!-- The coordinate frame called torso is attached to the lowest body of the model which is a parent of l_gripper, r_gripper and gaze. -->
  <link name="torso"/>
-<link name="Waist">
-    <inertial>
-      <origin xyz="-0.026391145 -5.8216364E-4 0.052632312" rpy="0.0 0.0 0.0"/>
-      <mass value="1.8008695"/>
-      <inertia ixx="0.0051032982"  ixy="-5.7170981E-5"  ixz="0.0016920543" iyy="0.006241636" iyz="1.7225949E-5" izz="0.0024517762" />
-    </inertial>
-    <visual>
-      <origin xyz="0 0 ${base_link_z_translation}" rpy="0 0 ${PI}"/>
-      <material name="dark_grey"/>
-      <geometry name="Waist_visual">
-        <mesh filename="package://coman_urdf/meshes/collada/torso0.stl" scale="${SF} ${SF} ${SF}"/>
-      </geometry>
-    </visual>
-    <collision>
-      <origin xyz="0 0 ${base_link_z_translation}" rpy="0 0 ${PI}"/>
-      <geometry name="Waist_collision">
-        <mesh filename="package://coman_urdf/meshes/collada/simple/simple_asm0001_collada_07_prt.stl" scale="${SF} ${SF} ${SF}"/>
-      </geometry>
-    </collision>
-</link>
   <link name ="DWL">
     <inertial>
@@ -95,9 +70,4 @@
   </link>
 <!-- JOINTS -->
-<joint name="base_joint" type="fixed">
-    <parent link="base_link"/>
-    <child link="Waist"/>
-    <origin xyz="0 0 0" rpy="0 0 0" />
-</joint>
 <joint name="torso_joint" type="fixed">
     <parent link="DWYTorso"/>

Commit message: Added missing link world

File: coman_urdf/urdf/coman_base.urdf.xacro (robot description, xacro)
@@ -38,4 +38,9 @@
     <origin xyz="0 0 0" rpy="0 0 0" />
 </joint>
+  <link name="world"/>
+  <joint name="reference" type="floating">
+    <parent link="world"/>
+    <child link="base_link"/>
+  </joint>
 <!-- ********************TORSO******************** -->
 <!-- first real link of the robot, inertial reference frame -->
