Commit message: Moved declaration of gazebo_yarp_plugins inside coman_robot.urdf.xacro. Now we do not need anymore to declarate them inside world files. Furthermore we have new file yarp_control.gazebo.xacro that automatically loads the right plugins for different version of coman that are selectable inside coman_config.urdf.xacro.

File: coman_urdf/urdf/coman_config.urdf.xacro (robot description, xacro)
@@ -21,25 +21,32 @@
 ####################################################
 ##
-##  FOREARMS SELECTION
+##  FOREARMS & HANDS SELECTION
 ##
 ##
 ## options:
 ## 1) no forearms
-## 2) 7dof forearms + soft hands
+## 2) 7dof forearms
+## 3) 7dof forearms + soft hands
 ##
 ####################################################
 # TODO: checks (must be mutually exclusive).. eventually, a menu!... documentation!
 #       at the moment just the only combinations that work are:
-#
-# 1) NO_FOREARMS + NO_HANDS
-#
+-->
+<!-- 1) NO_FOREARMS -->
+<!--
 <xacro:property name="GAZEBO_COMAN_USES_NO_FOREARMS" value="true" />
-<xacro:property name="GAZEBO_COMAN_USES_7DOF_FOREARMS_DRC_14" value="true" />
+<xacro:property name="GAZEBO_COMAN_USES_7DOF_FOREARMS_DRC_14" value="false" />
 <xacro:property name="GAZEBO_COMAN_USES_SOFTHANDS_DRC_sw1_14" value="false" />
-# 2) 7DOFS_FOREARMS + SOFTHANDS
 -->
+<!-- 2) 7DOFS_FOREARMS -->
 <xacro:property name="GAZEBO_COMAN_USES_NO_FOREARMS" value="false" />
 <xacro:property name="GAZEBO_COMAN_USES_7DOF_FOREARMS_DRC_14" value="true" />
 <xacro:property name="GAZEBO_COMAN_USES_SOFTHANDS_DRC_sw1_14" value="false" />
+<!-- 3) 7DOFS_FOREARMS + SOFT_HANDS -->
+<!--
+<xacro:property name="GAZEBO_COMAN_USES_NO_FOREARMS" value="false" />
+<xacro:property name="GAZEBO_COMAN_USES_7DOF_FOREARMS_DRC_14" value="true" />
+<xacro:property name="GAZEBO_COMAN_USES_SOFTHANDS_DRC_sw1_14" value="true" />
+-->
 <!--
 ####################################################

File: coman_urdf/urdf/coman_robot.urdf.xacro (robot description, xacro)
@@ -31,4 +31,6 @@
   </xacro:if>
   <xacro:include filename="$(find coman_urdf)/urdf/coman.gazebo.xacro" />
+<!-- YARP PLUGINS for GAZEBO SIMULATION -->
+  <xacro:include filename="$(find coman_urdf)/urdf/yarp_control.gazebo.xacro" />
   <origin xyz="0.0 0.0 0.521" rpy="0 0 0" />
 </robot>

Commit message: Added xtion stl. Missing in file. Deleted from models.

File: coman_urdf/urdf/coman_config.urdf.xacro (robot description, xacro)
@@ -123,4 +123,4 @@
 #
 -->
-<xacro:property name="GAZEBO_COMAN_USES_XTION" value="true" />
+<xacro:property name="GAZEBO_COMAN_USES_XTION" value="false" />
 </robot>

File: coman_urdf/urdf/config/coman_hands.urdf.xacro (robot description, xacro)
@@ -123,4 +123,4 @@
 #
 -->
-<xacro:property name="GAZEBO_COMAN_USES_XTION" value="true" />
+<xacro:property name="GAZEBO_COMAN_USES_XTION" value="false" />
 </robot>

Commit message: Simplified meshes for xtion. Set xtion flag default to false. Fixed warning in coman_slider.launch.

File: coman_urdf/urdf/coman_config.urdf.xacro (robot description, xacro)
@@ -41,4 +41,4 @@
 #
 -->
-<xacro:property name="GAZEBO_COMAN_USES_XTION" value="true" />
+<xacro:property name="GAZEBO_COMAN_USES_XTION" value="false" />
 </robot>

File: coman_urdf/urdf/sensors/xtion.urdf.xacro (robot description, xacro)
@@ -12,5 +12,5 @@
       <origin xyz="-0.020281504 0.0 -0.68662053" rpy="0 0 ${PI}"/>
       <geometry name="Xtion_body_visual">
-        <mesh filename="package://coman_urdf/meshes/collada/Xtion/xtion_base.stl" scale="0.03937 0.03937 0.03937" />
+        <mesh filename="package://coman_urdf/meshes/XtionBase.STL" scale="0.03937 0.03937 0.03937" />
       </geometry>
     </visual>
@@ -18,5 +18,5 @@
       <origin xyz="-0.020281504 0.0 -0.68662053" rpy="0 0 ${PI}"/>
       <geometry name="Xtion_body_collision">
-        <mesh filename="package://coman_urdf/meshes/collada/simple/Xtion/xtion_base.stl" scale="0.03937 0.03937 0.03937" />
+        <mesh filename="package://coman_urdf/meshes/simple/XtionBase.STL" scale="0.03937 0.03937 0.03937" />
       </geometry>
     </collision>
@@ -31,5 +31,5 @@
       <origin xyz="-0.0915 0.0 -1.2778" rpy="0 0 ${PI}"/>
       <geometry name="Xtion_cam_body_visual">
-        <mesh filename="package://coman_urdf/meshes/collada/Xtion/xtion_cam_body.stl" scale="0.001 0.001 0.001" />
+        <mesh filename="package://coman_urdf/meshes/XtionCamBody.STL" scale="0.001 0.001 0.001" />
       </geometry>
     </visual>
@@ -37,5 +37,5 @@
       <origin xyz="-0.0915 0.0 -1.2778" rpy="0 0 ${PI}"/>
       <geometry name="Xtion_cam_body_collision">
-        <mesh filename="package://coman_urdf/meshes/collada/simple/Xtion/xtion_cam_body.stl" scale="0.001 0.001 0.001" />
+        <mesh filename="package://coman_urdf/meshes/simple/XtionCamBody.STL" scale="0.001 0.001 0.001" />
       </geometry>
     </collision>

Commit message: Added new config model. Added ros imu sensor

File: coman_urdf/urdf/coman_config.urdf.xacro (robot description, xacro)
@@ -49,3 +49,17 @@
 -->
 <xacro:property name="GAZEBO_COMAN_USES_XTION" value="false" />
+<!--
+####################################################
+##
+##  USE GRASPFIX (IN ROS)
+####################################################
+-->
+<xacro:property name="GAZEBO_COMAN_USES_ROS_GRASPFIX" value="false" />
+<!--
+####################################################
+##
+##  USE ROS for IMU
+####################################################
+-->
+<xacro:property name="GAZEBO_COMAN_USES_ROS_IMU" value="false" />
 </robot>

File: coman_urdf/urdf/coman_robot.urdf.xacro (robot description, xacro)
@@ -12,7 +12,7 @@
 	<xacro:include filename="$(find coman_urdf)/urdf/gazebo/openni_kinect.gazebo.xacro" />
   </xacro:if>
-  <xacro:unless value="${GAZEBO_COMAN_USES_SOFTHANDS}">
+  <xacro:if value="${GAZEBO_COMAN_USES_ROS_GRASPFIX}">
 	<xacro:include filename="$(find coman_urdf)/urdf/gazebo/grasp_fix_plugin.xacro" />
-  </xacro:unless>
+  </xacro:if>
 <!-- YARP PLUGINS for GAZEBO SIMULATION -->
   <xacro:if value="${GAZEBO_COMAN_USES_YARP}">

File: coman_urdf/urdf/config/coman_cogimon.urdf.xacro (robot description, xacro)
@@ -1,6 +1,6 @@
 <?xml version="1.0"?>
 <robot xmlns:xacro="http://ros.org/wiki/xacro" name="COMAN">
-<xacro:property name="model_name" value="IIT Coman" />
-<xacro:property name="model_version" value="1.0" />
+<xacro:property name="model_name" value="IIT Coman COGIMON" />
+<xacro:property name="model_version" value="0.1" />
 <!--
 ####################################################
@@ -22,5 +22,5 @@
 -->
 <xacro:property name="GAZEBO_COMAN_USES_FOREARMS" value="true" />
-<xacro:property name="GAZEBO_COMAN_USES_SOFTHANDS" value="false" />
+<xacro:property name="GAZEBO_COMAN_USES_SOFTHANDS" value="true" />
 <!--
 ####################################################
@@ -29,5 +29,5 @@
 ####################################################
 -->
-<xacro:property name="GAZEBO_COMAN_USES_YARP" value="true" />
+<xacro:property name="GAZEBO_COMAN_USES_YARP" value="false" />
 <!--
 ####################################################
@@ -61,4 +61,4 @@
 ####################################################
 -->
-<xacro:property name="GAZEBO_COMAN_USES_ROS_IMU" value="false" />
+<xacro:property name="GAZEBO_COMAN_USES_ROS_IMU" value="true" />
 </robot>

File: coman_urdf/urdf/config/coman_no_forearms.urdf.xacro (robot description, xacro)
@@ -48,3 +48,17 @@
 -->
 <xacro:property name="GAZEBO_COMAN_USES_XTION" value="false" />
+<!--
+####################################################
+##
+##  USE GRASPFIX (IN ROS)
+####################################################
+-->
+<xacro:property name="GAZEBO_COMAN_USES_ROS_GRASPFIX" value="false" />
+<!--
+####################################################
+##
+##  USE ROS for IMU
+####################################################
+-->
+<xacro:property name="GAZEBO_COMAN_USES_ROS_IMU" value="false" />
 </robot>

File: coman_urdf/urdf/config/coman_softhand.urdf.xacro (robot description, xacro)
@@ -48,3 +48,17 @@
 -->
 <xacro:property name="GAZEBO_COMAN_USES_XTION" value="false" />
+<!--
+####################################################
+##
+##  USE GRASPFIX (IN ROS)
+####################################################
+-->
+<xacro:property name="GAZEBO_COMAN_USES_ROS_GRASPFIX" value="false" />
+<!--
+####################################################
+##
+##  USE ROS for IMU
+####################################################
+-->
+<xacro:property name="GAZEBO_COMAN_USES_ROS_IMU" value="false" />
 </robot>

File: coman_urdf/urdf/gazebo/grasp_fix_plugin.xacro (robot description, xacro)
@@ -9,5 +9,5 @@
 			<gripper_link>RSoftHandFingers</gripper_link>
 		</arm>
-                <arm>
+              <arm>
 			<arm_name>LArm</arm_name>
 			<palm_link>LWrMot2</palm_link>

File: coman_urdf/urdf/gazebo/microstrain_3dmgx2_imu.gazebo.xacro (robot description, xacro)
@@ -6,4 +6,19 @@
   This file groups files to use COMAN in GAZEBO
   -->
+<xacro:if value="${GAZEBO_COMAN_USES_ROS_IMU}">
+<gazebo>
+       <plugin name="imu_plugin" filename="libgazebo_ros_imu.so"> <!-- For now we use this...to change with the commented one in future-->
+       <!--plugin name="imu_plugin" filename="libgazebo_ros_imu_sensor.so"-->
+              <alwaysOn>true</alwaysOn>
+              <bodyName>imu_link</bodyName>
+              <frameName>imu_link</frameName>
+              <topicName>imu</topicName>
+              <serviceName>imu_service</serviceName>
+              <gaussianNoise>0.0</gaussianNoise>
+              <updateRate>20.0</updateRate>
+       </plugin>
+</gazebo>
+</xacro:if>
+<xacro:unless value="${GAZEBO_COMAN_USES_ROS_IMU}">
     <gazebo reference="imu_link">
         <sensor name="imu_sensor" type="imu">
@@ -38,3 +53,4 @@
         </sensor>
        </gazebo>
+</xacro:unless>
 </robot>

Commit message: enable xbot usage

File: coman_urdf/urdf/coman_config.urdf.xacro (robot description, xacro)
@@ -30,5 +30,12 @@
 ####################################################
 -->
-<xacro:property name="GAZEBO_COMAN_USES_YARP" value="true" />
+<xacro:property name="GAZEBO_COMAN_USES_YARP" value="false" />
+<!--
+####################################################
+##
+##  USE XBOT
+####################################################
+-->
+<xacro:property name="GAZEBO_COMAN_USES_XBOT" value="true" />
 <!--
 ####################################################

File: coman_urdf/urdf/coman_robot.urdf.xacro (robot description, xacro)
@@ -20,4 +20,8 @@
   </xacro:if>
   <xacro:include filename="$(find coman_urdf)/urdf/gazebo/force_torque.gazebo.xacro" />
+  <!-- XBOT PLUGINS for GAZEBO SIMULATION -->
+  <xacro:if value="${GAZEBO_COMAN_USES_XBOT}">
+         <xacro:include filename="$(find coman_urdf)/urdf/gazebo/xbot_control.gazebo.xacro" />
+  </xacro:if>
   <xacro:include filename="$(find coman_urdf)/urdf/gazebo/coman_materials.gazebo.xacro" />
   <origin xyz="0.0 0.0 0.521" rpy="0 0 0" />

File: coman_urdf/urdf/config/coman_cogimon.urdf.xacro (robot description, xacro)
@@ -33,4 +33,11 @@
 ####################################################
 ##
+##  USE XBOT
+####################################################
+-->
+<xacro:property name="GAZEBO_COMAN_USES_XBOT" value="true" />
+<!--
+####################################################
+##
 ##  Xtion SELECTION
 ##

File: coman_urdf/urdf/config/coman_hands.urdf.xacro (robot description, xacro)
@@ -29,5 +29,12 @@
 ####################################################
 -->
-<xacro:property name="GAZEBO_COMAN_USES_YARP" value="true" />
+<xacro:property name="GAZEBO_COMAN_USES_YARP" value="false" />
+<!--
+####################################################
+##
+##  USE XBOT
+####################################################
+-->
+<xacro:property name="GAZEBO_COMAN_USES_XBOT" value="true" />
 <!--
 ####################################################

File: coman_urdf/urdf/config/coman_no_forearms.urdf.xacro (robot description, xacro)
@@ -29,5 +29,12 @@
 ####################################################
 -->
-<xacro:property name="GAZEBO_COMAN_USES_YARP" value="true" />
+<xacro:property name="GAZEBO_COMAN_USES_YARP" value="false" />
+<!--
+####################################################
+##
+##  USE XBOT
+####################################################
+-->
+<xacro:property name="GAZEBO_COMAN_USES_XBOT" value="true" />
 <!--
 ####################################################

File: coman_urdf/urdf/config/coman_softhand.urdf.xacro (robot description, xacro)
@@ -29,5 +29,12 @@
 ####################################################
 -->
-<xacro:property name="GAZEBO_COMAN_USES_YARP" value="true" />
+<xacro:property name="GAZEBO_COMAN_USES_YARP" value="false" />
+<!--
+####################################################
+##
+##  USE XBOT
+####################################################
+-->
+<xacro:property name="GAZEBO_COMAN_USES_XBOT" value="true" />
 <!--
 ####################################################

File: coman_urdf/urdf/config/coman_xtion.urdf.xacro (robot description, xacro)
@@ -33,4 +33,11 @@
 ####################################################
 ##
+##  USE XBOT
+####################################################
+-->
+<xacro:property name="GAZEBO_COMAN_USES_XBOT" value="true" />
+<!--
+####################################################
+##
 ##  Xtion SELECTION
 ##

Commit message: updates and cleaning

File: coman_urdf/urdf/coman_config.urdf.xacro (robot description, xacro)
@@ -34,8 +34,8 @@
 ####################################################
 ##
-##  USE XBOT
+##  USE XBOTCORE
 ####################################################
 -->
-<xacro:property name="GAZEBO_COMAN_USES_XBOT" value="true" />
+<xacro:property name="GAZEBO_COMAN_USES_XBOTCORE" value="true" />
 <!--
 ####################################################

File: coman_urdf/urdf/coman_robot.urdf.xacro (robot description, xacro)
@@ -19,4 +19,7 @@
        <xacro:include filename="$(find coman_urdf)/urdf/gazebo/yarp_control.gazebo.xacro" />
   </xacro:if>
+  <xacro:if value="${GAZEBO_COMAN_USES_XBOTCORE}" >
+  	<xacro:include filename="$(find cogimon_urdf)/urdf/gazebo/xbot_control.gazebo.xacro" />
+  </xacro:if>
   <xacro:include filename="$(find coman_urdf)/urdf/gazebo/force_torque.gazebo.xacro" />
   <!-- XBOT PLUGINS for GAZEBO SIMULATION -->

File: coman_urdf/urdf/gazebo/xbot_control.gazebo.xacro (robot description, xacro)
@@ -2,7 +2,5 @@
 <robot xmlns:xacro="http://ros.org/wiki/xacro">
 <gazebo>
-    <plugin name="xbot_plugin_handler" filename="libGazeboXBotPlugin.so">
-       <path_to_config_file></path_to_config_file>
-    </plugin>
+    <plugin name="xbot_plugin_handler" filename="libGazeboXBotPlugin.so"/>
 </gazebo>
 </robot>

Commit message: set XTION option to true

File: coman_urdf/urdf/coman_config.urdf.xacro (robot description, xacro)
@@ -55,5 +55,5 @@
 #
 -->
-<xacro:property name="GAZEBO_COMAN_USES_XTION" value="false" />
+<xacro:property name="GAZEBO_COMAN_USES_XTION" value="true" />
 <!--
 ####################################################
