Commit message: Modified step width in simple_feet

File: coman_urdf/urdf/feet/simple_feet_DRC_sw1_14/accurate_FT_simple_foot_L_DRC_sw1_14.urdf.xacro (robot description, xacro)
@@ -10,5 +10,5 @@
      <origin xyz="0.03 0 -0.03" rpy="0 0 0" />
      <geometry>
-       <box size="0.2 0.12 0.04" />
+       <box size="0.2 0.1 0.04" />
      </geometry>
      <material name="Cyan">
@@ -19,5 +19,5 @@
      <origin xyz="0.03 0 -0.03" rpy="0 0 0"/>
      <geometry>
-       <box size="0.2 0.12 0.04" />
+       <box size="0.2 0.1 0.04" />
      </geometry>
    </collision>

File: coman_urdf/urdf/feet/simple_feet_DRC_sw1_14/accurate_FT_simple_foot_R_DRC_sw1_14.urdf.xacro (robot description, xacro)
@@ -10,5 +10,5 @@
      <origin xyz="0.03 0 -0.03" rpy="0 0 0" />
      <geometry>
-       <box size="0.2 0.12 0.04" />
+       <box size="0.2 0.1 0.04" />
      </geometry>
      <material name="Cyan">
@@ -19,5 +19,5 @@
      <origin xyz="0.03 0 -0.03" rpy="0 0 0"/>
      <geometry>
-       <box size="0.2 0.12 0.04" />
+       <box size="0.2 0.1 0.04" />
      </geometry>
    </collision>

File: coman_urdf/urdf/feet/simple_feet_DRC_sw1_14/simple_foot_L_DRC_sw1_14.urdf.xacro (robot description, xacro)
@@ -10,5 +10,5 @@
        <origin xyz="0.03 0 -0.09" rpy="0 0 0" />
        <geometry>
-         <box size="0.2 0.12 0.04" />
+         <box size="0.2 0.1 0.04" />
        </geometry>
        <material name="Cyan">
@@ -19,5 +19,5 @@
        <origin xyz="0.03 0 -0.09" rpy="0 0 0"/>
        <geometry>
-         <box size="0.2 0.12 0.04" />
+         <box size="0.2 0.1 0.04" />
        </geometry>
      </collision>

File: coman_urdf/urdf/feet/simple_feet_DRC_sw1_14/simple_foot_R_DRC_sw1_14.urdf.xacro (robot description, xacro)
@@ -10,5 +10,5 @@
      <origin xyz="0.03 0 -0.09" rpy="0 0 0" />
      <geometry>
-       <box size="0.2 0.12 0.04" />
+       <box size="0.2 0.1 0.04" />
      </geometry>
      <material name="Cyan">
@@ -19,5 +19,5 @@
      <origin xyz="0.03 0 -0.09" rpy="0 0 0"/>
      <geometry>
-       <box size="0.2 0.12 0.04" />
+       <box size="0.2 0.1 0.04" />
      </geometry>
    </collision>
