Commit message: Added new config

File: coman_urdf/urdf/config/coman_xtion.urdf.xacro (robot description, xacro)
@@ -1,5 +1,5 @@
 <?xml version="1.0"?>
 <robot xmlns:xacro="http://ros.org/wiki/xacro" name="COMAN">
-<xacro:property name="model_name" value="IIT Coman COGIMON" />
+<xacro:property name="model_name" value="IIT Coman Xtion" />
 <xacro:property name="model_version" value="0.1" />
 <!--
@@ -22,5 +22,5 @@
 -->
 <xacro:property name="GAZEBO_COMAN_USES_FOREARMS" value="true" />
-<xacro:property name="GAZEBO_COMAN_USES_SOFTHANDS" value="false" />
+<xacro:property name="GAZEBO_COMAN_USES_SOFTHANDS" value="true" />
 <!--
 ####################################################
@@ -47,5 +47,5 @@
 #
 -->
-<xacro:property name="GAZEBO_COMAN_USES_XTION" value="false" />
+<xacro:property name="GAZEBO_COMAN_USES_XTION" value="true" />
 <!--
 ####################################################
