Commit message: Hands and forearm meshes filesizes reduced

File: coman_urdf/urdf/forearms/7DOF_forearms_DRC_14/7DOF_forearms_DRC_14.urdf.xacro (robot description, xacro)
@@ -37,7 +37,7 @@
         </inertial>
         <visual>
-          <origin xyz="0 0 ${0.015 + Wrj1_to_FT}" rpy="-1.570796326795 0 1.570796326795"/>
+          <origin xyz="0 0 ${0.015 + Wrj1_to_FT}" rpy="3.14159265359 0 1.570796326795"/>
           <geometry name="LForearm_visual">
-            <mesh filename="package://coman_urdf/meshes/collada/forearms/forearm.dae" scale="0.001 0.001 0.001" />
+            <mesh filename="package://coman_urdf/meshes/collada/forearms/forearm_lowpoly.dae" scale="0.1 0.1 0.1" />
           </geometry>
         </visual>
@@ -120,7 +120,7 @@
         </inertial>
         <visual>
-          <origin xyz="0 0 ${0.015 + Wrj1_to_FT}" rpy="-1.570796326795 0 1.570796326795"/>
+          <origin xyz="0 0 ${0.015 + Wrj1_to_FT}" rpy="3.14159265359 0 1.570796326795"/>
           <geometry name="RForearm_visual">
-            <mesh filename="package://coman_urdf/meshes/collada/forearms/forearm.dae" scale="0.001 0.001 0.001" />
+            <mesh filename="package://coman_urdf/meshes/collada/forearms/forearm_lowpoly.dae" scale="0.1 0.1 0.1" />
           </geometry>
         </visual>

File: coman_urdf/urdf/soft_hand.urdf.xacro (robot description, xacro)
@@ -9,7 +9,7 @@
     </inertial>
     <visual>
-      <origin xyz="0 0.01 -0.04" rpy="0 0 3.14159265359"/>
+      <origin xyz="0.007 0.01 -0.04" rpy="${-3.14159265359/2} 0 ${3.14159265359}"/>
       <geometry name="RSoftHand_visual">
-        <mesh filename="package://coman_urdf/meshes/collada/forearms/R_soft_hand_open.dae" scale="1E-3 1E-3 1E-3" />
+        <mesh filename="package://coman_urdf/meshes/collada/forearms/R_soft_hand_open_lowpoly.dae" scale="0.1 0.1 0.1" />
       </geometry>
    </visual>
@@ -28,7 +28,7 @@
     </inertial>
     <visual>
-      <origin xyz="0.007 -0.012 -0.04" rpy="0 0 ${3.14159265359/2}"/>
+      <origin xyz="0.007 -0.012 -0.04" rpy="${-3.14159265359/2} 0 ${3.14159265359/2}"/>
       <geometry name="LSoftHand_visual">
-        <mesh filename="package://coman_urdf/meshes/collada/forearms/L_soft_hand_open.dae" scale="1E-3 1E-3 1E-3" />
+        <mesh filename="package://coman_urdf/meshes/collada/forearms/L_soft_hand_open_lowpoly.dae" scale="0.1 0.1 0.1" />
       </geometry>
    </visual>
