Commit message: Moved foot 2 cm up

File: coman_urdf/urdf/parts/subparts/simple_feet_DRC_sw1_14/accurate_FT_simple_foot_L_DRC_sw1_14.urdf.xacro (robot description, xacro)
@@ -8,5 +8,5 @@
       </inertial>
     <visual>
-     <origin xyz="0.03 0 -0.03" rpy="0 0 0" />
+     <origin xyz="0.03 0 -0.01" rpy="0 0 0" />
      <geometry>
        <box size="0.2 0.1 0.04" />
@@ -17,5 +17,5 @@
    </visual>
    <collision>
-     <origin xyz="0.03 0 -0.03" rpy="0 0 0"/>
+     <origin xyz="0.03 0 -0.01" rpy="0 0 0"/>
      <geometry>
        <box size="0.2 0.1 0.04" />

File: coman_urdf/urdf/parts/subparts/simple_feet_DRC_sw1_14/accurate_FT_simple_foot_R_DRC_sw1_14.urdf.xacro (robot description, xacro)
@@ -8,5 +8,5 @@
       </inertial>
     <visual>
-     <origin xyz="0.03 0 -0.03" rpy="0 0 0" />
+     <origin xyz="0.03 0 -0.01" rpy="0 0 0" />
      <geometry>
        <box size="0.2 0.1 0.04" />
@@ -17,5 +17,5 @@
    </visual>
    <collision>
-     <origin xyz="0.03 0 -0.03" rpy="0 0 0"/>
+     <origin xyz="0.03 0 -0.01" rpy="0 0 0"/>
      <geometry>
        <box size="0.2 0.1 0.04" />

File: coman_urdf/urdf/parts/subparts/simple_feet_DRC_sw1_14/simple_foot_L_DRC_sw1_14.urdf.xacro (robot description, xacro)
@@ -8,5 +8,5 @@
       </inertial>
       <visual>
-       <origin xyz="0.03 0 -0.09" rpy="0 0 0" />
+       <origin xyz="0.03 0 -0.07" rpy="0 0 0" />
        <geometry>
          <box size="0.2 0.1 0.04" />
@@ -17,5 +17,5 @@
      </visual>
      <collision>
-       <origin xyz="0.03 0 -0.09" rpy="0 0 0"/>
+       <origin xyz="0.03 0 -0.07" rpy="0 0 0"/>
        <geometry>
          <box size="0.2 0.1 0.04" />

File: coman_urdf/urdf/parts/subparts/simple_feet_DRC_sw1_14/simple_foot_R_DRC_sw1_14.urdf.xacro (robot description, xacro)
@@ -8,5 +8,5 @@
       </inertial>
     <visual>
-     <origin xyz="0.03 0 -0.09" rpy="0 0 0" />
+     <origin xyz="0.03 0 -0.07" rpy="0 0 0" />
      <geometry>
        <box size="0.2 0.1 0.04" />
@@ -17,5 +17,5 @@
    </visual>
    <collision>
-     <origin xyz="0.03 0 -0.09" rpy="0 0 0"/>
+     <origin xyz="0.03 0 -0.07" rpy="0 0 0"/>
      <geometry>
        <box size="0.2 0.1 0.04" />

Commit message: CHanged color to simple feet

File: coman_urdf/urdf/parts/subparts/simple_feet_DRC_sw1_14/accurate_FT_simple_foot_L_DRC_sw1_14.urdf.xacro (robot description, xacro)
@@ -12,8 +12,6 @@
        <box size="0.2 0.1 0.04" />
      </geometry>
-     <material name="Cyan">
-       <color rgba="0 1.0 1.0 1.0"/>
-     </material>
-   </visual>
+     <material name="dark_gray"/>
+    </visual>
    <collision>
      <origin xyz="0.03 0 -0.01" rpy="0 0 0"/>

File: coman_urdf/urdf/parts/subparts/simple_feet_DRC_sw1_14/accurate_FT_simple_foot_R_DRC_sw1_14.urdf.xacro (robot description, xacro)
@@ -12,7 +12,5 @@
        <box size="0.2 0.1 0.04" />
      </geometry>
-     <material name="Cyan">
-       <color rgba="0 1.0 1.0 1.0"/>
-     </material>
+     <material name="dark_gray"/>
    </visual>
    <collision>

File: coman_urdf/urdf/parts/subparts/simple_feet_DRC_sw1_14/simple_foot_L_DRC_sw1_14.urdf.xacro (robot description, xacro)
@@ -12,7 +12,5 @@
          <box size="0.2 0.1 0.04" />
        </geometry>
-       <material name="Cyan">
-         <color rgba="0 1.0 1.0 1.0"/>
-       </material>
+       <material name="dark_gray"/>
      </visual>
      <collision>

File: coman_urdf/urdf/parts/subparts/simple_feet_DRC_sw1_14/simple_foot_R_DRC_sw1_14.urdf.xacro (robot description, xacro)
@@ -12,7 +12,5 @@
        <box size="0.2 0.1 0.04" />
      </geometry>
-     <material name="Cyan">
-       <color rgba="0 1.0 1.0 1.0"/>
-     </material>
+     <material name="dark_gray"/>
    </visual>
    <collision>
