Commit message: relaxed joints limits for coman

File: coman_urdf/urdf/parts/7DOF_forearms_DRC_14.urdf.xacro (robot description, xacro)
@@ -149,5 +149,5 @@
     <origin xyz="-0.015 0.0 ${-0.051 - Wrj1_to_FT}" rpy="0 0 0"/>
     <axis xyz="0 0 1" />
-    <limit velocity="4.0" effort="5" lower="-1.5708" upper="1.5708" />
+    <limit effort="200" lower="-3.14" upper="3.14" velocity="4.0"/>
     <dynamics friction="0" damping="0.03"/>
   </joint>
@@ -157,5 +157,5 @@
     <origin xyz="0 0 ${-0.14368 + Wrj1_to_FT}" rpy="0 0 0"/>
     <axis xyz="0 1 0"/>
-    <limit velocity="4.0" effort="5" lower="-0.524" upper="0.524" />
+    <limit effort="200" lower="-3.14" upper="3.14" velocity="4.0"/>
     <dynamics friction="0" damping="0.03"/>
   </joint>
@@ -165,5 +165,5 @@
     <origin xyz="0 0 0.0" rpy="0 0 0"/>
     <axis xyz="1 0 0"/>
-    <limit velocity="4.0" effort="5" lower="-0.785375" upper="1.395" />
+    <limit effort="200" lower="-3.14" upper="3.14" velocity="4.0"/>
     <dynamics friction="0" damping="0.03"/>
   </joint>
@@ -179,5 +179,5 @@
     <origin xyz="-0.015 0.0 ${-0.051 - Wrj1_to_FT}" rpy="0 0 0"/>
     <axis xyz="0 0 1" />
-    <limit velocity="4.0" effort="5" lower="-1.5708" upper="1.5708" />
+    <limit effort="200" lower="-3.14" upper="3.14" velocity="4.0"/>
     <dynamics friction="0" damping="0.03"/>
   </joint>
@@ -187,5 +187,5 @@
     <origin xyz="0 0 ${-0.14368 + Wrj1_to_FT}" rpy="0 0 0"/>
     <axis xyz="0 1 0"/>
-    <limit velocity="4.0" effort="5" lower="-0.524" upper="0.524" />
+    <limit effort="200" lower="-3.14" upper="3.14" velocity="4.0"/>
     <dynamics friction="0" damping="0.03"/>
   </joint>
@@ -195,5 +195,5 @@
     <origin xyz="0 0 0.0" rpy="0 0 0"/>
     <axis xyz="1 0 0"/>
-    <limit velocity="4.0" effort="5" lower="-1.395" upper="0.785375" />
+    <limit effort="200" lower="-3.14" upper="3.14" velocity="4.0"/>
     <dynamics friction="0" damping="0.03"/>
   </joint>

File: coman_urdf/urdf/parts/arms.urdf.xacro (robot description, xacro)
@@ -173,5 +173,5 @@
     <origin xyz="-0.014976503999999998 -0.0825 0.15770847" rpy="0 0 0" />
     <axis xyz="0 1 0" />
-    <limit velocity="4.0" effort="50" lower="-3.4034" upper="1.6581" />
+    <limit effort="200" lower="-3.14" upper="3.14" velocity="4.0"/>
     <dynamics friction="0" damping="3.0"/>
 </joint>
@@ -181,5 +181,5 @@
     <origin xyz="0.0 -0.07329999999999999 0.0" rpy="0 0 0" />
     <axis xyz="1 0 0" />
-    <limit velocity="4.0" effort="50" lower="-2.094" upper="0.31415" />
+    <limit effort="200" lower="-3.14" upper="3.14" velocity="4.0"/>
     <dynamics friction="0" damping="3.0"/>
 </joint>
@@ -189,5 +189,5 @@
     <origin xyz="0.0 0.0 -0.04480846999999999" rpy="0 0 0" />
     <axis xyz="0 0 1" />
-    <limit velocity="4.0" effort="50" lower="-1.5708" upper="1.5708" />
+    <limit effort="200" lower="-3.14" upper="3.14" velocity="4.0"/>
     <dynamics friction="0" damping="3.0"/>
 </joint>
@@ -197,5 +197,5 @@
     <origin xyz="0.015 0.0 -0.13519152999999998" rpy="0 0 0" />
     <axis xyz="0 1 0" />
-    <limit velocity="4.0" effort="50" lower="-2.3562" upper="0.0" />
+    <limit effort="200" lower="-3.14" upper="3.14" velocity="4.0"/>
     <dynamics friction="0" damping="3.0"/>
   </joint>
@@ -206,5 +206,5 @@
     <origin xyz="-0.014976503999999998 0.0825 0.15770847" rpy="0 0 0" />
     <axis xyz="0 1 0" />
-    <limit velocity="4.0" effort="50" lower="-3.4034" upper="1.6581" />
+    <limit effort="200" lower="-3.14" upper="3.14" velocity="4.0"/>
     <dynamics friction="0" damping="3.0"/>
 </joint>
@@ -214,5 +214,5 @@
     <origin xyz="0.0 0.07329999999999999 0.0" rpy="0 0 0" />
     <axis xyz="1 0 0" />
-    <limit velocity="4.0" effort="50" lower="-0.31415" upper="2.094" />
+    <limit effort="200" lower="-3.14" upper="3.14" velocity="4.0"/>
     <dynamics friction="0" damping="3.0"/>
 </joint>
@@ -222,5 +222,5 @@
     <origin xyz="0.0 0.0 -0.04480846999999999" rpy="0 0 0" />
     <axis xyz="0 0 1" />
-    <limit velocity="4.0" effort="50" lower="-1.5708" upper="1.5708" />
+    <limit effort="200" lower="-3.14" upper="3.14" velocity="4.0"/>
     <dynamics friction="0" damping="3.0"/>
 </joint>
@@ -230,5 +230,5 @@
     <origin xyz="0.015 0.0 -0.13519152999999998" rpy="0 0 0" />
     <axis xyz="0 1 0" />
-    <limit velocity="4.0" effort="50" lower="-2.3562" upper="0.0" />
+    <limit effort="200" lower="-3.14" upper="3.14" velocity="4.0"/>
     <dynamics friction="0" damping="3.0"/>
   </joint>

File: coman_urdf/urdf/parts/legs.urdf.xacro (robot description, xacro)
@@ -260,5 +260,5 @@
     <origin xyz="0.0 -0.023 0.0" rpy="0 0 0" />
     <axis xyz="0 1 0" />
-    <limit velocity="4.0" effort="50" lower="-1.9199" upper="0.7854" />
+    <limit effort="200" lower="-3.14" upper="3.14" velocity="4.0"/>
     <dynamics friction="0" damping="3.0"/>
   </joint>
@@ -268,5 +268,5 @@
     <origin xyz="0.0 -0.0496 0.0" rpy="0 0 0" />
     <axis xyz="1 0 0" />
-    <limit velocity="4.0" effort="50" lower="-1.0472" upper="0.4363" />
+    <limit effort="200" lower="-3.14" upper="3.14" velocity="4.0"/>
     <dynamics friction="0" damping="3.0"/>
   </joint>
@@ -276,5 +276,5 @@
     <origin xyz="0.0 0.0 -0.1024" rpy="0 0 0" />
     <axis xyz="0 0 1" />
-    <limit velocity="4.0" effort="50" lower="-0.8727" upper="0.8727" />
+    <limit effort="200" lower="-3.14" upper="3.14" velocity="4.0"/>
     <dynamics friction="0" damping="3.0"/>
   </joint>
@@ -284,5 +284,5 @@
     <origin xyz="0.0 0.0 -0.1234" rpy="0 0 0" />
     <axis xyz="0 1 0" />
-    <limit velocity="4.0" effort="50" lower="-0.1745" upper="1.9199" />
+    <limit effort="200" lower="-3.14" upper="3.14" velocity="4.0"/>
     <dynamics friction="0" damping="3.0"/>
   </joint>
@@ -292,5 +292,5 @@
     <origin xyz="0.0 0.0 -0.201" rpy="0 0 0" />
     <axis xyz="1 0 0" />
-    <limit velocity="4.0" effort="50" lower="-0.6109" upper="0.6109" />
+    <limit effort="200" lower="-3.14" upper="3.14" velocity="4.0"/>
     <dynamics friction="0" damping="3.0"/>
   </joint>
@@ -301,5 +301,5 @@
       <origin xyz="0.0 0.0 0.0" rpy="0 0 0" />
       <axis xyz="0 1 0" />
-      <limit velocity="4.0" effort="50" lower="-1.2217" upper="1.2217" />
+      <limit effort="200" lower="-3.14" upper="3.14" velocity="4.0"/>
       <dynamics friction="0" damping="3.0"/>
     </joint>
@@ -311,5 +311,5 @@
       <origin xyz="0.0 0.0 0.0" rpy="0 0 0" />
       <axis xyz="0 1 0" />
-      <limit velocity="4.0" effort="50" lower="-1.2217" upper="1.2217" />
+      <limit effort="200" lower="-3.14" upper="3.14" velocity="4.0"/>
       <dynamics friction="0" damping="3.0"/>
     </joint>
@@ -329,5 +329,5 @@
     <origin xyz="0.0 0.023 0.0" rpy="0 0 0" />
     <axis xyz="0 1 0" />
-    <limit velocity="4.0" effort="50" lower="-1.9199" upper="0.7854" />
+    <limit effort="200" lower="-3.14" upper="3.14" velocity="4.0"/>
     <dynamics friction="0" damping="3.0"/>
   </joint>
@@ -337,5 +337,5 @@
     <origin xyz="0.0 0.0496 0.0" rpy="0 0 0" />
     <axis xyz="1 0 0" />
-    <limit velocity="4.0" effort="50" lower="-0.4363" upper="1.0472" />
+    <limit effort="200" lower="-3.14" upper="3.14" velocity="4.0"/>
     <dynamics friction="0" damping="3.0"/>
   </joint>
@@ -345,5 +345,5 @@
     <origin xyz="0.0 0.0 -0.1024" rpy="0 0 0" />
     <axis xyz="0 0 1" />
-    <limit velocity="4.0" effort="50" lower="-0.8727" upper="0.8727" />
+    <limit effort="200" lower="-3.14" upper="3.14" velocity="4.0"/>
     <dynamics friction="0" damping="3.0"/>
   </joint>
@@ -353,5 +353,5 @@
     <origin xyz="0.0 0.0 -0.1234" rpy="0 0 0" />
     <axis xyz="0 1 0" />
-    <limit velocity="4.0" effort="50" lower="-0.1745" upper="1.9199" />
+    <limit effort="200" lower="-3.14" upper="3.14" velocity="4.0"/>
     <dynamics friction="0" damping="3.0"/>
   </joint>
@@ -361,5 +361,5 @@
     <origin xyz="0.0 0.0 -0.201" rpy="0 0 0" />
     <axis xyz="1 0 0" />
-    <limit velocity="4.0" effort="50" lower="-0.6109" upper="0.6109" />
+    <limit effort="200" lower="-3.14" upper="3.14" velocity="4.0"/>
     <dynamics friction="0" damping="3.0"/>
   </joint>
@@ -370,5 +370,5 @@
       <origin xyz="0.0 0.0 0.0" rpy="0 0 0" />
       <axis xyz="0 1 0" />
-      <limit velocity="4.0" effort="50" lower="-1.2217" upper="1.2217" />
+      <limit effort="200" lower="-3.14" upper="3.14" velocity="4.0"/>
       <dynamics friction="0" damping="3.0"/>
     </joint>
@@ -380,5 +380,5 @@
       <origin xyz="0.0 0.0 0.0" rpy="0 0 0" />
       <axis xyz="0 1 0" />
-      <limit velocity="4.0" effort="50" lower="-1.2217" upper="1.2217" />
+      <limit effort="200" lower="-3.14" upper="3.14" velocity="4.0"/>
       <dynamics friction="0" damping="3.0"/>
     </joint>

File: coman_urdf/urdf/parts/soft_hand.urdf.xacro (robot description, xacro)
@@ -108,5 +108,5 @@
         <origin xyz="0 0 -0.04" rpy="0 0 0"/>
         <axis xyz="1 0 0" />
-        <limit velocity="4.0" effort="5" lower="0.0" upper="1.57075" />
+        <limit effort="200" lower="-3.14" upper="3.14" velocity="4.0"/>
         <dynamics friction="0" damping="3.0"/>
 </joint>
@@ -116,5 +116,5 @@
         <origin xyz="0 0 -0.04" rpy="0 0 0"/>
         <axis xyz="-1 0 0" />
-        <limit velocity="4.0" effort="5" lower="0.0" upper="1.57075" />
+        <limit effort="200" lower="-3.14" upper="3.14" velocity="4.0"/>
         <dynamics friction="0" damping="3.0"/>
 </joint>

File: coman_urdf/urdf/parts/torso.urdf.xacro (robot description, xacro)
@@ -110,5 +110,5 @@
     <origin xyz="0.020281504 0 0.11912053" rpy="0 0 0" />
     <axis xyz="${cos_20} 0 ${sin_20}" />
-    <limit velocity="4.0" effort="50" lower="-0.5236" upper="0.5235" />
+    <limit effort="200" lower="-3.14" upper="3.14" velocity="4.0"/>
     <!-- dynamics friction="0" damping="0.3"/ -->
     <dynamics friction="0" damping="3.0"/>
@@ -119,5 +119,5 @@
     <origin xyz="0 0 0" rpy="0 0 0" />
     <axis xyz="0 1 0" />
-    <limit velocity="4.0" effort="50" lower="-0.3491" upper="0.8727" />
+    <limit effort="200" lower="-3.14" upper="3.14" velocity="4.0"/>
     <dynamics friction="0" damping="3.0"/>
   </joint>
@@ -127,5 +127,5 @@
     <origin xyz="0 0 0.04749999" rpy="0 0 0" />
     <axis xyz="0 0 1" />
-    <limit velocity="4.0" effort="50" lower="-1.3963" upper="1.3962" />
+    <limit effort="200" lower="-3.14" upper="3.14" velocity="4.0"/>
     <dynamics friction="0" damping="3.0"/>
   </joint>
