Commit message: Added smaller meshes for torso.

File: coman_urdf/urdf/parts/torso.urdf.xacro (robot description, xacro)
@@ -19,5 +19,5 @@
       <material name="dark_grey"/>
       <geometry name="DWL_visual">
-        <mesh filename="package://coman_urdf/meshes/collada/torso1.stl" scale="${SF} ${SF} ${SF}" />
+        <mesh filename="package://coman_urdf/meshes/Torso1.STL" scale="${SF} ${SF} ${SF}" />
       </geometry>
     </visual>
@@ -25,5 +25,5 @@
       <origin xyz="-0.020281504 0 -0.63912053" rpy="0 0 ${PI}"/>
       <geometry name="DWL_collision">
-        <mesh filename="package://coman_urdf/meshes/collada/simple/simple_asm0001_collada_09_prt.stl" scale="${SF} ${SF} ${SF}" />
+        <mesh filename="package://coman_urdf/meshes/simple/Torso1.STL" scale="${SF} ${SF} ${SF}" />
       </geometry>
     </collision>
@@ -39,5 +39,5 @@
       <material name="dark_grey"/>
       <geometry name="DWS_visual">
-        <mesh filename="package://coman_urdf/meshes/collada/torso2.stl" scale="${SF} ${SF} ${SF}" />
+        <mesh filename="package://coman_urdf/meshes/Torso2.STL" scale="${SF} ${SF} ${SF}" />
       </geometry>
     </visual>
@@ -45,5 +45,5 @@
       <origin xyz="-0.020281504 0 -0.63912053" rpy="0 0 ${PI}"/>
       <geometry name="DWS_collision">
-        <mesh filename="package://coman_urdf/meshes/collada/simple/simple_asm0001_collada_08_prt.stl" scale="${SF} ${SF} ${SF}" />
+        <mesh filename="package://coman_urdf/meshes/simple/Torso2.STL" scale="${SF} ${SF} ${SF}" />
       </geometry>
     </collision>
@@ -59,5 +59,5 @@
       <material name="red"/>
       <geometry name="DWYTorso_visual">
-        <mesh filename="package://coman_urdf/meshes/collada/torso3.stl" scale="${SF} ${SF} ${SF}" />
+        <mesh filename="package://coman_urdf/meshes/Torso3.STL" scale="${SF} ${SF} ${SF}" />
       </geometry>
     </visual>
@@ -65,5 +65,5 @@
       <origin xyz="-0.020281504 0.0 -0.68662053" rpy="0 0 ${PI}"/>
       <geometry name="DWYTorso_collision">
-        <mesh filename="package://coman_urdf/meshes/collada/simple/simple_asm0001_collada_10_prt.stl" scale="${SF} ${SF} ${SF}" />
+        <mesh filename="package://coman_urdf/meshes/simple/Torso3.STL" scale="${SF} ${SF} ${SF}" />
       </geometry>
     </collision>
