Commit message: Simplified meshes for arms.

File: coman_urdf/urdf/parts/arms.urdf.xacro (robot description, xacro)
@@ -15,5 +15,5 @@
       <material name="dark_grey"/>
       <geometry name="RShp_visual">
-        <mesh filename="package://coman_urdf/meshes/collada/rarm0.stl" scale="${SF} ${SF} ${SF}" />
+        <mesh filename="package://coman_urdf/meshes/Arm0.STL" scale="${SF} ${SF} ${SF}" />
       </geometry>
     </visual>
@@ -21,5 +21,5 @@
       <origin xyz="-0.005305 0.0825 -0.844329" rpy="0 0 ${PI}"/>
       <geometry name="RShp_collision">
-        <mesh filename="package://coman_urdf/meshes/collada/simple/simple_asm0001_collada_24_prt.stl" scale="${SF} ${SF} ${SF}" />
+        <mesh filename="package://coman_urdf/meshes/simple/Arm0.STL" scale="${SF} ${SF} ${SF}" />
       </geometry>
     </collision>
@@ -35,5 +35,5 @@
       <material name="dark_grey"/>
       <geometry name="RShr_visual">
-        <mesh filename="package://coman_urdf/meshes/collada/rarm1.stl" scale="${SF} ${SF} ${SF}" />
+        <mesh filename="package://coman_urdf/meshes/Arm1.STL" scale="${SF} ${SF} ${SF}" />
       </geometry>
     </visual>
@@ -41,5 +41,5 @@
       <origin xyz="-0.005305 0.1558 -0.844329" rpy="0 0 ${PI}"/>
       <geometry name="RShr_collision">
-        <mesh filename="package://coman_urdf/meshes/collada/simple/simple_asm0001_collada_23_prt.stl" scale="${SF} ${SF} ${SF}" />
+        <mesh filename="package://coman_urdf/meshes/simple/Arm1.STL" scale="${SF} ${SF} ${SF}" />
       </geometry>
     </collision>
@@ -55,5 +55,5 @@
       <material name="dark_grey"/>
       <geometry name="RShy_visual">
-        <mesh filename="package://coman_urdf/meshes/collada/rarm2.stl" scale="${SF} ${SF} ${SF}" />
+        <mesh filename="package://coman_urdf/meshes/Arm2.STL" scale="${SF} ${SF} ${SF}" />
       </geometry>
     </visual>
@@ -61,5 +61,5 @@
       <origin xyz="-0.005305 0.1558 -0.79952053" rpy="0 0 ${PI}"/>
       <geometry name="RShy_collision">
-        <mesh filename="package://coman_urdf/meshes/collada/simple/simple_asm0001_collada_22_prt.stl" scale="${SF} ${SF} ${SF}" />
+        <mesh filename="package://coman_urdf/meshes/simple/Arm2.STL" scale="${SF} ${SF} ${SF}" />
       </geometry>
     </collision>
@@ -75,5 +75,5 @@
           <material name="dark_grey"/>
           <geometry name="RElb_visual">
-            <mesh filename="package://coman_urdf/meshes/collada/forearms/elbow.stl" scale="1.0 1.0 1.0" />
+            <mesh filename="package://coman_urdf/meshes/Elbow.STL" scale="1.0 1.0 1.0" />
           </geometry>
         </visual>
@@ -81,5 +81,5 @@
           <origin xyz="0 0 0" rpy="-1.570796326795 1.570796326795 0"/>
           <geometry name="RElb_collision">
-            <mesh filename="package://coman_urdf/meshes/collada/simple/forearms/elbow.stl" scale="1.0 1.0 1.0" />
+            <mesh filename="package://coman_urdf/meshes/simple/Elbow.STL" scale="1.0 1.0 1.0" />
           </geometry>
         </collision>
@@ -96,5 +96,5 @@
       <material name="dark_grey"/>
       <geometry name="LShp_visual">
-        <mesh filename="package://coman_urdf/meshes/collada/larm0.stl" scale="${SF} ${SF} ${SF}" />
+        <mesh filename="package://coman_urdf/meshes/Arm0.STL" scale="${SF} -${SF} ${SF}" />
       </geometry>
     </visual>
@@ -102,5 +102,5 @@
       <origin xyz="-0.005305 -0.0825 -0.844329" rpy="0 0 ${PI}"/>
       <geometry name="LShp_collision">
-        <mesh filename="package://coman_urdf/meshes/collada/simple/simple_asm0001_collada_14_prt.stl" scale="${SF} ${SF} ${SF}" />
+        <mesh filename="package://coman_urdf/meshes/simple/Arm0.STL" scale="${SF} -${SF} ${SF}" />
       </geometry>
     </collision>
@@ -116,5 +116,5 @@
       <material name="dark_grey"/>
       <geometry name="LShr_visual">
-        <mesh filename="package://coman_urdf/meshes/collada/larm1.stl" scale="${SF} ${SF} ${SF}" />
+        <mesh filename="package://coman_urdf/meshes/Arm1.STL" scale="${SF} -${SF} ${SF}" />
       </geometry>
     </visual>
@@ -122,5 +122,5 @@
       <origin xyz="-0.005305 -0.1558 -0.844329" rpy="0 0 ${PI}"/>
       <geometry name="LShr_collision">
-        <mesh filename="package://coman_urdf/meshes/collada/simple/simple_asm0001_collada_13_prt.stl" scale="${SF} ${SF} ${SF}" />
+        <mesh filename="package://coman_urdf/meshes/simple/Arm1.STL" scale="${SF} -${SF} ${SF}" />
       </geometry>
     </collision>
@@ -136,5 +136,5 @@
       <material name="dark_grey"/>
       <geometry name="LShy_visual">
-        <mesh filename="package://coman_urdf/meshes/collada/larm2.stl" scale="${SF} ${SF} ${SF}" />
+        <mesh filename="package://coman_urdf/meshes/Arm2.STL" scale="${SF} -${SF} ${SF}" />
       </geometry>
     </visual>
@@ -142,5 +142,5 @@
       <origin xyz="-0.005305 -0.1558 -0.79952053" rpy="0 0 ${PI}"/>
       <geometry name="LShy_collision">
-        <mesh filename="package://coman_urdf/meshes/collada/simple/simple_asm0001_collada_12_prt.stl" scale="${SF} ${SF} ${SF}" />
+        <mesh filename="package://coman_urdf/meshes/simple/Arm2.STL" scale="${SF} -${SF} ${SF}" />
       </geometry>
     </collision>
@@ -156,5 +156,5 @@
           <material name="dark_grey"/>
           <geometry name="LElb_visual">
-            <mesh filename="package://coman_urdf/meshes/collada/forearms/elbow.stl" scale="1.0 1.0 1.0" />
+            <mesh filename="package://coman_urdf/meshes/Elbow.STL" scale="1.0 1.0 1.0" />
           </geometry>
         </visual>
@@ -162,5 +162,5 @@
           <origin xyz="0 0 0" rpy="-1.570796326795 1.570796326795 0"/>
           <geometry name="LElb_collision">
-            <mesh filename="package://coman_urdf/meshes/collada/simple/forearms/elbow.stl" scale="1.0 1.0 1.0" />
+            <mesh filename="package://coman_urdf/meshes/simple/Elbow.STL" scale="1.0 1.0 1.0" />
           </geometry>
         </collision>
