Commit message: Simplified meshes for forearms

File: coman_urdf/urdf/parts/forearms.urdf.xacro (robot description, xacro)
@@ -21,5 +21,5 @@
           <material name="dark_grey"/>
           <geometry name="LForearm_visual">
-            <mesh filename="package://coman_urdf/meshes/collada/forearms/forearm0.stl" scale="0.1 0.1 0.1" />
+            <mesh filename="package://coman_urdf/meshes/Forearm0.STL" scale="0.1 0.1 0.1" />
           </geometry>
         </visual>
@@ -27,5 +27,5 @@
           <origin xyz="0 0 ${0.015 + Wrj1_to_FT}" rpy="0 3.14159265359 1.570796326795"/>
           <geometry name="LForearm_collision">
-            <mesh filename="package://coman_urdf/meshes/collada/simple/forearms/forearm.stl" scale="1.0 1.0 1.0" />
+            <mesh filename="package://coman_urdf/meshes/simple/Forearm0.STL" scale="1.0 1.0 1.0" />
           </geometry>
         </collision>
@@ -43,5 +43,5 @@
           <material name="grey"/>
           <geometry name="LWrMot2_visual">
-            <mesh filename="package://coman_urdf/meshes/collada/forearms/forearm1.stl" scale="0.001 0.001 0.001" />
+            <mesh filename="package://coman_urdf/meshes/Forearm1.STL" scale="0.001 0.001 0.001" />
           </geometry>
         </visual>
@@ -49,5 +49,5 @@
           <origin xyz="0.025 0 0" rpy="0 1.570796326795 3.14159265359"/>
           <geometry name="LWrMot2_collision">
-            <mesh filename="package://coman_urdf/meshes/collada/simple/forearms/simple_fa_asm_3_right_sw0001.stl" scale="0.001 0.001 0.001" />
+            <mesh filename="package://coman_urdf/meshes/simple/Forearm1.STL" scale="0.001 0.001 0.001" />
           </geometry>
         </collision>
@@ -65,5 +65,5 @@
           <material name="grey"/>
           <geometry name="LWrMot3_visual">
-            <mesh filename="package://coman_urdf/meshes/collada/forearms/forearm2.stl" scale="0.001 0.001 0.001" />
+            <mesh filename="package://coman_urdf/meshes/Forearm2.STL" scale="0.001 0.001 0.001" />
           </geometry>
         </visual>
@@ -71,5 +71,5 @@
           <origin xyz="0.025 -0.012 -0.02" rpy="0 3.14159265359 1.570796326795"/>
           <geometry name="LWrMot3_collision">
-            <mesh filename="package://coman_urdf/meshes/collada/simple/forearms/simple_fa_hand_interface_rig_sw0001.stl" scale="0.001 0.001 0.001" />
+            <mesh filename="package://coman_urdf/meshes/simple/Forearm2.STL" scale="0.001 0.001 0.001" />
           </geometry>
         </collision>
@@ -88,5 +88,5 @@
           <material name="dark_grey"/>
           <geometry name="RForearm_visual">
-            <mesh filename="package://coman_urdf/meshes/collada/forearms/forearm0.stl" scale="0.1 0.1 0.1" />
+            <mesh filename="package://coman_urdf/meshes/Forearm0.STL" scale="0.1 0.1 0.1" />
           </geometry>
         </visual>
@@ -94,5 +94,5 @@
           <origin xyz="0 0 ${0.015 + Wrj1_to_FT}" rpy="0 3.14159265359 1.570796326795"/>
           <geometry name="RForearm_collision">
-            <mesh filename="package://coman_urdf/meshes/collada/simple/forearms/forearm.stl" scale="1.0 1.0 1.0" />
+            <mesh filename="package://coman_urdf/meshes/simple/Forearm0.STL" scale="1.0 1.0 1.0" />
           </geometry>
         </collision>
@@ -110,5 +110,5 @@
           <material name="grey"/>
           <geometry name="RWrMot2_visual">
-            <mesh filename="package://coman_urdf/meshes/collada/forearms/forearm1.stl" scale="0.001 0.001 0.001" />
+            <mesh filename="package://coman_urdf/meshes/Forearm1.STL" scale="0.001 0.001 0.001" />
           </geometry>
         </visual>
@@ -116,5 +116,5 @@
           <origin xyz="0.025 0 0" rpy="0 1.570796326795 3.14159265359"/>
           <geometry name="RWrMot2_collision">
-            <mesh filename="package://coman_urdf/meshes/collada/simple/forearms/simple_fa_asm_3_right_sw0001.stl" scale="0.001 0.001 0.001" />
+            <mesh filename="package://coman_urdf/meshes/simple/Forearm1.STL" scale="0.001 0.001 0.001" />
           </geometry>
         </collision>
@@ -132,5 +132,5 @@
           <material name="grey"/>
           <geometry name="RWrMot3_visual">
-            <mesh filename="package://coman_urdf/meshes/collada/forearms/forearm2.stl" scale="0.001 0.001 0.001" />
+            <mesh filename="package://coman_urdf/meshes/Forearm2.STL" scale="0.001 0.001 0.001" />
           </geometry>
         </visual>
@@ -138,5 +138,5 @@
           <origin xyz="0.025 -0.012 -0.02" rpy="0 3.14159265359 1.570796326795"/>
           <geometry name="RWrMot3_collision">
-            <mesh filename="package://coman_urdf/meshes/collada/simple/forearms/simple_fa_hand_interface_rig_sw0001.stl" scale="0.001 0.001 0.001" />
+            <mesh filename="package://coman_urdf/meshes/simple/Forearm2.STL" scale="0.001 0.001 0.001" />
           </geometry>
         </collision>
