Commit message: Added some variables in no_forearms.urdf.xacro

File: coman_urdf/urdf/parts/no_forearms.urdf.xacro (robot description, xacro)
@@ -2,4 +2,7 @@
 <robot xmlns:xacro="http://ros.org/wiki/xacro">
 <xacro:property name="Wrj1_to_FT" value="0.0568" />
+<xacro:property name="PI" value="3.14159265359" />
+<xacro:property name="PI_2" value="1.57079632679" />
+<xacro:property name="SF" value="0.03937" /> <!-- Scale factor for meshes -->
 <!-- ***********LINKS*********** -->
 <!-- ***********LEFT FOREARM***********-->
@@ -11,13 +14,13 @@
       </inertial>
       <visual>
-        <origin xyz="-0.0055 -0.1558 -0.6175" rpy="0 0 3.14159265359"/>
+        <origin xyz="-0.0055 -0.1558 -0.6175" rpy="0 0 ${PI}"/>
         <geometry name="LForearm_visual">
-          <mesh filename="package://coman_urdf/meshes/collada/forearm_old.dae" scale="0.03937 0.03937 0.03937" />
+          <mesh filename="package://coman_urdf/meshes/collada/forearm_old.dae" scale="${SF} ${SF} ${SF}" />
         </geometry>
       </visual>
       <collision>
-        <origin xyz="-0.0055 -0.1558 -0.6175" rpy="0 0 3.14159265359"/>
+        <origin xyz="-0.0055 -0.1558 -0.6175" rpy="0 0 ${PI}"/>
         <geometry name="LForearm_collision">
-          <mesh filename="package://coman_urdf/meshes/collada/simple/forearm_old.dae" scale="0.03937 0.03937 0.03937" />
+          <mesh filename="package://coman_urdf/meshes/collada/simple/forearm_old.dae" scale="${SF} ${SF} ${SF}" />
         </geometry>
       </collision>
@@ -31,13 +34,13 @@
     </inertial>
       <visual>
-        <origin xyz="-0.0055 -0.1558 -0.6175" rpy="0 0 3.14159265359"/>
+        <origin xyz="-0.0055 -0.1558 -0.6175" rpy="0 0 ${PI}"/>
         <geometry name="RForearm_visual">
-          <mesh filename="package://coman_urdf/meshes/collada/forearm_old.dae" scale="0.03937 0.03937 0.03937" />
+          <mesh filename="package://coman_urdf/meshes/collada/forearm_old.dae" scale="${SF} ${SF} ${SF}" />
         </geometry>
       </visual>
       <collision>
-        <origin xyz="-0.0055 -0.1558 -0.6175" rpy="0 0 3.14159265359"/>
+        <origin xyz="-0.0055 -0.1558 -0.6175" rpy="0 0 ${PI}"/>
         <geometry name="RForearm_collision">
-          <mesh filename="package://coman_urdf/meshes/collada/simple/forearm_old.dae" scale="0.03937 0.03937 0.03937" />
+          <mesh filename="package://coman_urdf/meshes/collada/simple/forearm_old.dae" scale="${SF} ${SF} ${SF}" />
         </geometry>
       </collision>

Commit message: Simplified meshes for old forearms

File: coman_urdf/urdf/parts/no_forearms.urdf.xacro (robot description, xacro)
@@ -17,5 +17,5 @@
         <material name="dark_grey"/>
         <geometry name="LForearm_visual">
-          <mesh filename="package://coman_urdf/meshes/collada/forearm_old.stl" scale="${SF} ${SF} ${SF}" />
+          <mesh filename="package://coman_urdf/meshes/ForearmOld.STL" scale="${SF} ${SF} ${SF}" />
         </geometry>
       </visual>
@@ -23,5 +23,5 @@
         <origin xyz="-0.0055 -0.1558 -0.6175" rpy="0 0 ${PI}"/>
         <geometry name="LForearm_collision">
-          <mesh filename="package://coman_urdf/meshes/collada/simple/forearm_old.dae" scale="${SF} ${SF} ${SF}" />
+          <mesh filename="package://coman_urdf/meshes/simple/ForearmOld.STL" scale="${SF} ${SF} ${SF}" />
         </geometry>
       </collision>
@@ -38,5 +38,5 @@
         <material name="dark_grey"/>
         <geometry name="RForearm_visual">
-          <mesh filename="package://coman_urdf/meshes/collada/forearm_old.stl" scale="${SF} ${SF} ${SF}" />
+          <mesh filename="package://coman_urdf/meshes/ForearmOld.STL" scale="${SF} ${SF} ${SF}" />
         </geometry>
       </visual>
@@ -44,5 +44,5 @@
         <origin xyz="-0.0055 -0.1558 -0.6175" rpy="0 0 ${PI}"/>
         <geometry name="RForearm_collision">
-          <mesh filename="package://coman_urdf/meshes/collada/simple/forearm_old.dae" scale="${SF} ${SF} ${SF}" />
+          <mesh filename="package://coman_urdf/meshes/simple/ForearmOld.STL" scale="${SF} ${SF} ${SF}" />
         </geometry>
       </collision>
