Commit message: changed axis of rotation of fake left hand, changed PID gains

File: coman_urdf/urdf/parts/soft_hand.urdf.xacro (robot description, xacro)
@@ -113,6 +113,6 @@
         <child link="LSoftHand"/>
         <origin xyz="0 0 -0.04" rpy="0 0 0"/>
-        <axis xyz="1 0 0" />
-        <limit velocity="4.0" effort="5" lower="-1.57075" upper="0.0" />
+        <axis xyz="-1 0 0" />
+        <limit velocity="4.0" effort="5" lower="0.0" upper="1.57075" />
         <dynamics friction="0" damping="3.0"/>
 </joint>

Commit message: pisa iit soft hand articulated included

File: coman_urdf/urdf/parts/soft_hand.urdf.xacro (robot description, xacro)
@@ -2,6 +2,16 @@
 <robot xmlns:xacro="http://ros.org/wiki/xacro" name="SoftHand">
 <xacro:if value="${GAZEBO_COMAN_USES_SOFTHANDS_DRC_sw1_14}">
-<!-- LINKS -->
-<link name="RSoftHand">
+  <xacro:include filename="$(find soft_hand_description)/model/soft_hand.urdf.xacro"/>
+  <!-- RIGHT HAND -->
+  <xacro:soft_hand parent="RWrMot3" name="RSoftHand" withAdaptiveTransmission="true" useMimicTag="true" left="false">
+    <origin xyz="0.0 0.0 -0.038" rpy="3.141592 0 1.5707"/>
+  </xacro:soft_hand>
+  <!-- LEFT HAND -->
+  <xacro:soft_hand parent="LWrMot3" name="LSoftHand" withAdaptiveTransmission="true" useMimicTag="true" left="true">
+    <origin xyz="0.0 -0.0 -0.038" rpy="3.141592 0 -1.5707"/>
+  </xacro:soft_hand>
+  <!-- Keeping all as backup -->
+  <!-- LINKS
+  <link name="RSoftHand">
     <inertial>
       <origin xyz="0 0 0" rpy="0 0 0"/>
@@ -15,11 +25,11 @@
         <mesh filename="package://coman_urdf/meshes/collada/forearms/Rsofthand_fix.stl" scale="0.1 0.1 0.1" />
       </geometry>
-   </visual>
-   <collision>
+    </visual>
+    <collision>
       <origin xyz="0 0.01 -0.04" rpy="0 0 3.14159265359"/>
       <geometry name="RSoftHand_collision">
         <mesh filename="package://coman_urdf/meshes/collada/simple/forearms/R_soft_hand_open.stl" scale="1E-3 1E-3 1E-3" />
       </geometry>
-   </collision>
+    </collision>
   </link>
   <link name="LSoftHand">
@@ -43,5 +53,6 @@
    </collision>
   </link>
-<!-- JOINTS -->
+  -->
+  <!-- JOINTS
   <joint name="r_handj" type="fixed">
         <parent link="RWrMot3"/>
@@ -54,4 +65,5 @@
         <origin xyz="0 0 -0.07" rpy="0 0 0"/>
   </joint>
+  -->
 </xacro:if>
 <xacro:unless value="${GAZEBO_COMAN_USES_SOFTHANDS_DRC_sw1_14}">

Commit message: changed hand shape

File: coman_urdf/urdf/parts/soft_hand.urdf.xacro (robot description, xacro)
@@ -67,5 +67,5 @@
      <origin xyz="0 0 0" rpy="0 0 0" />
      <geometry>
-        <box size="0.07 0.07 0.07" />
+        <sphere radius="0.03"/>
      </geometry>
      <material name="Cyan">
@@ -76,5 +76,5 @@
      <origin xyz="0 0 0" rpy="0 0 0"/>
      <geometry>
-       <box size="0.07 0.07 0.07" />
+       <sphere radius="0.03"/>
      </geometry>
    </collision>
@@ -89,5 +89,5 @@
      <origin xyz="0 0 0" rpy="0 0 0" />
      <geometry>
-        <box size="0.07 0.07 0.07" />
+        <sphere radius="0.03"/>
      </geometry>
      <material name="Cyan">
@@ -98,5 +98,5 @@
      <origin xyz="0 0 0" rpy="0 0 0"/>
      <geometry>
-       <box size="0.07 0.07 0.07" />
+       <sphere radius="0.03"/>
      </geometry>
    </collision>

Commit message: Added simplified meshes for sofhand.

File: coman_urdf/urdf/parts/soft_hand.urdf.xacro (robot description, xacro)
@@ -13,5 +13,5 @@
       <material name="dark_grey"/>
       <geometry name="RSoftHand_visual">
-        <mesh filename="package://coman_urdf/meshes/collada/forearms/Rsofthand_fix.stl" scale="0.1 0.1 0.1" />
+        <mesh filename="package://coman_urdf/meshes/SoftHandOpen.STL" scale="0.1 0.1 0.1" />
       </geometry>
    </visual>
@@ -19,5 +19,5 @@
       <origin xyz="0 0.01 -0.04" rpy="0 0 3.14159265359"/>
       <geometry name="RSoftHand_collision">
-        <mesh filename="package://coman_urdf/meshes/collada/simple/forearms/R_soft_hand_open.stl" scale="1E-3 1E-3 1E-3" />
+        <mesh filename="package://coman_urdf/meshes/simple/SoftHandOpen.STL" scale="1E-3 1E-3 1E-3" />
       </geometry>
    </collision>
@@ -30,14 +30,14 @@
     </inertial>
     <visual>
-      <origin xyz="0.007 -0.012 -0.04" rpy="${-3.14159265359/2} 0 ${3.14159265359/2}"/>
+      <origin xyz="0.007 -0.01 -0.04" rpy="${-3.14159265359/2} 0 0"/>
       <material name="dark_grey"/>
       <geometry name="LSoftHand_visual">
-        <mesh filename="package://coman_urdf/meshes/collada/forearms/Lsofthand_fix.stl" scale="0.1 0.1 0.1" />
+        <mesh filename="package://coman_urdf/meshes/SoftHandOpen.STL" scale="-0.1 0.1 0.1" />
       </geometry>
    </visual>
    <collision>
-     <origin xyz="0.007 -0.012 -0.04" rpy="0 0 ${3.14159265359/2}"/>
+     <origin xyz="0.007 -0.01 -0.04" rpy="0 0 0"/>
       <geometry name="LSoftHand_collision">
-        <mesh filename="package://coman_urdf/meshes/collada/simple/forearms/L_soft_hand_open.stl" scale="1E-3 1E-3 1E-3" />
+        <mesh filename="package://coman_urdf/meshes/simple/SoftHandOpen.STL" scale="-1E-3 1E-3 1E-3" />
       </geometry>
    </collision>

Commit message: changed signs on hands

File: coman_urdf/urdf/parts/soft_hand.urdf.xacro (robot description, xacro)
@@ -159,6 +159,6 @@
         <child link="RSoftHandFingers"/>
         <origin xyz="0 0.06 0.0" rpy="0 0 0"/>
-        <axis xyz="0 1 0" />
-        <limit velocity="4.0" effort="50" lower="-0.05" upper="0.0" />
+        <axis xyz="0 -1 0" />
+        <limit velocity="4.0" effort="50" lower="0.0" upper="0.05" />
         <dynamics friction="0" damping="3.0"/>
 </joint>

File: coman_urdf/urdf/sensors/imu.urdf.xacro (robot description, xacro)
@@ -2,4 +2,5 @@
 <robot xmlns:xacro="http://ros.org/wiki/xacro">
 <xacro:property name="PI" value="3.14159265359" />
+<xacro:property name="PI_2" value="1.57079632679" />
 <link name="imu_link">
     <inertial>
@@ -19,5 +20,5 @@
     <child link="imu_link"/>
     <!--origin xyz="-0.072 -0.0068 0.044" rpy="0 ${PI} 0"/-->
-    <origin xyz="-0.072 -0.0068 0.044" rpy="0 0 0"/>
+    <origin xyz="-0.072 -0.0068 0.044" rpy="${PI_2} 0 ${PI_2}"/>
 </joint>
 </robot>
