Commit message: added camera link

File: coman_urdf/urdf/gazebo/openni_kinect.gazebo.xacro (robot description, xacro)
@@ -1,9 +1,9 @@
 <?xml version="1.0"?>
 <robot xmlns:xacro="http://ros.org/wiki/xacro">
-<gazebo reference="gaze">
+<gazebo reference="Xtion_cam_body">
         <sensor name="openni_camera_camera" type="depth">
           <always_on>1</always_on>
           <visualize>1</visualize>
-          <camera name="__default__">
+	  <camera name="__default__">
             <horizontal_fov>1.047</horizontal_fov>
             <image>

File: coman_urdf/urdf/sensors/xtion.urdf.xacro (robot description, xacro)
@@ -41,4 +41,5 @@
     </collision>
 </link>
+<link name="camera_link"/>
 <!-- JOINTS -->
 <joint name="Xtion_body_joint" type="fixed">
@@ -61,9 +62,9 @@
 	<origin xyz="0.015 0 0.022" rpy="0 0 0" />
 </joint>
-<!--joint name="camera_link_joint" type="fixed">
-    		<parent link="gaze"/>
-    		<child link="camera_link"/-->
-    		<!--origin xyz="0.004 0.06 0.019" rpy="0.00 0.003 0.0" /--> <!--Real xtion pro live-->
-        <!--origin xyz="0.0 0.0 0.0" rpy="-1.57 0.0 -1.57" /--> <!--Simulated xtion pro live-->
-  	<!--/joint-->
+<joint name="camera_link_joint" type="fixed">
+	<parent link="Xtion_cam_body"/>
+	<child link="camera_link"/>
+	<!--origin xyz="0.004 0.06 0.019" rpy="0.00 0.003 0.0" /--> <!--Real xtion pro live-->
+	<origin xyz="0.0 0.0 0.0" rpy="-1.57 0.0 -1.57" /> <!--Simulated xtion pro live-->
+</joint>
 </robot>
