Commit message: Added meshes of right arm.

File: coman_urdf/urdf/gazebo/coman_materials.gazebo.xacro (robot description, xacro)
@@ -13,3 +13,18 @@
   <material>Gazebo/Red</material>
 </gazebo>
+<gazebo reference="RShp">
+  <material>Gazebo/DarkGrey</material>
+</gazebo>
+<gazebo reference="RShr">
+  <material>Gazebo/DarkGrey</material>
+</gazebo>
+<gazebo reference="RShy">
+  <material>Gazebo/DarkGrey</material>
+</gazebo>
+<gazebo reference="RElb">
+  <material>Gazebo/DarkGrey</material>
+</gazebo>
+<gazebo reference="LElb">
+  <material>Gazebo/DarkGrey</material>
+</gazebo>
 </robot>

File: coman_urdf/urdf/parts/arms.urdf.xacro (robot description, xacro)
@@ -13,6 +13,7 @@
     <visual>
       <origin xyz="-0.005305 0.0825 -0.844329" rpy="0 0 ${PI}"/>
+      <material name="dark_grey"/>
       <geometry name="RShp_visual">
-        <mesh filename="package://coman_urdf/meshes/collada/asm0001_collada_24_prt.dae" scale="${SF} ${SF} ${SF}" />
+        <mesh filename="package://coman_urdf/meshes/collada/rarm0.stl" scale="${SF} ${SF} ${SF}" />
       </geometry>
     </visual>
@@ -32,6 +33,7 @@
     <visual>
       <origin xyz="-0.005305 0.1558 -0.844329" rpy="0 0 ${PI}"/>
+      <material name="dark_grey"/>
       <geometry name="RShr_visual">
-        <mesh filename="package://coman_urdf/meshes/collada/asm0001_collada_23_prt.dae" scale="${SF} ${SF} ${SF}" />
+        <mesh filename="package://coman_urdf/meshes/collada/rarm1.stl" scale="${SF} ${SF} ${SF}" />
       </geometry>
     </visual>
@@ -51,6 +53,7 @@
     <visual>
       <origin xyz="-0.005305 0.1558 -0.79952053" rpy="0 0 ${PI}"/>
+      <material name="dark_grey"/>
       <geometry name="RShy_visual">
-        <mesh filename="package://coman_urdf/meshes/collada/asm0001_collada_22_prt.dae" scale="${SF} ${SF} ${SF}" />
+        <mesh filename="package://coman_urdf/meshes/collada/rarm2.stl" scale="${SF} ${SF} ${SF}" />
       </geometry>
     </visual>
@@ -70,6 +73,7 @@
         <visual>
           <origin xyz="0 0 0" rpy="-1.570796326795 1.570796326795 0"/>
+          <material name="dark_grey"/>
           <geometry name="RElb_visual">
-            <mesh filename="package://coman_urdf/meshes/collada/forearms/elbow.dae" scale="1.0 1.0 1.0" />
+            <mesh filename="package://coman_urdf/meshes/collada/forearms/elbow.stl" scale="1.0 1.0 1.0" />
           </geometry>
         </visual>
@@ -147,6 +151,7 @@
         <visual>
           <origin xyz="0 0 0" rpy="-1.570796326795 1.570796326795 0"/>
+          <material name="dark_grey"/>
           <geometry name="LElb_visual">
-            <mesh filename="package://coman_urdf/meshes/collada/forearms/elbow.dae" scale="1.0 1.0 1.0" />
+            <mesh filename="package://coman_urdf/meshes/collada/forearms/elbow.stl" scale="1.0 1.0 1.0" />
           </geometry>
         </visual>

Commit message: Added left arm.

File: coman_urdf/urdf/gazebo/coman_materials.gazebo.xacro (robot description, xacro)
@@ -25,4 +25,13 @@
   <material>Gazebo/DarkGrey</material>
 </gazebo>
+<gazebo reference="LShp">
+  <material>Gazebo/DarkGrey</material>
+</gazebo>
+<gazebo reference="LShr">
+  <material>Gazebo/DarkGrey</material>
+</gazebo>
+<gazebo reference="LShy">
+  <material>Gazebo/DarkGrey</material>
+</gazebo>
 <gazebo reference="LElb">
   <material>Gazebo/DarkGrey</material>

File: coman_urdf/urdf/parts/arms.urdf.xacro (robot description, xacro)
@@ -94,6 +94,7 @@
     <visual>
       <origin xyz="-0.005305 -0.0825 -0.844329" rpy="0 0 ${PI}"/>
+      <material name="dark_grey"/>
       <geometry name="LShp_visual">
-        <mesh filename="package://coman_urdf/meshes/collada/asm0001_collada_14_prt.dae" scale="${SF} ${SF} ${SF}" />
+        <mesh filename="package://coman_urdf/meshes/collada/larm0.stl" scale="${SF} ${SF} ${SF}" />
       </geometry>
     </visual>
@@ -113,6 +114,7 @@
     <visual>
       <origin xyz="-0.005305 -0.1558 -0.844329" rpy="0 0 ${PI}"/>
+      <material name="dark_grey"/>
       <geometry name="LShr_visual">
-        <mesh filename="package://coman_urdf/meshes/collada/asm0001_collada_13_prt.dae" scale="${SF} ${SF} ${SF}" />
+        <mesh filename="package://coman_urdf/meshes/collada/larm1.stl" scale="${SF} ${SF} ${SF}" />
       </geometry>
     </visual>
@@ -132,6 +134,7 @@
     <visual>
       <origin xyz="-0.005305 -0.1558 -0.79952053" rpy="0 0 ${PI}"/>
+      <material name="dark_grey"/>
       <geometry name="LShy_visual">
-        <mesh filename="package://coman_urdf/meshes/collada/asm0001_collada_12_prt.dae" scale="${SF} ${SF} ${SF}" />
+        <mesh filename="package://coman_urdf/meshes/collada/larm2.stl" scale="${SF} ${SF} ${SF}" />
       </geometry>
     </visual>

Commit message: Added right leg up to foot (not included).

File: coman_urdf/urdf/gazebo/coman_materials.gazebo.xacro (robot description, xacro)
@@ -37,3 +37,18 @@
   <material>Gazebo/DarkGrey</material>
 </gazebo>
+<gazebo reference="RHipMot">
+  <material>Gazebo/DarkGrey</material>
+</gazebo>
+<gazebo reference="RThighUpLeg">
+  <material>Gazebo/DarkGrey</material>
+</gazebo>
+<gazebo reference="RThighLowLeg">
+  <material>Gazebo/DarkGrey</material>
+</gazebo>
+<gazebo reference="RLowLeg">
+  <material>Gazebo/DarkGrey</material>
+</gazebo>
+<gazebo reference="RFootmot">
+  <material>Gazebo/DarkGrey</material>
+</gazebo>
 </robot>

File: coman_urdf/urdf/parts/legs.urdf.xacro (robot description, xacro)
@@ -14,6 +14,7 @@
     <visual>
       <origin xyz="0.0 0.023 -0.52" rpy="0 0 ${PI}"/>
+      <material name="dark_grey"/>
       <geometry name="RHipMot_visual">
-        <mesh filename="package://coman_urdf/meshes/collada/asm0001_collada_20_prt.dae" scale="${SF} ${SF} ${SF}" />
+        <mesh filename="package://coman_urdf/meshes/collada/rleg0.stl" scale="${SF} ${SF} ${SF}" />
       </geometry>
     </visual>
@@ -33,6 +34,7 @@
     <visual>
       <origin xyz="0.0 0.0726 -0.52" rpy="0 0 ${PI}"/>
+      <material name="dark_grey"/>
       <geometry name="RThighUpLeg_visual">
-        <mesh filename="package://coman_urdf/meshes/collada/asm0001_collada_19_prt.dae" scale="${SF} ${SF} ${SF}" />
+        <mesh filename="package://coman_urdf/meshes/collada/rleg1.stl" scale="${SF} ${SF} ${SF}" />
       </geometry>
     </visual>
@@ -52,6 +54,7 @@
     <visual>
       <origin xyz="0.0 0.0726 -0.4176" rpy="0 0 ${PI}"/>
+      <material name="dark_grey"/>
       <geometry name="RThighLowLeg_visual">
-        <mesh filename="package://coman_urdf/meshes/collada/asm0001_collada_18_prt.dae" scale="${SF} ${SF} ${SF}" />
+        <mesh filename="package://coman_urdf/meshes/collada/rleg2.stl" scale="${SF} ${SF} ${SF}" />
       </geometry>
     </visual>
@@ -71,6 +74,7 @@
     <visual>
       <origin xyz="0.0 0.0726 -0.2942" rpy="0 0 ${PI}"/>
+      <material name="dark_grey"/>
       <geometry name="RLowLeg_visual">
-        <mesh filename="package://coman_urdf/meshes/collada/asm0001_collada_17_prt.dae" scale="${SF} ${SF} ${SF}" />
+        <mesh filename="package://coman_urdf/meshes/collada/rleg3.stl" scale="${SF} ${SF} ${SF}" />
       </geometry>
     </visual>
@@ -90,6 +94,7 @@
     <visual>
       <origin xyz="0.0 0.0726 -0.0932" rpy="0 0 ${PI}"/>
+      <material name="dark_grey"/>
       <geometry name="RFootmot_visual">
-        <mesh filename="package://coman_urdf/meshes/collada/asm0001_collada_16_prt.dae" scale="${SF} ${SF} ${SF}" />
+        <mesh filename="package://coman_urdf/meshes/collada/rleg4.stl" scale="${SF} ${SF} ${SF}" />
       </geometry>
     </visual>

Commit message: Added partially left leg

File: coman_urdf/urdf/gazebo/coman_materials.gazebo.xacro (robot description, xacro)
@@ -52,3 +52,9 @@
   <material>Gazebo/DarkGrey</material>
 </gazebo>
+<gazebo reference="LHipMot">
+  <material>Gazebo/DarkGrey</material>
+</gazebo>
+<gazebo reference="LThighUpLeg">
+  <material>Gazebo/DarkGrey</material>
+</gazebo>
 </robot>

File: coman_urdf/urdf/parts/legs.urdf.xacro (robot description, xacro)
@@ -138,6 +138,7 @@
     <visual>
       <origin xyz="0.0 -0.023 -0.52" rpy="0 0 ${PI}"/>
+      <material name="dark_grey"/>
       <geometry name="RHipMot_visual">
-        <mesh filename="package://coman_urdf/meshes/collada/asm0001_collada_06_prt.dae" scale="${SF} ${SF} ${SF}" />
+        <mesh filename="package://coman_urdf/meshes/collada/lleg0.stl" scale="${SF} ${SF} ${SF}" />
       </geometry>
     </visual>
@@ -157,6 +158,7 @@
     <visual>
       <origin xyz="0.0 -0.0726 -0.52" rpy="0 0 ${PI}"/>
+      <material name="dark_grey"/>
       <geometry name="LThighUpLeg_visual">
-        <mesh filename="package://coman_urdf/meshes/collada/asm0001_collada_05_prt.dae" scale="${SF} ${SF} ${SF}" />
+        <mesh filename="package://coman_urdf/meshes/collada/lleg1.stl" scale="${SF} ${SF} ${SF}" />
       </geometry>
     </visual>

Commit message: Finished left leg. Still missing feet

File: coman_urdf/urdf/gazebo/coman_materials.gazebo.xacro (robot description, xacro)
@@ -58,3 +58,12 @@
   <material>Gazebo/DarkGrey</material>
 </gazebo>
+<gazebo reference="LThighLowLeg">
+  <material>Gazebo/DarkGrey</material>
+</gazebo>
+<gazebo reference="LLowLeg">
+  <material>Gazebo/DarkGrey</material>
+</gazebo>
+<gazebo reference="LFootmot">
+  <material>Gazebo/DarkGrey</material>
+</gazebo>
 </robot>

File: coman_urdf/urdf/parts/legs.urdf.xacro (robot description, xacro)
@@ -178,6 +178,7 @@
     <visual>
       <origin xyz="0.0 -0.0726 -0.4176" rpy="0 0 ${PI}"/>
+      <material name="dark_grey"/>
       <geometry name="LThighLowLeg_visual">
-        <mesh filename="package://coman_urdf/meshes/collada/asm0001_collada_04_prt.dae" scale="${SF} ${SF} ${SF}" />
+        <mesh filename="package://coman_urdf/meshes/collada/lleg2.stl" scale="${SF} ${SF} ${SF}" />
       </geometry>
     </visual>
@@ -197,6 +198,7 @@
     <visual>
       <origin xyz="0.0 -0.0726 -0.2942" rpy="0 0 ${PI}"/>
+      <material name="dark_grey"/>
       <geometry name="LLowLeg_visual">
-        <mesh filename="package://coman_urdf/meshes/collada/asm0001_collada_03_prt.dae" scale="${SF} ${SF} ${SF}" />
+        <mesh filename="package://coman_urdf/meshes/collada/lleg3.stl" scale="${SF} ${SF} ${SF}" />
       </geometry>
     </visual>
@@ -216,6 +218,7 @@
     <visual>
       <origin xyz="0.0 -0.0726 -0.0932" rpy="0 0 ${PI}"/>
+      <material name="dark_grey"/>
       <geometry name="LFootmot_visual">
-        <mesh filename="package://coman_urdf/meshes/collada/asm0001_collada_02_prt.dae" scale="${SF} ${SF} ${SF}" />
+        <mesh filename="package://coman_urdf/meshes/collada/lleg4.stl" scale="${SF} ${SF} ${SF}" />
       </geometry>
     </visual>

Commit message: Added stl of OLD forearm.

File: coman_urdf/urdf/gazebo/coman_materials.gazebo.xacro (robot description, xacro)
@@ -25,4 +25,7 @@
   <material>Gazebo/DarkGrey</material>
 </gazebo>
+<gazebo reference="RForearm">
+  <material>Gazebo/DarkGrey</material>
+</gazebo>
 <gazebo reference="LShp">
   <material>Gazebo/DarkGrey</material>
@@ -35,4 +38,7 @@
 </gazebo>
 <gazebo reference="LElb">
+  <material>Gazebo/DarkGrey</material>
+</gazebo>
+<gazebo reference="LForearm">
   <material>Gazebo/DarkGrey</material>
 </gazebo>

File: coman_urdf/urdf/parts/no_forearms.urdf.xacro (robot description, xacro)
@@ -15,6 +15,7 @@
       <visual>
         <origin xyz="-0.0055 -0.1558 -0.6175" rpy="0 0 ${PI}"/>
+        <material name="dark_grey"/>
         <geometry name="LForearm_visual">
-          <mesh filename="package://coman_urdf/meshes/collada/forearm_old.dae" scale="${SF} ${SF} ${SF}" />
+          <mesh filename="package://coman_urdf/meshes/collada/forearm_old.stl" scale="${SF} ${SF} ${SF}" />
         </geometry>
       </visual>
@@ -35,6 +36,7 @@
       <visual>
         <origin xyz="-0.0055 -0.1558 -0.6175" rpy="0 0 ${PI}"/>
+        <material name="dark_grey"/>
         <geometry name="RForearm_visual">
-          <mesh filename="package://coman_urdf/meshes/collada/forearm_old.dae" scale="${SF} ${SF} ${SF}" />
+          <mesh filename="package://coman_urdf/meshes/collada/forearm_old.stl" scale="${SF} ${SF} ${SF}" />
         </geometry>
       </visual>

Commit message: Added soft hands (fixed ver)

File: coman_urdf/urdf/gazebo/coman_materials.gazebo.xacro (robot description, xacro)
@@ -34,4 +34,7 @@
   <material>Gazebo/Grey</material>
 </gazebo>
+<gazebo reference="RSoftHand">
+  <material>Gazebo/DarkGrey</material>
+</gazebo>
 <gazebo reference="LShp">
   <material>Gazebo/DarkGrey</material>
@@ -54,4 +57,7 @@
 <gazebo reference="LWrMot3">
   <material>Gazebo/Grey</material>
+</gazebo>
+<gazebo reference="LSoftHand">
+  <material>Gazebo/DarkGrey</material>
 </gazebo>
 <gazebo reference="RHipMot">

File: coman_urdf/urdf/parts/soft_hand.urdf.xacro (robot description, xacro)
@@ -11,6 +11,7 @@
     <visual>
       <origin xyz="0.007 0.01 -0.04" rpy="${-3.14159265359/2} 0 ${3.14159265359}"/>
+      <material name="dark_grey"/>
       <geometry name="RSoftHand_visual">
-        <mesh filename="package://coman_urdf/meshes/collada/forearms/R_soft_hand_open_lowpoly.dae" scale="0.1 0.1 0.1" />
+        <mesh filename="package://coman_urdf/meshes/collada/forearms/Rsofthand_fix.stl" scale="0.1 0.1 0.1" />
       </geometry>
    </visual>
@@ -30,6 +31,7 @@
     <visual>
       <origin xyz="0.007 -0.012 -0.04" rpy="${-3.14159265359/2} 0 ${3.14159265359/2}"/>
+      <material name="dark_grey"/>
       <geometry name="LSoftHand_visual">
-        <mesh filename="package://coman_urdf/meshes/collada/forearms/L_soft_hand_open_lowpoly.dae" scale="0.1 0.1 0.1" />
+        <mesh filename="package://coman_urdf/meshes/collada/forearms/Lsofthand_fix.stl" scale="0.1 0.1 0.1" />
       </geometry>
    </visual>

Commit message: Added old feet

File: coman_urdf/urdf/gazebo/coman_materials.gazebo.xacro (robot description, xacro)
@@ -76,4 +76,7 @@
   <material>Gazebo/DarkGrey</material>
 </gazebo>
+<gazebo reference="RFoot">
+  <material>Gazebo/DarkGrey</material>
+</gazebo>
 <gazebo reference="LHipMot">
   <material>Gazebo/DarkGrey</material>
@@ -91,3 +94,6 @@
   <material>Gazebo/DarkGrey</material>
 </gazebo>
+<gazebo reference="LFoot">
+  <material>Gazebo/DarkGrey</material>
+</gazebo>
 </robot>

File: coman_urdf/urdf/parts/subparts/round_feet_13/accurate_FT_round_foot_L_13.urdf.xacro (robot description, xacro)
@@ -9,6 +9,7 @@
       <visual>
         <origin xyz="0.0 -0.0726 -0.0282" rpy="0 0 -3.14159265359"/>
+        <material name="dark_grey"/>
         <geometry name="LFoot_visual">
-          <mesh filename="package://coman_urdf/meshes/collada/asm0001_collada_01_prt.dae" scale="0.03937 0.03937 0.03937" />
+          <mesh filename="package://coman_urdf/meshes/collada/Lfoot.stl" scale="0.03937 0.03937 0.03937" />
         </geometry>
       </visual>

File: coman_urdf/urdf/parts/subparts/round_feet_13/accurate_FT_round_foot_R_13.urdf.xacro (robot description, xacro)
@@ -9,6 +9,7 @@
       <visual>
         <origin xyz="0.0 0.0726 -0.0282" rpy="0 0 -3.14159265359"/>
+        <material name="dark_grey"/>
         <geometry name="RFoot_visual">
-          <mesh filename="package://coman_urdf/meshes/collada/asm0001_collada_15_prt.dae" scale="0.03937 0.03937 0.03937" />
+          <mesh filename="package://coman_urdf/meshes/collada/Rfoot.stl" scale="0.03937 0.03937 0.03937" />
         </geometry>
       </visual>

File: coman_urdf/urdf/parts/subparts/round_feet_13/round_foot_L_13.urdf.xacro (robot description, xacro)
@@ -9,6 +9,7 @@
       <visual>
         <origin xyz="0.0 -0.0726 -0.0932" rpy="0 0 -3.14159265359"/>
+        <material name="dark_grey"/>
         <geometry name="LFoot_visual">
-          <mesh filename="package://coman_urdf/meshes/collada/asm0001_collada_01_prt.dae" scale="0.03937 0.03937 0.03937" />
+          <mesh filename="package://coman_urdf/meshes/collada/Lfoot.stl" scale="0.03937 0.03937 0.03937" />
         </geometry>
       </visual>

File: coman_urdf/urdf/parts/subparts/round_feet_13/round_foot_R_13.urdf.xacro (robot description, xacro)
@@ -9,6 +9,7 @@
       <visual>
         <origin xyz="0.0 0.0726 -0.0932" rpy="0 0 -3.14159265359"/>
+        <material name="dark_grey"/>
         <geometry name="RFoot_visual">
-          <mesh filename="package://coman_urdf/meshes/collada/asm0001_collada_15_prt.dae" scale="0.03937 0.03937 0.03937" />
+          <mesh filename="package://coman_urdf/meshes/collada/Rfoot.stl" scale="0.03937 0.03937 0.03937" />
         </geometry>
       </visual>

Commit message: Added stl of xtion

File: coman_urdf/urdf/gazebo/coman_materials.gazebo.xacro (robot description, xacro)
@@ -28,13 +28,17 @@
   <material>Gazebo/DarkGrey</material>
 </gazebo>
-<gazebo reference="RWrMot2">
-  <material>Gazebo/Grey</material>
-</gazebo>
-<gazebo reference="RWrMot3">
-  <material>Gazebo/Grey</material>
-</gazebo>
-<gazebo reference="RSoftHand">
-  <material>Gazebo/DarkGrey</material>
-</gazebo>
+<xacro:if value="${GAZEBO_COMAN_USES_7DOF_FOREARMS_DRC_14}">
+  <gazebo reference="RWrMot2">
+    <material>Gazebo/Grey</material>
+  </gazebo>
+  <gazebo reference="RWrMot3">
+    <material>Gazebo/Grey</material>
+  </gazebo>
+  <xacro:if value="${GAZEBO_COMAN_USES_SOFTHANDS_DRC_sw1_14}">
+    <gazebo reference="RSoftHand">
+      <material>Gazebo/DarkGrey</material>
+    </gazebo>
+  </xacro:if>
+</xacro:if>
 <gazebo reference="LShp">
   <material>Gazebo/DarkGrey</material>
@@ -52,13 +56,17 @@
   <material>Gazebo/DarkGrey</material>
 </gazebo>
-<gazebo reference="LWrMot2">
-  <material>Gazebo/Grey</material>
-</gazebo>
-<gazebo reference="LWrMot3">
-  <material>Gazebo/Grey</material>
-</gazebo>
-<gazebo reference="LSoftHand">
-  <material>Gazebo/DarkGrey</material>
-</gazebo>
+<xacro:if value="${GAZEBO_COMAN_USES_7DOF_FOREARMS_DRC_14}">
+  <gazebo reference="LWrMot2">
+    <material>Gazebo/Grey</material>
+  </gazebo>
+  <gazebo reference="LWrMot3">
+    <material>Gazebo/Grey</material>
+  </gazebo>
+  <xacro:if value="${GAZEBO_COMAN_USES_SOFTHANDS_DRC_sw1_14}">
+    <gazebo reference="LSoftHand">
+      <material>Gazebo/DarkGrey</material>
+    </gazebo>
+  </xacro:if>
+</xacro:if>
 <gazebo reference="RHipMot">
   <material>Gazebo/DarkGrey</material>

File: coman_urdf/urdf/sensors/xtion.urdf.xacro (robot description, xacro)
@@ -12,5 +12,5 @@
       <origin xyz="-0.020281504 0.0 -0.68662053" rpy="0 0 ${PI}"/>
       <geometry name="Xtion_body_visual">
-        <mesh filename="package://coman_urdf/meshes/collada/Xtion/xtion_base.dae" scale="0.03937 0.03937 0.03937" />
+        <mesh filename="package://coman_urdf/meshes/collada/Xtion/xtion_base.stl" scale="0.03937 0.03937 0.03937" />
       </geometry>
     </visual>
@@ -31,5 +31,5 @@
       <origin xyz="-0.0915 0.0 -1.2778" rpy="0 0 ${PI}"/>
       <geometry name="Xtion_cam_body_visual">
-        <mesh filename="package://coman_urdf/meshes/collada/Xtion/xtion_cam_body.dae" scale="0.001 0.001 0.001" />
+        <mesh filename="package://coman_urdf/meshes/collada/Xtion/xtion_cam_body.stl" scale="0.001 0.001 0.001" />
       </geometry>
     </visual>

Commit message: added material for xtion

File: coman_urdf/urdf/gazebo/coman_materials.gazebo.xacro (robot description, xacro)
@@ -105,3 +105,11 @@
   <material>Gazebo/DarkGrey</material>
 </gazebo>
+<xacro:if value="${GAZEBO_COMAN_USES_XTION}">
+  <gazebo reference="Xtion_body">
+    <material>Gazebo/DarkGrey</material>
+  </gazebo>
+  <gazebo reference="Xtion_cam_body">
+    <material>Gazebo/Grey</material>
+  </gazebo>
+</xacro:if>
 </robot>
