Commit message: Changed order of joints in torso also in srdf

File: coman_srdf/srdf/coman.srdf.xacro (robot description, xacro)
@@ -62,6 +62,6 @@
     </group>
     <group name="torso">
+        <joint name="WaistLat" />
         <joint name="WaistSag" />
-        <joint name="WaistLat" />
         <joint name="WaistYaw" />
     </group>

Commit message: new srdf structure, no more joint names here, only in the urdf

File: coman_srdf/srdf/coman.srdf.xacro (robot description, xacro)
@@ -11,58 +11,42 @@
     <!--CHAINS: When a chain is specified, all the links along the chain (including endpoints) are included in the group. Additionally, all the joints that are parents to included links are also included. This means that joints along the chain and the parent joint of the base link are included in the group-->
     <!--SUBGROUPS: Groups can also be formed by referencing to already defined group names-->
-<xacro:if value="${GAZEBO_COMAN_USES_7DOF_FOREARMS_DRC_14}">
+    <group name="base">
+        <link name="Waist"/>
+    </group>
+    <group name="sensors">
+        <joint name="l_ankle_joint"/>
+        <joint name="r_ankle_joint"/>
+    </group>
+    <xacro:if value="${GAZEBO_COMAN_USES_7DOF_FOREARMS_DRC_14}">
     <group name="left_arm">
-        <joint name="LShSag" />
-        <joint name="LShLat" />
-        <joint name="LShYaw" />
-        <joint name="LElbj" />
-        <joint name="LForearmPlate" />
-        <joint name="LWrj1" />
-        <joint name="LWrj2" />
+        <chain base_link="DWYTorso" tip_link="l_wrist"/>
     </group>
     <group name="right_arm">
-        <joint name="RShSag" />
-        <joint name="RShLat" />
-        <joint name="RShYaw" />
-        <joint name="RElbj" />
-        <joint name="RForearmPlate" />
-        <joint name="RWrj1" />
-        <joint name="RWrj2" />
+        <chain base_link="DWYTorso" tip_link="r_wrist"/>
     </group>
 </xacro:if>
 <xacro:unless value="${GAZEBO_COMAN_USES_7DOF_FOREARMS_DRC_14}">
     <group name="left_arm">
-        <joint name="LShSag" />
-        <joint name="LShLat" />
-        <joint name="LShYaw" />
-        <joint name="LElbj" />
+        <chain base_link="DWYTorso" tip_link="l_wrist"/>
     </group>
     <group name="right_arm">
-        <joint name="RShSag" />
-        <joint name="RShLat" />
-        <joint name="RShYaw" />
-        <joint name="RElbj" />
+        <chain base_link="DWYTorso" tip_link="r_wrist"/>
     </group>
 </xacro:unless>
     <group name="left_leg">
-        <joint name="LHipSag" />
-        <joint name="LHipLat" />
-        <joint name="LHipYaw" />
-        <joint name="LKneeSag" />
-        <joint name="LAnkLat" />
-        <joint name="LAnkSag" />
+        <chain base_link="Waist" tip_link="l_sole"/>
     </group>
     <group name="right_leg">
-        <joint name="RHipSag" />
-        <joint name="RHipLat" />
-        <joint name="RHipYaw" />
-        <joint name="RKneeSag" />
-        <joint name="RAnkLat" />
-        <joint name="RAnkSag" />
+        <chain base_link="Waist" tip_link="r_sole"/>
     </group>
     <group name="torso">
-        <joint name="WaistLat" />
-        <joint name="WaistSag" />
-        <joint name="WaistYaw" />
+        <chain base_link="Waist" tip_link="DWYTorso"/>
+    </group>
+    <group name="chains"> <!--THIS HAS TO BE THE LAST GROUP IN THE FILE -->
+        <group name="left_arm"/>
+        <group name="right_arm"/>
+        <group name="left_leg"/>
+        <group name="right_leg"/>
+        <group name="torso"/>
     </group>
 </robot>

Commit message: Added force_torque and imu sensors to coman.srdf.xacro

File: coman_srdf/srdf/coman.srdf.xacro (robot description, xacro)
@@ -18,20 +18,36 @@
         <joint name="r_ankle_joint"/>
     </group>
+    <group name="imu_sensors">
+    <!-- NEAREST JOINT TO IMU -->
+        <joint name="WaistSag"/>
+    </group>
     <xacro:if value="${GAZEBO_COMAN_USES_7DOF_FOREARMS_DRC_14}">
-    <group name="left_arm">
-        <chain base_link="DWYTorso" tip_link="l_wrist"/>
-    </group>
-    <group name="right_arm">
-        <chain base_link="DWYTorso" tip_link="r_wrist"/>
-    </group>
-</xacro:if>
-<xacro:unless value="${GAZEBO_COMAN_USES_7DOF_FOREARMS_DRC_14}">
-    <group name="left_arm">
-        <chain base_link="DWYTorso" tip_link="l_wrist"/>
-    </group>
-    <group name="right_arm">
-        <chain base_link="DWYTorso" tip_link="r_wrist"/>
-    </group>
-</xacro:unless>
+        <group name="left_arm">
+            <chain base_link="DWYTorso" tip_link="l_wrist"/>
+        </group>
+        <group name="right_arm">
+            <chain base_link="DWYTorso" tip_link="r_wrist"/>
+        </group>
+        <group name="force_torque_sensors">
+        <!-- NEAREST JOINT TO FORCE_TORQUE SENSOR -->
+            <joint name="LAnkSag"/>
+            <joint name="RAnkSag"/>
+            <joint name="LForearmPlate"/>
+            <joint name="RForearmPlate"/>
+        </group>
+    </xacro:if>
+    <xacro:unless value="${GAZEBO_COMAN_USES_7DOF_FOREARMS_DRC_14}">
+        <group name="left_arm">
+            <chain base_link="DWYTorso" tip_link="l_wrist"/>
+        </group>
+        <group name="right_arm">
+            <chain base_link="DWYTorso" tip_link="r_wrist"/>
+        </group>
+        <group name="force_torque_sensors">
+        <!-- NEAREST JOINT TO FORCE_TORQUE SENSOR -->
+            <joint name="LAnkSag"/>
+            <joint name="RAnkSag"/>
+        </group>
+    </xacro:unless>
     <group name="left_leg">
         <chain base_link="Waist" tip_link="l_sole"/>

Commit message: Fixed bug in ft_sensor_list in srdf

File: coman_srdf/srdf/coman.srdf.xacro (robot description, xacro)
@@ -14,8 +14,4 @@
         <link name="Waist"/>
     </group>
-    <group name="sensors">
-        <joint name="l_ankle_joint"/>
-        <joint name="r_ankle_joint"/>
-    </group>
     <group name="imu_sensors">
     <!-- NEAREST JOINT TO IMU -->
@@ -30,9 +26,12 @@
         </group>
         <group name="force_torque_sensors">
-        <!-- NEAREST JOINT TO FORCE_TORQUE SENSOR -->
-            <joint name="LAnkSag"/>
+        <!--<joint name="LAnkSag"/>
             <joint name="RAnkSag"/>
             <joint name="LForearmPlate"/>
-            <joint name="RForearmPlate"/>
+            <joint name="RForearmPlate"/>-->
+            <joint name="l_ankle_joint"/>
+            <joint name="r_ankle_joint"/>
+            <joint name="l_wrist_joint"/>
+            <joint name="r_wrist_joint"/>
         </group>
     </xacro:if>
@@ -46,6 +45,8 @@
         <group name="force_torque_sensors">
         <!-- NEAREST JOINT TO FORCE_TORQUE SENSOR -->
-            <joint name="LAnkSag"/>
-            <joint name="RAnkSag"/>
+            <!--<joint name="LAnkSag"/>
+            <joint name="RAnkSag"/>-->
+            <joint name="l_ankle_joint"/>
+            <joint name="r_ankle_joint"/>
         </group>
     </xacro:unless>
