Commit message: Deleted useless files

File: coman_srdf/srdf/coman.srdf.xacro (robot description, xacro)
@@ -18,5 +18,5 @@
         <joint name="WaistSag"/>
     </group>
-    <xacro:if value="${GAZEBO_COMAN_USES_7DOF_FOREARMS_DRC_14}">
+    <xacro:if value="${GAZEBO_COMAN_USES_FOREARMS}">
         <group name="left_arm">
             <chain base_link="DWYTorso" tip_link="l_wrist"/>
@@ -36,5 +36,5 @@
         </group>
     </xacro:if>
-    <xacro:unless value="${GAZEBO_COMAN_USES_7DOF_FOREARMS_DRC_14}">
+    <xacro:unless value="${GAZEBO_COMAN_USES_FOREARMS}">
         <group name="left_arm">
             <chain base_link="DWYTorso" tip_link="l_wrist"/>

File: coman_urdf/urdf/coman.urdf.xacro (robot description, xacro)
@@ -35,12 +35,12 @@
 <link name="l_wrist"/>
 <link name="r_wrist"/>
-<xacro:if value="${GAZEBO_COMAN_USES_NO_FOREARMS}">
-    <xacro:include filename="$(find coman_urdf)/urdf/parts/no_forearms.urdf.xacro" />
-</xacro:if>
-<xacro:if value="${GAZEBO_COMAN_USES_7DOF_FOREARMS_DRC_14}">
+<xacro:if value="${GAZEBO_COMAN_USES_FOREARMS}">
     <xacro:include filename="$(find coman_urdf)/urdf/parts/7DOF_forearms_DRC_14.urdf.xacro" />
 </xacro:if>
+<xacro:unless value="${GAZEBO_COMAN_USES_FOREARMS}">
+    <xacro:include filename="$(find coman_urdf)/urdf/parts/no_forearms.urdf.xacro" />
+</xacro:unless>
 <!-- ************ HANDS ************ -->
-<xacro:if value="${GAZEBO_COMAN_USES_7DOF_FOREARMS_DRC_14}">
+<xacro:if value="${GAZEBO_COMAN_USES_FOREARMS}">
     <xacro:include filename="$(find coman_urdf)/urdf/parts/soft_hand.urdf.xacro" />
     <!-- Reference frames in hands -->

File: coman_urdf/urdf/coman_config.urdf.xacro (robot description, xacro)
@@ -9,15 +9,8 @@
 ##
 ##
-## options:
-## 1) round feet
-## 2) simple feet
 ##
 ####################################################
-# TODO checks (must be mutually exclusive)
 -->
-<!-- 1) round feet -->
-<xacro:property name="GAZEBO_COMAN_USES_ROUND_FEET_13" value="false" />
-<!-- 2) simple feet -->
-<xacro:property name="GAZEBO_COMAN_USES_SIMPLE_FEET_DRC_sw1_14" value="true" />
+<xacro:property name="GAZEBO_COMAN_USES_ROUND_FEET" value="false" />
 <!--
 ####################################################
@@ -26,84 +19,9 @@
 ##
 ##
-## options:
-## 1) no forearms
-## 2) 7dof forearms
-## 3) 7dof forearms + soft hands
 ##
 ####################################################
-# TODO: checks (must be mutually exclusive).. eventually, a menu!... documentation!
-#       at the moment just the only combinations that work are:
 -->
-<!-- 1) NO_FOREARMS -->
-<!--
-<xacro:property name="GAZEBO_COMAN_USES_NO_FOREARMS" value="true" />
-<xacro:property name="GAZEBO_COMAN_USES_7DOF_FOREARMS_DRC_14" value="false" />
-<xacro:property name="GAZEBO_COMAN_USES_SOFTHANDS_DRC_sw1_14" value="false" />
--->
-<!-- 2) 7DOFS_FOREARMS -->
-<!--
-<xacro:property name="GAZEBO_COMAN_USES_NO_FOREARMS" value="false" />
-<xacro:property name="GAZEBO_COMAN_USES_7DOF_FOREARMS_DRC_14" value="true" />
-<xacro:property name="GAZEBO_COMAN_USES_SOFTHANDS_DRC_sw1_14" value="false" />
--->
-<!-- 3) 7DOFS_FOREARMS + SOFT_HANDS -->
-<xacro:property name="GAZEBO_COMAN_USES_NO_FOREARMS" value="false" />
-<xacro:property name="GAZEBO_COMAN_USES_7DOF_FOREARMS_DRC_14" value="true" />
-<xacro:property name="GAZEBO_COMAN_USES_SOFTHANDS_DRC_sw1_14" value="true" />
-<!--
-####################################################
-##
-##  MIDDLEWARE SELECTION
-##
-##
-## options:
-#  notice how, regardless of the middleware selected
-#  a bare version of the robot is created (.urdf)
-#  1) yarp
-#	The robot is created using yarp plugins for
-#	the IMU and F/T sensors. The controlboard
-#	plugins used to control joints and get
-#	encoder and torque information are to be
-#	inserted using the .world file, where the
-#	initial configuration for the joints can
-#	be specified (for example, look at the
-#	worlds folder)
-#  2) ros
-#	The sdf is created including ros plugins
-#
-##
-####################################################
-#
-# 1) yarp
-#
--->
-<xacro:property name="GAZEBO_COMAN_USES_ROS" value="false" />
-<!--
-#
-# 2) ros
-#
--->
-<xacro:property name="GAZEBO_COMAN_USES_YARP" value="true" />
-<!--
-####################################################
-##
-##  F/T SELECTION
-##
-##
-## options:
-## 1) accurate (ft sensors located at exact spot)
-#	FT sensors are defined as children of
-#	underactuated joints, added specifically
-#	to create a frame for accurate reading,
-#	and to take into account the bias given
-#	by the sensor's inertia.
-## 2) non-accurate (ft sensors at the nearest joint)
-##
-####################################################
-#
-# 1/2 (true/false)
-#
--->
-<xacro:property name="GAZEBO_COMAN_USES_ACCURATE_FT" value="false" />
+<xacro:property name="GAZEBO_COMAN_USES_FOREARMS" value="true" />
+<xacro:property name="GAZEBO_COMAN_USES_SOFTHANDS" value="true" />
 <!--
 ####################################################

File: coman_urdf/urdf/coman_robot.urdf.xacro (robot description, xacro)
@@ -15,4 +15,5 @@
   <xacro:include filename="$(find coman_urdf)/urdf/gazebo/yarp_control.gazebo.xacro" />
   <xacro:include filename="$(find coman_urdf)/urdf/gazebo/coman_materials.gazebo.xacro" />
+  <xacro:include filename="$(find coman_urdf)/urdf/gazebo/force_torque.gazebo.xacro" />
   <origin xyz="0.0 0.0 0.521" rpy="0 0 0" />
 </robot>

File: coman_urdf/urdf/config/coman_hands.urdf.xacro (robot description, xacro)
@@ -9,15 +9,8 @@
 ##
 ##
-## options:
-## 1) round feet
-## 2) simple feet
 ##
 ####################################################
-# TODO checks (must be mutually exclusive)
 -->
-<!-- 1) round feet -->
-<xacro:property name="GAZEBO_COMAN_USES_ROUND_FEET_13" value="false" />
-<!-- 2) simple feet -->
-<xacro:property name="GAZEBO_COMAN_USES_SIMPLE_FEET_DRC_sw1_14" value="true" />
+<xacro:property name="GAZEBO_COMAN_USES_ROUND_FEET" value="false" />
 <!--
 ####################################################
@@ -26,84 +19,8 @@
 ##
 ##
-## options:
-## 1) no forearms
-## 2) 7dof forearms
-## 3) 7dof forearms + soft hands
-##
 ####################################################
-# TODO: checks (must be mutually exclusive).. eventually, a menu!... documentation!
-#       at the moment just the only combinations that work are:
 -->
-<!-- 1) NO_FOREARMS -->
-<!--
-<xacro:property name="GAZEBO_COMAN_USES_NO_FOREARMS" value="true" />
-<xacro:property name="GAZEBO_COMAN_USES_7DOF_FOREARMS_DRC_14" value="false" />
-<xacro:property name="GAZEBO_COMAN_USES_SOFTHANDS_DRC_sw1_14" value="false" />
--->
-<!-- 2) 7DOFS_FOREARMS -->
-<xacro:property name="GAZEBO_COMAN_USES_NO_FOREARMS" value="false" />
-<xacro:property name="GAZEBO_COMAN_USES_7DOF_FOREARMS_DRC_14" value="true" />
-<xacro:property name="GAZEBO_COMAN_USES_SOFTHANDS_DRC_sw1_14" value="false" />
-<!-- 3) 7DOFS_FOREARMS + SOFT_HANDS -->
-<!--
-<xacro:property name="GAZEBO_COMAN_USES_NO_FOREARMS" value="false" />
-<xacro:property name="GAZEBO_COMAN_USES_7DOF_FOREARMS_DRC_14" value="true" />
-<xacro:property name="GAZEBO_COMAN_USES_SOFTHANDS_DRC_sw1_14" value="true" />
--->
-<!--
-####################################################
-##
-##  MIDDLEWARE SELECTION
-##
-##
-## options:
-#  notice how, regardless of the middleware selected
-#  a bare version of the robot is created (.urdf)
-#  1) yarp
-#	The robot is created using yarp plugins for
-#	the IMU and F/T sensors. The controlboard
-#	plugins used to control joints and get
-#	encoder and torque information are to be
-#	inserted using the .world file, where the
-#	initial configuration for the joints can
-#	be specified (for example, look at the
-#	worlds folder)
-#  2) ros
-#	The sdf is created including ros plugins
-#
-##
-####################################################
-#
-# 1) yarp
-#
--->
-<xacro:property name="GAZEBO_COMAN_USES_ROS" value="false" />
-<!--
-#
-# 2) ros
-#
--->
-<xacro:property name="GAZEBO_COMAN_USES_YARP" value="true" />
-<!--
-####################################################
-##
-##  F/T SELECTION
-##
-##
-## options:
-## 1) accurate (ft sensors located at exact spot)
-#	FT sensors are defined as children of
-#	underactuated joints, added specifically
-#	to create a frame for accurate reading,
-#	and to take into account the bias given
-#	by the sensor's inertia.
-## 2) non-accurate (ft sensors at the nearest joint)
-##
-####################################################
-#
-# 1/2 (true/false)
-#
--->
-<xacro:property name="GAZEBO_COMAN_USES_ACCURATE_FT" value="false" />
+<xacro:property name="GAZEBO_COMAN_USES_FOREARMS" value="true" />
+<xacro:property name="GAZEBO_COMAN_USES_SOFTHANDS" value="false" />
 <!--
 ####################################################

File: coman_urdf/urdf/config/coman_no_forearms.urdf.xacro (robot description, xacro)
@@ -9,15 +9,8 @@
 ##
 ##
-## options:
-## 1) round feet
-## 2) simple feet
 ##
 ####################################################
-# TODO checks (must be mutually exclusive)
 -->
-<!-- 1) round feet -->
-<xacro:property name="GAZEBO_COMAN_USES_ROUND_FEET_13" value="true" />
-<!-- 2) simple feet -->
-<xacro:property name="GAZEBO_COMAN_USES_SIMPLE_FEET_DRC_sw1_14" value="false" />
+<xacro:property name="GAZEBO_COMAN_USES_ROUND_FEET" value="true" />
 <!--
 ####################################################
@@ -26,84 +19,8 @@
 ##
 ##
-## options:
-## 1) no forearms
-## 2) 7dof forearms
-## 3) 7dof forearms + soft hands
-##
 ####################################################
-# TODO: checks (must be mutually exclusive).. eventually, a menu!... documentation!
-#       at the moment just the only combinations that work are:
 -->
-<!-- 1) NO_FOREARMS -->
-<xacro:property name="GAZEBO_COMAN_USES_NO_FOREARMS" value="true" />
-<xacro:property name="GAZEBO_COMAN_USES_7DOF_FOREARMS_DRC_14" value="false" />
-<xacro:property name="GAZEBO_COMAN_USES_SOFTHANDS_DRC_sw1_14" value="false" />
-<!-- 2) 7DOFS_FOREARMS -->
-<!--
-<xacro:property name="GAZEBO_COMAN_USES_NO_FOREARMS" value="false" />
-<xacro:property name="GAZEBO_COMAN_USES_7DOF_FOREARMS_DRC_14" value="true" />
-<xacro:property name="GAZEBO_COMAN_USES_SOFTHANDS_DRC_sw1_14" value="false" />
--->
-<!-- 3) 7DOFS_FOREARMS + SOFT_HANDS -->
-<!--
-<xacro:property name="GAZEBO_COMAN_USES_NO_FOREARMS" value="false" />
-<xacro:property name="GAZEBO_COMAN_USES_7DOF_FOREARMS_DRC_14" value="true" />
-<xacro:property name="GAZEBO_COMAN_USES_SOFTHANDS_DRC_sw1_14" value="true" />
--->
-<!--
-####################################################
-##
-##  MIDDLEWARE SELECTION
-##
-##
-## options:
-#  notice how, regardless of the middleware selected
-#  a bare version of the robot is created (.urdf)
-#  1) yarp
-#	The robot is created using yarp plugins for
-#	the IMU and F/T sensors. The controlboard
-#	plugins used to control joints and get
-#	encoder and torque information are to be
-#	inserted using the .world file, where the
-#	initial configuration for the joints can
-#	be specified (for example, look at the
-#	worlds folder)
-#  2) ros
-#	The sdf is created including ros plugins
-#
-##
-####################################################
-#
-# 1) yarp
-#
--->
-<xacro:property name="GAZEBO_COMAN_USES_ROS" value="false" />
-<!--
-#
-# 2) ros
-#
--->
-<xacro:property name="GAZEBO_COMAN_USES_YARP" value="true" />
-<!--
-####################################################
-##
-##  F/T SELECTION
-##
-##
-## options:
-## 1) accurate (ft sensors located at exact spot)
-#	FT sensors are defined as children of
-#	underactuated joints, added specifically
-#	to create a frame for accurate reading,
-#	and to take into account the bias given
-#	by the sensor's inertia.
-## 2) non-accurate (ft sensors at the nearest joint)
-##
-####################################################
-#
-# 1/2 (true/false)
-#
--->
-<xacro:property name="GAZEBO_COMAN_USES_ACCURATE_FT" value="false" />
+<xacro:property name="GAZEBO_COMAN_USES_FOREARMS" value="false" />
+<xacro:property name="GAZEBO_COMAN_USES_SOFTHANDS" value="false" />
 <!--
 ####################################################

File: coman_urdf/urdf/config/coman_softhand.urdf.xacro (robot description, xacro)
@@ -9,15 +9,8 @@
 ##
 ##
-## options:
-## 1) round feet
-## 2) simple feet
 ##
 ####################################################
-# TODO checks (must be mutually exclusive)
 -->
-<!-- 1) round feet -->
-<xacro:property name="GAZEBO_COMAN_USES_ROUND_FEET_13" value="false" />
-<!-- 2) simple feet -->
-<xacro:property name="GAZEBO_COMAN_USES_SIMPLE_FEET_DRC_sw1_14" value="true" />
+<xacro:property name="GAZEBO_COMAN_USES_ROUND_FEET" value="false" />
 <!--
 ####################################################
@@ -26,29 +19,8 @@
 ##
 ##
-## options:
-## 1) no forearms
-## 2) 7dof forearms
-## 3) 7dof forearms + soft hands
-##
 ####################################################
-# TODO: checks (must be mutually exclusive).. eventually, a menu!... documentation!
-#       at the moment just the only combinations that work are:
 -->
-<!-- 1) NO_FOREARMS -->
-<!--
-<xacro:property name="GAZEBO_COMAN_USES_NO_FOREARMS" value="true" />
-<xacro:property name="GAZEBO_COMAN_USES_7DOF_FOREARMS_DRC_14" value="false" />
-<xacro:property name="GAZEBO_COMAN_USES_SOFTHANDS_DRC_sw1_14" value="false" />
--->
-<!-- 2) 7DOFS_FOREARMS -->
-<!--
-<xacro:property name="GAZEBO_COMAN_USES_NO_FOREARMS" value="false" />
-<xacro:property name="GAZEBO_COMAN_USES_7DOF_FOREARMS_DRC_14" value="true" />
-<xacro:property name="GAZEBO_COMAN_USES_SOFTHANDS_DRC_sw1_14" value="false" />
--->
-<!-- 3) 7DOFS_FOREARMS + SOFT_HANDS -->
-<xacro:property name="GAZEBO_COMAN_USES_NO_FOREARMS" value="false" />
-<xacro:property name="GAZEBO_COMAN_USES_7DOF_FOREARMS_DRC_14" value="true" />
-<xacro:property name="GAZEBO_COMAN_USES_SOFTHANDS_DRC_sw1_14" value="true" />
+<xacro:property name="GAZEBO_COMAN_USES_FOREARMS" value="true" />
+<xacro:property name="GAZEBO_COMAN_USES_SOFTHANDS" value="true" />
 <!--
 ####################################################
@@ -88,25 +60,4 @@
 ####################################################
 ##
-##  F/T SELECTION
-##
-##
-## options:
-## 1) accurate (ft sensors located at exact spot)
-#	FT sensors are defined as children of
-#	underactuated joints, added specifically
-#	to create a frame for accurate reading,
-#	and to take into account the bias given
-#	by the sensor's inertia.
-## 2) non-accurate (ft sensors at the nearest joint)
-##
-####################################################
-#
-# 1/2 (true/false)
-#
--->
-<xacro:property name="GAZEBO_COMAN_USES_ACCURATE_FT" value="false" />
-<!--
-####################################################
-##
 ##  Xtion SELECTION
 ##

File: coman_urdf/urdf/gazebo/coman.gazebo.xacro (robot description, xacro)
@@ -9,6 +9,5 @@
      <fdir1>1 0 0</fdir1>
      <maxVel>1.0</maxVel>
-     <minDepth>0.00</minDepth>
-     <cfmDamping>1</cfmDamping>
+     <minDepth>0.0</minDepth>
    </gazebo>
    <gazebo reference="RFoot">
@@ -20,128 +19,98 @@
      <maxVel>1.0</maxVel>
      <minDepth>0.00</minDepth>
-     <cfmDamping>1</cfmDamping>
    </gazebo>
-<!-- contact model for hand surface -->
-<!--
-<xacro:if value="${GAZEBO_COMAN_USES_7DOF_FOREARMS_DRC_14}">
-    <xacro:if value="${GAZEBO_COMAN_USES_SOFTHANDS_DRC_sw1_14}">
-   <gazebo reference="LSoftHand">
-     <kp>1000000.0</kp>
-     <kd>100.0</kd>
-     <mu1>1.0</mu1>
-     <mu2>1.0</mu2>
-     <fdir1>1 0 0</fdir1>
-     <maxVel>1.0</maxVel>
-     <minDepth>0.00</minDepth>
-     <cfmDamping>1</cfmDamping>
-   </gazebo>
-   <gazebo reference="RSoftHand">
-     <kp>1000000.0</kp>
-     <kd>100.0</kd>
-     <mu1>1.0</mu1>
-     <mu2>1.0</mu2>
-     <fdir1>1 0 0</fdir1>
-     <maxVel>1.0</maxVel>
-     <minDepth>0.00</minDepth>
-     <cfmDamping>1</cfmDamping>
-   </gazebo>
-  </xacro:if>
-</xacro:if>
--->
 <!-- Other parameters... -->
    <gazebo reference="WaistSag">
-    <cfmDamping>1</cfmDamping>
+    <implicitSpringDamper>1</implicitSpringDamper>
     <provideFeedback>true</provideFeedback>
    </gazebo>
    <gazebo reference="WaistLat">
-    <cfmDamping>1</cfmDamping>
+    <implicitSpringDamper>1</implicitSpringDamper>
     <provideFeedback>true</provideFeedback>
    </gazebo>
    <gazebo reference="WaistYaw">
-    <cfmDamping>1</cfmDamping>
+    <implicitSpringDamper>1</implicitSpringDamper>
     <provideFeedback>true</provideFeedback>
    </gazebo>
    <gazebo reference="RHipSag">
-    <cfmDamping>1</cfmDamping>
+    <implicitSpringDamper>1</implicitSpringDamper>
     <provideFeedback>true</provideFeedback>
    </gazebo>
    <gazebo reference="RHipLat">
-    <cfmDamping>1</cfmDamping>
+    <implicitSpringDamper>1</implicitSpringDamper>
     <provideFeedback>true</provideFeedback>
    </gazebo>
    <gazebo reference="RHipYaw">
-    <cfmDamping>1</cfmDamping>
+    <implicitSpringDamper>1</implicitSpringDamper>
     <provideFeedback>true</provideFeedback>
    </gazebo>
    <gazebo reference="RKneeSag">
-    <cfmDamping>1</cfmDamping>
+    <implicitSpringDamper>1</implicitSpringDamper>
     <provideFeedback>true</provideFeedback>
    </gazebo>
    <gazebo reference="RAnkLat">
-    <cfmDamping>1</cfmDamping>
+    <implicitSpringDamper>1</implicitSpringDamper>
     <provideFeedback>true</provideFeedback>
    </gazebo>
    <gazebo reference="RAnkSag">
-    <cfmDamping>1</cfmDamping>
+    <implicitSpringDamper>1</implicitSpringDamper>
     <provideFeedback>true</provideFeedback>
   </gazebo>
    <gazebo reference="LHipSag">
-    <cfmDamping>1</cfmDamping>
+    <implicitSpringDamper>1</implicitSpringDamper>
     <provideFeedback>true</provideFeedback>
    </gazebo>
    <gazebo reference="LHipLat">
-    <cfmDamping>1</cfmDamping>
+    <implicitSpringDamper>1</implicitSpringDamper>
     <provideFeedback>true</provideFeedback>
    </gazebo>
    <gazebo reference="LHipYaw">
-    <cfmDamping>1</cfmDamping>
+    <implicitSpringDamper>1</implicitSpringDamper>
     <provideFeedback>true</provideFeedback>
    </gazebo>
    <gazebo reference="LKneeSag">
-    <cfmDamping>1</cfmDamping>
+    <implicitSpringDamper>1</implicitSpringDamper>
     <provideFeedback>true</provideFeedback>
    </gazebo>
    <gazebo reference="LAnkLat">
-    <cfmDamping>1</cfmDamping>
+    <implicitSpringDamper>1</implicitSpringDamper>
     <provideFeedback>true</provideFeedback>
    </gazebo>
    <gazebo reference="LAnkSag">
-    <cfmDamping>1</cfmDamping>
+    <implicitSpringDamper>1</implicitSpringDamper>
     <provideFeedback>true</provideFeedback>
    </gazebo>
    <gazebo reference="RShSag">
-    <cfmDamping>1</cfmDamping>
+    <implicitSpringDamper>1</implicitSpringDamper>
     <provideFeedback>true</provideFeedback>
    </gazebo>
    <gazebo reference="RShLat">
-    <cfmDamping>1</cfmDamping>
+    <implicitSpringDamper>1</implicitSpringDamper>
     <provideFeedback>true</provideFeedback>
    </gazebo>
    <gazebo reference="RShYaw">
-    <cfmDamping>1</cfmDamping>
+    <implicitSpringDamper>1</implicitSpringDamper>
     <provideFeedback>true</provideFeedback>
    </gazebo>
    <gazebo reference="RElbj">
-    <cfmDamping>1</cfmDamping>
+    <implicitSpringDamper>1</implicitSpringDamper>
     <provideFeedback>true</provideFeedback>
    </gazebo>
-<xacro:if value="${GAZEBO_COMAN_USES_7DOF_FOREARMS_DRC_14}">
+<xacro:if value="${GAZEBO_COMAN_USES_FOREARMS}">
    <gazebo reference="RForearmPlate">
-    <cfmDamping>1</cfmDamping>
+    <implicitSpringDamper>1</implicitSpringDamper>
     <provideFeedback>true</provideFeedback>
    </gazebo>
    <gazebo reference="RWrj1">
-    <cfmDamping>1</cfmDamping>
+    <implicitSpringDamper>1</implicitSpringDamper>
     <provideFeedback>true</provideFeedback>
    </gazebo>
    <gazebo reference="RWrj2">
-    <cfmDamping>1</cfmDamping>
+    <implicitSpringDamper>1</implicitSpringDamper>
     <provideFeedback>true</provideFeedback>
    </gazebo>
-</xacro:if>
-<xacro:if value="${GAZEBO_COMAN_USES_7DOF_FOREARMS_DRC_14}">
-    <xacro:unless value="${GAZEBO_COMAN_USES_SOFTHANDS_DRC_sw1_14}">
+    <xacro:unless value="${GAZEBO_COMAN_USES_SOFTHANDS}">
       <gazebo reference="r_handj">
-        <cfmDamping>1</cfmDamping>
+        <implicitSpringDamper>1</implicitSpringDamper>
         <provideFeedback>true</provideFeedback>
       </gazebo>
@@ -149,37 +118,35 @@
 </xacro:if>
    <gazebo reference="LShSag">
-    <cfmDamping>1</cfmDamping>
+    <implicitSpringDamper>1</implicitSpringDamper>
     <provideFeedback>true</provideFeedback>
    </gazebo>
    <gazebo reference="LShLat">
-    <cfmDamping>1</cfmDamping>
+    <implicitSpringDamper>1</implicitSpringDamper>
     <provideFeedback>true</provideFeedback>
    </gazebo>
    <gazebo reference="LShYaw">
-    <cfmDamping>1</cfmDamping>
+    <implicitSpringDamper>1</implicitSpringDamper>
     <provideFeedback>true</provideFeedback>
    </gazebo>
    <gazebo reference="LElbj">
-    <cfmDamping>1</cfmDamping>
+    <implicitSpringDamper>1</implicitSpringDamper>
     <provideFeedback>true</provideFeedback>
    </gazebo>
-<xacro:if value="${GAZEBO_COMAN_USES_7DOF_FOREARMS_DRC_14}">
+<xacro:if value="${GAZEBO_COMAN_USES_FOREARMS}">
    <gazebo reference="LForearmPlate">
-    <cfmDamping>1</cfmDamping>
+    <implicitSpringDamper>1</implicitSpringDamper>
     <provideFeedback>true</provideFeedback>
    </gazebo>
    <gazebo reference="LWrj1">
-    <cfmDamping>1</cfmDamping>
+    <implicitSpringDamper>1</implicitSpringDamper>
     <provideFeedback>true</provideFeedback>
    </gazebo>
    <gazebo reference="LWrj2">
-    <cfmDamping>1</cfmDamping>
+    <implicitSpringDamper>1</implicitSpringDamper>
     <provideFeedback>true</provideFeedback>
    </gazebo>
-</xacro:if>
-<xacro:if value="${GAZEBO_COMAN_USES_7DOF_FOREARMS_DRC_14}">
-    <xacro:unless value="${GAZEBO_COMAN_USES_SOFTHANDS_DRC_sw1_14}">
+    <xacro:unless value="${GAZEBO_COMAN_USES_SOFTHANDS}">
       <gazebo reference="l_handj">
-        <cfmDamping>1</cfmDamping>
+        <implicitSpringDamper>1</implicitSpringDamper>
         <provideFeedback>true</provideFeedback>
       </gazebo>

File: coman_urdf/urdf/gazebo/coman_materials.gazebo.xacro (robot description, xacro)
@@ -28,5 +28,5 @@
   <material>Gazebo/DarkGrey</material>
 </gazebo>
-<xacro:if value="${GAZEBO_COMAN_USES_7DOF_FOREARMS_DRC_14}">
+<xacro:if value="${GAZEBO_COMAN_USES_FOREARMS}">
   <gazebo reference="RWrMot2">
     <material>Gazebo/Grey</material>
@@ -35,5 +35,5 @@
     <material>Gazebo/Grey</material>
   </gazebo>
-  <xacro:if value="${GAZEBO_COMAN_USES_SOFTHANDS_DRC_sw1_14}">
+  <xacro:if value="${GAZEBO_COMAN_USES_SOFTHANDS}">
     <gazebo reference="RSoftHand">
       <material>Gazebo/DarkGrey</material>
@@ -56,5 +56,5 @@
   <material>Gazebo/DarkGrey</material>
 </gazebo>
-<xacro:if value="${GAZEBO_COMAN_USES_7DOF_FOREARMS_DRC_14}">
+<xacro:if value="${GAZEBO_COMAN_USES_FOREARMS}">
   <gazebo reference="LWrMot2">
     <material>Gazebo/Grey</material>
@@ -63,5 +63,5 @@
     <material>Gazebo/Grey</material>
   </gazebo>
-  <xacro:if value="${GAZEBO_COMAN_USES_SOFTHANDS_DRC_sw1_14}">
+  <xacro:if value="${GAZEBO_COMAN_USES_SOFTHANDS}">
     <gazebo reference="LSoftHand">
       <material>Gazebo/DarkGrey</material>
