Commit message: Deleted useless files

File: coman_urdf/urdf/gazebo/microstrain_3dmgx2_imu.gazebo.xacro (robot description, xacro)
@@ -6,22 +6,4 @@
   This file groups files to use COMAN in GAZEBO
   -->
-  <xacro:if value="$(optenv GAZEBO_COMAN_USES_ROS false)">
-    <gazebo>
-        <plugin name="quadrotor_imu_sim" filename="libhector_gazebo_ros_imu.so">
-          <updateRate>100.0</updateRate>
-          <bodyName>imu_link</bodyName>
-          <topicName>COMAN/raw_imu</topicName>
-          <rpyOffsets>0 0 0</rpyOffsets> <!-- deprecated -->
-          <gaussianNoise>0</gaussianNoise>  <!-- deprecated -->
-          <accelDrift>0.5 0.5 0.5</accelDrift>
-          <accelGaussianNoise>0.35 0.35 0.3</accelGaussianNoise>
-          <rateDrift>0.1 0.1 0.1</rateDrift>
-          <rateGaussianNoise>0.05 0.05 0.015</rateGaussianNoise>
-          <headingDrift>0.1</headingDrift>
-          <headingGaussianNoise>0.05</headingGaussianNoise>
-        </plugin>
-      </gazebo>
-  </xacro:if>
-  <xacro:if value="$(optenv GAZEBO_COMAN_USES_YARP true)">
     <gazebo reference="imu_link">
         <sensor name="imu_sensor" type="imu">
@@ -54,4 +36,3 @@
         </sensor>
        </gazebo>
-  </xacro:if>
 </robot>

File: coman_urdf/urdf/gazebo/yarp_control.gazebo.xacro (robot description, xacro)
@@ -35,5 +35,5 @@
 </plugin>
 <!-- ARMS -->
-<xacro:if value="${GAZEBO_COMAN_USES_7DOF_FOREARMS_DRC_14}">
+<xacro:if value="${GAZEBO_COMAN_USES_FOREARMS}">
 	<plugin name="coman_yarp_gazebo_plugin_left_arm" filename="libgazebo_yarp_controlboard.so">
 		<yarpConfigurationFile>model://coman_urdf/conf/coman/coman_gazebo_left_arm.ini</yarpConfigurationFile>
@@ -57,5 +57,5 @@
     </plugin>
 	<!-- HANDS -->
-	<xacro:unless value="${GAZEBO_COMAN_USES_SOFTHANDS_DRC_sw1_14}">
+	<xacro:unless value="${GAZEBO_COMAN_USES_SOFTHANDS}">
 		<plugin name="coman_yarp_gazebo_plugin_left_hand" filename="libgazebo_yarp_controlboard.so">
 			<yarpConfigurationFile>model://coman_urdf/conf/coman/coman_gazebo_left_hand.ini</yarpConfigurationFile>
@@ -68,5 +68,5 @@
 	</xacro:unless>
 </xacro:if>
-<xacro:if value="${GAZEBO_COMAN_USES_NO_FOREARMS}">
+<xacro:unless value="${GAZEBO_COMAN_USES_FOREARMS}">
 	<plugin name="coman_yarp_gazebo_plugin_left_arm" filename="libgazebo_yarp_controlboard.so">
 		<yarpConfigurationFile>model://coman_urdf/conf/coman_no_forearms/coman_gazebo_left_arm.ini</yarpConfigurationFile>
@@ -89,5 +89,5 @@
         <yarpConfigurationFile>model://coman_urdf/conf/coman_no_forearms/coman_gazebo_right_arm_torque.ini</yarpConfigurationFile>
     </plugin>
-</xacro:if>
+</xacro:unless>
 <!-- Plugin to apply external wrenches to the robot -->
 <plugin name="coman_yarp_gazebo_plugin_external_wrench" filename="libgazebo_yarp_externalwrench.so"/>

File: coman_urdf/urdf/parts/legs.urdf.xacro (robot description, xacro)
@@ -106,27 +106,48 @@
     </collision>
   </link>
-<xacro:unless value="${GAZEBO_COMAN_USES_ACCURATE_FT}">
-    <xacro:if value="${GAZEBO_COMAN_USES_ROUND_FEET_13}">
-      <xacro:include filename="$(find coman_urdf)/urdf/parts/subparts/round_feet_13/round_foot_R_13.urdf.xacro" />
-    </xacro:if>
-    <xacro:if value="${GAZEBO_COMAN_USES_SIMPLE_FEET_DRC_sw1_14}">
-      <xacro:include filename="$(find coman_urdf)/urdf/parts/subparts/simple_feet_DRC_sw1_14/simple_foot_R_DRC_sw1_14.urdf.xacro" />
-    </xacro:if>
+  <xacro:if value="${GAZEBO_COMAN_USES_ROUND_FEET}">
+    <link name ="RFoot">
+      <inertial>
+        <origin xyz="0.00969210464 -0.0090460227 -0.043062308" rpy="0 0 0"/>
+        <mass value="0.66646684"/>
+        <inertia ixx="0.0012944808"  ixy="-9.2387693E-5"  ixz="2.0080105E-4" iyy="0.0015851846" iyz="2.7599327E-4" izz="0.0013326766" />
+      </inertial>
+      <visual>
+        <origin xyz="0.0 0.0726 -0.0932" rpy="0 0 -3.14159265359"/>
+        <material name="dark_grey"/>
+        <geometry name="RFoot_visual">
+          <mesh filename="package://coman_urdf/meshes/RoundFoot.STL" scale="0.03937 0.03937 0.03937" />
+        </geometry>
+      </visual>
+      <collision>
+        <origin xyz="0.0 0.0726 -0.0932" rpy="0 0 -3.14159265359"/>
+        <geometry name="RFoot_collision">
+          <mesh filename="package://coman_urdf/meshes/simple/RoundFoot.STL" scale="0.03937 0.03937 0.03937" />
+        </geometry>
+      </collision>
+    </link>
+  </xacro:if>
+  <xacro:unless value="${GAZEBO_COMAN_USES_ROUND_FEET}">
+    <link name ="RFoot">
+      <inertial>
+        <origin xyz="0.00969210464 -0.0090460227 -0.043062308" rpy="0 0 0"/>
+        <mass value="0.66646684"/>
+        <inertia ixx="0.0012944808"  ixy="-9.2387693E-5"  ixz="2.0080105E-4" iyy="0.0015851846" iyz="2.7599327E-4" izz="0.0013326766" />
+      </inertial>
+    <visual>
+     <origin xyz="0.03 0 -0.07" rpy="0 0 0" />
+     <geometry>
+       <box size="0.2 0.1 0.04" />
+     </geometry>
+     <material name="dark_gray"/>
+   </visual>
+   <collision>
+     <origin xyz="0.03 0 -0.07" rpy="0 0 0"/>
+     <geometry>
+       <box size="0.2 0.1 0.04" />
+     </geometry>
+   </collision>
+  </link>
   </xacro:unless>
-  <xacro:if value="${GAZEBO_COMAN_USES_ACCURATE_FT}">
-    <link name ="RFootFTSensor">
-      <inertial>
-        <origin xyz="0.0 -0.0 -0.0325" rpy="0 0 0"/>
-        <mass value="0.280"/>
-        <inertia ixx="0.0012944808"  ixy="0.0"  ixz="2.0080105E-4" iyy="0.0015851846" iyz="2.7599327E-4" izz="0.0013326766" />
-      </inertial>
-    </link>
-    <xacro:if value="${GAZEBO_COMAN_USES_ROUND_FEET_13}">
-      <xacro:include filename="$(find coman_urdf)/urdf/parts/subparts/round_feet_13/accurate_FT_round_foot_R_13.urdf.xacro" />
-    </xacro:if>
-    <xacro:if value="${GAZEBO_COMAN_USES_SIMPLE_FEET_DRC_sw1_14}">
-      <xacro:include filename="$(find coman_urdf)/urdf/parts/subparts/simple_feet_DRC_sw1_14/accurate_FT_simple_foot_R_DRC_sw1_14.urdf.xacro" />
-    </xacro:if>
-  </xacro:if>
 <!-- ********************LEFT LEG******************** -->
   <link name ="LHipMot">
@@ -230,27 +251,48 @@
     </collision>
   </link>
-  <xacro:unless value="${GAZEBO_COMAN_USES_ACCURATE_FT}">
-    <xacro:if value="${GAZEBO_COMAN_USES_ROUND_FEET_13}">
-      <xacro:include filename="$(find coman_urdf)/urdf/parts/subparts/round_feet_13/round_foot_L_13.urdf.xacro" />
-    </xacro:if>
-    <xacro:if value="${GAZEBO_COMAN_USES_SIMPLE_FEET_DRC_sw1_14}">
-      <xacro:include filename="$(find coman_urdf)/urdf/parts/subparts/simple_feet_DRC_sw1_14/simple_foot_L_DRC_sw1_14.urdf.xacro" />
-    </xacro:if>
+  <xacro:if value="${GAZEBO_COMAN_USES_ROUND_FEET}">
+    <link name ="LFoot">
+      <inertial>
+        <origin xyz="0.0096921046 0.0090460227 -0.043062308" rpy="0 0 0"/>
+        <mass value="0.66646684"/>
+        <inertia ixx="0.0012944808"  ixy="9.2387693E-5"  ixz="2.0080105E-4" iyy="0.0015851846" iyz="-2.7599327E-4" izz="0.0013326766" />
+      </inertial>
+      <visual>
+        <origin xyz="0.0 -0.0726 -0.0932" rpy="0 0 -3.14159265359"/>
+        <material name="dark_grey"/>
+        <geometry name="LFoot_visual">
+          <mesh filename="package://coman_urdf/meshes/RoundFoot.STL" scale="0.03937 -0.03937 0.03937" />
+        </geometry>
+      </visual>
+      <collision>
+        <origin xyz="0.0 -0.0726 -0.0932" rpy="0 0 -3.14159265359"/>
+        <geometry name="LFoot_collision">
+          <mesh filename="package://coman_urdf/meshes/simple/RoundFoot.STL" scale="0.03937 -0.03937 0.03937" />
+        </geometry>
+      </collision>
+    </link>
+  </xacro:if>
+  <xacro:unless value="${GAZEBO_COMAN_USES_ROUND_FEET}">
+    <link name ="LFoot">
+      <inertial>
+        <origin xyz="0.0096921046 0.0090460227 -0.043062308" rpy="0 0 0"/>
+        <mass value="0.66646684"/>
+        <inertia ixx="0.0012944808"  ixy="9.2387693E-5"  ixz="2.0080105E-4" iyy="0.0015851846" iyz="-2.7599327E-4" izz="0.0013326766" />
+      </inertial>
+      <visual>
+       <origin xyz="0.03 0 -0.07" rpy="0 0 0" />
+       <geometry>
+         <box size="0.2 0.1 0.04" />
+       </geometry>
+       <material name="dark_gray"/>
+     </visual>
+     <collision>
+       <origin xyz="0.03 0 -0.07" rpy="0 0 0"/>
+       <geometry>
+         <box size="0.2 0.1 0.04" />
+       </geometry>
+     </collision>
+    </link>
   </xacro:unless>
-  <xacro:if value="${GAZEBO_COMAN_USES_ACCURATE_FT}">
-    <link name ="LFootFTSensor">
-      <inertial>
-        <origin xyz="0.0 -0.0 -0.0325" rpy="0 0 0"/>
-        <mass value="0.280"/>
-        <inertia ixx="0.0012944808"  ixy="-9.2387693E-5"  ixz="2.0080105E-4" iyy="0.0015851846" iyz="2.7599327E-4" izz="0.0013326766" />
-      </inertial>
-    </link>
-    <xacro:if value="${GAZEBO_COMAN_USES_ROUND_FEET_13}">
-      <xacro:include filename="$(find coman_urdf)/urdf/parts/subparts/round_feet_13/accurate_FT_round_foot_L_13.urdf.xacro" />
-    </xacro:if>
-    <xacro:if value="${GAZEBO_COMAN_USES_SIMPLE_FEET_DRC_sw1_14}">
-      <xacro:include filename="$(find coman_urdf)/urdf/parts/subparts/simple_feet_DRC_sw1_14/accurate_FT_simple_foot_L_DRC_sw1_14.urdf.xacro" />
-    </xacro:if>
-  </xacro:if>
 <!-- JOINTS -->
 <!-- ********************RIGHT LEG******************** -->
@@ -295,6 +337,5 @@
     <dynamics friction="0" damping="3.0"/>
   </joint>
- <xacro:unless value="${GAZEBO_COMAN_USES_ACCURATE_FT}">
-    <joint name="RAnkSag" type="revolute">
+  <joint name="RAnkSag" type="revolute">
       <parent link="RFootmot"/>
       <child link="RFoot"/>
@@ -303,24 +344,5 @@
       <limit velocity="4.0" effort="50" lower="-1.2217" upper="1.2217" />
       <dynamics friction="0" damping="3.0"/>
-    </joint>
-  </xacro:unless>
-  <xacro:if value="${GAZEBO_COMAN_USES_ACCURATE_FT}">
-    <joint name="RAnkSag" type="revolute">
-      <parent link="RFootmot"/>
-      <child link="RFootFTSensor"/>
-      <origin xyz="0.0 0.0 0.0" rpy="0 0 0" />
-      <axis xyz="0 1 0" />
-      <limit velocity="4.0" effort="50" lower="-1.2217" upper="1.2217" />
-      <dynamics friction="0" damping="3.0"/>
-    </joint>
-    <joint name="RAnkSagFT" type="revolute">
-      <parent link="RFootFTSensor"/>
-      <child link="RFoot"/>
-      <origin xyz="0.0 0.0 -0.065" rpy="0 0 0" />
-      <axis xyz="0 1 0" />
-      <limit velocity="0.0" effort="0" lower="-0.0" upper="0.0" />
-      <dynamics friction="0" damping="3.0"/>
-    </joint>
-  </xacro:if>
+  </joint>
 <!-- ********************LEFT LEG******************** -->
   <joint name="LHipSag" type="revolute">
@@ -364,6 +386,5 @@
     <dynamics friction="0" damping="3.0"/>
   </joint>
-<xacro:unless value="${GAZEBO_COMAN_USES_ACCURATE_FT}">
-    <joint name="LAnkSag" type="revolute">
+  <joint name="LAnkSag" type="revolute">
       <parent link="LFootmot"/>
       <child link="LFoot"/>
@@ -372,23 +393,4 @@
       <limit velocity="4.0" effort="50" lower="-1.2217" upper="1.2217" />
       <dynamics friction="0" damping="3.0"/>
-    </joint>
-  </xacro:unless>
-  <xacro:if value="${GAZEBO_COMAN_USES_ACCURATE_FT}">
-    <joint name="LAnkSag" type="revolute">
-      <parent link="LFootmot"/>
-      <child link="LFootFTSensor"/>
-      <origin xyz="0.0 0.0 0.0" rpy="0 0 0" />
-      <axis xyz="0 1 0" />
-      <limit velocity="4.0" effort="50" lower="-1.2217" upper="1.2217" />
-      <dynamics friction="0" damping="3.0"/>
-    </joint>
-    <joint name="LAnkSagFT" type="revolute">
-      <parent link="LFootFTSensor"/>
-      <child link="LFoot"/>
-      <origin xyz="0.0 0.0 -0.065" rpy="0 0 0" />
-      <axis xyz="0 1 0" />
-      <limit velocity="0.0" effort="0" lower="-0.0" upper="0.0" />
-      <dynamics friction="0" damping="3.0"/>
-    </joint>
-  </xacro:if>
+  </joint>
 </robot>

File: coman_urdf/urdf/parts/soft_hand.urdf.xacro (robot description, xacro)
@@ -1,5 +1,5 @@
 <?xml version="1.0"?>
 <robot xmlns:xacro="http://ros.org/wiki/xacro" name="SoftHand">
-<xacro:if value="${GAZEBO_COMAN_USES_SOFTHANDS_DRC_sw1_14}">
+<xacro:if value="${GAZEBO_COMAN_USES_SOFTHANDS}">
 <!-- LINKS -->
 <link name="RSoftHand">
@@ -55,5 +55,5 @@
   </joint>
 </xacro:if>
-<xacro:unless value="${GAZEBO_COMAN_USES_SOFTHANDS_DRC_sw1_14}">
+<xacro:unless value="${GAZEBO_COMAN_USES_SOFTHANDS}">
 <!-- LINKS -->
 <!-- ## WRONG NUMBERS FOR... ok lasciamo perde... FIX THEM!! ## -->

Commit message: Fixed name of arm ft sensor ports

File: coman_srdf/srdf/coman.srdf.xacro (robot description, xacro)
@@ -26,12 +26,8 @@
         </group>
         <group name="force_torque_sensors">
-        <!--<joint name="LAnkSag"/>
-            <joint name="RAnkSag"/>
-            <joint name="LForearmPlate"/>
-            <joint name="RForearmPlate"/>-->
             <joint name="l_ankle_joint"/>
-            <joint name="r_ankle_joint"/>
-            <joint name="l_wrist_joint"/>
-            <joint name="r_wrist_joint"/>
+    	    <joint name="r_ankle_joint"/>
+    	    <joint name="l_arm_ft_joint"/>
+    	    <joint name="r_arm_ft_joint"/>
         </group>
     </xacro:if>

Commit message: Added proper ref frames for ft in legs. Changed srdf and config files accordly

File: coman_srdf/srdf/coman.srdf.xacro (robot description, xacro)
@@ -26,6 +26,6 @@
         </group>
         <group name="force_torque_sensors">
-            <joint name="l_ankle_joint"/>
-    	    <joint name="r_ankle_joint"/>
+            <joint name="l_leg_ft_joint"/>
+    	    <joint name="r_leg_ft_joint"/>
     	    <joint name="l_arm_ft_joint"/>
     	    <joint name="r_arm_ft_joint"/>

File: coman_urdf/urdf/coman.urdf.xacro (robot description, xacro)
@@ -53,4 +53,16 @@
     <xacro:include filename="$(find coman_urdf)/urdf/parts/no_forearms.urdf.xacro" />
 </xacro:unless>
+    <link name="l_leg_ft"/>
+    <link name="r_leg_ft"/>
+    <joint name="l_leg_ft_joint" type="fixed">
+      <parent link="LFoot"/>
+      <child link="l_leg_ft"/>
+      <origin xyz="0 0 -0.065" rpy="0 0 0" />
+    </joint>
+    <joint name="r_leg_ft_joint" type="fixed">
+      <parent link="RFoot"/>
+      <child link="r_leg_ft"/>
+      <origin xyz="0 0 -0.065" rpy="0 0 0" />
+    </joint>
 <!-- ************ HANDS ************ -->
 <xacro:if value="${GAZEBO_COMAN_USES_FOREARMS}">

Commit message: Updated imu link

File: coman_srdf/srdf/coman.srdf.xacro (robot description, xacro)
@@ -16,5 +16,5 @@
     <group name="imu_sensors">
     <!-- NEAREST JOINT TO IMU -->
-        <joint name="WaistSag"/>
+        <link name="imu_link"/>
     </group>
     <xacro:if value="${GAZEBO_COMAN_USES_FOREARMS}">

Commit message: Added hands kinematic chains in srdf. Changed script to generate model_name_robot.urdf files. Added variable in config to add/delete YARP things in model.

File: coman_srdf/srdf/coman.srdf.xacro (robot description, xacro)
@@ -19,4 +19,12 @@
         <link name="imu_link"/>
     </group>
+    <xacro:unless value="${GAZEBO_COMAN_USES_SOFTHANDS}">
+       <group name="left_hand">
+           <chain base_link="LWrMot3" tip_link="LSoftHand"/>
+       </group>
+       <group name="right_hand">
+           <chain base_link="RWrMot3" tip_link="RSoftHand"/>
+       </group>
+    </xacro:unless>
     <xacro:if value="${GAZEBO_COMAN_USES_FOREARMS}">
         <group name="left_arm">
@@ -63,4 +71,8 @@
         <group name="right_leg"/>
         <group name="torso"/>
+<xacro:unless value="${GAZEBO_COMAN_USES_SOFTHANDS}">
+        <group name="left_hand"/>
+        <group name="right_hand"/>
+</xacro:unless>
     </group>
     <xacro:include filename="$(find coman_urdf)/urdf/gazebo/rtt_gazebo.gazebo.xacro" />

File: coman_urdf/urdf/coman_config.urdf.xacro (robot description, xacro)
@@ -27,4 +27,11 @@
 ####################################################
 ##
+##  USE YARP
+####################################################
+-->
+<xacro:property name="GAZEBO_COMAN_USES_YARP" value="true" />
+<!--
+####################################################
+##
 ##  Xtion SELECTION
 ##

File: coman_urdf/urdf/coman_robot.urdf.xacro (robot description, xacro)
@@ -13,7 +13,9 @@
   </xacro:if>
 <!-- YARP PLUGINS for GAZEBO SIMULATION -->
-  <xacro:include filename="$(find coman_urdf)/urdf/gazebo/yarp_control.gazebo.xacro" />
+  <xacro:if value="${GAZEBO_COMAN_USES_YARP}">
+       <xacro:include filename="$(find coman_urdf)/urdf/gazebo/yarp_control.gazebo.xacro" />
+       <xacro:include filename="$(find coman_urdf)/urdf/gazebo/force_torque.gazebo.xacro" />
+  </xacro:if>
   <xacro:include filename="$(find coman_urdf)/urdf/gazebo/coman_materials.gazebo.xacro" />
-  <xacro:include filename="$(find coman_urdf)/urdf/gazebo/force_torque.gazebo.xacro" />
   <origin xyz="0.0 0.0 0.521" rpy="0 0 0" />
 </robot>

File: coman_urdf/urdf/config/coman_hands.urdf.xacro (robot description, xacro)
@@ -26,4 +26,11 @@
 ####################################################
 ##
+##  USE YARP
+####################################################
+-->
+<xacro:property name="GAZEBO_COMAN_USES_YARP" value="true" />
+<!--
+####################################################
+##
 ##  Xtion SELECTION
 ##

File: coman_urdf/urdf/config/coman_no_forearms.urdf.xacro (robot description, xacro)
@@ -26,4 +26,11 @@
 ####################################################
 ##
+##  USE YARP
+####################################################
+-->
+<xacro:property name="GAZEBO_COMAN_USES_YARP" value="true" />
+<!--
+####################################################
+##
 ##  Xtion SELECTION
 ##

File: coman_urdf/urdf/config/coman_softhand.urdf.xacro (robot description, xacro)
@@ -26,33 +26,6 @@
 ####################################################
 ##
-##  MIDDLEWARE SELECTION
-##
-##
-## options:
-#  notice how, regardless of the middleware selected
-#  a bare version of the robot is created (.urdf)
-#  1) yarp
-#	The robot is created using yarp plugins for
-#	the IMU and F/T sensors. The controlboard
-#	plugins used to control joints and get
-#	encoder and torque information are to be
-#	inserted using the .world file, where the
-#	initial configuration for the joints can
-#	be specified (for example, look at the
-#	worlds folder)
-#  2) ros
-#	The sdf is created including ros plugins
-#
-##
+##  USE YARP
 ####################################################
-#
-# 1) yarp
-#
--->
-<xacro:property name="GAZEBO_COMAN_USES_ROS" value="false" />
-<!--
-#
-# 2) ros
-#
 -->
 <xacro:property name="GAZEBO_COMAN_USES_YARP" value="true" />

File: coman_urdf/urdf/gazebo/force_torque.gazebo.xacro (robot description, xacro)
@@ -18,7 +18,9 @@
 			       <update_rate>1000</update_rate>
                             <pose>0 0 0 0 0 0</pose>
+<xacro:if value="${GAZEBO_COMAN_USES_YARP}">
 			       <plugin name="RForearmPlate_FT_plugin" filename="libgazebo_yarp_forcetorque.so">
 				       <yarpConfigurationFile>model://coman_urdf/conf/coman/coman_gazebo_right_arm_ft.ini</yarpConfigurationFile>
 			       </plugin>
+</xacro:if>
 		       </sensor>
 	       </gazebo>
@@ -33,7 +35,9 @@
 			       <update_rate>1000</update_rate>
                             <pose>0 0 0 0 0 0</pose>
+<xacro:if value="${GAZEBO_COMAN_USES_YARP}">
 			       <plugin name="LForearmPlate_FT_plugin" filename="libgazebo_yarp_forcetorque.so">
 				       <yarpConfigurationFile>model://coman_urdf/conf/coman/coman_gazebo_left_arm_ft.ini</yarpConfigurationFile>
 			       </plugin>
+</xacro:if>
 		       </sensor>
 	       </gazebo>
@@ -49,7 +53,9 @@
 			<update_rate>1000</update_rate>
 			<pose>0 0 -0.065 0 0 0</pose>
+<xacro:if value="${GAZEBO_COMAN_USES_YARP}">
 			<plugin name="LAnkSag_FT_plugin" filename="libgazebo_yarp_forcetorque.so">
 				<yarpConfigurationFile>model://coman_urdf/conf/coman/coman_gazebo_left_leg_ft.ini</yarpConfigurationFile>
 			</plugin>
+</xacro:if>
 		</sensor>
 	</gazebo>
@@ -64,7 +70,9 @@
 			<update_rate>1000</update_rate>
 			<pose>0 0 -0.065 0 0 0</pose>
+<xacro:if value="${GAZEBO_COMAN_USES_YARP}">
 			<plugin name="RAnkSag_FT_plugin" filename="libgazebo_yarp_forcetorque.so">
 				<yarpConfigurationFile>model://coman_urdf/conf/coman/coman_gazebo_right_leg_ft.ini</yarpConfigurationFile>
 	        	</plugin>
+</xacro:if>
 		</sensor>
 	</gazebo>

File: coman_urdf/urdf/gazebo/microstrain_3dmgx2_imu.gazebo.xacro (robot description, xacro)
@@ -31,7 +31,9 @@
           -->
          </imu>
+<xacro:if value="${GAZEBO_COMAN_USES_YARP}">
          <plugin name="coman_yarp_gazebo_plugin_IMU" filename="libgazebo_yarp_imu.so">
            <yarpConfigurationFile>model://coman_urdf/conf/coman/coman_gazebo_inertial.ini</yarpConfigurationFile>
          </plugin>
+</xacro:if>
         </sensor>
        </gazebo>

File: coman_urdf/urdf/gazebo/rtt_gazebo.gazebo.xacro (robot description, xacro)
@@ -14,4 +14,16 @@
        <controller type="JointTorqueCtrl"/>
 </rtt-gazebo>
+<xacro:unless value="${GAZEBO_COMAN_USES_SOFTHANDS}">
+<rtt-gazebo reference="left_hand">
+       <controller type="JointPositionCtrl">
+              <gains reference="l_handj" P="10." D="0.01" I="0."/>
+       </controller>
+</rtt-gazebo>
+<rtt-gazebo reference="right_hand">
+       <controller type="JointPositionCtrl">
+              <gains reference="r_handj" P="10." D="0.01" I="0."/>
+       </controller>
+</rtt-gazebo>
+</xacro:unless>
 <rtt-gazebo reference="right_arm">
        <controller type="JointPositionCtrl">
