Commit message: Added a simple gripper to the model

File: coman_srdf/srdf/coman.srdf.xacro (robot description, xacro)
@@ -21,8 +21,8 @@
     <xacro:unless value="${GAZEBO_COMAN_USES_SOFTHANDS}">
        <group name="left_hand">
-           <chain base_link="LWrMot3" tip_link="LSoftHand"/>
+           <chain base_link="LWrMot3" tip_link="LSoftHandFingers"/>
        </group>
        <group name="right_hand">
-           <chain base_link="RWrMot3" tip_link="RSoftHand"/>
+           <chain base_link="RWrMot3" tip_link="RSoftHandFingers"/>
        </group>
     </xacro:unless>

File: coman_urdf/urdf/gazebo/coman.gazebo.xacro (robot description, xacro)
@@ -111,5 +111,5 @@
    </gazebo>
     <xacro:unless value="${GAZEBO_COMAN_USES_SOFTHANDS}">
-      <gazebo reference="r_handj">
+      <gazebo reference="r_handj2">
         <implicitSpringDamper>1</implicitSpringDamper>
         <provideFeedback>true</provideFeedback>
@@ -147,5 +147,5 @@
    </gazebo>
     <xacro:unless value="${GAZEBO_COMAN_USES_SOFTHANDS}">
-      <gazebo reference="l_handj">
+      <gazebo reference="l_handj2">
         <implicitSpringDamper>1</implicitSpringDamper>
         <provideFeedback>true</provideFeedback>

File: coman_urdf/urdf/gazebo/rtt_gazebo.gazebo.xacro (robot description, xacro)
@@ -17,10 +17,10 @@
 <rtt-gazebo reference="left_hand">
        <controller type="JointPositionCtrl">
-              <gains reference="l_handj" P="10." D="0.01" I="0."/>
+              <gains reference="l_handj2" P="10." D="0.01" I="0."/>
        </controller>
 </rtt-gazebo>
 <rtt-gazebo reference="right_hand">
        <controller type="JointPositionCtrl">
-              <gains reference="r_handj" P="10." D="0.01" I="0."/>
+              <gains reference="r_handj2" P="10." D="0.01" I="0."/>
        </controller>
 </rtt-gazebo>

File: coman_urdf/urdf/parts/soft_hand.urdf.xacro (robot description, xacro)
@@ -67,5 +67,5 @@
      <origin xyz="0 0 0" rpy="0 0 0" />
      <geometry>
-        <box size="0.07 0.07 0.07" />
+        <box size="0.07 0.01 0.07" />
      </geometry>
      <material name="Cyan">
@@ -76,5 +76,27 @@
      <origin xyz="0 0 0" rpy="0 0 0"/>
      <geometry>
-       <box size="0.07 0.07 0.07" />
+       <box size="0.07 0.01 0.07" />
+     </geometry>
+   </collision>
+  </link>
+  <link name="RSoftHandFingers">
+    <inertial>
+      <origin xyz="0 0 0" rpy="0 0 0"/>
+      <mass value="0.3"/>
+      <inertia ixx="0.001"  ixy="0"  ixz="0" iyy="0.001" iyz="0" izz="0.001" />
+    </inertial>
+    <visual>
+     <origin xyz="0 0 0" rpy="0 0 0" />
+     <geometry>
+        <box size="0.07 0.01 0.07" />
+     </geometry>
+     <material name="Cyan">
+       <color rgba="0 1.0 1.0 1.0"/>
+     </material>
+   </visual>
+   <collision>
+     <origin xyz="0 0 0" rpy="0 0 0"/>
+     <geometry>
+       <box size="0.07 0.01 0.07" />
      </geometry>
    </collision>
@@ -89,5 +111,5 @@
      <origin xyz="0 0 0" rpy="0 0 0" />
      <geometry>
-        <box size="0.07 0.07 0.07" />
+        <box size="0.07 0.01 0.07" />
      </geometry>
      <material name="Cyan">
@@ -98,23 +120,61 @@
      <origin xyz="0 0 0" rpy="0 0 0"/>
      <geometry>
-       <box size="0.07 0.07 0.07" />
+       <box size="0.07 0.01 0.07" />
+     </geometry>
+   </collision>
+  </link>
+  <link name="LSoftHandFingers">
+    <inertial>
+      <origin xyz="0 0 0" rpy="0 0 0"/>
+      <mass value="0.3"/>
+      <inertia ixx="0.001"  ixy="0"  ixz="0" iyy="0.001" iyz="0" izz="0.001" />
+    </inertial>
+    <visual>
+     <origin xyz="0 0 0" rpy="0 0 0" />
+     <geometry>
+        <box size="0.07 0.01 0.07" />
+     </geometry>
+     <material name="Cyan">
+       <color rgba="0 1.0 1.0 1.0"/>
+     </material>
+   </visual>
+   <collision>
+     <origin xyz="0 0 0" rpy="0 0 0"/>
+     <geometry>
+       <box size="0.07 0.01 0.07" />
      </geometry>
    </collision>
   </link>
 <!-- JOINTS -->
-<joint name="r_handj" type="revolute">
+<joint name="r_handj" type="fixed">
         <parent link="RWrMot3"/>
         <child link="RSoftHand"/>
-        <origin xyz="0 0 -0.04" rpy="0 0 0"/>
-        <axis xyz="1 0 0" />
+        <origin xyz="0 -0.03 -0.07" rpy="0 0 0"/>
+        <!--axis xyz="1 0 0" />
         <limit velocity="4.0" effort="5" lower="0.0" upper="1.57075" />
+        <dynamics friction="0" damping="3.0"/-->
+</joint>
+<joint name="r_handj2" type="prismatic">
+        <parent link="RSoftHand"/>
+        <child link="RSoftHandFingers"/>
+        <origin xyz="0 0.06 0.0" rpy="0 0 0"/>
+        <axis xyz="0 1 0" />
+        <limit velocity="4.0" effort="50" lower="-0.05" upper="0.0" />
         <dynamics friction="0" damping="3.0"/>
 </joint>
-<joint name="l_handj" type="revolute">
+<joint name="l_handj" type="fixed">
         <parent link="LWrMot3"/>
         <child link="LSoftHand"/>
-        <origin xyz="0 0 -0.04" rpy="0 0 0"/>
-        <axis xyz="-1 0 0" />
+        <origin xyz="0 0.03 -0.07" rpy="0 0 0"/>
+        <!--axis xyz="-1 0 0" />
         <limit velocity="4.0" effort="5" lower="0.0" upper="1.57075" />
+        <dynamics friction="0" damping="3.0"/-->
+</joint>
+<joint name="l_handj2" type="prismatic">
+        <parent link="LSoftHand"/>
+        <child link="LSoftHandFingers"/>
+        <origin xyz="0 -0.06 0.0" rpy="0 0 0"/>
+        <axis xyz="0 1 0" />
+        <limit velocity="4.0" effort="50" lower="0.0" upper="0.05" />
         <dynamics friction="0" damping="3.0"/>
 </joint>

Commit message: updates and cleaning

File: coman_srdf/srdf/coman.srdf.xacro (robot description, xacro)
@@ -76,4 +76,37 @@
 </xacro:unless>
     </group>
+	<xacro:if value="${GAZEBO_COMAN_USES_XBOTCORE}">
+		<group_state group="chains" name="home">
+        <joint name="WaistLat" value="0.0"/>
+        <joint name="WaistSag" value="0.0"/>
+        <joint name="WaistYaw" value="0.0"/>
+        <joint name="RShSag" value="0.5"/>
+        <joint name="RShLat" value="-0.5"/>
+        <joint name="RShYaw" value="0.30"/>
+        <joint name="RElbj" value="-1.57"/>
+        <joint name="RForearmPlate" value="0.0"/>
+        <joint name="RWrj1" value="-0.0"/>
+        <joint name="RWrj2" value="-0.0"/>
+        <joint name="LShSag" value="0.5"/>
+        <joint name="LShLat" value="0.5"/>
+        <joint name="LShYaw" value="-0.30"/>
+        <joint name="LElbj" value="-1.57"/>
+        <joint name="LForearmPlate" value="0.0"/>
+        <joint name="LWrj1" value="0.0"/>
+        <joint name="LWrj2" value="-0.0"/>
+        <joint name="RHipLat" value="0.0"/>
+        <joint name="RHipYaw" value="0.0"/>
+        <joint name="RHipSag" value="-0.45"/>
+        <joint name="RKneeSag" value="0.90"/>
+        <joint name="RAnkSag" value="-0.45"/>
+        <joint name="RAnkLat" value="-0.0"/>
+        <joint name="LHipLat" value="-0.0"/>
+        <joint name="LHipYaw" value="0.0"/>
+        <joint name="LHipSag" value="-0.45"/>
+        <joint name="LKneeSag" value="0.90"/>
+        <joint name="LAnkSag" value="-0.45"/>
+        <joint name="LAnkLat" value="0.0"/>
+  </group_state>
+	</xacro:if>
     <xacro:include filename="$(find coman_urdf)/urdf/gazebo/rtt_gazebo.gazebo.xacro" />
 </robot>

File: coman_urdf/urdf/coman_config.urdf.xacro (robot description, xacro)
@@ -30,5 +30,12 @@
 ####################################################
 -->
-<xacro:property name="GAZEBO_COMAN_USES_YARP" value="true" />
+<xacro:property name="GAZEBO_COMAN_USES_YARP" value="false" />
+<!--
+####################################################
+##
+##  USE XBOTCORE
+####################################################
+-->
+<xacro:property name="GAZEBO_COMAN_USES_XBOTCORE" value="true" />
 <!--
 ####################################################

File: coman_urdf/urdf/coman_robot.urdf.xacro (robot description, xacro)
@@ -19,4 +19,7 @@
        <xacro:include filename="$(find coman_urdf)/urdf/gazebo/yarp_control.gazebo.xacro" />
   </xacro:if>
+  <xacro:if value="${GAZEBO_COMAN_USES_XBOTCORE}" >
+  	<xacro:include filename="$(find cogimon_urdf)/urdf/gazebo/xbot_control.gazebo.xacro" />
+  </xacro:if>
   <xacro:include filename="$(find coman_urdf)/urdf/gazebo/force_torque.gazebo.xacro" />
   <xacro:include filename="$(find coman_urdf)/urdf/gazebo/coman_materials.gazebo.xacro" />

File: coman_urdf/urdf/gazebo/force_torque.gazebo.xacro (robot description, xacro)
@@ -9,5 +9,5 @@
 	<xacro:if value="${GAZEBO_COMAN_USES_FOREARMS}">
               <gazebo reference="RForearmPlate">
-	              <sensor type="force_torque" name="right_arm">
+	              <sensor type="force_torque" name="right_arm_ft">
 		              <force_torque>
                                    <frame>sensor</frame>
@@ -26,5 +26,5 @@
 	       </gazebo>
               <gazebo reference="LForearmPlate">
-	              <sensor type="force_torque" name="left_arm">
+	              <sensor type="force_torque" name="left_arm_ft">
 		              <force_torque>
                                    <frame>sensor</frame>
@@ -44,5 +44,5 @@
        </xacro:if>
        <gazebo reference="LAnkSag">
-		<sensor type="force_torque" name="left_leg">
+		<sensor type="force_torque" name="left_leg_ft">
                      <force_torque>
                        <frame>sensor</frame>
@@ -61,5 +61,5 @@
 	</gazebo>
 	<gazebo reference="RAnkSag">
-		<sensor type="force_torque" name="right_leg">
+		<sensor type="force_torque" name="right_leg_ft">
                      <force_torque>
                        <frame>sensor</frame>

Commit message: updated homing for mom experimets

File: coman_srdf/srdf/coman.srdf.xacro (robot description, xacro)
@@ -77,5 +77,67 @@
     </group>
 	<xacro:if value="${GAZEBO_COMAN_USES_XBOTCORE}">
-		<group_state group="chains" name="home">
+<group_state group="chains" name="home">
+    <joint name="WaistLat" value="0.0"/>
+    <joint name="WaistSag" value="0.0"/>
+    <joint name="WaistYaw" value="0.0"/>
+    <joint name="RShSag" value="0.7047622086892001"/>
+    <joint name="RShLat" value="-0.5677635252336075"/>
+    <joint name="RShYaw" value="0.2890564140758947"/>
+    <joint name="RElbj" value="-1.6532190021255193"/>
+    <joint name="RForearmPlate" value="-0.0003280309196516731"/>
+    <joint name="RWrj1" value="-0.008641640605188954"/>
+    <joint name="RWrj2" value="-0.0013920145156089084"/>
+    <joint name="LShSag" value="0.5545755010440612"/>
+    <joint name="LShLat" value="0.6179429857281579"/>
+    <joint name="LShYaw" value="-0.2412515368003296"/>
+    <joint name="LElbj" value="-1.7123663089414456"/>
+    <joint name="LForearmPlate" value="-0.0007051899703876909"/>
+    <joint name="LWrj1" value="-0.013205282554514752"/>
+    <joint name="LWrj2" value="0.0037545474284079597"/>
+    <joint name="RHipLat" value="-0.73156157875935218"/>
+    <joint name="RHipYaw" value="0."/>
+    <joint name="RHipSag" value="-0.1636185715937876"/>
+    <joint name="RKneeSag" value="1.1413767149293743"/>
+    <joint name="RAnkSag" value="-0.4421027118276261"/>
+    <joint name="RAnkLat" value="0.004101490304317014"/>
+    <joint name="LHipLat" value="0.73156157875935218"/>
+    <joint name="LHipYaw" value="0."/>
+    <joint name="LHipSag" value="-0.1636185715937876"/>
+    <joint name="LKneeSag" value="0.8076545504729606"/>
+    <joint name="LAnkSag" value="-0.4695127574050335"/>
+    <joint name="LAnkLat" value="0.0012525979207698662"/>
+  </group_state>
+<!--group_state group="chains" name="home">
+        <joint name="WaistLat" value="0.0"/>
+        <joint name="WaistSag" value="0.0"/>
+        <joint name="WaistYaw" value="0.0"/>
+        <joint name="RShSag" value="0.7047622086892001"/>
+        <joint name="RShLat" value="-0.5677635252336075"/>
+        <joint name="RShYaw" value="0.2890564140758947"/>
+        <joint name="RElbj" value="-1.6532190021255193"/>
+        <joint name="RForearmPlate" value="-0.0003280309196516731"/>
+        <joint name="RWrj1" value="-0.008641640605188954"/>
+        <joint name="RWrj2" value="-0.0013920145156089084"/>
+        <joint name="LShSag" value="0.5545755010440612"/>
+        <joint name="LShLat" value="0.6179429857281579"/>
+        <joint name="LShYaw" value="-0.2412515368003296"/>
+        <joint name="LElbj" value="-1.7123663089414456"/>
+        <joint name="LForearmPlate" value="-0.0007051899703876909"/>
+        <joint name="LWrj1" value="-0.013205282554514752"/>
+        <joint name="LWrj2" value="0.0037545474284079597"/>
+        <joint name="RHipLat" value="0.23156157875935218"/>
+        <joint name="RHipYaw" value="-0.08173321672018607"/>
+        <joint name="RHipSag" value="-0.1636185715937876"/>
+        <joint name="RKneeSag" value="1.1413767149293743"/>
+        <joint name="RAnkSag" value="-0.4421027118276261"/>
+        <joint name="RAnkLat" value="0.004101490304317014"/>
+        <joint name="LHipLat" value="-0.1841192194591785"/>
+        <joint name="LHipYaw" value="0.040708524744865394"/>
+        <joint name="LHipSag" value="-1.1891851384504697"/>
+        <joint name="LKneeSag" value="0.8076545504729606"/>
+        <joint name="LAnkSag" value="-0.4695127574050335"/>
+        <joint name="LAnkLat" value="0.0012525979207698662"/>
+</group_state-->
+  <!--group_state group="chains" name="home">
         <joint name="WaistLat" value="0.0"/>
         <joint name="WaistSag" value="0.0"/>
@@ -107,5 +169,5 @@
         <joint name="LAnkSag" value="-0.45"/>
         <joint name="LAnkLat" value="0.0"/>
-  </group_state>
+  </group_state-->
 	</xacro:if>
     <xacro:include filename="$(find coman_urdf)/urdf/gazebo/rtt_gazebo.gazebo.xacro" />

Commit message: COMAN_USES_XBOT

File: coman_srdf/srdf/coman.srdf.xacro (robot description, xacro)
@@ -76,5 +76,5 @@
 </xacro:unless>
     </group>
-	<xacro:if value="${GAZEBO_COMAN_USES_XBOTCORE}">
+	<xacro:if value="${GAZEBO_COMAN_USES_XBOT}">
 		<group_state group="chains" name="home">
         <joint name="WaistLat" value="0.0"/>

File: coman_urdf/urdf/coman_config.urdf.xacro (robot description, xacro)
@@ -37,5 +37,5 @@
 ####################################################
 -->
-<xacro:property name="GAZEBO_COMAN_USES_XBOTCORE" value="true" />
+<xacro:property name="GAZEBO_COMAN_USES_XBOT" value="true" />
 <!--
 ####################################################

File: coman_urdf/urdf/coman_robot.urdf.xacro (robot description, xacro)
@@ -19,7 +19,4 @@
        <xacro:include filename="$(find coman_urdf)/urdf/gazebo/yarp_control.gazebo.xacro" />
   </xacro:if>
-  <xacro:if value="${GAZEBO_COMAN_USES_XBOTCORE}" >
-  	<xacro:include filename="$(find cogimon_urdf)/urdf/gazebo/xbot_control.gazebo.xacro" />
-  </xacro:if>
   <xacro:include filename="$(find coman_urdf)/urdf/gazebo/force_torque.gazebo.xacro" />
   <!-- XBOT PLUGINS for GAZEBO SIMULATION -->
